Commit message: Remove unused sensors and fix link to mesh in xtion

File: tiago_description/urdf/sensors/openni.gazebo.xacro (robot description, xacro)
@@ -6,5 +6,5 @@
   To view a copy of this license, visit http://creativecommons.org/licenses/by-nc-nd/3.0/ or send a letter to
   Creative Commons, 444 Castro Street, Suite 900, Mountain View, California, 94041, USA.
-  ROS Gazebo plugin for RGBD sensor with Softkinetic specifications
+  ROS Gazebo plugin for RGBD sensor (OpenNI/Kinect/ASUS)
    * Publishes MONO8 format "depth" image & PointCloud
    * Publishes RGB8 format color image & 2nd copy of PointCloud (for registered)
@@ -12,34 +12,32 @@
 -->
 <robot xmlns:xacro="http://ros.org/wiki/xacro">
-  <xacro:macro name="softkinetic_ds311_rgbd_camera_gazebo" params="name">
+  <xacro:macro name="openni_camera_gazebo_v0" params="name">
     <gazebo reference="${name}_link">
-      <!-- IR + depth -->
       <sensor type="depth" name="${name}_frame_sensor">
         <always_on>true</always_on>
-        <update_rate>10.0</update_rate>
+        <update_rate>20.0</update_rate>
         <camera>
-          <horizontal_fov>${57.3 * deg_to_rad}</horizontal_fov>
+          <horizontal_fov>${57.0*M_PI/180.0}</horizontal_fov>
           <image>
             <format>R8G8B8</format>
-            <width>160</width>
-            <height>120</height>
+            <width>640</width>
+            <height>480</height>
           </image>
           <clip>
-            <near>0.1</near>
-            <far>4.0</far>
+            <near>0.01</near>
+            <far>5</far>
           </clip>
         </camera>
         <plugin name="${name}_frame_controller" filename="libgazebo_ros_openni_kinect.so">
           <alwaysOn>true</alwaysOn>
-          <updateRate>10.0</updateRate>
-          <cameraName>softkinetic_camera</cameraName>
+          <updateRate>20.0</updateRate>
+          <cameraName>${name}</cameraName>
           <imageTopicName>ir/image_raw</imageTopicName>
-          <cameraInfoTopicName>ir/camera_info</cameraInfoTopicName>
-          <depthImageTopicName>depth_registered/image_raw</depthImageTopicName>
-          <depthImageCameraInfoTopicName>depth_registered/camera_info</depthImageCameraInfoTopicName>
-          <pointCloudTopicName>depth_registered/points</pointCloudTopicName>
+          <cameraInfoTopicName>/ir/camera_info</cameraInfoTopicName>
+          <depthImageTopicName>depth/image_raw</depthImageTopicName>
+          <depthImageCameraInfoTopicName>depth/camera_info</depthImageCameraInfoTopicName>
+          <pointCloudTopicName>depth/points</pointCloudTopicName>
           <frameName>${name}_optical_frame</frameName>
-          <pointCloudCutoff>0.0</pointCloudCutoff>
-          <rangeMax>4.0</rangeMax>
+          <pointCloudCutoff>0.5</pointCloudCutoff>
           <distortionK1>0.00000001</distortionK1>
           <distortionK2>0.00000001</distortionK2>
@@ -49,10 +47,9 @@
         </plugin>
       </sensor>
-      <!-- RGB -->
       <sensor type="depth" name="${name}_frame_sensor">
         <always_on>true</always_on>
-        <update_rate>10.0</update_rate>
+        <update_rate>20.0</update_rate>
         <camera>
-          <horizontal_fov>${50.0 * deg_to_rad}</horizontal_fov>
+          <horizontal_fov>${57.0*M_PI/180.0}</horizontal_fov>
           <image>
             <format>R8G8B8</format>
@@ -61,18 +58,17 @@
           </image>
           <clip>
-            <near>0.1</near>
-            <far>4.0</far>
+            <near>0.01</near>
+            <far>5</far>
           </clip>
         </camera>
         <plugin name="${name}_frame_controller" filename="libgazebo_ros_openni_kinect.so">
           <alwaysOn>true</alwaysOn>
-          <updateRate>10.0</updateRate>
-          <cameraName>softkinetic_camera</cameraName>
-          <imageTopicName>rgb_data/image_raw</imageTopicName>
-          <cameraInfoTopicName>rgb_data/camera_info</cameraInfoTopicName>
-          <pointCloudTopicName>rgbd_data/points</pointCloudTopicName>
+          <updateRate>20.0</updateRate>
+          <cameraName>${name}</cameraName>
+          <imageTopicName>rgb/image_raw</imageTopicName>
+          <pointCloudTopicName>rgb/points</pointCloudTopicName>
+          <cameraInfoTopicName>rgb/camera_info</cameraInfoTopicName>
           <frameName>${name}_optical_frame</frameName>
-          <pointCloudCutoff>0.0</pointCloudCutoff>
-          <rangeMax>4.0</rangeMax>
+          <pointCloudCutoff>0.5</pointCloudCutoff>
           <distortionK1>0.00000001</distortionK1>
           <distortionK2>0.00000001</distortionK2>

File: tiago_description/urdf/sensors/xtion_pro_live.urdf.xacro (robot description, xacro)
@@ -18,10 +18,11 @@
 -->
 <robot xmlns:xacro="http://ros.org/wiki/xacro">
-  <xacro:include filename="$(find ant_description)/urdf/sensors/xtion_pro_live.gazebo.xacro" />
+  <xacro:include filename="$(find tiago_description)/urdf/sensors/openni.gazebo.xacro" />
   <!-- Macro -->
-  <xacro:macro name="xtion_pro_live" params="name parent *origin *optical_origin">
+  <xacro:macro name="xtion_pro_live" params="name parent *origin *calibration_origin">
+    <!-- BEGIN frames in the center of the camera -->
     <joint name="${name}_frame_joint" type="fixed">
       <insert_block name="origin" />
-      <parent link="${parent}_link"/>
+      <parent link="${parent}"/>
       <child link="${name}_link"/>
     </joint>
@@ -37,5 +38,5 @@
         <origin xyz="0 0 0" rpy="0 0 0"/>
         <geometry>
-          <mesh filename="package://ant_description/meshes/sensors/xtion_pro_live/xtion_pro_live.dae" />
+          <mesh filename="package://tiago_description/meshes/sensors/xtion_pro_live/xtion_pro_live.dae" />
         </geometry>
         <material name="Grey">
@@ -51,5 +52,5 @@
     </link>
     <joint name="${name}_optical_joint" type="fixed">
-      <insert_block name="optical_origin" />
+      <insert_block name="calibration_origin" />
       <parent link="${name}_link"/>
       <child link="${name}_optical_frame"/>
@@ -64,4 +65,33 @@
       </inertial>
     </link>
+    <!-- END frames in the center of the camera -->
+    <!-- BEGIN frames of the depth sensor -->
+    <joint name="${name}_depth_joint" type="fixed">
+      <origin xyz="0.0 0.049 0.0" rpy="0 0 0" />
+      <parent link="${name}_link" />
+      <child link="${name}_depth_frame"/>
+    </joint>
+    <link name="${name}_depth_frame"/>
+      <joint name="${name}_depth_optical_joint" type="fixed">
+        <origin xyz="0 0 0" rpy="${-M_PI/2} 0.0 ${-M_PI/2}" />
+        <parent link="${name}_depth_frame" />
+        <child link="${name}_depth_optical_frame"/>
+      </joint>
+    <link name="${name}_depth_optical_frame"/>
+    <!-- END frames of the depth sensor -->
+    <!-- BEGIN frames of the rgb sensor -->
+    <joint name="${name}_rgb_joint" type="fixed">
+      <origin xyz="0.0 0.022 0.0" rpy="0 0 0" />
+      <parent link="${name}_link" />
+      <child link="${name}_rgb_frame"/>
+    </joint>
+    <link name="${name}_rgb_frame"/>
+    <joint name="${name}_rgb_optical_joint" type="fixed">
+      <origin xyz="0 0 0" rpy="${-M_PI/2} 0.0 ${-M_PI/2}" />
+      <parent link="${name}_rgb_frame" />
+      <child link="${name}_rgb_optical_frame"/>
+    </joint>
+    <link name="${name}_rgb_optical_frame"/>
+    <!-- END frames of the rgb sensor -->
     <!-- extensions -->
     <xacro:openni_camera_gazebo_v0 name="${name}" />
