Commit message: added extrinsic camera calibration file changes

File: tiago_description/urdf/sensors/xtion_pro_live.urdf.xacro (robot description, xacro)
@@ -19,4 +19,5 @@
 <robot xmlns:xacro="http://ros.org/wiki/xacro">
   <xacro:include filename="$(find tiago_description)/urdf/sensors/openni.gazebo.xacro" />
+  <xacro:include filename="$(find tiago_description_calibration)/urdf/calibration/extrinsic_camera_calibration_constants.urdf.xacro" />
   <!-- Macro -->
   <xacro:macro name="xtion_pro_live" params="name parent camera_model *origin *optical_origin">
@@ -69,13 +70,5 @@
     <!-- frames of the depth sensor -->
     <joint name="${name}_depth_joint" type="fixed">
-      <xacro:if value="${camera_model == 'orbbec-astra'}">
-        <origin xyz="0.0 0.047 0.0" rpy="0 0 0" />
-      </xacro:if>
-      <xacro:if value="${camera_model == 'orbbec-astra-pro'}">
-        <origin xyz="0.0 0.047 0.0" rpy="0 0 0" />
-      </xacro:if>
-      <xacro:if value="${camera_model == 'asus-xtion'}">
-        <origin xyz="0.0 0.049 0.0" rpy="0 0 0" />
-      </xacro:if>
+      <xacro:camera_baseline_constants camera_model="${camera_model}" />
       <parent link="${name}_link" />
       <child link="${name}_depth_frame"/>
