Commit message: Fix y orientation error

File: tiago_description/urdf/sensors/orbbec_astra.urdf.xacro (robot description, xacro)
@@ -74,5 +74,5 @@
       <!-- This is the real origin as in the robot solidworks, it must match: 0.1015 0.095 0.008 -->
       <!-- Assuming we have 0.0908 0.08 0.0 from default camera_position, and rotated -90 deg on x.-->
-      <origin xyz="0.0107 -0.008 0.015" rpy="0 0 0" />
+      <origin xyz="0.0107 0.008 0.015" rpy="0 0 0" />
       <parent link="${name}_link" />
       <child link="${name}_orbbec_aux_joint_frame"/>

Commit message: depth frame for orbbec is referenced on the rgb frame

File: tiago_description/urdf/sensors/orbbec_astra.urdf.xacro (robot description, xacro)
@@ -90,5 +90,5 @@
     <joint name="${name}_depth_joint" type="fixed">
       <xacro:camera_baseline_constants camera_model="${camera_model}" />
-      <parent link="${name}_orbbec_aux_joint_frame" />
+      <parent link="${name}_rgb_frame" />
       <child link="${name}_depth_frame"/>
     </joint>

Commit message: Updated Changelog

File: tiago_description/urdf/sensors/orbbec_astra.urdf.xacro (robot description, xacro)
@@ -75,5 +75,7 @@
       <!-- This is the real origin as in the robot solidworks, it must match: 0.1015 0.095 0.008 -->
       <!-- Assuming we have 0.0908 0.08 0.0 from default camera_position, and rotated -90 deg on x.-->
-      <origin xyz="0.0107 0.008 0.015" rpy="0 0 0" />
+      <!-- Pending confirmation from Orbbec about the position of the frames, going with old defaults-->
+      <!-- <origin xyz="0.0107 0.008 0.015" rpy="0 0 0" />-->
+      <origin xyz="0 0 0" rpy="0 0 0" />
       <parent link="${name}_link" />
       <child link="${name}_orbbec_aux_joint_frame"/>
@@ -119,5 +121,5 @@
     <!-- frames of the rgb sensor -->
     <joint name="${name}_rgb_joint" type="fixed">
-      <origin xyz="-0.0006 0.0125 -0.015" rpy="0 0 0" />
+      <origin xyz="0.0 0.022 0.0" rpy="0 0 0" />
       <parent link="${name}_orbbec_aux_joint_frame" />
       <child link="${name}_rgb_frame"/>
