Commit message: Add arm and adjust torso

File: tiago_description/robots/tiago_full.urdf.xacro (robot description, xacro)
@@ -17,4 +17,6 @@
   <!-- Torso -->
   <xacro:include filename="$(find tiago_description)/urdf/torso/torso.urdf.xacro" />
+  <!-- Arm -->
+  <xacro:include filename="$(find tiago_description)/urdf/arm/arm.urdf.xacro" />
   <!-- Generic simulator_gazebo plugins -->
   <xacro:include filename="$(find tiago_description)/gazebo/gazebo.urdf.xacro" />
@@ -24,5 +26,6 @@
   <xacro:base name="base"/>
   <xacro:tiago_torso name="torso" parent="base"/>
-  <!--<xacro:reem_head  name="head"  parent="torso_2_link"/>
-  <xacro:reem_arm name="arm" parent="torso_2_link" side="right" reflect="1.0"  /> -->
+  <xacro:tiago_arm name="arm" parent="torso_lift_link"/>
+  <!-- <xacro:tiago_head  name="head"  parent="torso_lift_link"/> -->
+  <!-- <xacro:reem_hand  name="hand"  parent="arm_tool_link"/> -->
 </robot>

File: tiago_description/urdf/arm/arm.transmission.xacro (robot description, xacro)
@@ -8,12 +8,14 @@
 -->
 <robot xmlns:xacro="http://ros.org/wiki/xacro">
-  <xacro:macro name="reem_arm_simple_transmission" params="name side number reduction" >
-    <transmission name="${name}_${side}_${number}_trans">
+  <xacro:macro name="arm_simple_transmission" params="name number reduction" >
+    <transmission name="${name}_${number}_trans">
       <type>transmission_interface/SimpleTransmission</type>
-      <actuator name="${name}_${side}_${number}_motor" >
+      <actuator name="${name}_${number}_motor" >
         <mechanicalReduction>${reduction}</mechanicalReduction>
       </actuator>
-      <joint name="${name}_${side}_${number}_joint">
+      <joint name="${name}_${number}_joint">
         <hardwareInterface>hardware_interface/PositionJointInterface</hardwareInterface>
+        <hardwareInterface>hardware_interface/EffortJointInterface</hardwareInterface>
+        <hardwareInterface>hardware_interface/JointModeInterface</hardwareInterface>
       </joint>
     </transmission>

File: tiago_description/urdf/arm/arm.urdf.xacro (robot description, xacro)
@@ -1,5 +1,5 @@
 <?xml version="1.0"?>
 <!--
-  Copyright (c) 2011-2012, PAL Robotics, S.L.
+  Copyright (c) 2014, PAL Robotics, S.L.
   All rights reserved.
   This work is licensed under the Creative Commons Attribution-NonCommercial-NoDerivs 3.0 Unported License.
@@ -9,7 +9,7 @@
 <robot xmlns:xacro="http://ros.org/wiki/xacro">
   <!--File includes-->
-  <xacro:include filename="$(find reemc_description)/urdf/deg_to_rad.xacro" />
-  <xacro:include filename="$(find reemc_description)/urdf/arm/wrist.urdf.xacro" />
-  <xacro:include filename="$(find reemc_description)/urdf/arm/arm.transmission.xacro" />
+  <xacro:include filename="$(find tiago_description)/urdf/deg_to_rad.xacro" />
+  <xacro:include filename="$(find tiago_description)/urdf/arm/wrist.urdf.xacro" />
+  <xacro:include filename="$(find tiago_description)/urdf/arm/arm.transmission.xacro" />
   <!--Constant parameters-->
   <xacro:property name="arm_friction"       value="1.0" />
@@ -25,15 +25,12 @@
   <xacro:property name="arm_eps"            value="0.02" />
   <!-- TODO: Update dynamic models -->
-  <xacro:macro name="reem_arm" params="name parent side reflect">
+  <xacro:macro name="tiago_arm" params="name parent">
     <!--************************-->
     <!--        SHOULDER        -->
     <!--************************-->
-    <link name="${name}_${side}_1_link">
-      <inertial>
-        <origin xyz="0.00701 -0.00011 ${reflect*0.18627}" rpy="0 0 0"/>
+    <link name="${name}_1_link">
+      <inertial>
+        <origin xyz="0.00 -0.00011 0.18627" rpy="0 0 0"/>
         <mass value="1.53614" />
-<!--        <inertia ixx="0"  ixy="0"  ixz="0" iyy="0" iyz="0" izz="0" /> -->
-<!--         NOTE: Assuming cylinder centered at CoM with r=0.05, h=0.05 with axis parallel to x coordinate -->
-<!--        <inertia ixx="0.0026850"  ixy="0"  ixz="0" iyy="0.0017900" iyz="0" izz="0.0017900" /> -->
         <inertia ixx="0.00327313329"  ixy="-0.00000460054"  ixz="-0.00025121368" iyy="0.00316047802" iyz="0.00000313158" izz="0.00157642528" />
       </inertial>
@@ -41,5 +38,5 @@
         <origin xyz="0 0 0" rpy="0 0 0" />
         <geometry>
-          <mesh filename="package://reemc_description/meshes/arm/arm_1.dae" scale="1 1 ${-1*reflect}"/>
+          <mesh filename="package://tiago_description/meshes/arm/arm_1.dae" scale="1 1 -1"/>
         </geometry>
         <material name="DarkGrey" />
@@ -48,12 +45,12 @@
        <origin xyz="0 0 0" rpy="0 0 0" />
         <geometry>
-          <mesh filename="package://reemc_description/meshes/arm/arm_1_collision.stl" scale="1 1 ${-1*reflect}"/>
-        </geometry>
-      </collision>
-    </link>
-    <joint name="${name}_${side}_1_joint" type="revolute">
+          <mesh filename="package://tiago_description/meshes/arm/arm_1_collision.stl" scale="1 1 -1"/>
+        </geometry>
+      </collision>
+    </link>
+    <joint name="${name}_1_joint" type="revolute">
       <parent link="${parent}" />
-      <child link="${name}_${side}_1_link" />
-      <origin xyz="0 -0.31827 0" rpy="${(-165.0*reflect) * deg_to_rad} 0 0" />
+      <child link="${name}_1_link" />
+      <origin xyz="0.1 0.07 0" rpy="${0 * deg_to_rad} ${0 * deg_to_rad} ${-90 * deg_to_rad}" />
       <axis xyz="0 0 1" />
       <limit lower="${-45.0 * deg_to_rad}" upper="${180.0 * deg_to_rad}" effort="${arm_1_max_effort}" velocity="${arm_1_max_vel}" />
@@ -64,11 +61,8 @@
                          soft_upper_limit="${ 180.0 * deg_to_rad - arm_eps}" />
     </joint>
-   <link name="${name}_${side}_2_link">
-      <inertial>
-        <origin xyz="0.01435 -0.06294 ${reflect*0.01039}" rpy="0 0 0"/>
+   <link name="${name}_2_link">
+      <inertial>
+        <origin xyz="0.01435 -0.06294 ${0.01039}" rpy="0 0 0"/>
         <mass value="1.60393" />
-        <!--<inertia ixx="0"  ixy="0"  ixz="0" iyy="0" iyz="0" izz="0" />-->
-        <!-- NOTE: Assuming cylinder centered at CoM with r=0.05, h=0.05 with axis parallel to y coordinate -->
-        <!-- <inertia ixx="0.0013417"  ixy="0"  ixz="0" iyy="0.0020125" iyz="0" izz="0.0013417" /> -->
         <inertia ixx="0.0046195621"  ixy="-0.00056769245"  ixz="0.00018376961" iyy="0.00185384237" iyz="-0.00078286958" izz="0.0049356022" />
       </inertial>
@@ -76,19 +70,19 @@
         <origin xyz="0 0 0" rpy="0 0 0" />
         <geometry>
-          <mesh filename="package://reemc_description/meshes/arm/arm_2.dae" scale="1 1 ${-1*reflect}"/>
-        </geometry>
-        <material name="DarkGrey" />
-      </visual>
-      <collision>
-        <origin xyz="0 0 0" rpy="0 0 0" />
-        <geometry>
-          <mesh filename="package://reemc_description/meshes/arm/arm_2_collision.stl" scale="1 1 ${-1*reflect}"/>
-        </geometry>
-      </collision>
-    </link>
-    <joint name="${name}_${side}_2_joint" type="revolute">
-      <parent link="${name}_${side}_1_link" />
-      <child link="${name}_${side}_2_link" />
-      <origin xyz="0 0 ${0.21749 * reflect}" rpy="${-90.0 * reflect * deg_to_rad} ${-75.0 * reflect * deg_to_rad} ${90.0 * deg_to_rad}" />
+          <mesh filename="package://tiago_description/meshes/arm/arm_2.dae" scale="1 1 -1"/>
+        </geometry>
+        <material name="DarkGrey" />
+      </visual>
+      <collision>
+        <origin xyz="0 0 0" rpy="0 0 0" />
+        <geometry>
+          <mesh filename="package://tiago_description/meshes/arm/arm_2_collision.stl" scale="1 1 -1"/>
+        </geometry>
+      </collision>
+    </link>
+    <joint name="${name}_2_joint" type="revolute">
+      <parent link="${name}_1_link" />
+      <child link="${name}_2_link" />
+      <origin xyz="0.11 0 -0.08" rpy="${90.0 * deg_to_rad} ${0 * deg_to_rad} ${0 * deg_to_rad}" />
       <axis xyz="0 0 1" />
       <limit lower="${-15.0 * deg_to_rad}" upper="${120.0 * deg_to_rad}" effort="${arm_2_max_effort}" velocity="${arm_2_max_vel}" />
@@ -99,10 +93,8 @@
                          soft_upper_limit="${ 120.0 * deg_to_rad - arm_eps}" />
     </joint>
-    <link name="${name}_${side}_3_link">
-      <inertial>
-        <origin xyz="0.00606 -0.0113 ${reflect * 0.05748}" rpy="0 0 0"/>
+    <link name="${name}_3_link">
+      <inertial>
+        <origin xyz="0.00606 -0.0113 0.05748" rpy="0 0 0"/>
         <mass value="1.64293" />
-        <!--<inertia ixx="0"  ixy="0"  ixz="0" iyy="0" iyz="0" izz="0" />-->
-        <!-- NOTE: Assuming cylinder centered at CoM with r=0.05, h=0.05 with axis parallel to x coordinate -->
          <inertia ixx="0.00372686652"  ixy="-0.00008722874"  ixz="-0.00028800176" iyy="0.00344463026" iyz="0.00042776588" izz="0.00192229026" />
       </inertial>
@@ -110,19 +102,19 @@
         <origin xyz="0 0 0" rpy="0 0 0" />
         <geometry>
-          <mesh filename="package://reemc_description/meshes/arm/arm_3.dae" scale="1 1 ${-1*reflect}"/>
-        </geometry>
-        <material name="DarkGrey" />
-      </visual>
-      <collision>
-        <origin xyz="0 0 0" rpy="0 0 0" />
-        <geometry>
-          <mesh filename="package://reemc_description/meshes/arm/arm_3_collision.stl" scale="1 1 ${-1*reflect}"/>
-        </geometry>
-      </collision>
-    </link>
-    <joint name="${name}_${side}_3_joint" type="revolute">
-      <parent link="${name}_${side}_2_link" />
-      <child link="${name}_${side}_3_link" />
-      <origin xyz="0.02 -0.142 0" rpy="${90.0 * reflect * deg_to_rad} 0 0" />
+          <mesh filename="package://tiago_description/meshes/arm/arm_3.dae" scale="1 1 -1"/>
+        </geometry>
+        <material name="DarkGrey" />
+      </visual>
+      <collision>
+        <origin xyz="0 0 0" rpy="0 0 0" />
+        <geometry>
+          <mesh filename="package://tiago_description/meshes/arm/arm_3_collision.stl" scale="1 1 -1"/>
+        </geometry>
+      </collision>
+    </link>
+    <joint name="${name}_3_joint" type="revolute">
+      <parent link="${name}_2_link" />
+      <child link="${name}_3_link" />
+      <origin xyz="0.142 -0.02 0" rpy="${0.0 * deg_to_rad} ${-90.0 * deg_to_rad} 0" />
       <axis xyz="0 0 1" />
       <limit lower="${-135.0 * deg_to_rad}" upper="${157.5 * deg_to_rad}" effort="${arm_3_max_effort}" velocity="${arm_3_max_vel}" />
@@ -136,11 +128,8 @@
     <!--        ELBOW           -->
     <!--************************-->
-    <link name="${name}_${side}_4_link">
-      <inertial>
-        <origin xyz="-0.04129 0.0118 ${reflect * -0.01387}" rpy="0 0 0"/>
+    <link name="${name}_4_link">
+      <inertial>
+        <origin xyz="-0.04129 0.0118 -0.01387" rpy="0 0 0"/>
         <mass value="1.20222" />
-        <!--<inertia ixx="0"  ixy="0"  ixz="0" iyy="0" iyz="0" izz="0" />-->
-        <!-- NOTE: Assuming cylinder centered at CoM with r=0.05, h=0.05 with axis parallel to x coordinate -->
-        <!-- <inertia ixx="0.0012663"  ixy="0"  ixz="0" iyy="0.00084417" iyz="0" izz="0.00084417" /> -->
         <inertia ixx="0.00156355749"  ixy="-0.000353141"  ixz="0.00053402452" iyy="0.00277186194" iyz="-0.00015541973" izz="0.00307369106" />
       </inertial>
@@ -148,19 +137,19 @@
         <origin xyz="0 0 0" rpy="0 0 0" />
         <geometry>
-          <mesh filename="package://reemc_description/meshes/arm/arm_4.dae" scale="1 1 ${-1*reflect}"/>
-        </geometry>
-        <material name="DarkGrey" />
-      </visual>
-      <collision>
-        <origin xyz="0 0 0" rpy="0 0 0" />
-        <geometry>
-          <mesh filename="package://reemc_description/meshes/arm/arm_4_collision.stl" scale="1 1 ${-1*reflect}"/>
-        </geometry>
-      </collision>
-    </link>
-    <joint name="${name}_${side}_4_joint" type="revolute">
-      <parent link="${name}_${side}_3_link" />
-      <child link="${name}_${side}_4_link" />
-      <origin xyz="0 -0.02 ${0.088 * reflect}" rpy="0 ${90.0 * reflect * deg_to_rad} 0" />
+          <mesh filename="package://tiago_description/meshes/arm/arm_4.dae" scale="1 1 -1"/>
+        </geometry>
+        <material name="DarkGrey" />
+      </visual>
+      <collision>
+        <origin xyz="0 0 0" rpy="0 0 0" />
+        <geometry>
+          <mesh filename="package://tiago_description/meshes/arm/arm_4_collision.stl" scale="1 1 -1"/>
+        </geometry>
+      </collision>
+    </link>
+    <joint name="${name}_4_joint" type="revolute">
+      <parent link="${name}_3_link" />
+      <child link="${name}_4_link" />
+      <origin xyz="0 -0.02 -0.183" rpy="0 ${-90.0 * deg_to_rad} 0" />
       <axis xyz="0 0 1" />
       <limit lower="0" upper="${130.0 * deg_to_rad}" effort="${arm_4_max_effort}" velocity="${arm_4_max_vel}" />
@@ -171,30 +160,30 @@
                          soft_upper_limit="${ 130.0 * deg_to_rad - arm_eps}" />
     </joint>
-   <gazebo reference="${name}_${side}_1_link">
-     <mu1>0.9</mu1>
-     <mu2>0.9</mu2>
-   </gazebo>
-   <gazebo reference="${name}_${side}_2_link">
-     <mu1>0.9</mu1>
-     <mu2>0.9</mu2>
-   </gazebo>
-   <gazebo reference="${name}_${side}_3_link">
-     <mu1>0.9</mu1>
-     <mu2>0.9</mu2>
-   </gazebo>
-   <gazebo reference="${name}_${side}_4_link">
-     <mu1>0.9</mu1>
-     <mu2>0.9</mu2>
-   </gazebo>
-   <gazebo reference="${name}_${side}_1_joint">
-      <implicitSpringDamper>1</implicitSpringDamper>
-   </gazebo>
-   <gazebo reference="${name}_${side}_2_joint">
-      <implicitSpringDamper>1</implicitSpringDamper>
-   </gazebo>
-   <gazebo reference="${name}_${side}_3_joint">
-      <implicitSpringDamper>1</implicitSpringDamper>
-   </gazebo>
-   <gazebo reference="${name}_${side}_4_joint">
+   <gazebo reference="${name}_1_link">
+     <mu1>0.9</mu1>
+     <mu2>0.9</mu2>
+   </gazebo>
+   <gazebo reference="${name}_2_link">
+     <mu1>0.9</mu1>
+     <mu2>0.9</mu2>
+   </gazebo>
+   <gazebo reference="${name}_3_link">
+     <mu1>0.9</mu1>
+     <mu2>0.9</mu2>
+   </gazebo>
+   <gazebo reference="${name}_4_link">
+     <mu1>0.9</mu1>
+     <mu2>0.9</mu2>
+   </gazebo>
+   <gazebo reference="${name}_1_joint">
+      <implicitSpringDamper>1</implicitSpringDamper>
+   </gazebo>
+   <gazebo reference="${name}_2_joint">
+      <implicitSpringDamper>1</implicitSpringDamper>
+   </gazebo>
+   <gazebo reference="${name}_3_joint">
+      <implicitSpringDamper>1</implicitSpringDamper>
+   </gazebo>
+   <gazebo reference="${name}_4_joint">
       <implicitSpringDamper>1</implicitSpringDamper>
    </gazebo>
@@ -202,9 +191,9 @@
     <!--        WRIST           -->
     <!--************************-->
-    <xacro:reem_wrist name="arm" parent="${name}_${side}_4_link" side="${side}" reflect="${reflect}"  />
+    <xacro:wrist name="arm" parent="${name}_4_link" reflect="1"/>
     <!--***********************-->
     <!--        TOOL           -->
     <!--***********************-->
-    <link name="${name}_${side}_tool_link">
+    <link name="${name}_tool_link">
       <inertial>
         <mass value="0.1" />
@@ -225,14 +214,14 @@
       </collision>
     </link>
-    <joint name="${name}_${side}_tool_joint" type="fixed">
-      <parent link="${name}_${side}_7_link" />
-      <child link="${name}_${side}_tool_link" />
-      <origin xyz="0 0 ${reflect * 0.046}" rpy="${90.0 * deg_to_rad} ${-90.0 * reflect * deg_to_rad} 0" />
+    <joint name="${name}_tool_joint" type="fixed">
+      <parent link="${name}_7_link" />
+      <child link="${name}_tool_link" />
+      <origin xyz="0 0 0.046" rpy="${90.0 * deg_to_rad} ${-90.0 * deg_to_rad} 0" />
     </joint>
     <!-- extensions -->
-    <xacro:reem_arm_simple_transmission name="${name}" side="${side}" number="1" reduction="1.0" />
-    <xacro:reem_arm_simple_transmission name="${name}" side="${side}" number="2" reduction="1.0" />
-    <xacro:reem_arm_simple_transmission name="${name}" side="${side}" number="3" reduction="1.0" />
-    <xacro:reem_arm_simple_transmission name="${name}" side="${side}" number="4" reduction="1.0" />
+    <xacro:arm_simple_transmission name="${name}" number="1" reduction="1.0" />
+    <xacro:arm_simple_transmission name="${name}" number="2" reduction="1.0" />
+    <xacro:arm_simple_transmission name="${name}" number="3" reduction="1.0" />
+    <xacro:arm_simple_transmission name="${name}" number="4" reduction="1.0" />
   </xacro:macro>
 </robot>

File: tiago_description/urdf/arm/wrist.urdf.xacro (robot description, xacro)
@@ -9,6 +9,6 @@
 <robot xmlns:xacro="http://ros.org/wiki/xacro">
   <!--File includes-->
-  <xacro:include filename="$(find reemc_description)/urdf/deg_to_rad.xacro" />
-  <xacro:include filename="$(find reemc_description)/urdf/arm/wrist.transmission.xacro" />
+  <xacro:include filename="$(find tiago_description)/urdf/deg_to_rad.xacro" />
+  <xacro:include filename="$(find tiago_description)/urdf/arm/wrist.transmission.xacro" />
   <!--Constant parameters-->
   <xacro:property name="wrist_friction"       value="1.0" />
@@ -22,9 +22,9 @@
   <xacro:property name="wrist_eps"          value="0.02" />
   <!-- TODO: Update dynamic models -->
-  <xacro:macro name="reem_wrist" params="name parent side reflect">
+  <xacro:macro name="wrist" params="name parent reflect">
     <!--************************-->
     <!--        WRIST           -->
     <!--************************-->
-    <link name="${name}_${side}_5_link">
+    <link name="${name}_5_link">
       <inertial>
         <origin xyz="-0.00044 0.00012 ${reflect * 0.07445}" rpy="0 0 0"/>
@@ -38,5 +38,5 @@
         <origin xyz="0 0 0" rpy="0 0 0" />
         <geometry>
-          <mesh filename="package://reemc_description/meshes/arm/arm_5.dae" scale="1 1 ${-1*reflect}"/>
+          <mesh filename="package://tiago_description/meshes/arm/arm_5.dae" scale="1 1 ${-1*reflect}"/>
         </geometry>
         <material name="LightGrey" />
@@ -45,12 +45,12 @@
         <origin xyz="0 0 0" rpy="0 0 0" />
         <geometry>
-          <mesh filename="package://reemc_description/meshes/arm/arm_5_collision.stl" scale="1 1 ${-1*reflect}"/>
+          <mesh filename="package://tiago_description/meshes/arm/arm_5_collision.stl" scale="1 1 ${-1*reflect}"/>
         </geometry>
       </collision>
     </link>
-    <joint name="${name}_${side}_5_joint" type="revolute">
+    <joint name="${name}_5_joint" type="revolute">
       <parent link="${parent}" />
-      <child link="${name}_${side}_5_link" />
-      <origin xyz="-0.088 0.02 0" rpy="0 ${-90.0 * reflect * deg_to_rad} 0" />
+      <child link="${name}_5_link" />
+      <origin xyz="-0.1245 0.02 0" rpy="0 ${-90.0 * deg_to_rad} 0" />
       <axis xyz="0 0 1" />
       <limit lower="${-120.0 * deg_to_rad}" upper="${120.0 * deg_to_rad}" effort="${wrist_1_max_effort}" velocity="${wrist_1_max_vel}" /> <!--TODO: Check effort value!-->
@@ -61,5 +61,5 @@
                          soft_upper_limit="${ 120.0 * deg_to_rad - wrist_eps}" />
     </joint>
-    <link name="${name}_${side}_6_link">
+    <link name="${name}_6_link">
       <inertial>
         <origin xyz="-0.00005 -0.00252 ${reflect * 0.00007}" rpy="0 0 0"/>
@@ -73,5 +73,5 @@
         <origin xyz="0 0 0" rpy="0 0 0" />
         <geometry>
-          <mesh filename="package://reemc_description/meshes/arm/arm_6.dae" scale="1 1 ${-1*reflect}"/>
+          <mesh filename="package://tiago_description/meshes/arm/arm_6.dae" scale="1 1 ${-1*reflect}"/>
         </geometry>
         <material name="LightGrey" />
@@ -84,8 +84,8 @@
       </collision>
     </link>
-    <joint name="${name}_${side}_6_joint" type="revolute">
-      <parent link="${name}_${side}_5_link" />
-      <child link="${name}_${side}_6_link" />
-      <origin xyz="0 0 ${0.15 * reflect}" rpy="${-90.0 * reflect * deg_to_rad} 0 0" />
+    <joint name="${name}_6_joint" type="revolute">
+      <parent link="${name}_5_link" />
+      <child link="${name}_6_link" />
+      <origin xyz="0 0 0.15" rpy="${-90.0 * reflect * deg_to_rad} 0 0" />
       <axis xyz="0 0 1" />
       <limit lower="${-90.0 * deg_to_rad}" upper="${90.0 * deg_to_rad}" effort="${wrist_2_max_effort}" velocity="${wrist_2_max_vel}" />
@@ -96,5 +96,5 @@
                          soft_upper_limit="${ 90.0 * deg_to_rad - wrist_eps}" />
     </joint>
-    <link name="${name}_${side}_7_link">
+    <link name="${name}_7_link">
       <inertial>
         <!--TODO: Verify these inertial parameters-->
@@ -120,7 +120,7 @@
       </collision>
     </link>
-    <joint name="${name}_${side}_7_joint" type="revolute">
-      <parent link="${name}_${side}_6_link" />
-      <child link="${name}_${side}_7_link" />
+    <joint name="${name}_7_joint" type="revolute">
+      <parent link="${name}_6_link" />
+      <child link="${name}_7_link" />
       <origin xyz="0 0 0" rpy="${90.0 * reflect * deg_to_rad} 0 0" />
       <axis xyz="0 0 1" />
@@ -132,28 +132,28 @@
                          soft_upper_limit="${ 120.0 * deg_to_rad - wrist_eps}" />
     </joint>
-    <gazebo reference="${name}_${side}_5_link">
+    <gazebo reference="${name}_5_link">
       <mu1>0.9</mu1>
       <mu2>0.9</mu2>
     </gazebo>
-    <gazebo reference="${name}_${side}_6_link">
+    <gazebo reference="${name}_6_link">
       <mu1>0.9</mu1>
       <mu2>0.9</mu2>
     </gazebo>
-    <gazebo reference="${name}_${side}_7_link">
+    <gazebo reference="${name}_7_link">
       <mu1>0.9</mu1>
       <mu2>0.9</mu2>
     </gazebo>
-    <gazebo reference="${name}_${side}_5_joint">
+    <gazebo reference="${name}_5_joint">
         <implicitSpringDamper>1</implicitSpringDamper>
     </gazebo>
-    <gazebo reference="${name}_${side}_6_joint">
+    <gazebo reference="${name}_6_joint">
         <implicitSpringDamper>1</implicitSpringDamper>
     </gazebo>
-    <gazebo reference="${name}_${side}_7_joint">
+    <gazebo reference="${name}_7_joint">
         <implicitSpringDamper>1</implicitSpringDamper>
     </gazebo>
     <!-- extensions -->
-    <xacro:reem_wrist_simple_transmission name="${name}" side="${side}" number="5" reduction="1.0" />
-    <xacro:reem_wrist_differential_transmission name="${name}" side="${side}" number_1="6" number_2="7"
+    <xacro:wrist_simple_transmission name="${name}" number="5" reduction="1.0" />
+    <xacro:wrist_differential_transmission name="${name}" number_1="6" number_2="7"
                                                 act_reduction_1="-1.0" act_reduction_2="1.0"
                                                 jnt_reduction_1="-1.0" jnt_reduction_2="${-reflect}" />

File: tiago_description/urdf/torso/torso.urdf.xacro (robot description, xacro)
@@ -30,5 +30,5 @@
   </link>
   <joint name="${name}_fixed_joint" type="fixed">
-    <origin rpy="0 0 0" xyz="0 0 0.3" />
+    <origin rpy="0 0 0" xyz="-0.053 0 0.3" />
     <parent link="${parent}_link" />
     <child link="${name}_fixed_link" />
