Commit message: Add hey5 hand to tiago

File: tiago_description/robots/tiago_full.urdf.xacro (robot description, xacro)
@@ -19,4 +19,6 @@
   <!-- Arm -->
   <xacro:include filename="$(find tiago_description)/urdf/arm/arm.urdf.xacro" />
+  <!-- Hand -->
+  <xacro:include filename="$(find hey5_description)/urdf/hey5_hand.urdf.xacro" />
   <!-- Generic simulator_gazebo plugins -->
   <xacro:include filename="$(find tiago_description)/gazebo/gazebo.urdf.xacro" />
@@ -28,4 +30,6 @@
   <xacro:tiago_arm name="arm" parent="torso_lift_link"/>
   <!-- <xacro:tiago_head  name="head"  parent="torso_lift_link"/> -->
-  <!-- <xacro:reem_hand  name="hand"  parent="arm_tool_link"/> -->
+  <xacro:hey5_hand parent="arm_tool_link" name="hand" reflect="1">
+    <origin xyz="0 0 0" rpy="0 0 0"/>
+  </xacro:hey5_hand>
 </robot>

File: tiago_description/urdf/arm/arm.urdf.xacro (robot description, xacro)
@@ -217,5 +217,5 @@
       <parent link="${name}_7_link" />
       <child link="${name}_tool_link" />
-      <origin xyz="0 0 0.046" rpy="${90.0 * deg_to_rad} ${-90.0 * deg_to_rad} 0" />
+      <origin xyz="0 0 0.046" rpy="${90.0 * deg_to_rad} ${-90.0 * deg_to_rad} ${180 * deg_to_rad}" />
     </joint>
     <!-- extensions -->

File: tiago_description/urdf/arm/wrist.urdf.xacro (robot description, xacro)
@@ -52,5 +52,5 @@
       <parent link="${parent}" />
       <child link="${name}_5_link" />
-      <origin xyz="-0.1245 0.02 0" rpy="0 ${-90.0 * deg_to_rad} 0" />
+      <origin xyz="-0.1245 0.02 0" rpy="${-90 * deg_to_rad} ${180 * deg_to_rad} ${90 * deg_to_rad}" />
       <axis xyz="0 0 1" />
       <limit lower="${-120.0 * deg_to_rad}" upper="${120.0 * deg_to_rad}" effort="${wrist_1_max_effort}" velocity="${wrist_1_max_vel}" /> <!--TODO: Check effort value!-->

Commit message: Add preliminary head

File: tiago_description/robots/tiago_full.urdf.xacro (robot description, xacro)
@@ -21,4 +21,6 @@
   <!-- Hand -->
   <xacro:include filename="$(find hey5_description)/urdf/hey5_hand.urdf.xacro" />
+  <!-- Head -->
+  <xacro:include filename="$(find tiago_description)/urdf/head/head.urdf.xacro" />
   <!-- Generic simulator_gazebo plugins -->
   <xacro:include filename="$(find tiago_description)/gazebo/gazebo.urdf.xacro" />
@@ -28,4 +30,5 @@
   <xacro:base name="base"/>
   <xacro:tiago_torso name="torso" parent="base"/>
+  <xacro:head name="head" parent="torso_lift_link"/>
   <xacro:tiago_arm name="arm" parent="torso_lift_link"/>
   <!-- <xacro:tiago_head  name="head"  parent="torso_lift_link"/> -->

File: tiago_description/urdf/head/head.urdf.xacro (robot description, xacro)
@@ -11,5 +11,5 @@
   <xacro:include filename="$(find tiago_description)/urdf/deg_to_rad.xacro" />
   <xacro:include filename="$(find tiago_description)/urdf/head/head.transmission.xacro" />
-  <xacro:include filename="$(find tiago_description)/urdf/sensors/range.urdf.xacro" />
+  <xacro:include filename="$(find tiago_description)/urdf/sensors/xtion_pro_live.urdf.xacro" />
   <!--Constant parameters-->
   <xacro:property name="head_friction" value="1.0" />
@@ -20,25 +20,24 @@
   <!--     HEAD_1 (PAN)       -->
   <!--************************-->
-  <xacro:macro name="reem_head_1" params="name parent">
+  <xacro:macro name="head_1" params="name parent">
     <link name="${name}_link">
       <inertial>
         <origin xyz="0.01819	0.00248	-0.00517" rpy="0 0 0" />
         <mass value="1.11967" />
-        <!-- NOTE: Assuming cylinder with r=0.06, h=0.08 -->
-<!--         <inertia ixx="0.0014125"  ixy="0"  ixz="0" iyy="0.0014125" iyz="0" izz="0.0017738" /> -->
         <inertia ixx="0.00111370229"  ixy="0.00003992198"  ixz="-0.00012464155" iyy="0.00111361487" iyz="0.00001943162" izz="0.00114794061" />
       </inertial>
       <visual>
-        <origin rpy="0 0 0" xyz="-0.03 0 0"/> <!--TODO: Remove offset when good meshes arrive-->
+        <origin rpy="0 0 0" xyz="0.03 0 0"/>
         <geometry>
-          <mesh filename="package://reemc_description/meshes/head/head_1.dae" />
+          <box size="0.06 0.04 0.04"/>
         </geometry>
-        <material name="DarkGrey" />
+        <material name="Grey" />
       </visual>
       <collision>
-        <origin xyz="-0.03 0 0" rpy="0 0 0" />
+        <origin xyz="0.03 0 0" rpy="0 0 0" />
         <geometry>
-          <mesh filename="package://reemc_description/meshes/head/head_1_collision.stl" />
+          <box size="0.06 0.04 0.04"/>
         </geometry>
+        <material name="Grey" />
       </collision>
     </link>
@@ -46,5 +45,5 @@
       <parent link="${parent}"/>
       <child link="${name}_link"/>
-      <origin xyz="0.0 -0.42316 0" rpy="${90.0 * deg_to_rad} 0 0" />
+      <origin xyz="0 0 0.04" rpy="${0.0 * deg_to_rad} 0 0" />
       <axis xyz="0 0 1" />
       <limit lower="${-75.0 * deg_to_rad}" upper="${75.0 * deg_to_rad}" effort="3.4" velocity="${head_max_vel}" />
@@ -68,26 +67,24 @@
   <!--      HEAD_2 (TILT)     -->
   <!--************************-->
-  <xacro:macro name="reem_head_2" params="name parent">
+  <xacro:macro name="head_2" params="name parent">
     <link name="${name}_link">
       <inertial>
         <origin xyz="0.01183 -0.08098 0.00104" rpy="0 0 0" />
         <mass value="1.63134" />
-        <!-- NOTE: Assuming box with d=0.28433, w=0.20302, h=0.26741 -->
-<!--         <inertia ixx="0.011353"  ixy="0"  ixz="0" iyy="0.012294" iyz="0" izz="0.015345" /> -->
-        <!--NOTE: Low (0.1 or lower) diagonal inertia values make Gazebo 1.0.2 simulation unstable when head sensors are added.-->
         <inertia ixx="0.00640199093"  ixy="0.00012197067"  ixz="-0.00000897011" iyy="0.00676228591" iyz="-0.0000552329" izz="0.00614192438" />
       </inertial>
       <visual>
-        <origin rpy="0 0 0" xyz="-0.03 0 0"/> <!--TODO: Remove offset when good meshes arrive-->
+        <origin xyz="-0.035 0 0" rpy="0 0 0"/>
         <geometry>
-          <mesh filename="package://reemc_description/meshes/head/head_2.dae" />
+          <box size="0.035 0.035 0.05"/>
         </geometry>
-        <material name="LightGrey" />
+        <material name="DarkGrey" />
       </visual>
       <collision>
-        <origin xyz="-0.03 0 0" rpy="0 0 0" />
+        <origin xyz="-0.035 0 0" rpy="0 0 0" />
         <geometry>
-          <mesh filename="package://reemc_description/meshes/head/head_2_collision.stl" />
+          <box size="0.035 0.035 0.05"/>
         </geometry>
+        <material name="DarkGrey" />
       </collision>
     </link>
@@ -95,5 +92,5 @@
       <parent link="${parent}"/>
         <child link="${name}_link"/>
-      <origin xyz="0.0445 0 0" rpy="${-90.0 * deg_to_rad} 0 0" />
+      <origin xyz="0.0845 0 0.03" rpy="${-90.0 * deg_to_rad} 0 0" />
       <axis xyz="0 0 1" />
       <limit lower="${-15.0 * deg_to_rad}" upper="${45.0 * deg_to_rad}" effort="3.26" velocity="${head_max_vel}" />
@@ -105,7 +102,11 @@
     </joint>
   </xacro:macro>
-  <xacro:macro name="reem_head" params="name parent">
-    <xacro:reem_head_1 name="${name}_1" parent="${parent}" />
-    <xacro:reem_head_2 name="${name}_2" parent="${name}_1_link"/>
+  <xacro:macro name="head" params="name parent">
+    <xacro:head_1 name="${name}_1" parent="${parent}" />
+    <xacro:head_2 name="${name}_2" parent="${name}_1_link"/>
+    <xacro:xtion_pro_live name="xtion" parent="${name}_2">
+      <origin xyz="0 -0.03 0" rpy="${90 * deg_to_rad} 0 0" />
+      <origin xyz="0 -0.03 0" rpy="${90 * deg_to_rad} 0 0" />
+    </xacro:xtion_pro_live>
   </xacro:macro>
 </robot>

Commit message: Update inertias, Center of Mass' and related pids Hand commented until it works on gazebo

File: tiago_description/robots/tiago_full.urdf.xacro (robot description, xacro)
@@ -32,7 +32,8 @@
   <xacro:head name="head" parent="torso_lift_link"/>
   <xacro:tiago_arm name="arm" parent="torso_lift_link"/>
-  <!-- <xacro:tiago_head  name="head"  parent="torso_lift_link"/> -->
+  <!--
   <xacro:hey5_hand parent="arm_tool_link" name="hand" reflect="1">
     <origin xyz="0 0 0" rpy="0 0 0"/>
   </xacro:hey5_hand>
+  -->
 </robot>

File: tiago_description/urdf/arm/arm.urdf.xacro (robot description, xacro)
@@ -31,7 +31,7 @@
     <link name="${name}_1_link">
       <inertial>
-        <origin xyz="0.00 -0.00011 0.18627" rpy="0 0 0"/>
-        <mass value="1.53614" />
-        <inertia ixx="0.00327313329"  ixy="-0.00000460054"  ixz="-0.00025121368" iyy="0.00316047802" iyz="0.00000313158" izz="0.00157642528" />
+        <origin xyz="0.08375 0.00308 -0.04965" rpy="0 0 0"/>
+        <mass value="2.64731" />
+        <inertia ixx="0.01488823102"  ixy="0.00097928027"  ixz="-0.014599404" iyy="0.03785812845" iyz="-0.0008663619" izz="0.0261720489" />
       </inertial>
       <!-- M90 module -->
@@ -89,5 +89,5 @@
       <safety_controller k_position="20"
                          k_velocity="20"
-                         soft_lower_limit="${0 * deg_to_rad  + arm_eps}"
+                         soft_lower_limit="${0 * deg_to_rad}"
                          soft_upper_limit="${180.0 * deg_to_rad - arm_eps}" />
     </joint>
@@ -95,6 +95,6 @@
       <inertial>
         <origin xyz="0.01435 -0.06294 ${0.01039}" rpy="0 0 0"/>
-        <mass value="1.60393" />
-        <inertia ixx="0.0046195621"  ixy="-0.00056769245"  ixz="0.00018376961" iyy="0.00185384237" iyz="-0.00078286958" izz="0.0049356022" />
+        <mass value="1.58751" />
+        <inertia ixx="0.002253374"  ixy="-0.00185617271"  ixz="0.00023094382" iyy="0.01079198201" iyz="-0.00004741252" izz="0.0112248261" />
       </inertial>
       <visual>
@@ -126,7 +126,7 @@
     <link name="${name}_3_link">
       <inertial>
-        <origin xyz="0.00606 -0.0113 0.05748" rpy="0 0 0"/>
-        <mass value="1.64293" />
-         <inertia ixx="0.00372686652"  ixy="-0.00008722874"  ixz="-0.00028800176" iyy="0.00344463026" iyz="0.00042776588" izz="0.00192229026" />
+        <origin xyz="0.00557 -0.01042 -0.10388" rpy="0 0 0"/>
+        <mass value="1.79881" />
+         <inertia ixx="0.02682610467"  ixy="-0.00019692212"  ixz="-0.0015045329" iyy="0.02638053578" iyz="0.00263989274" izz="0.002385016" />
       </inertial>
       <visual>
@@ -175,7 +175,7 @@
     <link name="${name}_4_link">
       <inertial>
-        <origin xyz="-0.04129 0.0118 -0.01387" rpy="0 0 0"/>
-        <mass value="1.20222" />
-        <inertia ixx="0.00156355749"  ixy="-0.000353141"  ixz="0.00053402452" iyy="0.00277186194" iyz="-0.00015541973" izz="0.00307369106" />
+        <origin xyz="-0.06578 0.0126 0.01194" rpy="0 0 0"/>
+        <mass value="1.35076" />
+        <inertia ixx="0.00220509703"  ixy="-0.00165490069" ixz="-0.0002277335" iyy="0.01177626386" iyz="0.00003472435" izz="0.0120918757" />
       </inertial>
       <visual>

File: tiago_description/urdf/arm/wrist.urdf.xacro (robot description, xacro)
@@ -28,10 +28,7 @@
     <link name="${name}_5_link">
       <inertial>
-        <origin xyz="-0.00044 0.00012 ${reflect * 0.07445}" rpy="0 0 0"/>
-        <mass value="1.21524" />
-        <!-- <inertia ixx="0"  ixy="0"  ixz="0" iyy="0" iyz="0" izz="0" /> -->
-        <!-- NOTE: Assuming cylinder centered at CoM with r=0.05, h=0.1 with axis parallel to z coordinate -->
-<!--         <inertia ixx="0.0027096"  ixy="0"  ixz="0" iyy="0.0027096" iyz="0" izz="0.0023225" /> -->
-      <inertia ixx="0.00193499547"  ixy="-0.00000027528"  ixz="-0.00001268153" iyy="0.00177767506" iyz="-0.00000466638" izz="0.00057101196" />
+        <origin xyz="-0.00084 0.00001 ${reflect * 0.07797}" rpy="0 0 0"/>
+        <mass value="1.32698" />
+        <inertia ixx="0.01049566566"  ixy="-0.00000316264"  ixz="-0.00012548144" iyy="0.01028836655" iyz="0.0000027891" izz="0.00094419873" />
       </inertial>
       <visual>
@@ -63,10 +60,7 @@
     <link name="${name}_6_link">
       <inertial>
-        <origin xyz="-0.00005 -0.00252 ${reflect * 0.00007}" rpy="0 0 0"/>
-        <mass value="0.41597" />
-        <!-- <inertia ixx="0"  ixy="0"  ixz="0" iyy="0" iyz="0" izz="0" /> -->
-        <!-- NOTE: Assuming cylinder centered at CoM with r=0.02, h=0.08 with axis parallel to z coordinate -->
-<!--         <inertia ixx="0.0001615"  ixy="0"  ixz="0" iyy="0.0001615" iyz="0" izz="0.000051" /> -->
-         <inertia ixx="0.00020339659"  ixy="-0.00000071703"  ixz="-0.00000006654" iyy="0.00015240261" iyz="0.00000014315" izz="0.0001671881" />
+        <origin xyz="-0.000014 -0.00368 ${reflect * 0.00001}" rpy="0 0 0"/>
+        <mass value="0.35781" />
+         <inertia ixx="0.00016489507"  ixy="0.0000002779"  ixz="0.00000009308" iyy="0.00013154987" iyz="0.00000007106" izz="0.00011998795" />
       </inertial>
       <visual>
@@ -98,11 +92,7 @@
     <link name="${name}_7_link">
       <inertial>
-        <!--TODO: Verify these inertial parameters-->
-        <origin xyz="-0.00004 0 ${reflect * -0.02887}" rpy="0 0 0"/>
-        <mass value="0.06697" />
-       <!-- <inertia ixx="0"  ixy="0"  ixz="0" iyy="0" iyz="0" izz="0" /> -->
-        <!-- NOTE: Assuming point mass -->
-<!--         <inertia ixx="0"  ixy="0"  ixz="0" iyy="0" iyz="0" izz="0" /> -->
-         <inertia ixx="0.0000123718"  ixy="0.00000000002"  ixz="0.00000002403" iyy="0.00001242132" iyz="0.00000000001" izz="0.0000059514" />
+        <origin xyz="0 -0.00005 ${reflect * -0.01573}" rpy="0 0 0"/>
+        <mass value="0.10721" />
+         <inertia ixx="0.00008977003"  ixy="-0.00000000001"  ixz="0.0" iyy="0.00008968773" iyz="-0.00000021816" izz="0.00000951878" />
       </inertial>
       <visual>

File: tiago_description/urdf/head/head.urdf.xacro (robot description, xacro)
@@ -23,7 +23,7 @@
     <link name="${name}_link">
       <inertial>
-        <origin xyz="0.01819	0.00248	-0.00517" rpy="0 0 0" />
-        <mass value="1.11967" />
-        <inertia ixx="0.00111370229"  ixy="0.00003992198"  ixz="-0.00012464155" iyy="0.00111361487" iyz="0.00001943162" izz="0.00114794061" />
+        <origin xyz="0.0208 -0.00025 0.0215" rpy="0 0 0" />
+        <mass value="0.09793" />
+        <inertia ixx="0.00005844626"  ixy="-0.00000051494"  ixz="0.00004662971" iyy="0.00001161435" iyz="0.0" izz="0.00005236593" />
       </inertial>
       <visual>
@@ -47,5 +47,5 @@
       <origin xyz="0.193 0 0.04" rpy="${0.0 * deg_to_rad} 0 0" />
       <axis xyz="0 0 1" />
-      <limit lower="${-90.0 * deg_to_rad}" upper="${90.0 * deg_to_rad}" effort="3.4" velocity="${head_max_vel}" />
+      <limit lower="${-90.0 * deg_to_rad}" upper="${90.0 * deg_to_rad}" effort="5.197" velocity="${head_max_vel}" />
       <dynamics damping="${head_damping}" friction="${head_friction}"/>
       <safety_controller k_position="20"
@@ -70,7 +70,7 @@
     <link name="${name}_link">
       <inertial>
-        <origin xyz="0.01183 -0.08098 0.00104" rpy="0 0 0" />
-        <mass value="1.63134" />
-        <inertia ixx="0.00640199093"  ixy="0.00012197067"  ixz="-0.00000897011" iyy="0.00676228591" iyz="-0.0000552329" izz="0.00614192438" />
+        <origin xyz="0.04149 -0.01221 0.001" rpy="0 0 0" />
+        <mass value="0.24875" />
+        <inertia ixx="0.0000498057"  ixy="-0.00012697329"  ixz="0.00000011444" iyy="0.00044922137" iyz="-0.00000065525" izz="0.00048113173" />
       </inertial>
     </link>
@@ -80,5 +80,5 @@
       <origin xyz="0.0355 0 0.023" rpy="${-90.0 * deg_to_rad} 0 0" />
       <axis xyz="0 0 1" />
-      <limit lower="${-90 * deg_to_rad}" upper="${45.0 * deg_to_rad}" effort="3.26" velocity="${head_max_vel}" />
+      <limit lower="${-90 * deg_to_rad}" upper="${45.0 * deg_to_rad}" effort="2.77" velocity="${head_max_vel}" />
       <dynamics damping="${head_damping}" friction="${head_friction}"/>
       <safety_controller k_position="20"

File: tiago_description/urdf/torso/torso.urdf.xacro (robot description, xacro)
@@ -10,9 +10,9 @@
   <link name="${name}_fixed_link">
     <inertial>
-      <origin rpy="0 0 0" xyz="0.053 0.55187 -0.00188" />
-      <mass value="7.19400" />
-      <inertia ixx="0.16941095831" ixy="-0.00114443001"   ixz="0.00090167218"
-               iyy="0.15113888533" iyz="-0.00744737659"
-               izz="0.04165307088" />
+      <origin rpy="0 0 0" xyz="0.00635 -0.01673 0.10662" />
+      <mass value="14.52876" />
+      <inertia ixx="0.17621875653" ixy="-0.00154333947"   ixz="0.00980172504"
+               iyy="0.18995293862" iyz="-0.0259201152"
+               izz="0.03571737542" />
     </inertial>
   <visual>
@@ -39,9 +39,9 @@
   <link name="${name}_lift_link">
     <inertial>
-      <origin rpy="0 0 0" xyz="-0.060142360276412 0.00304133533168627 0.343272867034157" />
-      <mass value="10.81628746254819" />
-      <inertia ixx="0.0641960264706125" ixy="0.001128617953499" ixz="0.00203364821006436"
-               iyy="0.061658561971383" iyz="-3.14401755382909E-05"
-               izz="0.0376084656328484" />
+      <origin rpy="0 0 0" xyz="0.02909 0.01068 -0.14826" />
+      <mass value="8.62177" />
+      <inertia ixx="0.19639986797" ixy="0.00528625771" ixz="-0.04018414421"
+               iyy="0.212736527" iyz="-0.01564349386"
+               izz="0.02479371908" />
     </inertial>
     <!-- Lifting body -->
@@ -81,5 +81,5 @@
     <child link="${name}_lift_link" />
     <axis xyz="0 0 1" />
-    <limit effort="450" lower="0.0" upper="0.35" velocity="0.1" />
+    <limit effort="2000" lower="0.0" upper="0.35" velocity="0.01" />
     <calibration rising="0.0" />
     <dynamics damping="1000" />

Commit message: Don't append _link to parent value

File: tiago_description/robots/tiago_full.urdf.xacro (robot description, xacro)
@@ -29,5 +29,5 @@
   <!-- Now we can start using the macros included above to define the actual robot -->
   <xacro:base name="base"/>
-  <xacro:tiago_torso name="torso" parent="base"/>
+  <xacro:tiago_torso name="torso" parent="base_link"/>
   <xacro:head name="head" parent="torso_lift_link"/>
   <xacro:tiago_arm name="arm" parent="torso_lift_link"/>

File: tiago_description/urdf/torso/torso.urdf.xacro (robot description, xacro)
@@ -33,5 +33,5 @@
   <joint name="${name}_fixed_joint" type="fixed">
     <origin rpy="0 0 0" xyz="-0.068 0 0.2235" />
-    <parent link="${parent}_link" />
+    <parent link="${parent}" />
     <child link="${name}_fixed_link" />
     <axis xyz="0 0 0" />
