Commit message: Add safety box around the hand

File: tiago_description/robots/tiago_titanium.urdf.xacro (robot description, xacro)
@@ -32,3 +32,29 @@
     <origin xyz="0 0 0" rpy="0 0 0"/>
   </xacro:hey5_hand>
+  <joint name="hand_safety_box_joint" type="fixed">
+    <parent link="arm_tool_link"/>
+    <child link="hand_safety_box"/>
+    <origin xyz="0.1 0.02 0.02" rpy="0 0 0"/>
+  </joint>
+  <link name="hand_safety_box">
+    <inertial>
+      <origin xyz="0 0 0" rpy="0 0 0"/>
+      <mass value="0.0001" />
+      <inertia ixx="0.0001"  ixy="0"  ixz="0" iyy="0.0001" iyz="0" izz="0.0001" />
+    </inertial>
+    <!--
+    <visual>
+      <origin xyz="0 0 0" rpy="0 0 0" />
+      <geometry>
+        <box size="0.2 0.115 0.18" />
+      </geometry>
+    </visual>
+    -->
+    <collision>
+      <origin xyz="0 0 0" rpy="0 0 0" />
+      <geometry>
+        <box size="0.2 0.115 0.18" />
+      </geometry>
+    </collision>
+  </link>
 </robot>

Commit message: Add force torque sensor

File: tiago_description/robots/tiago_titanium.urdf.xacro (robot description, xacro)
@@ -24,4 +24,6 @@
   <!-- Materials for visualization -->
   <xacro:include filename="$(find tiago_description)/urdf/materials.urdf.xacro" />
+  <!-- Force Torque sensor -->
+  <xacro:include filename="$(find tiago_description)/urdf/sensors/ftsensor.urdf.xacro" />
   <!-- Now we can start using the macros included above to define the actual robot -->
   <xacro:base_sensors name="base" hokuyo="false" sick551="false" sick561="true" sick571="false" sonars="false" microphone="false"/>
@@ -29,9 +31,10 @@
   <xacro:head name="head" parent="torso_lift_link"/>
   <xacro:tiago_arm name="arm" parent="torso_lift_link"/>
-  <xacro:hey5_hand parent="arm_tool_link" name="hand" reflect="1">
+  <xacro:ft_sensor name="wrist" parent="arm_tool_link" />
+  <xacro:hey5_hand parent="wrist_ft_tool_link" name="hand" reflect="1">
     <origin xyz="0 0 0" rpy="0 0 0"/>
   </xacro:hey5_hand>
   <joint name="hand_safety_box_joint" type="fixed">
-    <parent link="arm_tool_link"/>
+    <parent link="wrist_ft_tool_link"/>
     <child link="hand_safety_box"/>
     <origin xyz="0.1 0.02 0.02" rpy="0 0 0"/>
