Commit message: fixes #13516

File: tiago_description/robots/tiago_steel.urdf.xacro (robot description, xacro)
@@ -28,5 +28,5 @@
   <xacro:tiago_torso name="torso" parent="base_link"/>
   <xacro:head name="head" parent="torso_lift_link"/>
-  <xacro:tiago_arm name="arm" parent="torso_lift_link"/>
+  <xacro:tiago_arm name="arm" parent="torso_lift_link" wrist_6_range="90.0"/>
   <xacro:tiago_gripper parent="arm_tool_link" name="gripper">
     <origin xyz="0 0 0" rpy="${90*deg_to_rad} 0 0"/>

File: tiago_description/robots/tiago_titanium.urdf.xacro (robot description, xacro)
@@ -28,5 +28,5 @@
   <xacro:tiago_torso name="torso" parent="base_link"/>
   <xacro:head name="head" parent="torso_lift_link"/>
-  <xacro:tiago_arm name="arm" parent="torso_lift_link"/>
+  <xacro:tiago_arm name="arm" parent="torso_lift_link" wrist_6_range="81"/>
   <xacro:hey5_hand parent="arm_tool_link" name="hand" reflect="1">
     <origin xyz="0 0 0" rpy="0 0 0"/>

File: tiago_description/robots/tiago_titanium_chessboard.urdf.xacro (robot description, xacro)
@@ -28,5 +28,5 @@
   <xacro:tiago_torso name="torso" parent="base_link"/>
   <xacro:head name="head" parent="torso_lift_link"/>
-  <xacro:tiago_arm name="arm" parent="torso_lift_link"/>
+  <xacro:tiago_arm name="arm" parent="torso_lift_link" wrist_6_range="81"/>
   <!-- <xacro:hey5_hand parent="arm_tool_link" name="hand" reflect="1">
     <origin xyz="0 0 0" rpy="0 0 0"/>

File: tiago_description/urdf/arm/arm.urdf.xacro (robot description, xacro)
@@ -24,5 +24,5 @@
   <xacro:property name="arm_4_max_effort"   value="17.86" />
   <xacro:property name="arm_eps"            value="0.02" />
-  <xacro:macro name="tiago_arm" params="name parent">
+  <xacro:macro name="tiago_arm" params="name parent wrist_6_range">
     <!--************************-->
     <!--        SHOULDER        -->
@@ -211,5 +211,5 @@
     <!--        WRIST           -->
     <!--************************-->
-    <xacro:wrist name="arm" parent="${name}_4_link" reflect="1"/>
+    <xacro:wrist name="arm" parent="${name}_4_link" reflect="1" wrist_6_range="${wrist_6_range}"/>
     <!--***********************-->
     <!--        TOOL           -->

File: tiago_description/urdf/arm/wrist.urdf.xacro (robot description, xacro)
@@ -21,5 +21,5 @@
   <xacro:property name="wrist_3_max_effort"   value="6.6" />
   <xacro:property name="wrist_eps"          value="0.02" />
-  <xacro:macro name="wrist" params="name parent reflect">
+  <xacro:macro name="wrist" params="name parent reflect wrist_6_range">
     <!--************************-->
     <!--        WRIST           -->
@@ -86,10 +86,10 @@
       <origin xyz="0 0 0.15" rpy="${0.0 * deg_to_rad} ${-90.0 * deg_to_rad} ${-90.0 * deg_to_rad}" />
       <axis xyz="0 0 1" />
-      <limit lower="${-90.0 * deg_to_rad}" upper="${90.0 * deg_to_rad}" effort="${wrist_2_max_effort}" velocity="${wrist_2_max_vel}" />
+      <limit lower="${-wrist_6_range * deg_to_rad}" upper="${wrist_6_range * deg_to_rad}" effort="${wrist_2_max_effort}" velocity="${wrist_2_max_vel}" />
       <dynamics friction="${wrist_friction}" damping="${wrist_damping}"/>
       <safety_controller k_position="20"
                          k_velocity="20"
-                         soft_lower_limit="${-90.0 * deg_to_rad + wrist_eps}"
-                         soft_upper_limit="${ 90.0 * deg_to_rad - wrist_eps}" />
+                         soft_lower_limit="${-wrist_6_range * deg_to_rad + wrist_eps}"
+                         soft_upper_limit="${ wrist_6_range * deg_to_rad - wrist_eps}" />
     </joint>
     <link name="${name}_7_link">

Commit message: Changed previous gripper to newer one

File: tiago_description/robots/tiago_steel.urdf.xacro (robot description, xacro)
@@ -19,5 +19,5 @@
   <xacro:include filename="$(find tiago_description)/urdf/head/head.urdf.xacro" />
   <!-- Gripper -->
-  <xacro:include filename="$(find tiago_description)/urdf/gripper/gripper.urdf.xacro" />
+  <xacro:include filename="$(find pal_gripper_description)/urdf/gripper.urdf.xacro" />
   <!-- Generic simulator_gazebo plugins -->
   <xacro:include filename="$(find tiago_description)/gazebo/gazebo.urdf.xacro" />
@@ -29,6 +29,6 @@
   <xacro:head name="head" parent="torso_lift_link"/>
   <xacro:tiago_arm name="arm" parent="torso_lift_link" wrist_6_range="90.0"/>
-  <xacro:tiago_gripper parent="arm_tool_link" name="gripper">
-    <origin xyz="0 0 0" rpy="${90*deg_to_rad} 0 0"/>
-  </xacro:tiago_gripper>
+  <xacro:pal_gripper parent="arm_tool_link" name="gripper">
+    <origin xyz="0.01 0 0" rpy="${90*deg_to_rad} 0 ${-90*deg_to_rad}"/>
+  </xacro:pal_gripper>
 </robot>

Commit message: Corrected the pose of the gripper

File: tiago_description/robots/tiago_steel.urdf.xacro (robot description, xacro)
@@ -30,5 +30,5 @@
   <xacro:tiago_arm name="arm" parent="torso_lift_link" wrist_6_range="90.0"/>
   <xacro:pal_gripper parent="arm_tool_link" name="gripper">
-    <origin xyz="0.01 0 0" rpy="${90*deg_to_rad} 0 ${-90*deg_to_rad}"/>
+    <origin xyz="0.01 0 0" rpy="${90*deg_to_rad} ${90*deg_to_rad} ${-90*deg_to_rad}"/>
   </xacro:pal_gripper>
 </robot>
