Commit message: Updated changelog

File: tiago_description/robots/tiago_titanium_chessboard.urdf.xacro (robot description, xacro)
@@ -34,4 +34,4 @@
   <!-- Chessboard for eye-hand calibration -->
   <xacro:include filename="$(find tiago_description)/urdf/chessboard/chessboard.urdf.xacro" />
-  <xacro:chessboard name="arm_chessboard" parent="arm_7_link" origin="0 -0.10 0.19" rpy="1.5708  -0   1.5708"/>
+  <xacro:chessboard name="arm_chessboard" parent="arm_7_link" origin="-0.1 0.0 0.19" rpy="1.5708  -0   0"/>
 </robot>

File: tiago_description/urdf/chessboard/chessboard.urdf.xacro (robot description, xacro)
@@ -22,4 +22,11 @@
         <material name="DarkGrey" />
       </visual>
+      <collision>
+        <origin xyz="0 0 0" rpy="0 0 0" />
+        <geometry>
+          <mesh filename="package://tiago_description/meshes/chessboard/chessboard.dae"/>
+        </geometry>
+        <material name="DarkGrey" />
+      </collision>
     </link>
     <joint name="${name}_joint" type="fixed">
