Commit message: add fingertip force sensors

File: tiago_description/robots/tiago_schunk.urdf.xacro (robot description, xacro)
@@ -24,4 +24,6 @@
   <!-- Gripper -->
   <xacro:include filename="$(find pal_wsg_gripper_description)/urdf/gripper.urdf.xacro" />
+  <!-- Fingertips sensors -->
+  <xacro:include filename="$(find pal_wsg_gripper_description)/urdf/fingertip_sensor.urdf.xacro" />
   <!-- Generic simulator_gazebo plugins -->
   <xacro:include filename="$(find tiago_description)/gazebo/gazebo.urdf.xacro" />
@@ -36,3 +38,10 @@
     <origin xyz="0.01 0 0" rpy="${90*deg_to_rad} ${90*deg_to_rad} ${-90*deg_to_rad}"/>
   </xacro:pal_wsg_gripper>
+  <!-- Fingertip sensors -->
+  <xacro:fingertip_sensor name="gripper_left" parent="gripper_left_finger">
+    <origin xyz="0.035 0 -0.1465" rpy="0 ${-90*deg_to_rad} 0"/>
+  </xacro:fingertip_sensor>
+  <xacro:fingertip_sensor name="gripper_right" parent="gripper_right_finger">
+    <origin xyz="-0.035 0 -0.1465" rpy="0 ${90*deg_to_rad} 0"/>
+  </xacro:fingertip_sensor>
 </robot>
