Commit message: Add head and migrate controller launch

File: tiago_description/robots/tiago.urdf.xacro (robot description, xacro)
@@ -13,4 +13,5 @@
     <xacro:arg name="ft_sensor" default="schunk-ft"/> <!-- false, schunk-ft -->
     <xacro:arg name="laser_model" default="sick-571"/> <!-- false, hokuyo, sick-551, sick-561, sick-571-->
+    <xacro:arg name="camera_model" default="orbbec-astra"/> <!-- false, orbbec-astra, orbbec-astra-pro, asus-xtion -->
     <xacro:arg name="has_thermal_camera" default="false"/>
     <xacro:arg name="multiple" default="false"/>
@@ -18,6 +19,20 @@
     <xacro:property name="end_effector" value="$(arg end_effector)" />
     <xacro:property name="ft_sensor" value="$(arg ft_sensor)" />
+    <xacro:property name="laser_model" value="$(arg laser_model)" />
+    <xacro:property name="camera_model" value="$(arg camera_model)" />
     <xacro:property name="is_multiple" value="$(arg multiple)" />
     <xacro:property name="nsp" value="$(arg namespace)" />
+  <xacro:if value="${end_effector not in ['false', 'pal-gripper', 'pal-hey5', 'schunk-wsg']}">
+    <xacro:wrong_end_effector/>
+  </xacro:if>
+  <xacro:if value="${ft_sensor not in ['false', 'schunk-ft']}">
+    <xacro:wrong_ft_sensor/>
+  </xacro:if>
+  <xacro:if value="${laser_model not in ['false', 'sick-551', 'sick-561', 'sick-571', 'hokuyo']}">
+    <xacro:wrong_laser_model/>
+  </xacro:if>
+  <xacro:if value="${camera_model not in ['false', 'orbbec-astra', 'orbbec-astra-pro', 'asus-xtion']}">
+    <xacro:wrong_camera_model/>
+  </xacro:if>
         <!-- The properties below are modified using empy http://www.alcyone.com/software/empy/
              from the create_robot.py tool. Handle them with care -->
@@ -66,5 +81,5 @@
   <xacro:base_sensors name="base" laser_model="$(arg laser_model)" sonars="true" microphone="true"/>
   <xacro:tiago_torso name="torso" parent="base_link"/>
-  <xacro:head name="head" parent="torso_lift_link"/>
+  <xacro:head name="head" parent="torso_lift_link" camera_model="$(arg camera_model)"/>
   <xacro:if value="${has_arm}">
 	  <xacro:tiago_arm name="arm" parent="torso_lift_link" wrist_6_range="${wrist_6_range}"/>

File: tiago_description/urdf/head/head.urdf.xacro (robot description, xacro)
@@ -111,8 +111,8 @@
     <xacro:head_transmission name="${name}" reduction="1" offset_value="${head_2_joint_offset}"/>
   </xacro:macro>
-  <xacro:macro name="head" params="name parent">
+  <xacro:macro name="head" params="name parent camera_model">
     <xacro:head_1 name="${name}_1" parent="${parent}" />
     <xacro:head_2 name="${name}_2" parent="${name}_1_link"/>
-    <xacro:xtion_pro_live name="xtion" parent="${name}_2">
+    <xacro:xtion_pro_live name="xtion" parent="${name}_2" camera_model="${camera_model}">
       <origin xyz="${camera_position_x} ${camera_position_y} ${camera_position_z}" rpy="${camera_orientation_r} ${camera_orientation_p} ${camera_orientation_y}" />
       <!-- optical origin -->

File: tiago_description/urdf/sensors/xtion_pro_live.urdf.xacro (robot description, xacro)
@@ -20,5 +20,5 @@
   <xacro:include filename="$(find tiago_description)/urdf/sensors/openni.gazebo.xacro" />
   <!-- Macro -->
-  <xacro:macro name="xtion_pro_live" params="name parent *origin *optical_origin">
+  <xacro:macro name="xtion_pro_live" params="name parent camera_model *origin *optical_origin">
     <!-- frames in the center of the camera -->
     <joint name="${name}_joint" type="fixed">
@@ -69,5 +69,13 @@
     <!-- frames of the depth sensor -->
     <joint name="${name}_depth_joint" type="fixed">
-      <origin xyz="0.0 0.049 0.0" rpy="0 0 0" />
+      <xacro:if value="${camera_model == 'orbbec-astra'}">
+        <origin xyz="0.0 0.047 0.0" rpy="0 0 0" />
+      </xacro:if>
+      <xacro:if value="${camera_model == 'orbbec-astra-pro'}">
+        <origin xyz="0.0 0.047 0.0" rpy="0 0 0" />
+      </xacro:if>
+      <xacro:if value="${camera_model == 'asus-xtion'}">
+        <origin xyz="0.0 0.049 0.0" rpy="0 0 0" />
+      </xacro:if>
       <parent link="${name}_link" />
       <child link="${name}_depth_frame"/>

Commit message: Move end_effector xacro code for reusing

File: tiago_description/robots/tiago.urdf.xacro (robot description, xacro)
@@ -38,10 +38,8 @@
              from the create_robot.py tool. Handle them with care -->
    <property name="has_arm"                 value="$(arg arm)"/>
-   <property name="has_hey5"                value="${end_effector == 'pal-hey5'}"/>
-   <property name="has_gripper"             value="${end_effector == 'pal-gripper'}"/>
-   <property name="has_schunk_wsg"          value="${end_effector == 'schunk-wsg'}"/>
    <property name="has_schunk_ft"           value="${ft_sensor == 'schunk-ft'}"/>
    <property name="has_ft_sensor"           value="${has_schunk_ft}"/> <!-- This should be OR'ed with other FT sensors-->
    <property name="end_effector_link"       value="${'wrist_ft_tool_link' if has_ft_sensor else 'arm_tool_link'}"/>
+   <property name="end_effector_name"       value="${'hand' if end_effector == 'pal-hey5' else 'gripper'}"/>
    <property name="wrist_6_range"           value="${ 81 if has_ft_sensor else 90 }"/>
    <property name="head_link_name"          value="head_2_link"/>
@@ -54,17 +52,5 @@
     <!-- Arm -->
     <xacro:include filename="$(find tiago_description)/urdf/arm/arm.urdf.xacro" />
-  </xacro:if>
-  <!-- Hand -->
-  <xacro:if value="${has_hey5}">
-    <xacro:include filename="$(find hey5_description)/urdf/hey5_hand.urdf.xacro" />
-  </xacro:if>
-  <!-- Gripper -->
-  <xacro:if value="${has_gripper}">
-   <xacro:include filename="$(find pal_gripper_description)/urdf/gripper.urdf.xacro" />
-  </xacro:if>
-  <!-- Schunk WSG -->
-  <xacro:if value="${has_schunk_wsg}">
-      <xacro:include filename="$(find pal_wsg_gripper_description)/urdf/gripper.urdf.xacro" />
-      <xacro:include filename="$(find pal_wsg_gripper_description)/urdf/fingertip_sensor.urdf.xacro" />
+    <xacro:include filename="$(find tiago_description)/urdf/end_effector/end_effector.urdf.xacro" />
   </xacro:if>
   <!-- Force Torque sensor -->
@@ -84,59 +70,9 @@
   <xacro:if value="${has_arm}">
 	  <xacro:tiago_arm name="arm" parent="torso_lift_link" wrist_6_range="${wrist_6_range}"/>
+      <xacro:tiago_end_effector name="${end_effector_name}" parent="${end_effector_link}" type="${end_effector}" reflect="1"/>
   </xacro:if>
   <!-- Force Torque sensor -->
   <xacro:if value="${has_ft_sensor}">
       <xacro:ft_sensor name="wrist" parent="arm_tool_link" />
-  </xacro:if>
-  <!-- Gripper -->
-  <xacro:if value="${has_gripper}">
-      <xacro:pal_gripper parent="${end_effector_link}" name="gripper">
-        <origin xyz="0.01 0 0" rpy="${90*deg_to_rad} ${90*deg_to_rad} ${-90*deg_to_rad}"/>
-      </xacro:pal_gripper>
-  </xacro:if>
-  <!-- Schunk WSG -->
-  <xacro:if value="${has_schunk_wsg}">
-      <xacro:pal_wsg_gripper parent="${end_effector_link}" name="gripper">
-        <origin xyz="0.01 0 0" rpy="${90*deg_to_rad} ${90*deg_to_rad} ${-90*deg_to_rad}"/>
-      </xacro:pal_wsg_gripper>
-      <!-- Fingertip sensors -->
-      <xacro:fingertip_sensor name="gripper_left" parent="gripper_left_finger">
-        <origin xyz="0.035 0 -0.1465" rpy="0 ${-90*deg_to_rad} 0"/>
-      </xacro:fingertip_sensor>
-      <xacro:fingertip_sensor name="gripper_right" parent="gripper_right_finger">
-        <origin xyz="-0.035 0 -0.1465" rpy="0 ${90*deg_to_rad} 0"/>
-      </xacro:fingertip_sensor>
-  </xacro:if>
-  <!-- Hand -->
-  <xacro:if value="${has_hey5}">
-          <xacro:hey5_hand parent="${end_effector_link}" name="hand" reflect="1">
-		<origin xyz="0 0 0" rpy="0 0 0"/>
-	  </xacro:hey5_hand>
-	  <joint name="hand_safety_box_joint" type="fixed">
-		<parent link="${end_effector_link}"/>
-		<child link="hand_safety_box"/>
-		<origin xyz="0.1 0.02 0.02" rpy="0 0 0"/>
-	  </joint>
-	  <link name="hand_safety_box">
-		<inertial>
-		  <origin xyz="0 0 0" rpy="0 0 0"/>
-		  <mass value="0.0001" />
-		  <inertia ixx="0.0001"  ixy="0"  ixz="0" iyy="0.0001" iyz="0" izz="0.0001" />
-		</inertial>
-		<!--
-		<visual>
-		  <origin xyz="0 0 0" rpy="0 0 0" />
-		  <geometry>
-		    <box size="0.2 0.115 0.18" />
-		  </geometry>
-		</visual>
-		-->
-		<collision>
-		  <origin xyz="0 0 0" rpy="0 0 0" />
-		  <geometry>
-		    <box size="0.2 0.115 0.18" />
-		  </geometry>
-		</collision>
-	  </link>
   </xacro:if>
   <!-- Thermal camera -->

Commit message: Parametrize arm origin

File: tiago_description/robots/tiago.urdf.xacro (robot description, xacro)
@@ -69,5 +69,7 @@
   <xacro:head name="head" parent="torso_lift_link" camera_model="$(arg camera_model)"/>
   <xacro:if value="${has_arm}">
-	  <xacro:tiago_arm name="arm" parent="torso_lift_link" wrist_6_range="${wrist_6_range}"/>
+	  <xacro:tiago_arm name="arm" parent="torso_lift_link" wrist_6_range="${wrist_6_range}">
+        <origin xyz="0.15505 0.014 -0.151" rpy="0 0 ${-90 * deg_to_rad}" />
+      </xacro:tiago_arm>
       <xacro:tiago_end_effector name="${end_effector_name}" parent="${end_effector_link}" type="${end_effector}" reflect="1"/>
   </xacro:if>

File: tiago_description/urdf/arm/arm.urdf.xacro (robot description, xacro)
@@ -25,5 +25,5 @@
   <xacro:property name="arm_4_max_effort"   value="17.86" />
   <xacro:property name="arm_eps"            value="0.07" />
-  <xacro:macro name="tiago_arm" params="name parent wrist_6_range">
+  <xacro:macro name="tiago_arm" params="name parent wrist_6_range *origin">
     <!--************************-->
     <!--        SHOULDER        -->
@@ -55,5 +55,5 @@
       <parent link="${parent}" />
       <child link="${name}_1_link" />
-      <origin xyz="0.15505 0.014 -0.151" rpy="0 0 ${-90 * deg_to_rad}" />
+      <xacro:insert_block name="origin"/>
       <axis xyz="0 0 1" />
       <limit lower="${0.0 * deg_to_rad}" upper="${157.5 * deg_to_rad}" effort="${arm_1_max_effort}" velocity="${arm_1_max_vel}" />
@@ -209,5 +209,5 @@
     <!--        WRIST           -->
     <!--************************-->
-    <xacro:wrist name="arm" parent="${name}_4_link" reflect="1" wrist_6_range="${wrist_6_range}"/>
+   <xacro:wrist name="${name}" parent="${name}_4_link" reflect="1" wrist_6_range="${wrist_6_range}"/>
     <!--***********************-->
     <!--        TOOL           -->

Commit message: Fix xacro warnings

File: tiago_description/robots/tiago.urdf.xacro (robot description, xacro)
@@ -37,11 +37,11 @@
         <!-- The properties below are modified using empy http://www.alcyone.com/software/empy/
              from the create_robot.py tool. Handle them with care -->
-   <property name="has_arm"                 value="$(arg arm)"/>
-   <property name="has_schunk_ft"           value="${ft_sensor == 'schunk-ft'}"/>
-   <property name="has_ft_sensor"           value="${has_schunk_ft}"/> <!-- This should be OR'ed with other FT sensors-->
-   <property name="end_effector_link"       value="${'wrist_ft_tool_link' if has_ft_sensor else 'arm_tool_link'}"/>
-   <property name="end_effector_name"       value="${'hand' if end_effector == 'pal-hey5' else 'gripper'}"/>
-   <property name="wrist_6_range"           value="${ 81 if has_ft_sensor else 90 }"/>
-   <property name="head_link_name"          value="head_2_link"/>
+   <xacro:property name="has_arm"                 value="$(arg arm)"/>
+   <xacro:property name="has_schunk_ft"           value="${ft_sensor == 'schunk-ft'}"/>
+   <xacro:property name="has_ft_sensor"           value="${has_schunk_ft}"/> <!-- This should be OR'ed with other FT sensors-->
+   <xacro:property name="end_effector_link"       value="${'wrist_ft_tool_link' if has_ft_sensor else 'arm_tool_link'}"/>
+   <xacro:property name="end_effector_name"       value="${'hand' if end_effector == 'pal-hey5' else 'gripper'}"/>
+   <xacro:property name="wrist_6_range"           value="${ 81 if has_ft_sensor else 90 }"/>
+   <xacro:property name="head_link_name"          value="head_2_link"/>
   <!-- The following included files set up definitions of parts of the robot body -->
   <!-- Base -->

Commit message: Fixes for tiago dual

File: tiago_description/robots/tiago.urdf.xacro (robot description, xacro)
@@ -69,5 +69,5 @@
   <xacro:head name="head" parent="torso_lift_link" camera_model="$(arg camera_model)"/>
   <xacro:if value="${has_arm}">
-	  <xacro:tiago_arm name="arm" parent="torso_lift_link" wrist_6_range="${wrist_6_range}">
+	  <xacro:tiago_arm name="arm" parent="torso_lift_link" wrist_6_range="${wrist_6_range}" reflect="1">
         <origin xyz="0.15505 0.014 -0.151" rpy="0 0 ${-90 * deg_to_rad}" />
       </xacro:tiago_arm>

File: tiago_description/urdf/arm/arm.urdf.xacro (robot description, xacro)
@@ -25,5 +25,6 @@
   <xacro:property name="arm_4_max_effort"   value="17.86" />
   <xacro:property name="arm_eps"            value="0.07" />
-  <xacro:macro name="tiago_arm" params="name parent wrist_6_range *origin">
+  <!-- reflect: Set to 1 for a right arm, or to -1 for a left arm-->
+  <xacro:macro name="tiago_arm" params="name parent wrist_6_range reflect *origin">
     <!--************************-->
     <!--        SHOULDER        -->
@@ -126,5 +127,5 @@
       <parent link="${name}_2_link" />
       <child link="${name}_3_link" />
-      <origin xyz="0.0895 0.0 0.0015"
+      <origin xyz="0.0895 0.0 ${reflect*0.0015}"
               rpy="${-90.0 * deg_to_rad} ${0.0 * deg_to_rad} ${90.0 * deg_to_rad}"/>
       <axis xyz="0 0 1" />
@@ -209,5 +210,5 @@
     <!--        WRIST           -->
     <!--************************-->
-   <xacro:wrist name="${name}" parent="${name}_4_link" reflect="1" wrist_6_range="${wrist_6_range}"/>
+   <xacro:wrist name="${name}" parent="${name}_4_link" reflect="${reflect}" wrist_6_range="${wrist_6_range}"/>
     <!--***********************-->
     <!--        TOOL           -->

File: tiago_description/urdf/arm/wrist.urdf.xacro (robot description, xacro)
@@ -50,5 +50,5 @@
       <parent link="${parent}" />
       <child link="${name}_5_link" />
-      <origin xyz="-0.162 0.02 0.027" rpy="${0.0 * deg_to_rad} ${-90.0 * deg_to_rad} ${0.0 * deg_to_rad}" />
+      <origin xyz="-0.162 0.02 0.027" rpy="${90.0 * deg_to_rad} ${reflect * -90.0 * deg_to_rad} ${-90.0 * deg_to_rad}" />
       <axis xyz="0 0 1" />
       <limit lower="${-120.0 * deg_to_rad}" upper="${120.0 * deg_to_rad}" effort="${wrist_1_max_effort}" velocity="${wrist_1_max_vel}" />

Commit message: Modify arm 1, 2 and 3 for TIAGo Dual

File: tiago_description/robots/tiago.urdf.xacro (robot description, xacro)
@@ -69,5 +69,5 @@
   <xacro:head name="head" parent="torso_lift_link" camera_model="$(arg camera_model)"/>
   <xacro:if value="${has_arm}">
-	  <xacro:tiago_arm name="arm" parent="torso_lift_link" wrist_6_range="${wrist_6_range}" reflect="1">
+	  <xacro:tiago_arm name="arm" parent="torso_lift_link" wrist_6_range="${wrist_6_range}" reflect="1" tiago_dual="-1">
         <origin xyz="0.15505 0.014 -0.151" rpy="0 0 ${-90 * deg_to_rad}" />
       </xacro:tiago_arm>

File: tiago_description/urdf/arm/arm.urdf.xacro (robot description, xacro)
@@ -26,5 +26,6 @@
   <xacro:property name="arm_eps"            value="0.07" />
   <!-- reflect: Set to 1 for a right arm, or to -1 for a left arm-->
-  <xacro:macro name="tiago_arm" params="name parent wrist_6_range reflect *origin">
+  <!-- tiago_dual: Set to 1 for tiago dual, -1 for original tiago, changes joints 1 and 2 -->
+  <xacro:macro name="tiago_arm" params="name parent wrist_6_range reflect tiago_dual *origin">
     <!--************************-->
     <!--        SHOULDER        -->
@@ -43,5 +44,5 @@
         <origin xyz="0 0 0" rpy="0 0 0" />
         <geometry>
-          <mesh filename="package://tiago_description/meshes/arm/arm_1.stl" scale="1 1 ${reflect}"/>
+          <mesh filename="package://tiago_description/meshes/arm/arm_1.stl" scale="1 ${-1 * tiago_dual} ${reflect}"/>
         </geometry>
         <material name="White"/>
@@ -50,5 +51,5 @@
         <origin xyz="0 0 0" rpy="0 0 0" />
         <geometry>
-          <mesh filename="package://tiago_description/meshes/arm/arm_1_collision.dae" scale="1 1 ${reflect}"/>
+          <mesh filename="package://tiago_description/meshes/arm/arm_1_collision.dae" scale="1 ${-1 * tiago_dual} ${reflect}"/>
         </geometry>
       </collision>
@@ -59,10 +60,12 @@
       <xacro:insert_block name="origin"/>
       <axis xyz="0 0 1" />
-      <limit lower="${0.0 * deg_to_rad}" upper="${157.5 * deg_to_rad}" effort="${arm_1_max_effort}" velocity="${arm_1_max_vel}" />
-      <dynamics friction="${arm_friction}" damping="${arm_damping}"/>
-      <safety_controller k_position="20"
-                         k_velocity="20"
-                         soft_lower_limit="${0.0 * deg_to_rad + arm_eps}"
-                         soft_upper_limit="${157.5 * deg_to_rad - arm_eps}" />
+      <xacro:property name="arm_1_upper_limit"       value="${180.0 if tiago_dual == 1 else 157.5}"/>
+      <xacro:property name="arm_1_lower_limit"       value="${22.5 if tiago_dual == 1 else 0.0}"/>
+      <limit lower="${arm_1_lower_limit * deg_to_rad}" upper="${arm_1_upper_limit * deg_to_rad}" effort="${arm_1_max_effort}" velocity="${arm_1_max_vel}" />
+      <dynamics friction="${arm_friction}" damping="${arm_damping}"/>
+      <safety_controller k_position="20"
+                         k_velocity="20"
+                         soft_lower_limit="${arm_1_lower_limit * deg_to_rad + arm_eps}"
+                         soft_upper_limit="${arm_1_upper_limit * deg_to_rad - arm_eps}" />
     </joint>
    <link name="${name}_2_link">
@@ -93,13 +96,14 @@
       <parent link="${name}_1_link" />
       <child link="${name}_2_link" />
-      <origin xyz="0.125 0.0195 ${reflect * -0.031}"
-              rpy="${reflect * 90.0 * deg_to_rad} 0.0 0.0"/>
-      <axis xyz="0 0 1" />
-      <limit lower="${-90.0 * deg_to_rad}" upper="${62.5 * deg_to_rad}" effort="${arm_2_max_effort}" velocity="${arm_2_max_vel}" />
+      <origin xyz="0.125 ${tiago_dual * -0.0195} ${reflect * -0.031}"
+              rpy="${reflect * tiago_dual * -90.0 * deg_to_rad} 0.0 0.0"/>
+      <axis xyz="0 0 1" />
+      <xacro:property name="arm_2_upper_limit"       value="${90.0 if tiago_dual == 1 else 62.5}"/>
+      <limit lower="${-90.0 * deg_to_rad}" upper="${arm_2_upper_limit * deg_to_rad}" effort="${arm_2_max_effort}" velocity="${arm_2_max_vel}" />
       <dynamics friction="${arm_friction}" damping="${arm_damping}"/>
       <safety_controller k_position="20"
                          k_velocity="20"
                          soft_lower_limit="${-90.0 * deg_to_rad  + arm_eps}"
-                         soft_upper_limit="${ 62.5 * deg_to_rad - arm_eps}" />
+                         soft_upper_limit="${ arm_2_upper_limit * deg_to_rad - arm_eps}" />
     </joint>
     <link name="${name}_3_link">
@@ -131,10 +135,12 @@
               rpy="${-90.0 * deg_to_rad} ${(90.0 - reflect * 90.0) * deg_to_rad} ${reflect * 90.0 * deg_to_rad}"/>
       <axis xyz="0 0 1" />
-      <limit lower="${-202.5 * deg_to_rad}" upper="${90.0 * deg_to_rad}" effort="${arm_3_max_effort}" velocity="${arm_3_max_vel}" />
-      <dynamics friction="${arm_friction}" damping="${arm_damping}"/>
-      <safety_controller k_position="20"
-                         k_velocity="20"
-                         soft_lower_limit="${-202.5 * deg_to_rad + arm_eps}"
-                         soft_upper_limit="${ 90.0 * deg_to_rad - arm_eps}" />
+      <xacro:property name="arm_3_lower_limit"       value="${-45. if tiago_dual == 1 else -202.5}"/>
+      <xacro:property name="arm_3_upper_limit"       value="${225 if tiago_dual == 1 else 90.0}"/>
+      <limit lower="${arm_3_lower_limit * deg_to_rad}" upper="${arm_3_upper_limit * deg_to_rad}" effort="${arm_3_max_effort}" velocity="${arm_3_max_vel}" />
+      <dynamics friction="${arm_friction}" damping="${arm_damping}"/>
+      <safety_controller k_position="20"
+                         k_velocity="20"
+                         soft_lower_limit="${arm_3_lower_limit * deg_to_rad + arm_eps}"
+                         soft_upper_limit="${ arm_3_upper_limit * deg_to_rad - arm_eps}" />
     </joint>
     <!--************************-->
