Commit message: parse arm joint offsets through the macro

File: tiago_description/robots/tiago.urdf.xacro (robot description, xacro)
@@ -53,4 +53,5 @@
     <xacro:include filename="$(find tiago_description)/urdf/arm/arm.urdf.xacro" />
     <xacro:include filename="$(find tiago_description)/urdf/end_effector/end_effector.urdf.xacro" />
+    <xacro:include filename="$(find tiago_description_calibration)/urdf/calibration/calibration_constants.urdf.xacro" />
   </xacro:if>
   <!-- Force Torque sensor -->
@@ -69,5 +70,5 @@
   <xacro:head name="head" parent="torso_lift_link" camera_model="$(arg camera_model)"/>
   <xacro:if value="${has_arm}">
-	  <xacro:tiago_arm name="arm" parent="torso_lift_link" wrist_6_range="${wrist_6_range}" reflect="1" tiago_dual="-1">
+	  <xacro:tiago_arm name="arm" parent="torso_lift_link" wrist_6_range="${wrist_6_range}" reflect="1" tiago_dual="-1" arm_1_offset="${arm_1_joint_offset}" arm_2_offset="${arm_2_joint_offset}" arm_3_offset="${arm_3_joint_offset}" arm_4_offset="${arm_4_joint_offset}" arm_5_offset="${arm_5_joint_offset}" arm_6_offset="${arm_6_joint_offset}" arm_7_offset="${arm_7_joint_offset}">
         <origin xyz="0.15505 0.014 -0.151" rpy="0 0 ${-90 * deg_to_rad}" />
       </xacro:tiago_arm>

File: tiago_description/urdf/arm/arm.urdf.xacro (robot description, xacro)
@@ -12,5 +12,4 @@
   <xacro:include filename="$(find tiago_description)/urdf/arm/wrist.urdf.xacro" />
   <xacro:include filename="$(find tiago_description)/urdf/arm/arm.transmission.xacro" />
-  <xacro:include filename="$(find tiago_description_calibration)/urdf/calibration/calibration_constants.urdf.xacro" />
   <!--Constant parameters-->
   <xacro:property name="arm_friction"       value="1.0" />
@@ -27,5 +26,5 @@
   <!-- reflect: Set to 1 for a right arm, or to -1 for a left arm-->
   <!-- tiago_dual: Set to 1 for tiago dual, -1 for original tiago, changes joints 1 and 2 -->
-  <xacro:macro name="tiago_arm" params="name parent wrist_6_range reflect tiago_dual *origin">
+  <xacro:macro name="tiago_arm" params="name parent wrist_6_range reflect tiago_dual *origin arm_1_offset arm_2_offset arm_3_offset arm_4_offset arm_5_offset arm_6_offset arm_7_offset">
     <!--************************-->
     <!--        SHOULDER        -->
@@ -218,5 +217,5 @@
     <!--        WRIST           -->
     <!--************************-->
-   <xacro:wrist name="${name}" parent="${name}_4_link" reflect="${reflect}" wrist_6_range="${wrist_6_range}"/>
+   <xacro:wrist name="${name}" parent="${name}_4_link" reflect="${reflect}" wrist_6_range="${wrist_6_range}" arm_5_offset="${arm_5_offset}" arm_6_offset="${arm_6_offset}" arm_7_offset="${arm_7_offset}"/>
     <!--***********************-->
     <!--        TOOL           -->
@@ -247,8 +246,8 @@
     </joint>
     <!-- extensions -->
-    <xacro:arm_simple_transmission name="${name}" number="1" reduction="1.0" offset_value="$${${name}_1_joint_offset}"/>
-    <xacro:arm_simple_transmission name="${name}" number="2" reduction="1.0" offset_value="$${${name}_2_joint_offset}"/>
-    <xacro:arm_simple_transmission name="${name}" number="3" reduction="1.0" offset_value="$${${name}_3_joint_offset}"/>
-    <xacro:arm_simple_transmission name="${name}" number="4" reduction="1.0" offset_value="$${${name}_4_joint_offset}"/>
+    <xacro:arm_simple_transmission name="${name}" number="1" reduction="1.0" offset_value="${arm_1_offset}"/>
+    <xacro:arm_simple_transmission name="${name}" number="2" reduction="1.0" offset_value="${arm_2_offset}"/>
+    <xacro:arm_simple_transmission name="${name}" number="3" reduction="1.0" offset_value="${arm_3_offset}"/>
+    <xacro:arm_simple_transmission name="${name}" number="4" reduction="1.0" offset_value="${arm_4_offset}"/>
   </xacro:macro>
 </robot>

File: tiago_description/urdf/arm/wrist.transmission.xacro (robot description, xacro)
@@ -9,7 +9,5 @@
 -->
 <robot xmlns:xacro="http://ros.org/wiki/xacro">
-  <!--File includes-->
-  <xacro:include filename="$(find tiago_description_calibration)/urdf/calibration/calibration_constants.urdf.xacro" />
-  <xacro:macro name="wrist_simple_transmission" params="name number reduction" >
+  <xacro:macro name="wrist_simple_transmission" params="name number reduction offset" >
     <transmission name="${name}_${number}_trans">
       <type>transmission_interface/SimpleTransmission</type>
@@ -18,5 +16,5 @@
       </actuator>
       <joint name="${name}_${number}_joint">
-        <offset>$${${name}_${number}_joint_offset}</offset>
+        <offset>${offset}</offset>
         <hardwareInterface>hardware_interface/JointStateInterface</hardwareInterface>
         <hardwareInterface>hardware_interface/PositionJointInterface</hardwareInterface>
@@ -26,5 +24,5 @@
   </xacro:macro>
   <xacro:macro name="wrist_differential_transmission"
-               params="name number_1 number_2 act_reduction_1 act_reduction_2 jnt_reduction_1 jnt_reduction_2" >
+               params="name number_1 number_2 act_reduction_1 act_reduction_2 jnt_reduction_1 jnt_reduction_2 number_1_offset number_2_offset" >
   <transmission name="${name}_wrist_trans">
       <type>transmission_interface/DifferentialTransmission</type>
@@ -39,5 +37,5 @@
       <joint name="${name}_${number_1}_joint">
         <role>joint1</role>
-        <offset>$${${name}_${number_1}_joint_offset}</offset>
+        <offset>${number_1_offset}</offset>
         <mechanicalReduction>${jnt_reduction_1}</mechanicalReduction>
         <hardwareInterface>hardware_interface/JointStateInterface</hardwareInterface>
@@ -48,5 +46,5 @@
       <joint name="${name}_${number_2}_joint">
         <role>joint2</role>
-        <offset>$${${name}_${number_2}_joint_offset}</offset>
+        <offset>${number_2_offset}</offset>
         <mechanicalReduction>${jnt_reduction_2}</mechanicalReduction>
         <hardwareInterface>hardware_interface/JointStateInterface</hardwareInterface>

File: tiago_description/urdf/arm/wrist.urdf.xacro (robot description, xacro)
@@ -21,5 +21,5 @@
   <xacro:property name="wrist_3_max_effort"   value="6.6" />
   <xacro:property name="wrist_eps"          value="0.02" />
-  <xacro:macro name="wrist" params="name parent reflect wrist_6_range">
+  <xacro:macro name="wrist" params="name parent reflect wrist_6_range arm_5_offset arm_6_offset arm_7_offset">
     <!--************************-->
     <!--        WRIST           -->
@@ -137,8 +137,9 @@
     </gazebo>
     <!-- extensions -->
-    <xacro:wrist_simple_transmission name="${name}" number="5" reduction="1.0" />
+    <xacro:wrist_simple_transmission name="${name}" number="5" reduction="1.0" offset="${arm_5_offset}"/>
     <xacro:wrist_differential_transmission name="${name}" number_1="6" number_2="7"
                                                 act_reduction_1="-1.0" act_reduction_2="1.0"
-                                                jnt_reduction_1="1.0" jnt_reduction_2="${-reflect}" />
+                                                jnt_reduction_1="1.0" jnt_reduction_2="${-reflect}"
+                                                number_1_offset="${arm_6_offset}" number_2_offset="${arm_7_offset}"/>
   </xacro:macro>
 </robot>

File: tiago_description/urdf/head/head.urdf.xacro (robot description, xacro)
@@ -69,5 +69,5 @@
     </gazebo>
     <!-- extensions -->
-    <xacro:head_transmission name="${name}" reduction="1" offset_value="$${${name}_joint_offset}"/>
+    <xacro:head_transmission name="${name}" reduction="1" offset_value="${head_1_joint_offset}"/>
   </xacro:macro>
   <!--************************-->
@@ -109,5 +109,5 @@
                          soft_upper_limit="${head_2_upper_limit * deg_to_rad}" />
     </joint>
-    <xacro:head_transmission name="${name}" reduction="1" offset_value="$${${name}_joint_offset}"/>
+    <xacro:head_transmission name="${name}" reduction="1" offset_value="${head_2_joint_offset}"/>
   </xacro:macro>
   <xacro:macro name="head" params="name parent camera_model">

Commit message: add wrist_model arg

File: tiago_description/robots/tiago.urdf.xacro (robot description, xacro)
@@ -10,4 +10,5 @@
         name="tiago" >
     <xacro:arg name="arm" default="true"/> <!-- true, false -->
+    <xacro:arg name="wrist_model" default="wrist-2010"/>
     <xacro:arg name="end_effector" default="pal-hey5"/> <!-- false, pal-gripper, pal-hey5, schunk-wsg-->
     <xacro:arg name="ft_sensor" default="schunk-ft"/> <!-- false, schunk-ft -->
@@ -17,4 +18,5 @@
     <xacro:arg name="multiple" default="false"/>
     <xacro:arg name="namespace" default=""/>
+    <xacro:property name="wrist_model" value="$(arg wrist_model)" />
     <xacro:property name="end_effector" value="$(arg end_effector)" />
     <xacro:property name="ft_sensor" value="$(arg ft_sensor)" />
@@ -23,4 +25,7 @@
     <xacro:property name="is_multiple" value="$(arg multiple)" />
     <xacro:property name="nsp" value="$(arg namespace)" />
+  <xacro:if value="${wrist_model not in ['wrist-2010', 'wrist-2017']}">
+    <xacro:wrong_wrist_model/>
+  </xacro:if>
   <xacro:if value="${end_effector not in ['false', False, 'pal-gripper', 'pal-hey5', 'schunk-wsg']}">
     <xacro:wrong_end_effector/>
@@ -42,5 +47,10 @@
    <xacro:property name="end_effector_link"       value="${'wrist_ft_tool_link' if has_ft_sensor else 'arm_tool_link'}"/>
    <xacro:property name="end_effector_name"       value="${'hand' if end_effector == 'pal-hey5' else 'gripper'}"/>
-   <xacro:property name="wrist_6_range"           value="${ 81 if has_ft_sensor else 90 }"/>
+   <xacro:if value="${wrist_model == 'wrist-2010'}">
+     <xacro:property name="wrist_6_range"           value="${ 81 if has_ft_sensor else 90 }"/>
+   </xacro:if>
+   <xacro:if value="${wrist_model == 'wrist-2017'}">
+     <xacro:property name="wrist_6_range"           value="81"/>
+   </xacro:if>
    <xacro:property name="head_link_name"          value="head_2_link"/>
   <!-- The following included files set up definitions of parts of the robot body -->

Commit message: Allow using custom end-effector

File: tiago_description/robots/tiago.urdf.xacro (robot description, xacro)
@@ -28,5 +28,5 @@
     <xacro:wrong_wrist_model/>
   </xacro:if>
-  <xacro:if value="${end_effector not in ['false', False, 'pal-gripper', 'pal-hey5', 'schunk-wsg']}">
+  <xacro:if value="${end_effector not in ['false', False, 'pal-gripper', 'pal-hey5', 'schunk-wsg', 'custom']}">
     <xacro:wrong_end_effector/>
   </xacro:if>

File: tiago_description/urdf/end_effector/end_effector.urdf.xacro (robot description, xacro)
@@ -19,4 +19,5 @@
   -->
   <xacro:macro name="tiago_end_effector" params="name parent type reflect">
+  <!-- PAL Gripper -->
   <xacro:if value="${type == 'pal-gripper'}">
     <xacro:include filename="$(find pal_gripper_description)/urdf/gripper.urdf.xacro" />
@@ -72,4 +73,11 @@
     </link>
   </xacro:if>
+  <!-- Custom -->
+  <xacro:if value="${type == 'custom'}">
+    <xacro:include filename="$(find custom_ee_description)/urdf/end-effector.urdf.xacro" />
+    <xacro:end_effector parent="${parent}">
+      <origin xyz="0.01 0 0" rpy="${90*deg_to_rad} ${90*deg_to_rad} ${-90*deg_to_rad}"/>
+    </xacro:end_effector>
+  </xacro:if>
   </xacro:macro>
 </robot>

Commit message: Change wrist tool link position with wrist 2017

File: tiago_description/robots/tiago.urdf.xacro (robot description, xacro)
@@ -47,10 +47,4 @@
    <xacro:property name="end_effector_link"       value="${'wrist_ft_tool_link' if has_ft_sensor else 'arm_tool_link'}"/>
    <xacro:property name="end_effector_name"       value="${'hand' if end_effector == 'pal-hey5' else 'gripper'}"/>
-   <xacro:if value="${wrist_model == 'wrist-2010'}">
-     <xacro:property name="wrist_6_range"           value="${ 81 if has_ft_sensor else 90 }"/>
-   </xacro:if>
-   <xacro:if value="${wrist_model == 'wrist-2017'}">
-     <xacro:property name="wrist_6_range"           value="81"/>
-   </xacro:if>
    <xacro:property name="head_link_name"          value="head_2_link"/>
   <!-- The following included files set up definitions of parts of the robot body -->
@@ -80,5 +74,5 @@
   <xacro:head name="head" parent="torso_lift_link" camera_model="$(arg camera_model)"/>
   <xacro:if value="${has_arm}">
-	  <xacro:tiago_arm name="arm" parent="torso_lift_link" wrist_6_range="${wrist_6_range}" reflect="1" tiago_dual="-1" arm_1_offset="${arm_1_joint_offset}" arm_2_offset="${arm_2_joint_offset}" arm_3_offset="${arm_3_joint_offset}" arm_4_offset="${arm_4_joint_offset}" arm_5_offset="${arm_5_joint_offset}" arm_6_offset="${arm_6_joint_offset}" arm_7_offset="${arm_7_joint_offset}">
+	  <xacro:tiago_arm name="arm" parent="torso_lift_link" wrist_model="${wrist_model}" has_ft_sensor="${has_ft_sensor}" reflect="1" tiago_dual="-1" arm_1_offset="${arm_1_joint_offset}" arm_2_offset="${arm_2_joint_offset}" arm_3_offset="${arm_3_joint_offset}" arm_4_offset="${arm_4_joint_offset}" arm_5_offset="${arm_5_joint_offset}" arm_6_offset="${arm_6_joint_offset}" arm_7_offset="${arm_7_joint_offset}">
         <origin xyz="0.15505 0.014 -0.151" rpy="0 0 ${-90 * deg_to_rad}" />
       </xacro:tiago_arm>

File: tiago_description/urdf/arm/arm.urdf.xacro (robot description, xacro)
@@ -26,5 +26,5 @@
   <!-- reflect: Set to 1 for a right arm, or to -1 for a left arm-->
   <!-- tiago_dual: Set to 1 for tiago dual, -1 for original tiago, changes joints 1 and 2 -->
-  <xacro:macro name="tiago_arm" params="name parent wrist_6_range reflect tiago_dual *origin arm_1_offset arm_2_offset arm_3_offset arm_4_offset arm_5_offset arm_6_offset arm_7_offset">
+  <xacro:macro name="tiago_arm" params="name parent wrist_model has_ft_sensor reflect tiago_dual *origin arm_1_offset arm_2_offset arm_3_offset arm_4_offset arm_5_offset arm_6_offset arm_7_offset">
     <!--************************-->
     <!--        SHOULDER        -->
@@ -217,4 +217,10 @@
     <!--        WRIST           -->
     <!--************************-->
+   <xacro:if value="${wrist_model == 'wrist-2010'}">
+     <xacro:property name="wrist_6_range"           value="${ 81 if has_ft_sensor else 90 }"/>
+   </xacro:if>
+   <xacro:if value="${wrist_model == 'wrist-2017'}">
+     <xacro:property name="wrist_6_range"           value="81"/>
+   </xacro:if>
    <xacro:wrist name="${name}" parent="${name}_4_link" reflect="${reflect}" wrist_6_range="${wrist_6_range}" arm_5_offset="${arm_5_offset}" arm_6_offset="${arm_6_offset}" arm_7_offset="${arm_7_offset}"/>
     <!--***********************-->
@@ -240,8 +246,14 @@
       </collision>
     </link>
+    <xacro:if value="${wrist_model == 'wrist-2010'}">
+      <xacro:property name="tool_link_z_offset"           value="0.046"/>
+    </xacro:if>
+    <xacro:if value="${wrist_model == 'wrist-2017'}">
+     <xacro:property name="tool_link_z_offset"           value="${ 0.046 if has_ft_sensor else 0.06825 }"/>
+    </xacro:if>
     <joint name="${name}_tool_joint" type="fixed">
       <parent link="${name}_7_link" />
       <child link="${name}_tool_link" />
-      <origin xyz="0 0 ${reflect*0.046}" rpy="${90.0 * deg_to_rad} ${reflect * -90.0 * deg_to_rad} ${180 * deg_to_rad}" />
+        <origin xyz="0 0 ${reflect * tool_link_z_offset}" rpy="${90.0 * deg_to_rad} ${reflect * -90.0 * deg_to_rad} ${180 * deg_to_rad}" />
     </joint>
     <!-- extensions -->

Commit message: pass the camera origin as an argument to head

File: tiago_description/robots/tiago.urdf.xacro (robot description, xacro)
@@ -72,5 +72,8 @@
   <xacro:base_sensors name="base" laser_model="$(arg laser_model)" sonars="true" microphone="true"/>
   <xacro:tiago_torso name="torso" parent="base_link"/>
-  <xacro:head name="head" parent="torso_lift_link" camera_model="$(arg camera_model)"/>
+  <xacro:head name="head" parent="torso_lift_link" camera_model="$(arg camera_model)">
+    <!-- Camera origin Post Eye-Hand Calibration -->
+    <origin xyz="${camera_position_x} ${camera_position_y} ${camera_position_z}" rpy="${camera_orientation_r} ${camera_orientation_p} ${camera_orientation_y}" />
+  </xacro:head>
   <xacro:if value="${has_arm}">
 	  <xacro:tiago_arm name="arm" parent="torso_lift_link" wrist_model="${wrist_model}" has_ft_sensor="${has_ft_sensor}" reflect="1" tiago_dual="-1" arm_1_offset="${arm_1_joint_offset}" arm_2_offset="${arm_2_joint_offset}" arm_3_offset="${arm_3_joint_offset}" arm_4_offset="${arm_4_joint_offset}" arm_5_offset="${arm_5_joint_offset}" arm_6_offset="${arm_6_joint_offset}" arm_7_offset="${arm_7_joint_offset}">

File: tiago_description/urdf/head/head.urdf.xacro (robot description, xacro)
@@ -13,5 +13,4 @@
   <xacro:include filename="$(find tiago_description)/urdf/sensors/xtion_pro_live.urdf.xacro" />
   <xacro:include filename="$(find tiago_description)/urdf/sensors/orbbec_astra.urdf.xacro" />
-  <xacro:include filename="$(find tiago_description_calibration)/urdf/calibration/calibration_constants.urdf.xacro" />
   <!--Constant parameters-->
   <xacro:property name="head_friction" value="1.0" />
@@ -112,10 +111,10 @@
     <xacro:head_transmission name="${name}" reduction="1" offset_value="${head_2_joint_offset}"/>
   </xacro:macro>
-  <xacro:macro name="head" params="name parent camera_model">
+  <xacro:macro name="head" params="name parent camera_model *camera_origin">
     <xacro:head_1 name="${name}_1" parent="${parent}" />
     <xacro:head_2 name="${name}_2" parent="${name}_1_link"/>
     <xacro:if value="${camera_model == 'asus-xtion'}">
       <xacro:xtion_pro_live name="xtion" parent="${name}_2" camera_model="${camera_model}">
-        <origin xyz="${camera_position_x} ${camera_position_y} ${camera_position_z}" rpy="${camera_orientation_r} ${camera_orientation_p} ${camera_orientation_y}" />
+        <xacro:insert_block name="camera_origin"/>
         <!-- optical origin -->
         <origin xyz="0 0 0" rpy="${-90 * deg_to_rad} ${0 * deg_to_rad} ${-90 * deg_to_rad}" />
@@ -124,5 +123,5 @@
     <xacro:if value="${camera_model in ['orbbec-astra', 'orbbec-astra-pro']}">
       <xacro:orbbec_astra name="xtion" parent="${name}_2" camera_model="${camera_model}">
-        <origin xyz="${camera_position_x} ${camera_position_y} ${camera_position_z}" rpy="${camera_orientation_r} ${camera_orientation_p} ${camera_orientation_y}" />
+        <xacro:insert_block name="camera_origin"/>
         <!-- optical origin -->
         <origin xyz="0 0 0" rpy="${-90 * deg_to_rad} ${0 * deg_to_rad} ${-90 * deg_to_rad}" />
