Commit message: parse package name instead of individual elements and load files respective to package

File: tiago_description/robots/tiago.urdf.xacro (robot description, xacro)
@@ -72,8 +72,5 @@
   <xacro:base_sensors name="base" laser_model="$(arg laser_model)" sonars="true" microphone="true"/>
   <xacro:tiago_torso name="torso" parent="base_link"/>
-  <xacro:head name="head" parent="torso_lift_link" camera_model="$(arg camera_model)">
-    <!-- Camera origin Post Eye-Hand Calibration -->
-    <origin xyz="${camera_position_x} ${camera_position_y} ${camera_position_z}" rpy="${camera_orientation_r} ${camera_orientation_p} ${camera_orientation_y}" />
-  </xacro:head>
+  <xacro:head name="head" parent="torso_lift_link" camera_model="$(arg camera_model)" description_calibration_package="tiago_description_calibration"/>
   <xacro:if value="${has_arm}">
 	  <xacro:tiago_arm name="arm" parent="torso_lift_link" wrist_model="${wrist_model}" has_ft_sensor="${has_ft_sensor}" reflect="1" tiago_dual="-1" arm_1_offset="${arm_1_joint_offset}" arm_2_offset="${arm_2_joint_offset}" arm_3_offset="${arm_3_joint_offset}" arm_4_offset="${arm_4_joint_offset}" arm_5_offset="${arm_5_joint_offset}" arm_6_offset="${arm_6_joint_offset}" arm_7_offset="${arm_7_joint_offset}">

File: tiago_description/urdf/head/head.urdf.xacro (robot description, xacro)
@@ -111,10 +111,12 @@
     <xacro:head_transmission name="${name}" reduction="1" offset_value="${head_2_joint_offset}"/>
   </xacro:macro>
-  <xacro:macro name="head" params="name parent camera_model *camera_origin">
+  <xacro:macro name="head" params="name parent camera_model description_calibration_package:=tiago_description_calibration">
+    <!-- includes -->
+    <xacro:include filename="$(find ${description_calibration_package})/urdf/calibration/calibration_constants.urdf.xacro" />
     <xacro:head_1 name="${name}_1" parent="${parent}" />
     <xacro:head_2 name="${name}_2" parent="${name}_1_link"/>
     <xacro:if value="${camera_model == 'asus-xtion'}">
-      <xacro:xtion_pro_live name="xtion" parent="${name}_2" camera_model="${camera_model}">
-        <xacro:insert_block name="camera_origin"/>
+      <xacro:xtion_pro_live name="xtion" parent="${name}_2" camera_model="${camera_model}" extrinsic_package="${description_calibration_package}">
+        <origin xyz="${camera_position_x} ${camera_position_y} ${camera_position_z}" rpy="${camera_orientation_r} ${camera_orientation_p} ${camera_orientation_y}" />
         <!-- optical origin -->
         <origin xyz="0 0 0" rpy="${-90 * deg_to_rad} ${0 * deg_to_rad} ${-90 * deg_to_rad}" />
@@ -122,6 +124,6 @@
     </xacro:if>
     <xacro:if value="${camera_model in ['orbbec-astra', 'orbbec-astra-pro']}">
-      <xacro:orbbec_astra name="xtion" parent="${name}_2" camera_model="${camera_model}">
-        <xacro:insert_block name="camera_origin"/>
+      <xacro:orbbec_astra name="xtion" parent="${name}_2" camera_model="${camera_model}" extrinsic_package="${description_calibration_package}">
+        <origin xyz="${camera_position_x} ${camera_position_y} ${camera_position_z}" rpy="${camera_orientation_r} ${camera_orientation_p} ${camera_orientation_y}" />
         <!-- optical origin -->
         <origin xyz="0 0 0" rpy="${-90 * deg_to_rad} ${0 * deg_to_rad} ${-90 * deg_to_rad}" />

File: tiago_description/urdf/sensors/orbbec_astra.urdf.xacro (robot description, xacro)
@@ -20,7 +20,8 @@
 <robot xmlns:xacro="http://ros.org/wiki/xacro">
   <xacro:include filename="$(find tiago_description)/urdf/sensors/openni.gazebo.xacro" />
-  <xacro:include filename="$(find tiago_description_calibration)/urdf/calibration/extrinsic_camera_calibration_constants.urdf.xacro" />
   <!-- Macro -->
-  <xacro:macro name="orbbec_astra" params="name parent camera_model *origin *optical_origin">
+  <xacro:macro name="orbbec_astra" params="name parent camera_model *origin *optical_origin extrinsic_package:=tiago_description_calibration">
+    <!-- includes -->
+    <xacro:include filename="$(find ${extrinsic_package})/urdf/calibration/extrinsic_camera_calibration_constants.urdf.xacro" />
     <!-- frames in the center of the camera -->
     <joint name="${name}_joint" type="fixed">

File: tiago_description/urdf/sensors/xtion_pro_live.urdf.xacro (robot description, xacro)
@@ -19,7 +19,8 @@
 <robot xmlns:xacro="http://ros.org/wiki/xacro">
   <xacro:include filename="$(find tiago_description)/urdf/sensors/openni.gazebo.xacro" />
-  <xacro:include filename="$(find tiago_description_calibration)/urdf/calibration/extrinsic_camera_calibration_constants.urdf.xacro" />
   <!-- Macro -->
-  <xacro:macro name="xtion_pro_live" params="name parent camera_model *origin *optical_origin">
+  <xacro:macro name="xtion_pro_live" params="name parent camera_model *origin *optical_origin extrinsic_package:=tiago_description_calibration">
+    <!-- includes -->
+    <xacro:include filename="$(find ${extrinsic_package})/urdf/calibration/extrinsic_camera_calibration_constants.urdf.xacro" />
     <!-- frames in the center of the camera -->
     <joint name="${name}_joint" type="fixed">

Commit message: Add master calibration compatibility for eye hand and extrinsic

File: tiago_description/robots/tiago.urdf.xacro (robot description, xacro)
@@ -17,4 +17,6 @@
     <xacro:arg name="has_thermal_camera" default="false"/>
     <xacro:arg name="multiple" default="false"/>
+    <xacro:arg name="description_calibration_dir" default="$(find tiago_description_calibration)/urdf/calibration"/>
+    <xacro:arg name="extrinsic_calibration_dir" default="$(find tiago_description_calibration)/urdf/calibration"/>
     <xacro:arg name="namespace" default=""/>
     <xacro:property name="wrist_model" value="$(arg wrist_model)" />
@@ -50,4 +52,5 @@
    <xacro:property name="end_effector_name"       value="${'hand' if end_effector == 'pal-hey5' else 'gripper'}"/>
    <xacro:property name="head_link_name"          value="head_2_link"/>
+   <xacro:property name="description_calibration_dir"       value="${arg description_calibration_dir}"/>
   <!-- The following included files set up definitions of parts of the robot body -->
   <!-- Base -->
@@ -59,5 +62,5 @@
     <xacro:include filename="$(find tiago_description)/urdf/arm/arm.urdf.xacro" />
     <xacro:include filename="$(find tiago_description)/urdf/end_effector/end_effector.urdf.xacro" />
-    <xacro:include filename="$(find tiago_description_calibration)/urdf/calibration/calibration_constants.urdf.xacro" />
+  <xacro:include filename="$(arg description_calibration_dir)/calibration_constants.urdf.xacro" />
   </xacro:if>
   <!-- Force Torque sensor -->
@@ -74,5 +77,7 @@
   <xacro:base_sensors name="base" laser_model="$(arg laser_model)" sonars="true" microphone="true"/>
   <xacro:tiago_torso name="torso" parent="base_link"/>
-  <xacro:head name="head" parent="torso_lift_link" camera_model="$(arg camera_model)" description_calibration_package="tiago_description_calibration"/>
+  <xacro:head name="head" parent="torso_lift_link" camera_model="$(arg camera_model)"
+	  description_calibration_dir="$(arg description_calibration_dir)"
+	  extrinsic_calibration_dir="$(arg extrinsic_calibration_dir)"/>
   <xacro:if value="${has_arm}">
 	  <xacro:tiago_arm name="arm" parent="torso_lift_link" wrist_model="${wrist_model}" has_ft_sensor="${has_ft_sensor}" reflect="1" tiago_dual="-1" arm_1_offset="${arm_1_joint_offset}" arm_2_offset="${arm_2_joint_offset}" arm_3_offset="${arm_3_joint_offset}" arm_4_offset="${arm_4_joint_offset}" arm_5_offset="${arm_5_joint_offset}" arm_6_offset="${arm_6_joint_offset}" arm_7_offset="${arm_7_joint_offset}">

File: tiago_description/urdf/head/head.urdf.xacro (robot description, xacro)
@@ -111,11 +111,11 @@
     <xacro:head_transmission name="${name}" reduction="1" offset_value="${head_2_joint_offset}"/>
   </xacro:macro>
-  <xacro:macro name="head" params="name parent camera_model description_calibration_package">
+  <xacro:macro name="head" params="name parent camera_model description_calibration_dir extrinsic_calibration_dir">
     <!-- includes -->
-    <xacro:include filename="$(find ${description_calibration_package})/urdf/calibration/calibration_constants.urdf.xacro" />
+    <xacro:include filename="$(arg description_calibration_dir)/calibration_constants.urdf.xacro" />
     <xacro:head_1 name="${name}_1" parent="${parent}" />
     <xacro:head_2 name="${name}_2" parent="${name}_1_link"/>
     <xacro:if value="${camera_model == 'asus-xtion'}">
-      <xacro:xtion_pro_live name="xtion" parent="${name}_2" camera_model="${camera_model}" extrinsic_package="${description_calibration_package}">
+      <xacro:xtion_pro_live name="xtion" parent="${name}_2" camera_model="${camera_model}" extrinsic_calibration_dir="${extrinsic_calibration_dir}">
         <origin xyz="${camera_position_x} ${camera_position_y} ${camera_position_z}" rpy="${camera_orientation_r} ${camera_orientation_p} ${camera_orientation_y}" />
         <!-- optical origin -->
@@ -124,5 +124,5 @@
     </xacro:if>
     <xacro:if value="${camera_model in ['orbbec-astra', 'orbbec-astra-pro']}">
-      <xacro:orbbec_astra name="xtion" parent="${name}_2" camera_model="${camera_model}" extrinsic_package="${description_calibration_package}">
+      <xacro:orbbec_astra name="xtion" parent="${name}_2" camera_model="${camera_model}" extrinsic_calibration_dir="${extrinsic_calibration_dir}">
         <origin xyz="${camera_position_x} ${camera_position_y} ${camera_position_z}" rpy="${camera_orientation_r} ${camera_orientation_p} ${camera_orientation_y}" />
         <!-- optical origin -->

Commit message: Add the option of disabling arm_safety_eps via launch file

File: tiago_description/robots/tiago.urdf.xacro (robot description, xacro)
@@ -20,4 +20,5 @@
     <xacro:arg name="extrinsic_calibration_dir" default="$(find tiago_description_calibration)/urdf/calibration"/>
     <xacro:arg name="namespace" default=""/>
+    <xacro:arg name="no_safety_eps" default="false"/>
     <xacro:property name="wrist_model" value="$(arg wrist_model)" />
     <xacro:property name="end_effector" value="$(arg end_effector)" />
@@ -27,4 +28,5 @@
     <xacro:property name="is_multiple" value="$(arg multiple)" />
     <xacro:property name="nsp" value="$(arg namespace)" />
+    <xacro:property name="no_safety_eps" value="$(arg no_safety_eps)" />
   <xacro:if value="$(arg arm)">
     <xacro:if value="${wrist_model not in ['wrist-2010', 'wrist-2017']}">
@@ -81,5 +83,5 @@
 	  extrinsic_calibration_dir="$(arg extrinsic_calibration_dir)"/>
   <xacro:if value="${has_arm}">
-	  <xacro:tiago_arm name="arm" parent="torso_lift_link" wrist_model="${wrist_model}" has_ft_sensor="${has_ft_sensor}" reflect="1" tiago_dual="-1" arm_1_offset="${arm_1_joint_offset}" arm_2_offset="${arm_2_joint_offset}" arm_3_offset="${arm_3_joint_offset}" arm_4_offset="${arm_4_joint_offset}" arm_5_offset="${arm_5_joint_offset}" arm_6_offset="${arm_6_joint_offset}" arm_7_offset="${arm_7_joint_offset}">
+	  <xacro:tiago_arm name="arm" parent="torso_lift_link" wrist_model="${wrist_model}" has_ft_sensor="${has_ft_sensor}" reflect="1" tiago_dual="-1" arm_1_offset="${arm_1_joint_offset}" arm_2_offset="${arm_2_joint_offset}" arm_3_offset="${arm_3_joint_offset}" arm_4_offset="${arm_4_joint_offset}" arm_5_offset="${arm_5_joint_offset}" arm_6_offset="${arm_6_joint_offset}" arm_7_offset="${arm_7_joint_offset}" no_safety_eps="${no_safety_eps}">
         <origin xyz="0.15505 0.014 -0.151" rpy="0 0 ${-90 * deg_to_rad}" />
       </xacro:tiago_arm>

File: tiago_description/urdf/arm/arm.urdf.xacro (robot description, xacro)
@@ -23,8 +23,8 @@
   <xacro:property name="arm_3_max_effort"   value="26" />
   <xacro:property name="arm_4_max_effort"   value="26" />
-  <xacro:property name="arm_eps"            value="0.07" />
   <!-- reflect: Set to 1 for a right arm, or to -1 for a left arm-->
   <!-- tiago_dual: Set to 1 for tiago dual, -1 for original tiago, changes joints 1 and 2 -->
-  <xacro:macro name="tiago_arm" params="name parent wrist_model has_ft_sensor reflect tiago_dual *origin arm_1_offset arm_2_offset arm_3_offset arm_4_offset arm_5_offset arm_6_offset arm_7_offset">
+  <xacro:macro name="tiago_arm" params="name parent wrist_model has_ft_sensor reflect tiago_dual *origin arm_1_offset arm_2_offset arm_3_offset arm_4_offset arm_5_offset arm_6_offset arm_7_offset no_safety_eps:=${no_safety_eps}">
+   <xacro:property name="arm_eps"       value="${0.00 if no_safety_eps else 0.07}"/>
     <!--************************-->
     <!--        SHOULDER        -->
@@ -217,5 +217,5 @@
     <!--        WRIST           -->
     <!--************************-->
-   <xacro:wrist name="${name}" parent="${name}_4_link" reflect="${reflect}" wrist_model="${wrist_model}" has_ft_sensor="${has_ft_sensor}" arm_5_offset="${arm_5_offset}" arm_6_offset="${arm_6_offset}" arm_7_offset="${arm_7_offset}"/>
+   <xacro:wrist name="${name}" parent="${name}_4_link" reflect="${reflect}" wrist_model="${wrist_model}" has_ft_sensor="${has_ft_sensor}" arm_5_offset="${arm_5_offset}" arm_6_offset="${arm_6_offset}" arm_7_offset="${arm_7_offset}"  no_safety_eps="${no_safety_eps}"/>
     <!--***********************-->
     <!--        TOOL           -->

Commit message: added no safety eps to head

File: tiago_description/robots/tiago.urdf.xacro (robot description, xacro)
@@ -81,5 +81,6 @@
   <xacro:head name="head" parent="torso_lift_link" camera_model="$(arg camera_model)"
 	  description_calibration_dir="$(arg description_calibration_dir)"
-	  extrinsic_calibration_dir="$(arg extrinsic_calibration_dir)"/>
+	  extrinsic_calibration_dir="$(arg extrinsic_calibration_dir)"
+    no_safety_eps="${no_safety_eps}"/>
   <xacro:if value="${has_arm}">
 	  <xacro:tiago_arm name="arm" parent="torso_lift_link" wrist_model="${wrist_model}" has_ft_sensor="${has_ft_sensor}" reflect="1" tiago_dual="-1" arm_1_offset="${arm_1_joint_offset}" arm_2_offset="${arm_2_joint_offset}" arm_3_offset="${arm_3_joint_offset}" arm_4_offset="${arm_4_joint_offset}" arm_5_offset="${arm_5_joint_offset}" arm_6_offset="${arm_6_joint_offset}" arm_7_offset="${arm_7_joint_offset}" no_safety_eps="${no_safety_eps}">

File: tiago_description/urdf/head/head.urdf.xacro (robot description, xacro)
@@ -17,5 +17,4 @@
   <xacro:property name="head_damping"  value="0.5" />
   <xacro:property name="head_max_vel"  value="3.0" />
-  <xacro:property name="head_eps"      value="0.07" />
   <xacro:property name="head_1_lower_limit" value="-75"/>
   <xacro:property name="head_1_upper_limit" value="75"/>
@@ -25,5 +24,6 @@
   <!--     HEAD_1 (PAN)       -->
   <!--************************-->
-  <xacro:macro name="head_1" params="name parent">
+  <xacro:macro name="head_1" params="name parent no_safety_eps:=False">
+    <xacro:property name="head_eps"      value="${0.00 if no_safety_eps else 0.07}" />
     <link name="${name}_link">
       <inertial>

Commit message: All joints now form part of a single ros2_control system

File: tiago_description/robots/tiago.urdf.xacro (robot description, xacro)
@@ -74,4 +74,6 @@
   <!-- Generic simulator_gazebo plugins -->
   <xacro:include filename="$(find tiago_description)/gazebo/gazebo.urdf.xacro" />
+  <!-- ros2_control -->
+  <xacro:include filename="$(find tiago_description)/ros2_control/ros2_control.urdf.xacro" />
   <!-- Materials for visualization -->
   <xacro:include filename="$(find tiago_description)/urdf/materials.urdf.xacro" />

File: tiago_description/urdf/torso/torso.ros2_control.xacro (robot description, xacro)
@@ -8,29 +8,24 @@
 -->
 <robot xmlns:xacro="http://ros.org/wiki/xacro">
-  <!-- Torso Joint -->
-  <xacro:macro name="torso_ros2_control" params="name reduction" >
-    <ros2_control name="${name}" type="system">
-      <hardware>
-        <plugin>gazebo_ros2_control/GazeboSystem</plugin>
-      </hardware>
+  <xacro:macro name="ros2_control_torso" params="name reduction" >
+    <joint name="${name}_joint">
+      <command_interface name="position" />
+      <state_interface name="position" />
+      <state_interface name="velocity" />
+      <state_interface name="effort" />
+    </joint>
+    <!-- @TODO transmissions for ros2 system -->
+    <!--
+    <transmission name="${name}_trans">
+      <type>transmission_interface/SimpleTransmission</type>
+      <actuator name="${name}_motor" >
+        <mechanicalReduction>${reduction}</mechanicalReduction>
+      </actuator>
       <joint name="${name}_joint">
-        <command_interface name="position" />
-        <state_interface name="position" />
-        <state_interface name="velocity" />
+        <hardwareInterface>hardware_interface/PositionJointInterface</hardwareInterface>
+        <hardwareInterface>hardware_interface/JointStateInterface</hardwareInterface>
       </joint>
-      <!-- @TODO transmissions for ros2 system -->
-      <!--
-      <transmission name="${name}_trans">
-        <type>transmission_interface/SimpleTransmission</type>
-        <actuator name="${name}_motor" >
-          <mechanicalReduction>${reduction}</mechanicalReduction>
-        </actuator>
-        <joint name="${name}_joint">
-          <hardwareInterface>hardware_interface/PositionJointInterface</hardwareInterface>
-          <hardwareInterface>hardware_interface/JointStateInterface</hardwareInterface>
-        </joint>
-      </transmission>
-      -->
-    </ros2_control>
+    </transmission>
+    -->
   </xacro:macro>
 </robot>

File: tiago_description/urdf/torso/torso.urdf.xacro (robot description, xacro)
@@ -11,5 +11,4 @@
   <xacro:include filename="$(find tiago_description)/urdf/deg_to_rad.xacro" />
   <xacro:include filename="$(find tiago_description)/urdf/torso/torso.transmission.xacro" />
-  <xacro:include filename="$(find tiago_description)/urdf/torso/torso.ros2_control.xacro" />
   <!--Constant parameters-->
   <xacro:property name="torso_max_vel"  value="0.07" />
@@ -135,6 +134,4 @@
                          soft_upper_limit="0.35" />
   </joint>
-  <!-- ROS Control -->
-  <xacro:torso_ros2_control name="torso_lift" reduction="1.0"/>
  </xacro:macro>
 </robot>

Commit message: Add IMU and FT ROS2 Control sensors

File: tiago_description/robots/tiago.urdf.xacro (robot description, xacro)
@@ -69,4 +69,5 @@
   <xacro:if value="${has_ft_sensor}">
     <xacro:include filename="$(find tiago_description)/urdf/sensors/ftsensor.urdf.xacro" />
+    <xacro:include filename="$(find tiago_description)/urdf/sensors/ftsensor.gazebo.xacro" />
   </xacro:if>
   <!-- Head -->
@@ -123,3 +124,6 @@
       </inertial>
   </link>
+  <xacro:if value="${has_ft_sensor}">
+    <xacro:force_torque_sensor_gazebo joint_name="wrist_ft_joint" update_rate="100"/>
+  </xacro:if>
 </robot>

File: tiago_description/ros2_control/ros2_control.urdf.xacro (robot description, xacro)
@@ -24,4 +24,5 @@
     </xacro:if>
   </xacro:if>
+  <xacro:include filename="$(find pmb2_description)/urdf/sensors/sensors.ros2_control.xacro"/>
   <!-- calibration offsets -->
   <xacro:include filename="$(arg description_calibration_dir)/calibration_constants.urdf.xacro" />
@@ -33,4 +34,6 @@
     <xacro:ros2_control_wheel side="right" />
     <xacro:ros2_control_wheel side="left" />
+    <!-- IMU -->
+    <xacro:ros2_control_imu name="base_imu_sensor"/>
     <!-- torso -->
     <xacro:ros2_control_torso name="torso_lift" reduction="1.0" />
@@ -56,4 +59,9 @@
       </xacro:if>
     </xacro:if>
+    <!-- Force Torque sensor -->
+    <xacro:if value="${has_ft_sensor}">
+      <xacro:include filename="$(find tiago_description)/urdf/sensors/sensors.ros2_control.xacro"/>
+      <xacro:ros2_control_force_torque_sensor name="wrist_ft_joint_force_torque"/>
+    </xacro:if>
   </ros2_control>
 </robot>

File: tiago_description/urdf/sensors/ftsensor.gazebo.xacro (robot description, xacro)
@@ -7,19 +7,17 @@
   Creative Commons, 444 Castro Street, Suite 900, Mountain View, California, 94041, USA.
 -->
-<robot name="reemc" xmlns:xacro="http://ros.org/wiki/xacro">
-<xacro:macro name="reemc_force_torque_sensor" params="name update_rate">
-  <gazebo reference="${name}">
-    <sensor name="${name}_contact_sensor" type="contact">
-      <pose>0.105 0.071 0 0 0 0</pose>
-      <always_on>1</always_on>
+<robot xmlns:xacro="http://ros.org/wiki/xacro">
+  <xacro:macro name="force_torque_sensor_gazebo" params="joint_name update_rate">
+  <gazebo reference="${joint_name}">
+    <preserveFixedJoint>true</preserveFixedJoint> <!-- in case this is in a fixed joint -->
+    <sensor name="${joint_name}_force_torque" type="force_torque">
       <update_rate>${update_rate}</update_rate>
-      <contact>
-        <collision>${name}_collision</collision>
-      </contact>
+      <visualize>true</visualize>
+      <force_torque>
+        <frame>child</frame>
+        <measure_direction>child_to_parent</measure_direction>
+      </force_torque>
     </sensor>
-  </gazebo>
-  <gazebo reference="${name}">
-    <provideFeedback>1</provideFeedback>
-  </gazebo>
+</gazebo>
 </xacro:macro>
 </robot>

Commit message: integrate the new robotiq-85 and robotiq-140 grippers

File: tiago_description/robots/tiago.urdf.xacro (robot description, xacro)
@@ -34,5 +34,5 @@
     </xacro:if>
   </xacro:if>
-  <xacro:if value="${end_effector not in ['false', False, 'pal-gripper', 'pal-hey5', 'schunk-wsg', 'custom']}">
+  <xacro:if value="${end_effector not in ['false', False, 'pal-gripper', 'pal-hey5', 'schunk-wsg', 'robotiq-85', 'robotiq-140', 'custom']}">
     <xacro:wrong_end_effector/>
   </xacro:if>

File: tiago_description/urdf/end_effector/end_effector.urdf.xacro (robot description, xacro)
@@ -73,4 +73,18 @@
     </link>
   </xacro:if>
+  <!-- Robotiq 2F-85 Gripper -->
+  <xacro:if value="${type == 'robotiq-85'}">
+    <xacro:include filename="$(find pal_robotiq_85_description)/urdf/robotiq_85_gripper.urdf.xacro" />
+    <xacro:robotiq_85_gripper prefix="${name}_" parent="${parent}" >
+      <origin xyz="0.01 0 0" rpy="${90*deg_to_rad} ${0*deg_to_rad} ${90*deg_to_rad}"/>
+    </xacro:robotiq_85_gripper>
+  </xacro:if>
+  <!-- Robotiq 2F-140 Gripper -->
+  <xacro:if value="${type == 'robotiq-140'}">
+    <xacro:include filename="$(find pal_robotiq_140_description)/urdf/robotiq_140_gripper.urdf.xacro" />
+    <xacro:robotiq_140_gripper prefix="${name}_" parent="${parent}" >
+      <origin xyz="0.01 0 0" rpy="${90*deg_to_rad} ${0*deg_to_rad} ${90*deg_to_rad}"/>
+    </xacro:robotiq_140_gripper>
+  </xacro:if>
   <!-- Custom -->
   <xacro:if value="${type == 'custom' and not is_dual}">
