Commit message: Rename some tiago hw options, add camera_model and add tests

File: tiago_description/robots/tiago.urdf.xacro (robot description, xacro)
@@ -9,10 +9,10 @@
 <robot  xmlns:xacro="http://ros.org/wiki/xacro"
         name="tiago" >
-    <xacro:arg name="arm" default="true"/> <!-- true, false -->
+    <xacro:arg name="arm" default="right-arm"/> <!-- right-arm, left-arm, no-arm -->
     <xacro:arg name="wrist_model" default="wrist-2010"/>
-    <xacro:arg name="end_effector" default="pal-hey5"/> <!-- false, pal-gripper, pal-hey5, schunk-wsg-->
-    <xacro:arg name="ft_sensor" default="schunk-ft"/> <!-- false, schunk-ft -->
-    <xacro:arg name="laser_model" default="sick-571"/> <!-- false, hokuyo, sick-551, sick-561, sick-571-->
-    <xacro:arg name="camera_model" default="orbbec-astra"/> <!-- false, orbbec-astra, orbbec-astra-pro, asus-xtion -->
+    <xacro:arg name="end_effector" default="pal-hey5"/> <!-- no-end-effector, pal-gripper, pal-hey5, schunk-wsg-->
+    <xacro:arg name="ft_sensor" default="schunk-ft"/> <!-- no-ft-sensor, schunk-ft -->
+    <xacro:arg name="laser_model" default="sick-571"/> <!-- no-laser, hokuyo, sick-551, sick-561, sick-571-->
+    <xacro:arg name="camera_model" default="orbbec-astra"/> <!-- no-camera, orbbec-astra, orbbec-astra-pro, asus-xtion -->
     <xacro:arg name="has_thermal_camera" default="false"/>
     <xacro:arg name="multiple" default="false"/>
@@ -21,4 +21,8 @@
     <xacro:arg name="namespace" default=""/>
     <xacro:arg name="no_safety_eps" default="false"/>
+    <xacro:property name="arm" value="$(arg arm)" />
+    <xacro:if value="${arm not in ['right-arm', 'left-arm', 'no-arm']}">
+      <xacro:wrong_arm/>
+    </xacro:if>
     <xacro:property name="wrist_model" value="$(arg wrist_model)" />
     <xacro:property name="end_effector" value="$(arg end_effector)" />
@@ -29,26 +33,26 @@
     <xacro:property name="nsp" value="$(arg namespace)" />
     <xacro:property name="no_safety_eps" value="$(arg no_safety_eps)" />
-  <xacro:if value="$(arg arm)">
+    <xacro:property name="has_arm" value="${arm != 'no-arm'}"/>
+  <xacro:if value="${has_arm}">
     <xacro:if value="${wrist_model not in ['wrist-2010', 'wrist-2017']}">
       <xacro:wrong_wrist_model/>
     </xacro:if>
   </xacro:if>
-  <xacro:if value="${end_effector not in ['false', False, 'pal-gripper', 'pal-hey5', 'schunk-wsg', 'custom']}">
+  <xacro:if value="${end_effector not in ['no-end-effector', 'pal-gripper', 'pal-hey5', 'schunk-wsg', 'custom']}">
     <xacro:wrong_end_effector/>
   </xacro:if>
-  <xacro:if value="${ft_sensor not in ['false', False, 'schunk-ft']}">
+  <xacro:if value="${ft_sensor not in ['no-ft-sensor', 'schunk-ft']}">
     <xacro:wrong_ft_sensor/>
   </xacro:if>
-  <xacro:if value="${laser_model not in ['false', False, 'sick-551', 'sick-561', 'sick-571', 'hokuyo']}">
+  <xacro:if value="${laser_model not in ['no-laser', 'sick-551', 'sick-561', 'sick-571', 'hokuyo']}">
     <xacro:wrong_laser_model/>
   </xacro:if>
-  <xacro:if value="${camera_model not in ['false', False, 'orbbec-astra', 'orbbec-astra-pro', 'asus-xtion']}">
+  <xacro:if value="${camera_model not in ['no-camera', 'orbbec-astra', 'orbbec-astra-pro', 'asus-xtion']}">
     <xacro:wrong_camera_model/>
   </xacro:if>
         <!-- The properties below are modified using empy http://www.alcyone.com/software/empy/
              from the create_robot.py tool. Handle them with care -->
-   <xacro:property name="has_arm"                 value="$(arg arm)"/>
    <xacro:property name="has_schunk_ft"           value="${ft_sensor == 'schunk-ft'}"/>
-   <xacro:property name="has_ft_sensor"           value="${has_schunk_ft}"/> <!-- This should be OR'ed with other FT sensors-->
+   <xacro:property name="has_ft_sensor"           value="${has_arm and has_schunk_ft}"/> <!-- This should be OR'ed with other FT sensors-->
    <xacro:property name="end_effector_link"       value="${'wrist_ft_tool_link' if has_ft_sensor else 'arm_tool_link'}"/>
    <xacro:property name="end_effector_name"       value="${'hand' if end_effector == 'pal-hey5' else 'gripper'}"/>
@@ -64,5 +68,5 @@
     <xacro:include filename="$(find tiago_description)/urdf/arm/arm.urdf.xacro" />
     <xacro:include filename="$(find tiago_description)/urdf/end_effector/end_effector.urdf.xacro" />
-  <xacro:include filename="$(arg description_calibration_dir)/calibration_constants.urdf.xacro" />
+    <xacro:include filename="$(arg description_calibration_dir)/calibration_constants.urdf.xacro" />
   </xacro:if>
   <!-- Force Torque sensor -->

File: tiago_description/ros2_control/ros2_control.urdf.xacro (robot description, xacro)
@@ -12,5 +12,5 @@
   <xacro:arg name="end_effector" default="pal-hey5"/>
   <xacro:arg name="description_calibration_dir" default="$(find tiago_description_calibration)/urdf/calibration" />
-  <xacro:property name="has_arm" value="$(arg arm)" />
+  <xacro:property name="has_arm" value="${arm != 'no-arm'}" />
   <xacro:property name="end_effector" value="$(arg end_effector)" />
   <xacro:include filename="$(find pmb2_description)/urdf/wheels/wheel.ros2_control.xacro" />

Commit message: Creating tiago with omni_base robot

File: tiago_description/robots/tiago.urdf.xacro (robot description, xacro)
@@ -26,4 +26,5 @@
     <xacro:arg name="namespace" default=""/>
     <xacro:arg name="no_safety_eps" default="false"/>
+    <xacro:arg name="base_type" default="pmb2"/> <!-- pmb2, omni_base -->
     <xacro:property name="wrist_model" value="$(arg wrist_model)" />
     <xacro:property name="end_effector" value="$(arg end_effector)" />
@@ -33,4 +34,5 @@
     <xacro:property name="is_multiple" value="$(arg multiple)" />
     <xacro:property name="nsp" value="$(arg namespace)" />
+    <xacro:property name="base_type" value="$(arg base_type)" />
     <xacro:property name="no_safety_eps" value="$(arg no_safety_eps)" />
   <xacro:if value="$(arg arm)">
@@ -51,4 +53,7 @@
     <xacro:wrong_camera_model/>
   </xacro:if>
+  <xacro:if value="${base_type not in ['pmb2', 'omni_base']}">
+    <xacro:wrong_base_type/>
+  </xacro:if>
         <!-- The properties below are modified using empy http://www.alcyone.com/software/empy/
              from the create_robot.py tool. Handle them with care -->
@@ -62,5 +67,5 @@
   <!-- The following included files set up definitions of parts of the robot body -->
   <!-- Base -->
-  <xacro:include filename="$(find pmb2_description)/urdf/base/base_sensors.urdf.xacro" />
+  <xacro:include filename="$(find ${base_type}_description)/urdf/base/base_sensors.urdf.xacro" />
   <!-- Torso -->
   <xacro:include filename="$(find tiago_description)/urdf/torso/torso.urdf.xacro" />
@@ -77,10 +82,17 @@
   <!-- Head -->
   <xacro:include filename="$(find tiago_description)/urdf/head/head.urdf.xacro" />
-  <!-- Generic simulator_gazebo plugins -->
-  <xacro:include filename="$(find tiago_description)/gazebo/gazebo.urdf.xacro" />
   <!-- Materials for visualization -->
   <xacro:include filename="$(find tiago_description)/urdf/materials.urdf.xacro" />
   <!-- Now we can start using the macros included above to define the actual robot -->
-  <xacro:base_sensors name="base" laser_model="$(arg laser_model)" sonars="true" microphone="true"/>
+  <xacro:if value="${base_type == 'pmb2'}">
+    <!-- Generic simulator_gazebo plugins -->
+    <xacro:include filename="$(find tiago_description)/gazebo/gazebo.urdf.xacro" />
+    <xacro:base_sensors name="base" laser_model="$(arg laser_model)" sonars="true" microphone="true"/>
+  </xacro:if>
+  <xacro:if value="${base_type == 'omni_base'}">
+    <!-- Generic simulator_gazebo plugins -->
+    <xacro:include filename="$(find tiago_description)/gazebo/gazebo_omni.urdf.xacro" />
+    <xacro:base_sensors name="base" front_laser_model="$(arg laser_model)" rear_laser_model="$(arg laser_model)"/>
+  </xacro:if>
   <xacro:tiago_torso name="torso" parent="base_link"/>
   <xacro:head name="head" parent="torso_lift_link" camera_model="$(arg camera_model)"

Commit message: Update eval function, generate scripts

File: tiago_description/robots/tiago.urdf.xacro (robot description, xacro)
@@ -41,5 +41,5 @@
     </xacro:if>
   </xacro:if>
-  <xacro:if value="${end_effector not in ['false', False, 'pal-gripper', 'pal-hey5', 'schunk-wsg', 'robotiq-2f-85', 'robotiq-2f-140', 'custom']}">
+  <xacro:if value="${end_effector not in ['false', False, 'pal-gripper', 'pal-hey5', 'schunk-wsg', 'robotiq-2f-85', 'robotiq-2f-140', 'custom', 'no-ee']}">
     <xacro:wrong_end_effector/>
   </xacro:if>
@@ -61,4 +61,5 @@
    <xacro:property name="has_schunk_ft"           value="${ft_sensor == 'schunk-ft'}"/>
    <xacro:property name="has_ft_sensor"           value="${has_schunk_ft}"/> <!-- This should be OR'ed with other FT sensors-->
+   <xacro:property name="has_end_effector"        value="${end_effector != 'false'}"/>
    <xacro:property name="end_effector_link"       value="${'wrist_ft_tool_link' if has_ft_sensor else 'arm_tool_link'}"/>
    <xacro:property name="end_effector_name"       value="${'hand' if end_effector == 'pal-hey5' else 'gripper'}"/>
@@ -102,5 +103,5 @@
         <origin xyz="0.15505 0.014 -0.151" rpy="0 0 ${-90 * deg_to_rad}" />
       </xacro:tiago_arm>
-      <xacro:tiago_end_effector name="${end_effector_name}" parent="${end_effector_link}" type="${end_effector}" reflect="1"/>
+      <xacro:tiago_end_effector name="${end_effector_name}" parent="${end_effector_link}" type="${end_effector}" has_end_effector="${has_end_effector}" reflect="1"/>
   </xacro:if>
   <!-- Force Torque sensor -->

File: tiago_description/urdf/end_effector/end_effector.urdf.xacro (robot description, xacro)
@@ -23,5 +23,27 @@
     - reflect: Set to 1 for a right end effector, or to -1 for a left end effector
   -->
-  <xacro:macro name="tiago_end_effector" params="name parent type reflect is_dual:=false">
+  <xacro:macro name="tiago_end_effector" params="name parent type has_end_effector reflect is_dual:=false">
+  <!-- No end-effector -->
+  <xacro:unless value="${has_end_effector}">
+    <xacro:include filename="$(find custom_ee_description)/urdf/end-effector.urdf.xacro" />
+    <xacro:end_effector parent="${parent}">
+      <origin xyz="0.01 0 0" rpy="${90*deg_to_rad} ${90*deg_to_rad} ${-90*deg_to_rad}"/>
+    </xacro:end_effector>
+  </xacro:unless>
+    <!-- No end-effector dual-->
+  <xacro:unless value="${has_end_effector and is_dual}">
+    <xacro:if value="${reflect == 1}"> <!-- If right -->
+    <xacro:include filename="$(find custom_dual_ee_description)/urdf/end-effector-right.urdf.xacro" />
+    <xacro:end_effector_right parent="${parent}">
+      <origin xyz="0.01 0 0" rpy="${90*deg_to_rad} ${90*deg_to_rad} ${-90*deg_to_rad}"/>
+    </xacro:end_effector_right>
+    </xacro:if>
+    <xacro:if value="${reflect == -1}"> <!-- If left -->
+    <xacro:include filename="$(find custom_dual_ee_description)/urdf/end-effector-left.urdf.xacro" />
+    <xacro:end_effector_left parent="${parent}">
+      <origin xyz="0.01 0 0" rpy="${90*deg_to_rad} ${90*deg_to_rad} ${-90*deg_to_rad}"/>
+    </xacro:end_effector_left>
+    </xacro:if>
+  </xacro:unless>
   <!-- PAL Gripper -->
   <xacro:if value="${type == 'pal-gripper'}">

Commit message: Update eval function, generate scripts

File: tiago_description/robots/tiago.urdf.xacro (robot description, xacro)
@@ -41,5 +41,5 @@
     </xacro:if>
   </xacro:if>
-  <xacro:if value="${end_effector not in ['false', False, 'pal-gripper', 'pal-hey5', 'schunk-wsg', 'robotiq-2f-85', 'robotiq-2f-140', 'robotiq-epick', 'custom']}">
+  <xacro:if value="${end_effector not in ['false', False, 'pal-gripper', 'pal-hey5', 'schunk-wsg', 'robotiq-2f-85', 'robotiq-2f-140', 'robotiq-epick', 'custom', 'no-ee']}">
     <xacro:wrong_end_effector/>
   </xacro:if>

File: tiago_description/urdf/end_effector/end_effector.urdf.xacro (robot description, xacro)
@@ -23,5 +23,9 @@
     - reflect: Set to 1 for a right end effector, or to -1 for a left end effector
   -->
-  <xacro:macro name="tiago_end_effector" params="name parent type reflect is_dual:=false">
+  <xacro:macro name="tiago_end_effector" params="name parent type has_end_effector reflect is_dual:=false">
+  <!-- No end-effector -->
+  <xacro:if value="${not has_end_effector}">
+    <!-- Add nothing -->
+  </xacro:if>
   <!-- PAL Gripper -->
   <xacro:if value="${type == 'pal-gripper'}">

Commit message: Update eval function, generate scripts

File: tiago_description/robots/tiago.urdf.xacro (robot description, xacro)
@@ -41,5 +41,5 @@
     </xacro:if>
   </xacro:if>
-  <xacro:if value="${end_effector not in ['false', False, 'pal-gripper', 'pal-hey5', 'schunk-wsg', 'robotiq-2f-85', 'robotiq-2f-140', 'robotiq-epick', 'custom']}">
+  <xacro:if value="${end_effector not in ['false', False, 'pal-gripper', 'pal-hey5', 'schunk-wsg', 'robotiq-2f-85', 'robotiq-2f-140', 'robotiq-epick', 'custom', 'no-ee']}">
     <xacro:wrong_end_effector/>
   </xacro:if>
@@ -61,4 +61,5 @@
    <xacro:property name="has_schunk_ft"           value="${ft_sensor == 'schunk-ft'}"/>
    <xacro:property name="has_ft_sensor"           value="${has_schunk_ft}"/> <!-- This should be OR'ed with other FT sensors-->
+   <xacro:property name="has_end_effector"        value="${end_effector != 'false'}"/>
    <xacro:property name="end_effector_link"       value="${'wrist_ft_tool_link' if has_ft_sensor else 'arm_tool_link'}"/>
    <xacro:property name="end_effector_name"       value="${'hand' if end_effector == 'pal-hey5' else 'gripper'}"/>
@@ -102,5 +103,5 @@
         <origin xyz="0.15505 0.014 -0.151" rpy="0 0 ${-90 * deg_to_rad}" />
       </xacro:tiago_arm>
-      <xacro:tiago_end_effector name="${end_effector_name}" parent="${end_effector_link}" type="${end_effector}" reflect="1"/>
+      <xacro:tiago_end_effector name="${end_effector_name}" parent="${end_effector_link}" type="${end_effector}" has_end_effector="${has_end_effector}" reflect="1"/>
   </xacro:if>
   <!-- Force Torque sensor -->

File: tiago_description/urdf/end_effector/end_effector.urdf.xacro (robot description, xacro)
@@ -23,5 +23,27 @@
     - reflect: Set to 1 for a right end effector, or to -1 for a left end effector
   -->
-  <xacro:macro name="tiago_end_effector" params="name parent type reflect is_dual:=false">
+  <xacro:macro name="tiago_end_effector" params="name parent type has_end_effector reflect is_dual:=false">
+  <!-- No end-effector -->
+  <xacro:unless value="${has_end_effector}">
+    <xacro:include filename="$(find custom_ee_description)/urdf/end-effector.urdf.xacro" />
+    <xacro:end_effector parent="${parent}">
+      <origin xyz="0.01 0 0" rpy="${90*deg_to_rad} ${90*deg_to_rad} ${-90*deg_to_rad}"/>
+    </xacro:end_effector>
+  </xacro:unless>
+    <!-- No end-effector dual-->
+  <xacro:unless value="${has_end_effector and is_dual}">
+    <xacro:if value="${reflect == 1}"> <!-- If right -->
+    <xacro:include filename="$(find custom_dual_ee_description)/urdf/end-effector-right.urdf.xacro" />
+    <xacro:end_effector_right parent="${parent}">
+      <origin xyz="0.01 0 0" rpy="${90*deg_to_rad} ${90*deg_to_rad} ${-90*deg_to_rad}"/>
+    </xacro:end_effector_right>
+    </xacro:if>
+    <xacro:if value="${reflect == -1}"> <!-- If left -->
+    <xacro:include filename="$(find custom_dual_ee_description)/urdf/end-effector-left.urdf.xacro" />
+    <xacro:end_effector_left parent="${parent}">
+      <origin xyz="0.01 0 0" rpy="${90*deg_to_rad} ${90*deg_to_rad} ${-90*deg_to_rad}"/>
+    </xacro:end_effector_left>
+    </xacro:if>
+  </xacro:unless>
   <!-- PAL Gripper -->
   <xacro:if value="${type == 'pal-gripper'}">

Commit message: made some changes

File: tiago_description/robots/tiago.urdf.xacro (robot description, xacro)
@@ -61,4 +61,5 @@
    <xacro:property name="has_schunk_ft"           value="${ft_sensor == 'schunk-ft'}"/>
    <xacro:property name="has_ft_sensor"           value="${has_schunk_ft}"/> <!-- This should be OR'ed with other FT sensors-->
+   <xacro:property name="has_end_effector"        value="${end_effector != 'false'}"/>
    <xacro:property name="end_effector_link"       value="${'wrist_ft_tool_link' if has_ft_sensor else 'arm_tool_link'}"/>
    <xacro:property name="end_effector_name"       value="${'hand' if end_effector == 'pal-hey5' else 'gripper'}"/>
@@ -102,5 +103,5 @@
         <origin xyz="0.15505 0.014 -0.151" rpy="0 0 ${-90 * deg_to_rad}" />
       </xacro:tiago_arm>
-      <xacro:tiago_end_effector name="${end_effector_name}" parent="${end_effector_link}" type="${end_effector}" reflect="1"/>
+      <xacro:tiago_end_effector name="${end_effector_name}" parent="${end_effector_link}" type="${end_effector}" has_end_effector="${has_end_effector}" reflect="1"/>
   </xacro:if>
   <!-- Force Torque sensor -->

Commit message: add no-ee to urdf

File: tiago_description/robots/tiago.urdf.xacro (robot description, xacro)
@@ -41,5 +41,5 @@
     </xacro:if>
   </xacro:if>
-  <xacro:if value="${end_effector not in ['false', False, 'pal-gripper', 'pal-hey5', 'schunk-wsg', 'robotiq-2f-85', 'robotiq-2f-140', 'custom']}">
+  <xacro:if value="${end_effector not in ['false', False, 'pal-gripper', 'pal-hey5', 'schunk-wsg', 'robotiq-2f-85', 'robotiq-2f-140', 'custom', 'no-ee']}">
     <xacro:wrong_end_effector/>
   </xacro:if>

File: tiago_description/urdf/end_effector/end_effector.urdf.xacro (robot description, xacro)
@@ -24,28 +24,7 @@
   -->
   <xacro:macro name="tiago_end_effector" params="name parent type has_end_effector reflect is_dual:=false">
-  <!-- For now the custom end-effector is used in the case of no end-effector -->
+  <!-- No end-effector -->
   <xacro:if value="${not has_end_effector}">
-    <!-- No end-effector single-->
-    <xacro:if values="${not is_dual}">
-      <xacro:include filename="$(find custom_ee_description)/urdf/end-effector.urdf.xacro" />
-      <xacro:end_effector parent="${parent}">
-        <origin xyz="0.01 0 0" rpy="${90*deg_to_rad} ${90*deg_to_rad} ${-90*deg_to_rad}"/>
-      </xacro:end_effector>
-    </xacro:if>
-  <!-- No end-effector dual -->
-    <xacro:if value="${is_dual}">
-      <xacro:if value="${reflect == 1}">
-        <xacro:include filename="$(find custom_dual_ee_description)/urdf/end-effector-right.urdf.xacro" />
-        <xacro:end_effector_right parent="${parent}">
-          <origin xyz="0.01 0 0" rpy="${90*deg_to_rad} ${90*deg_to_rad} ${-90*deg_to_rad}"/>
-        </xacro:end_effector_right>
-      </xacro:if>
-      <xacro:if value="${reflect == -1}">
-        <xacro:include filename="$(find custom_dual_ee_description)/urdf/end-effector-left.urdf.xacro" />
-        <xacro:end_effector_left parent="${parent}">
-          <origin xyz="0.01 0 0" rpy="${90*deg_to_rad} ${90*deg_to_rad} ${-90*deg_to_rad}"/>
-        </xacro:end_effector_left>
-      </xacro:if>
-    </xacro:if>
+    <!-- Add nothing -->
   </xacro:if>
   <!-- PAL Gripper -->

Commit message: Apply 5 suggestion(s) to 4 file(s)

File: tiago_description/robots/tiago.urdf.xacro (robot description, xacro)
@@ -61,5 +61,5 @@
    <xacro:property name="has_schunk_ft"           value="${ft_sensor == 'schunk-ft'}"/>
    <xacro:property name="has_ft_sensor"           value="${has_schunk_ft}"/> <!-- This should be OR'ed with other FT sensors-->
-   <xacro:property name="has_end_effector"        value="${end_effector != 'false'}"/>
+   <xacro:property name="has_end_effector"        value="${end_effector not in ['false', False, 'no-ee']}"/>
    <xacro:property name="end_effector_link"       value="${'wrist_ft_tool_link' if has_ft_sensor else 'arm_tool_link'}"/>
    <xacro:property name="end_effector_name"       value="${'hand' if end_effector == 'pal-hey5' else 'gripper'}"/>
