Commit message: add use_sim arg

File: tiago_description/robots/tiago.urdf.xacro (robot description, xacro)
@@ -21,4 +21,5 @@
     <xacro:arg name="namespace" default=""/>
     <xacro:arg name="no_safety_eps" default="false"/>
+    <xacro:arg name="use_sim" default="true"/>
     <xacro:property name="arm" value="$(arg arm)" />
     <xacro:if value="${arm not in ['right-arm', 'left-arm', 'no-arm']}">
@@ -81,4 +82,6 @@
   <!-- ros2_control -->
   <xacro:include filename="$(find tiago_description)/ros2_control/ros2_control.urdf.xacro" />
+  <xacro:tiago_ros2_control
+    use_sim="$(arg use_sim)" />
   <!-- Materials for visualization -->
   <xacro:include filename="$(find tiago_description)/urdf/materials.urdf.xacro" />

File: tiago_description/ros2_control/ros2_control.urdf.xacro (robot description, xacro)
@@ -9,66 +9,77 @@
 <robot xmlns:xacro="http://ros.org/wiki/xacro"
        name="tiago" >
-  <xacro:arg name="arm" default="true" />
-  <xacro:arg name="end_effector" default="pal-hey5"/>
-  <xacro:arg name="description_calibration_dir" default="$(find tiago_description_calibration)/urdf/calibration" />
-  <xacro:property name="has_arm" value="${arm != 'no-arm'}" />
-  <xacro:property name="end_effector" value="$(arg end_effector)" />
-  <xacro:include filename="$(find pmb2_description)/urdf/wheels/wheel.ros2_control.xacro" />
-  <xacro:include filename="$(find tiago_description)/urdf/torso/torso.ros2_control.xacro" />
-  <xacro:include filename="$(find tiago_description)/urdf/head/head.ros2_control.xacro" />
-  <xacro:if value="${has_arm}">
-    <xacro:include filename="$(find tiago_description)/urdf/arm/arm.ros2_control.xacro" />
-    <xacro:include filename="$(find tiago_description)/urdf/arm/wrist.ros2_control.xacro" />
-    <xacro:if value="${end_effector == 'pal-gripper'}">
-      <xacro:include filename="$(find pal_gripper_description)/urdf/gripper.ros2_control.xacro" />
-    </xacro:if>
-    <xacro:if value="${end_effector == 'pal-hey5'}">
-      <xacro:include filename="$(find tiago_description)/urdf/end_effector/pal-hey5.ros2_control.xacro" />
-    </xacro:if>
-  </xacro:if>
-  <xacro:include filename="$(find pmb2_description)/urdf/sensors/sensors.ros2_control.xacro"/>
-  <!-- calibration offsets -->
-  <xacro:include filename="$(arg description_calibration_dir)/calibration_constants.urdf.xacro" />
-  <ros2_control name="ros2_control_tiago_system" type="system">
-    <hardware>
-      <plugin>gazebo_ros2_control/GazeboSystem</plugin>
-    </hardware>
-    <!-- wheels -->
-    <xacro:ros2_control_wheel side="right" />
-    <xacro:ros2_control_wheel side="left" />
-    <!-- IMU -->
-    <xacro:ros2_control_imu name="base_imu_sensor"/>
-    <!-- torso -->
-    <xacro:ros2_control_torso name="torso_lift" reduction="1.0" />
-    <!-- head -->
-    <xacro:ros2_control_head name="head_1" reduction="1.0" offset="${head_1_joint_offset}" />
-    <xacro:ros2_control_head name="head_2" reduction="1.0" offset="${head_2_joint_offset}" />
+  <xacro:macro name="tiago_ros2_control" params="use_sim:=^|true">
+    <xacro:arg name="arm" default="true" />
+    <xacro:arg name="end_effector" default="pal-hey5"/>
+    <xacro:arg name="description_calibration_dir" default="$(find tiago_description_calibration)/urdf/calibration" />
+    <xacro:property name="has_arm" value="${arm != 'no-arm'}" />
+    <xacro:property name="end_effector" value="$(arg end_effector)" />
+    <xacro:include filename="$(find pmb2_description)/urdf/wheels/wheel.ros2_control.xacro" />
+    <xacro:include filename="$(find tiago_description)/urdf/torso/torso.ros2_control.xacro" />
+    <xacro:include filename="$(find tiago_description)/urdf/head/head.ros2_control.xacro" />
     <xacro:if value="${has_arm}">
-      <!-- arm -->
-      <xacro:ros2_control_arm name="arm_1" reduction="1.0" offset="${arm_1_joint_offset}" />
-      <xacro:ros2_control_arm name="arm_2" reduction="1.0" offset="${arm_2_joint_offset}" />
-      <xacro:ros2_control_arm name="arm_3" reduction="1.0" offset="${arm_3_joint_offset}" />
-      <xacro:ros2_control_arm name="arm_4" reduction="1.0" offset="${arm_4_joint_offset}" />
-      <!-- wrist -->
-      <xacro:ros2_control_wrist_rotational name="arm_5" reduction="1.0" offset="${arm_5_joint_offset}" />
-      <xacro:ros2_control_wrist_differential name_1="arm_6" name_2="arm_7"
-                                             act_reduction_1="-1.0" act_reduction_2="1.0"
-                                             jnt_reduction_1="1.0" jnt_reduction_2="1.0"
-                                             number_1_offset="${arm_6_joint_offset}" number_2_offset="${arm_7_joint_offset}" />
+      <xacro:include filename="$(find tiago_description)/urdf/arm/arm.ros2_control.xacro" />
+      <xacro:include filename="$(find tiago_description)/urdf/arm/wrist.ros2_control.xacro" />
       <xacro:if value="${end_effector == 'pal-gripper'}">
-        <!-- pal-gripper -->
-        <xacro:ros2_control_gripper name="gripper_left_finger" reduction="1.0" />
-        <xacro:ros2_control_gripper name="gripper_right_finger" reduction="1.0" />
+        <xacro:include filename="$(find pal_gripper_description)/urdf/gripper.ros2_control.xacro" />
       </xacro:if>
       <xacro:if value="${end_effector == 'pal-hey5'}">
-        <!-- pal-hey5 -->
-        <xacro:ros2_control_hey5 name="hand"/>
+        <xacro:include filename="$(find tiago_description)/urdf/end_effector/pal-hey5.ros2_control.xacro" />
       </xacro:if>
     </xacro:if>
-    <!-- Force Torque sensor -->
-    <xacro:if value="${has_ft_sensor}">
-      <xacro:include filename="$(find tiago_description)/urdf/sensors/sensors.ros2_control.xacro"/>
-      <xacro:ros2_control_force_torque_sensor name="wrist_ft_joint_force_torque"/>
-    </xacro:if>
-  </ros2_control>
+    <xacro:include filename="$(find pmb2_description)/urdf/sensors/sensors.ros2_control.xacro"/>
+    <!-- calibration offsets -->
+    <xacro:include filename="$(arg description_calibration_dir)/calibration_constants.urdf.xacro" />
+    <ros2_control name="ros2_control_tiago_system" type="system">
+      <hardware>
+        <xacro:if value="$(arg use_sim)">
+          <plugin>gazebo_ros2_control/GazeboSystem</plugin>
+        </xacro:if>
+        <xacro:unless value="$(arg use_sim)">
+          <plugin>robot_control/RobotControl</plugin>
+        </xacro:unless>
+      </hardware>
+      <!-- wheels -->
+      <xacro:ros2_control_wheel side="right" />
+      <xacro:ros2_control_wheel side="left" />
+      <!-- IMU -->
+      <xacro:if value="$(arg use_sim)">
+        <xacro:ros2_control_imu name="base_imu_sensor"/>
+      </xacro:if>
+      <!-- torso -->
+      <xacro:ros2_control_torso name="torso_lift" reduction="1.0" />
+      <!-- head -->
+      <xacro:ros2_control_head name="head_1" reduction="1.0" offset="${head_1_joint_offset}" />
+      <xacro:ros2_control_head name="head_2" reduction="1.0" offset="${head_2_joint_offset}" />
+      <xacro:if value="${has_arm}">
+        <!-- arm -->
+        <xacro:ros2_control_arm name="arm_1" reduction="1.0" offset="${arm_1_joint_offset}" />
+        <xacro:ros2_control_arm name="arm_2" reduction="1.0" offset="${arm_2_joint_offset}" />
+        <xacro:ros2_control_arm name="arm_3" reduction="1.0" offset="${arm_3_joint_offset}" />
+        <xacro:ros2_control_arm name="arm_4" reduction="1.0" offset="${arm_4_joint_offset}" />
+        <!-- wrist -->
+        <xacro:ros2_control_wrist_rotational name="arm_5" reduction="1.0" offset="${arm_5_joint_offset}" />
+        <xacro:ros2_control_wrist_differential name_1="arm_6" name_2="arm_7"
+                                               act_reduction_1="-1.0" act_reduction_2="1.0"
+                                               jnt_reduction_1="1.0" jnt_reduction_2="1.0"
+                                               number_1_offset="${arm_6_joint_offset}" number_2_offset="${arm_7_joint_offset}" />
+        <xacro:if value="${end_effector == 'pal-gripper'}">
+          <!-- pal-gripper -->
+          <xacro:ros2_control_gripper name="gripper_left_finger" reduction="1.0" />
+          <xacro:ros2_control_gripper name="gripper_right_finger" reduction="1.0" />
+        </xacro:if>
+        <xacro:if value="${end_effector == 'pal-hey5'}">
+          <!-- pal-hey5 -->
+          <xacro:ros2_control_hey5 name="hand"/>
+        </xacro:if>
+      </xacro:if>
+      <!-- Force Torque sensor -->
+      <xacro:if value="${has_ft_sensor}">
+        <xacro:include filename="$(find tiago_description)/urdf/sensors/sensors.ros2_control.xacro"/>
+        <xacro:if value="$(arg use_sim)">
+          <xacro:ros2_control_force_torque_sensor name="wrist_ft_joint_force_torque"/>
+        </xacro:if>
+      </xacro:if>
+    </ros2_control>
+  </xacro:macro>
 </robot>

Commit message: Added fixed_torso parameter to main xacro

File: tiago_description/robots/tiago.urdf.xacro (robot description, xacro)
@@ -27,4 +27,5 @@
     <xacro:arg name="no_safety_eps" default="false"/>
     <xacro:arg name="base_type" default="pmb2"/> <!-- pmb2, omni_base -->
+    <xacro:arg name="fixed_torso" default="false" />
     <xacro:property name="wrist_model" value="$(arg wrist_model)" />
     <xacro:property name="end_effector" value="$(arg end_effector)" />
@@ -36,4 +37,5 @@
     <xacro:property name="base_type" value="$(arg base_type)" />
     <xacro:property name="no_safety_eps" value="$(arg no_safety_eps)" />
+    <xacro:property name="fixed_torso" value="$(arg fixed_torso)" />
   <xacro:if value="$(arg arm)">
     <xacro:if value="${wrist_model not in ['wrist-2010', 'wrist-2017']}">

Commit message: Set use_sim_time false as default

File: tiago_description/robots/tiago.urdf.xacro (robot description, xacro)
@@ -26,5 +26,5 @@
     <xacro:arg name="namespace" default=""/>
     <xacro:arg name="no_safety_eps" default="false"/>
-    <xacro:arg name="use_sim" default="true"/>
+    <xacro:arg name="use_sim" default="false"/>
     <xacro:property name="arm" value="$(arg arm)" />
     <xacro:if value="${arm not in ['right-arm', 'no-arm']}">

File: tiago_description/ros2_control/ros2_control.urdf.xacro (robot description, xacro)
@@ -14,5 +14,5 @@
 <robot xmlns:xacro="http://ros.org/wiki/xacro"
        name="tiago" >
-  <xacro:macro name="tiago_ros2_control" params="use_sim:=^|true">
+  <xacro:macro name="tiago_ros2_control" params="use_sim:=^|false">
     <xacro:arg name="arm" default="true" />
     <xacro:arg name="end_effector" default="pal-hey5"/>

Commit message: adding robotiq_grippers as possibles end_effectors

File: tiago_description/robots/tiago.urdf.xacro (robot description, xacro)
@@ -45,5 +45,5 @@
     </xacro:if>
   </xacro:if>
-  <xacro:if value="${end_effector not in ['no-end-effector', 'pal-gripper', 'pal-hey5', 'custom']}">
+  <xacro:if value="${end_effector not in ['no-end-effector', 'pal-gripper', 'pal-hey5', 'custom', 'robotiq-2f-85', 'robotiq-2f-140', 'robotiq-epick']}">
     <xacro:wrong_end_effector/>
   </xacro:if>

File: tiago_description/ros2_control/ros2_control.urdf.xacro (robot description, xacro)
@@ -31,4 +31,10 @@
       <xacro:if value="${end_effector == 'pal-hey5'}">
         <xacro:include filename="$(find pal_hey5_description)/urdf/pal_hey5.ros2_control.xacro" />
+      </xacro:if>
+      <xacro:if value="${end_effector == 'pal-robtiq-2f-85'}">
+        <xacro:include filename="$(find pal_robotiq_description)/urdf/pal_robotiq.ros2_control.xacro" />
+      </xacro:if>
+      <xacro:if value="${end_effector == 'pal-robtiq-2f-140'}">
+        <xacro:include filename="$(find pal_robotiq_description)/urdf/pal_robotiq.ros2_control.xacro" />
       </xacro:if>
     </xacro:if>

File: tiago_description/urdf/end_effector/end_effector.urdf.xacro (robot description, xacro)
@@ -30,4 +30,25 @@
       <origin xyz="0.01 0 0" rpy="${90*deg_to_rad} ${90*deg_to_rad} ${-90*deg_to_rad}"/>
     </xacro:pal_gripper>
+  </xacro:if>
+  <!-- Robotiq 2F-85 Gripper -->
+  <xacro:if value="${type == 'robotiq-2f-85'}">
+    <xacro:include filename="$(find pal_robotiq_85_description)/urdf/robotiq_85_gripper.urdf.xacro" />
+    <xacro:robotiq_85_gripper prefix="${name}_" parent="${parent}" >
+      <origin xyz="0.01 0 0" rpy="${90*deg_to_rad} ${0*deg_to_rad} ${90*deg_to_rad}"/>
+    </xacro:robotiq_85_gripper>
+  </xacro:if>
+  <!-- Robotiq 2F-140 Gripper -->
+  <xacro:if value="${type == 'robotiq-2f-140'}">
+    <xacro:include filename="$(find pal_robotiq_140_description)/urdf/robotiq_140_gripper.urdf.xacro" />
+    <xacro:robotiq_140_gripper prefix="${name}_" parent="${parent}" >
+      <origin xyz="0.01 0 0" rpy="${90*deg_to_rad} ${0*deg_to_rad} ${90*deg_to_rad}"/>
+    </xacro:robotiq_140_gripper>
+  </xacro:if>
+  <!-- Robotiq Epick Gripper -->
+  <xacro:if value="${type == 'robotiq-epick'}">
+    <xacro:include filename="$(find pal_robotiq_epick_description)/urdf/robotiq_epick_model_macro.xacro" />
+    <xacro:epick_hand  prefix="${name}_" parent="${parent}">
+      <origin xyz="0.01 0 0" rpy="${90*deg_to_rad} ${0*deg_to_rad} ${90*deg_to_rad}"/>
+    </xacro:epick_hand>
   </xacro:if>
   <!-- Hand -->

Commit message: Add screen parameter and screen stl file in the urdf

File: tiago_description/robots/tiago.urdf.xacro (robot description, xacro)
@@ -29,4 +29,5 @@
     <xacro:arg name="fixed_torso" default="false" />
     <xacro:arg name="gazebo_control_period" default="0.001"/> <!-- 1000Hz or 100 Hz-->
+    <xacro:arg name="has_screen" default="false"/> <!-- True, False -->
     <xacro:property name="wrist_model" value="$(arg wrist_model)" />
     <xacro:property name="end_effector" value="$(arg end_effector)" />
@@ -40,4 +41,5 @@
     <xacro:property name="fixed_torso" value="$(arg fixed_torso)" />
     <xacro:property name="gazebo_control_period" value="$(arg gazebo_control_period)" />
+    <xacro:property name="has_screen" value="$(arg has_screen)" />
   <xacro:if value="$(arg arm)">
     <xacro:if value="${wrist_model not in ['wrist-2010', 'wrist-2017']}">
@@ -100,5 +102,5 @@
     <xacro:base_sensors name="base" front_laser_model="$(arg laser_model)" rear_laser_model="$(arg laser_model)"/>
   </xacro:if>
-  <xacro:tiago_torso name="torso" parent="base_link"/>
+  <xacro:tiago_torso name="torso" parent="base_link" has_screen="$(arg has_screen)"/>
   <xacro:head name="head" parent="torso_lift_link" camera_model="$(arg camera_model)"
 	  description_calibration_dir="$(arg description_calibration_dir)"

File: tiago_description/urdf/torso/torso.urdf.xacro (robot description, xacro)
@@ -18,5 +18,5 @@
   <xacro:property name="torso_max_vel"  value="0.07" />
   <xacro:property name="torso_eps"      value="0.02" />
-  <xacro:macro name="tiago_torso" params="name parent">
+  <xacro:macro name="tiago_torso" params="name parent has_screen">
   <!-- Bottom fixed part of column -->
   <link name="${name}_fixed_link">
@@ -149,4 +149,34 @@
     <xacro:torso_simple_transmission name="torso_lift" reduction="1.0" />
   </xacro:unless>
+  <xacro:if value="$(arg has_screen)">
+    <link name="${name}_screen_link">
+      <inertial>
+        <origin xyz="0.00004923 0.000001  -0.00000308" rpy="0.00000 0.00000 0.00000"/>
+        <mass value="0.96841"/>
+        <inertia ixx="0.0" ixy="1.0" ixz="0.0"
+                iyy="0.24926900000" iyz="0.00828100000"
+                izz="0.09039500000"/>
+      </inertial>
+      <visual>
+        <origin rpy="3.14159 0 0" xyz="-0.0425 0.1275 0.065" />
+        <geometry>
+          <mesh filename="package://tiago_description/meshes/torso/tiago_screen.STL" scale="0.001 0.001 0.001"/>
+        </geometry>
+        <material name="White"/>
+      </visual>
+      <collision>
+        <origin rpy="3.14159 0 0" xyz="-0.040 0.1275 0.065" />
+        <geometry>
+          <mesh filename="package://tiago_description/meshes/torso/tiago_screen.STL" scale="0.001 0.001 0.001"/>
+        </geometry>
+        <material name="LightGrey"/>
+      </collision>
+    </link>
+    <joint name="${name}_screen_joint" type="fixed">
+      <origin rpy="0.0 0.0 1.57" xyz="-0.02 0.125 -0.27" />
+      <parent link="${name}_lift_link" />
+      <child link="${name}_screen_link" />
+    </joint>
+  </xacro:if>
  </xacro:macro>
 </robot>

Commit message: Fix Issue #27: Add fixed joint for base_sonar_01_link to resolve TF error

File: tiago_description/robots/tiago.urdf.xacro (robot description, xacro)
@@ -110,4 +110,10 @@
   <!-- Base -->
   <xacro:include filename="$(find ${base_type}_description)/urdf/base/base_sensors.urdf.xacro" />
+    <!-- Fixed joint to mount the sonar sensor (base_sonar_01_link) -->
+  <joint name="sonar_mount_joint" type="fixed">
+    <origin xyz="0.2 0.0 0.15" rpy="0 0 0"/>
+    <parent link="base_link"/>
+    <child link="base_sonar_01_link"/>
+  </joint>
   <!-- Torso -->
   <xacro:include filename="$(find tiago_description)/urdf/torso/torso.urdf.xacro" />

Commit message: Add gazebo_version xacro argument

File: tiago_description/robots/tiago.urdf.xacro (robot description, xacro)
@@ -51,4 +51,5 @@
   <xacro:arg name="namespace" default=""/>
   <xacro:arg name="is_public_sim" default="false"/>
+  <xacro:arg name="gazebo_version" default="classic"/>
   <!-- PROPERTIES -->
   <!-- HW configuration -->
@@ -105,4 +106,5 @@
   <xacro:property name="namespace" value="$(arg namespace)" />
   <xacro:property name="is_public_sim" value="$(arg is_public_sim)" />
+  <xacro:property name="gazebo_version" value="$(arg gazebo_version)" />
   <!-- INCLUDES -->
   <!-- Tools -->

Commit message: add calibration_tool parameter

File: tiago_description/robots/tiago.urdf.xacro (robot description, xacro)
@@ -43,4 +43,6 @@
   <!-- false, true -->
   <xacro:arg name="no_safety_eps" default="false"/>
+  <!-- False, True -->
+  <xacro:arg name="calibration_tool" default="False" />
   <!-- Calibration -->
   <xacro:arg name="eye_hand_calibration_dir" default="$(find tiago_description)/urdf/calibration"/>
@@ -64,4 +66,5 @@
   <xacro:property name="has_screen" value="$(arg has_screen)" />
   <xacro:property name="no_safety_eps" value="$(arg no_safety_eps)" />
+  <xacro:property name="calibration_tool" value="$(arg calibration_tool)"/>
   <!-- HW configuration check -->
   <xacro:if value="${base_type not in ['pmb2', 'omni_base']}">

File: tiago_description/urdf/calibration/eye_hand_calibration.urdf.xacro (robot description, xacro)
@@ -27,5 +27,5 @@
   <xacro:property name="arm_4_joint_offset" value="0.0" />
   <xacro:property name="arm_5_joint_offset" value="0.0" />
-  <xacro:property name="arm_6_joint_offset" value="0.0" />
+  <xacro:property name="arm_6_joint_offset" value="-0.0" />
   <xacro:property name="arm_7_joint_offset" value="0.0" />
   <xacro:property name="head_1_joint_offset" value="0.0" />

File: tiago_description/urdf/end_effector/end_effector.urdf.xacro (robot description, xacro)
@@ -30,5 +30,5 @@
     <!-- PAL Gripper -->
     <xacro:if value="${end_effector == 'pal-gripper'}">
-      <xacro:pal_gripper parent="${parent}" name="${name}">
+      <xacro:pal_gripper parent="${parent}" name="${name}" calibration_tool="${calibration_tool}">
         <origin xyz="0 0 0" rpy="${90*deg_to_rad} ${90*deg_to_rad} ${-90*deg_to_rad}"/>
       </xacro:pal_gripper>
