Commit message: rename frame

File: tiago_description/urdf/chessboard/chessboard.gazebo.xacro (robot description, xacro)
@@ -9,5 +9,5 @@
 <robot xmlns:xacro="http://ros.org/wiki/xacro">
   <xacro:macro name="chessboard_gazebo" params="name texture">
-    <gazebo reference="chessboard_${name}_link">
+    <gazebo reference="${name}_link">
       <material>${texture}</material>
     </gazebo>

File: tiago_description/urdf/chessboard/chessboard.urdf.xacro (robot description, xacro)
@@ -9,5 +9,5 @@
 <robot xmlns:xacro="http://ros.org/wiki/xacro">
   <xacro:macro name="chessboard" params="name parent origin rpy">
-    <link name="chessboard_${name}_link">
+    <link name="${name}_link">
       <inertial>
         <origin xyz="0 0 0" rpy="0 0 0" />
@@ -28,7 +28,7 @@
       </collision>
     </link>
-    <joint name="chessboard_${name}_joint" type="fixed">
+    <joint name="${name}_joint" type="fixed">
       <parent link="${parent}" />
-      <child link="chessboard_${name}_link" />
+      <child link="${name}_link" />
       <origin xyz="${origin}" rpy="${rpy}" />
     </joint>
