Commit message: remove collision in calibration chessboard

File: tiago_description/urdf/chessboard/chessboard.urdf.xacro (robot description, xacro)
@@ -16,4 +16,5 @@
       </inertial>
       <visual>
+        <origin xyz="0 0 0" rpy="0 0 0" />
         <geometry>
           <mesh filename="package://tiago_description/meshes/chessboard/chessboard.dae"/>
@@ -21,10 +22,4 @@
         <material name="DarkGrey" />
       </visual>
-      <collision>
-        <origin xyz="0 0 0" rpy="0 0 0" />
-        <geometry>
-	  <box size="0.21 0.24 0.000000001"/>
-        </geometry>
-      </collision>
     </link>
     <joint name="${name}_joint" type="fixed">
