Commit message: Gripper parts color

File: tiago_description/urdf/gripper/gripper.gazebo.xacro (robot description, xacro)
@@ -37,4 +37,5 @@
       <maxVel>1.0</maxVel>
       <minDepth>0.00</minDepth>
+      <material>Gazebo/Black</material>
     </gazebo>
     <gazebo reference="${name}_joint">

File: tiago_description/urdf/gripper/gripper.urdf.xacro (robot description, xacro)
@@ -23,7 +23,5 @@
         <mesh filename="package://tiago_description/meshes/gripper/gripper_link.stl"/>
       </geometry>
-      <material name="">
-        <color rgba="1 1 1 1" />
-      </material>
+      <material name="White"/>
     </visual>
     <collision>
@@ -34,4 +32,7 @@
     </collision>
   </link>
+  <gazebo reference="${name}_link">
+    <material>Gazebo/White</material>
+  </gazebo>
   <joint name="${name}_joint" type="fixed">
     <insert_block name="origin"/>
@@ -53,7 +54,5 @@
         <mesh filename="package://tiago_description/meshes/gripper/gripper_finger_link.stl" scale="1 -1 1"/>
       </geometry>
-      <material name="">
-        <color rgba="0 0 0 1" />
-      </material>
+      <material name="Black"/>
     </visual>
     <collision>
@@ -86,7 +85,5 @@
         <mesh filename="package://tiago_description/meshes/gripper/gripper_finger_link.stl"/>
       </geometry>
-      <material name="">
-        <color rgba="0 0 0 1" />
-      </material>
+      <material name="Black"/>
     </visual>
     <collision>
