Commit message: Change finger names and add controller + first gains

File: tiago_description/urdf/gripper/gripper.urdf.xacro (robot description, xacro)
@@ -37,5 +37,5 @@
     <axis xyz="0 0 0" />
   </joint>
-  <link name="right_gripper_finger_link">
+  <link name="gripper_right_finger_link">
     <inertial>
       <origin rpy="0 0 0" xyz="0.0018 -0.00508 0" />
@@ -61,8 +61,8 @@
     </collision>
   </link>
-  <joint name="right_gripper_joint" type="prismatic">
+  <joint name="gripper_right_joint" type="prismatic">
     <origin rpy="0 0 0" xyz="0.111 0 0" />
     <parent link="gripper_link" />
-    <child link="right_gripper_finger_link" />
+    <child link="gripper_right_finger_link" />
     <axis xyz="0 -1 0" />
     <limit effort="28.0" lower="0.0" upper="0.045" velocity="0.1" />
@@ -70,5 +70,5 @@
     <dynamics damping="2500" />
   </joint>
-  <link name="left_gripper_finger_link">
+  <link name="gripper_left_finger_link">
     <inertial>
       <origin rpy="0 0 0" xyz="0.0018 0.00508 0" />
@@ -94,8 +94,8 @@
     </collision>
   </link>
-  <joint name="left_gripper_joint" type="prismatic">
+  <joint name="gripper_left_joint" type="prismatic">
     <origin rpy="0 0 0" xyz="0.111 0 0" />
     <parent link="gripper_link" />
-    <child link="left_gripper_finger_link" />
+    <child link="gripper_left_finger_link" />
     <axis xyz="0 1 0" />
     <limit effort="28.0" lower="0.0" upper="0.045" velocity="0.1" />
@@ -103,6 +103,6 @@
     <dynamics damping="2500" />
   </joint>
-  <xacro:gripper_simple_transmission name="right_gripper" reduction="1.0"/>
-  <xacro:gripper_simple_transmission name="left_gripper" reduction="1.0"/>
+  <xacro:gripper_simple_transmission name="gripper_left" reduction="1.0"/>
+  <xacro:gripper_simple_transmission name="gripper_right" reduction="1.0"/>
  </xacro:macro>
 </robot>

Commit message: Change gripper joint names and add pids

File: tiago_description/urdf/gripper/gripper.urdf.xacro (robot description, xacro)
@@ -61,5 +61,5 @@
     </collision>
   </link>
-  <joint name="gripper_right_joint" type="prismatic">
+  <joint name="gripper_right_finger_joint" type="prismatic">
     <origin rpy="0 0 0" xyz="0.111 0 0" />
     <parent link="gripper_link" />
@@ -94,5 +94,5 @@
     </collision>
   </link>
-  <joint name="gripper_left_joint" type="prismatic">
+  <joint name="gripper_left_finger_joint" type="prismatic">
     <origin rpy="0 0 0" xyz="0.111 0 0" />
     <parent link="gripper_link" />
@@ -103,6 +103,6 @@
     <dynamics damping="2500" />
   </joint>
-  <xacro:gripper_simple_transmission name="gripper_left" reduction="1.0"/>
-  <xacro:gripper_simple_transmission name="gripper_right" reduction="1.0"/>
+  <xacro:gripper_simple_transmission name="gripper_left_finger" reduction="1.0"/>
+  <xacro:gripper_simple_transmission name="gripper_right_finger" reduction="1.0"/>
  </xacro:macro>
 </robot>

Commit message: Changes to fix finger shaking. Much better than before.

File: tiago_description/urdf/gripper/gripper.urdf.xacro (robot description, xacro)
@@ -11,5 +11,5 @@
   <link name="gripper_link">
     <inertial>
-      <inertia ixx="0.00039" ixy="0.0" ixz="0.0" iyy="0.00039" iyz="-1e-05" izz="0.00066" />
+      <inertia ixx="0.00039" ixy="1E-07" ixz="1E-07" iyy="0.00039" iyz="-1e-05" izz="0.00066" />
       <mass value="0.4218" />
       <origin rpy="0.0 0.0 0.0" xyz="0.04724 0.00159 0.00064" />
@@ -40,8 +40,8 @@
     <inertial>
       <origin rpy="0 0 0" xyz="0.0018 -0.00508 0" />
-      <mass value="0.008" />
-      <inertia ixx="5.11E-03" ixy="3.30E-09" ixz="-1.24E-12"
-               iyy="2.94E-03" iyz="7.57E-12"
-               izz="2.63E-03" />
+      <mass value="0.1" />
+      <inertia ixx="5.11E-01" ixy="3.30E-09" ixz="-1.24E-12"
+               iyy="2.94E-01" iyz="7.57E-12"
+               izz="2.63E-01" />
     </inertial>
     <visual>
@@ -73,8 +73,8 @@
     <inertial>
       <origin rpy="0 0 0" xyz="0.0018 0.00508 0" />
-      <mass value="0.008" />
-      <inertia ixx="5.11E-03" ixy="-3.30E-09" ixz="1.24E-12"
-               iyy="2.94E-03" iyz="7.57E-12"
-               izz="2.63E-03" />
+      <mass value="0.1" />
+      <inertia ixx="5.11E-01" ixy="-3.30E-09" ixz="1.24E-12"
+               iyy="2.94E-01" iyz="7.57E-12"
+               izz="2.63E-01" />
     </inertial>
     <visual>

Commit message: Tweak inertial params

File: tiago_description/urdf/gripper/gripper.urdf.xacro (robot description, xacro)
@@ -11,5 +11,7 @@
   <link name="gripper_link">
     <inertial>
-      <inertia ixx="0.00039" ixy="1E-07" ixz="1E-07" iyy="0.00039" iyz="-1e-05" izz="0.00066" />
+      <inertia ixx="0.00039" ixy="0" ixz="0"
+               iyy="0.00039" iyz="0"
+               izz="0.00066" />
       <mass value="0.4218" />
       <origin rpy="0.0 0.0 0.0" xyz="0.04724 0.00159 0.00064" />
@@ -41,7 +43,7 @@
       <origin rpy="0 0 0" xyz="0.0018 -0.00508 0" />
       <mass value="0.1" />
-      <inertia ixx="5.11E-01" ixy="3.30E-09" ixz="-1.24E-12"
-               iyy="2.94E-01" iyz="7.57E-12"
-               izz="2.63E-01" />
+      <inertia ixx="0.00001" ixy="0" ixz="0"
+               iyy="0.00001" iyz="0"
+               izz="0.00001" />
     </inertial>
     <visual>
@@ -74,7 +76,7 @@
       <origin rpy="0 0 0" xyz="0.0018 0.00508 0" />
       <mass value="0.1" />
-      <inertia ixx="5.11E-01" ixy="-3.30E-09" ixz="1.24E-12"
-               iyy="2.94E-01" iyz="7.57E-12"
-               izz="2.63E-01" />
+      <inertia ixx="0.0001" ixy="0" ixz="0"
+               iyy="0.0001" iyz="0"
+               izz="0.0001" />
     </inertial>
     <visual>
@@ -99,5 +101,5 @@
     <child link="gripper_left_finger_link" />
     <axis xyz="0 1 0" />
-    <limit effort="28.0" lower="0.0" upper="0.045" velocity="0.1" />
+    <limit effort="28.0" lower="0" upper="0.045" velocity="0.1" />
     <calibration rising="0.0" />
     <dynamics damping="2500" />

File: tiago_description/urdf/head/head.urdf.xacro (robot description, xacro)
@@ -25,5 +25,7 @@
         <origin xyz="0.0208 -0.00025 0.0215" rpy="0 0 0" />
         <mass value="0.09793" />
-        <inertia ixx="0.00005844626"  ixy="-0.00000051494"  ixz="0.00004662971" iyy="0.00001161435" iyz="0.0" izz="0.00005236593" />
+        <inertia ixx="0.00005844626"  ixy="-0.00000051494"  ixz="0.00004662971"
+                 iyy="0.00001161435" iyz="0.000000001"
+                 izz="0.00005236593" />
       </inertial>
       <visual>
@@ -72,5 +74,7 @@
         <origin xyz="0.04149 -0.01221 0.001" rpy="0 0 0" />
         <mass value="0.24875" />
-        <inertia ixx="0.0000498057"  ixy="-0.00012697329"  ixz="0.00000011444" iyy="0.00044922137" iyz="-0.00000065525" izz="0.00048113173" />
+        <inertia ixx="0.0000498057" ixy="0" ixz="0"
+                 iyy="0.0004492213" iyz="0"
+                 izz="0.00048113173" />
       </inertial>
       <visual>

File: tiago_description/urdf/sensors/xtion_pro_live.urdf.xacro (robot description, xacro)
@@ -56,5 +56,13 @@
       <child link="${name}_optical_frame"/>
     </joint>
-    <link name="${name}_optical_frame"/>
+    <link name="${name}_optical_frame">
+      <inertial>
+        <origin xyz="0 0 0" rpy="0 0 0"/>
+        <mass value="0.001"/>
+        <inertia ixx="0.00001" ixy="0" ixz="0"
+                 iyy="0.00001" iyz="0"
+                 izz="0.00001"/>
+      </inertial>
+    </link>
     <!-- frames of the depth sensor -->
     <joint name="${name}_depth_joint" type="fixed">
@@ -63,5 +71,13 @@
       <child link="${name}_depth_frame"/>
     </joint>
-    <link name="${name}_depth_frame"/>
+    <link name="${name}_depth_frame">
+      <inertial>
+        <origin xyz="0 0 0" rpy="0 0 0"/>
+        <mass value="0.001"/>
+        <inertia ixx="0.00001" ixy="0" ixz="0"
+                 iyy="0.00001" iyz="0"
+                 izz="0.00001"/>
+      </inertial>
+    </link>
     <joint name="${name}_depth_optical_joint" type="fixed">
       <origin xyz="0 0 0" rpy="${-90.0 * deg_to_rad} 0.0 ${-90.0 * deg_to_rad}" />
@@ -69,5 +85,13 @@
       <child link="${name}_depth_optical_frame"/>
     </joint>
-    <link name="${name}_depth_optical_frame"/>
+    <link name="${name}_depth_optical_frame">
+      <inertial>
+        <origin xyz="0 0 0" rpy="0 0 0"/>
+        <mass value="0.001"/>
+        <inertia ixx="0.00001" ixy="0" ixz="0"
+                 iyy="0.00001" iyz="0"
+                 izz="0.00001"/>
+      </inertial>
+    </link>
     <!-- frames of the rgb sensor -->
     <joint name="${name}_rgb_joint" type="fixed">
@@ -76,5 +100,13 @@
       <child link="${name}_rgb_frame"/>
     </joint>
-    <link name="${name}_rgb_frame"/>
+    <link name="${name}_rgb_frame">
+      <inertial>
+        <origin xyz="0 0 0" rpy="0 0 0"/>
+        <mass value="0.001"/>
+        <inertia ixx="0.00001" ixy="0" ixz="0"
+                 iyy="0.00001" iyz="0"
+                 izz="0.00001"/>
+      </inertial>
+    </link>
     <joint name="${name}_rgb_optical_joint" type="fixed">
       <origin xyz="0 0 0" rpy="${-90.0 * deg_to_rad} 0.0 ${-90.0 * deg_to_rad}" />
@@ -82,5 +114,13 @@
       <child link="${name}_rgb_optical_frame"/>
     </joint>
-    <link name="${name}_rgb_optical_frame"/>
+    <link name="${name}_rgb_optical_frame">
+      <inertial>
+        <origin xyz="0 0 0" rpy="0 0 0"/>
+        <mass value="0.001"/>
+        <inertia ixx="0.00001" ixy="0" ixz="0"
+                 iyy="0.00001" iyz="0"
+                 izz="0.00001"/>
+      </inertial>
+    </link>
     <!-- extensions -->
     <xacro:openni_camera_gazebo_v0 name="${name}" />

File: tiago_description/urdf/torso/torso.urdf.xacro (robot description, xacro)
@@ -13,7 +13,7 @@
       <origin rpy="0 0 0" xyz="0.01929 -0.01317 0.0798" />
       <mass value="7.22876" />
-      <inertia ixx="0.17621875653" ixy="-0.00154333947"   ixz="0.00980172504"
-               iyy="0.18995293862" iyz="-0.0259201152"
-               izz="0.03571737542" />
+      <inertia ixx="0.16941095831" ixy="-0.00114443001" ixz="0.00090167218"
+               iyy="0.15113888533" iyz="-0.00744737659"
+               izz="0.04165307088" />
     </inertial>
   <visual>
@@ -40,9 +40,14 @@
   <link name="${name}_lift_link">
     <inertial>
-      <origin rpy="0 0 0" xyz="0.04761 0.01408 -0.12387" />
+      <origin rpy="0 0 0" xyz="-0.04761 0.01408 -0.12387" />
       <mass value="6.54467" />
-      <inertia ixx="0.19639986797" ixy="0.00528625771" ixz="-0.04018414421"
-               iyy="0.212736527" iyz="-0.01564349386"
-               izz="0.02479371908" />
+      <!--
+      <inertia ixx="0.19792" ixy="0" ixz="0"
+               iyy="0.21204" iyz="0"
+               izz="0.00332" />
+               -->
+      <inertia ixx="0.0641960264706125" ixy="0.001128617953499" ixz="0.00203364821006436"
+               iyy="0.061658561971383" iyz="-3.14401755382909E-05"
+               izz="0.0376084656328484" />
     </inertial>
     <!-- Lifting body -->

Commit message: Added grasping frame

File: tiago_description/urdf/gripper/gripper.urdf.xacro (robot description, xacro)
@@ -106,4 +106,19 @@
     <dynamics damping="2500" />
   </joint>
+  <!-- Grasping frame -->
+  <joint name="gripper_grasping_frame_joint" type="fixed">
+    <parent link="gripper_link" />
+    <child link="gripper_grasping_frame" />
+    <origin xyz="0.12 0 0" rpy="0 0 0" />
+  </joint>
+  <link name="gripper_grasping_frame">
+    <inertial>
+      <origin xyz="0 0 0" rpy="0 0 0" />
+      <mass value="0.0001" />
+      <inertia ixx="0.00001" ixy="0.0" ixz="0.0"
+               iyy="0.00001" iyz="0.0"
+               izz="0.00001" />
+    </inertial>
+  </link>
   <xacro:gripper_simple_transmission name="gripper_left_finger" reduction="1.0"/>
   <xacro:gripper_simple_transmission name="gripper_right_finger" reduction="1.0"/>

Commit message: Refactor gripper to ${name}

File: tiago_description/urdf/gripper/gripper.urdf.xacro (robot description, xacro)
@@ -10,5 +10,5 @@
   <xacro:property name="torso_eps"      value="0.02" />
   <xacro:macro name="tiago_gripper" params="name parent *origin">
-  <link name="gripper_link">
+  <link name="${name}_link">
     <inertial>
       <inertia ixx="0.00039" ixy="0" ixz="0"
@@ -34,11 +34,11 @@
     </collision>
   </link>
-  <joint name="gripper_joint" type="fixed">
+  <joint name="${name}_joint" type="fixed">
     <insert_block name="origin"/>
     <parent link="${parent}" />
-    <child link="gripper_link" />
+    <child link="${name}_link" />
     <axis xyz="0 0 0" />
   </joint>
-  <link name="gripper_right_finger_link">
+  <link name="${name}_right_finger_link">
     <inertial>
       <origin rpy="0 0 0" xyz="0.0018 -0.00508 0" />
@@ -64,8 +64,8 @@
     </collision>
   </link>
-  <joint name="gripper_right_finger_joint" type="prismatic">
+  <joint name="${name}_right_finger_joint" type="prismatic">
     <origin rpy="0 0 0" xyz="0.111 0 0" />
-    <parent link="gripper_link" />
-    <child link="gripper_right_finger_link" />
+    <parent link="${name}_link" />
+    <child link="${name}_right_finger_link" />
     <axis xyz="0 -1 0" />
     <limit effort="28.0" lower="0.0" upper="0.045" velocity="0.1" />
@@ -73,5 +73,5 @@
     <dynamics damping="2500" />
   </joint>
-  <link name="gripper_left_finger_link">
+  <link name="${name}_left_finger_link">
     <inertial>
       <origin rpy="0 0 0" xyz="0.0018 0.00508 0" />
@@ -97,8 +97,8 @@
     </collision>
   </link>
-  <joint name="gripper_left_finger_joint" type="prismatic">
+  <joint name="${name}_left_finger_joint" type="prismatic">
     <origin rpy="0 0 0" xyz="0.111 0 0" />
-    <parent link="gripper_link" />
-    <child link="gripper_left_finger_link" />
+    <parent link="${name}_link" />
+    <child link="${name}_left_finger_link" />
     <axis xyz="0 1 0" />
     <limit effort="28.0" lower="0" upper="0.045" velocity="0.1" />
@@ -107,10 +107,10 @@
   </joint>
   <!-- Grasping frame -->
-  <joint name="gripper_grasping_frame_joint" type="fixed">
-    <parent link="gripper_link" />
-    <child link="gripper_grasping_frame" />
+  <joint name="${name}_grasping_frame_joint" type="fixed">
+    <parent link="${name}_link" />
+    <child link="${name}_grasping_frame" />
     <origin xyz="0.12 0 0" rpy="0 0 0" />
   </joint>
-  <link name="gripper_grasping_frame">
+  <link name="${name}_grasping_frame">
     <inertial>
       <origin xyz="0 0 0" rpy="0 0 0" />
@@ -121,9 +121,9 @@
     </inertial>
   </link>
-  <xacro:gripper_simple_transmission name="gripper_left_finger" reduction="1.0"/>
-  <xacro:gripper_simple_transmission name="gripper_right_finger" reduction="1.0"/>
-  <xacro:finger_gazebo name="gripper_left_finger"/>
-  <xacro:finger_gazebo name="gripper_right_finger"/>
-  <xacro:gripper_grasping_hack name="gripper"/>
+  <xacro:gripper_simple_transmission name="${name}_left_finger" reduction="1.0"/>
+  <xacro:gripper_simple_transmission name="${name}_right_finger" reduction="1.0"/>
+  <xacro:finger_gazebo name="${name}_left_finger"/>
+  <xacro:finger_gazebo name="${name}_right_finger"/>
+  <xacro:gripper_grasping_hack name="${name}"/>
  </xacro:macro>
 </robot>

Commit message: Update gripper length to approx real one

File: tiago_description/urdf/gripper/gripper.urdf.xacro (robot description, xacro)
@@ -49,5 +49,5 @@
     </inertial>
     <visual>
-      <origin rpy="0 0 0" xyz="0 0 0" />
+      <origin rpy="0 0 0" xyz="0.03 0 0" />
       <geometry>
         <mesh filename="package://tiago_description/meshes/gripper/gripper_finger_link.stl" scale="1 -1 1"/>
@@ -82,5 +82,5 @@
     </inertial>
     <visual>
-      <origin rpy="0 0 0" xyz="0 0 0" />
+      <origin rpy="0 0 0" xyz="0.03 0 0" />
       <geometry>
         <mesh filename="package://tiago_description/meshes/gripper/gripper_finger_link.stl"/>

Commit message: Update gripper finger

File: tiago_description/urdf/gripper/gripper.urdf.xacro (robot description, xacro)
@@ -49,5 +49,5 @@
     </inertial>
     <visual>
-      <origin rpy="0 0 0" xyz="0.03 0 0" />
+      <origin rpy="0 0 0" xyz="0 0 0" />
       <geometry>
         <mesh filename="package://tiago_description/meshes/gripper/gripper_finger_link.stl" scale="1 -1 1"/>
@@ -58,12 +58,12 @@
     </visual>
     <collision>
-      <origin rpy="0 0 0" xyz="0 -0.005 0" />
+      <origin rpy="0 0 0" xyz="0.0725 0 0" />
       <geometry>
-        <box size="0.06 0.01 0.022" />
+        <box size="0.145 0.015 0.04" />
       </geometry>
     </collision>
   </link>
   <joint name="${name}_right_finger_joint" type="prismatic">
-    <origin rpy="0 0 0" xyz="0.111 0 0" />
+    <origin rpy="0 0 0" xyz="0.07 0 0" />
     <parent link="${name}_link" />
     <child link="${name}_right_finger_link" />
@@ -82,5 +82,5 @@
     </inertial>
     <visual>
-      <origin rpy="0 0 0" xyz="0.03 0 0" />
+      <origin rpy="0 0 0" xyz="0 0 0" />
       <geometry>
         <mesh filename="package://tiago_description/meshes/gripper/gripper_finger_link.stl"/>
@@ -91,12 +91,12 @@
     </visual>
     <collision>
-      <origin rpy="0 0 0" xyz="0 0.005 0" />
+      <origin rpy="0 0 0" xyz="0.0725 -0 0" />
       <geometry>
-        <box size="0.06 0.01 0.022" />
+        <box size="0.145 0.015 0.04" />
       </geometry>
     </collision>
   </link>
   <joint name="${name}_left_finger_joint" type="prismatic">
-    <origin rpy="0 0 0" xyz="0.111 0 0" />
+    <origin rpy="0 0 0" xyz="0.07 0 0" />
     <parent link="${name}_link" />
     <child link="${name}_left_finger_link" />

Commit message: Update limits

File: tiago_description/urdf/gripper/gripper.urdf.xacro (robot description, xacro)
@@ -69,5 +69,5 @@
     <child link="${name}_right_finger_link" />
     <axis xyz="0 -1 0" />
-    <limit effort="28.0" lower="0.0" upper="0.045" velocity="0.1" />
+    <limit effort="28.0" lower="0.0" upper="0.05" velocity="0.1" />
     <calibration rising="0.0" />
     <dynamics damping="2500" />
@@ -102,5 +102,5 @@
     <child link="${name}_left_finger_link" />
     <axis xyz="0 1 0" />
-    <limit effort="28.0" lower="0" upper="0.045" velocity="0.1" />
+    <limit effort="28.0" lower="0" upper="0.05" velocity="0.1" />
     <calibration rising="0.0" />
     <dynamics damping="2500" />

Commit message: fix inertial matrices and remove grasp hack

File: tiago_description/urdf/gripper/gripper.urdf.xacro (robot description, xacro)
@@ -12,7 +12,10 @@
   <link name="${name}_link">
     <inertial>
-      <inertia ixx="0.00039" ixy="0" ixz="0"
-               iyy="0.00039" iyz="0"
-               izz="0.00066" />
+<!--      <inertia ixx="0.291026" ixy="0.003769" ixz="0.000179"
+               iyy="0.126426" iyz="0.0"
+               izz="0.374198" /> -->
+      <inertia ixx="0.001920326" ixy="0.00002487" ixz="0.000001181"
+               iyy="0.000834218" iyz="0.0"
+               izz="0.002469134" />
       <mass value="0.4218" />
       <origin rpy="0.0 0.0 0.0" xyz="0.04724 0.00159 0.00064" />
@@ -45,7 +48,7 @@
       <origin rpy="0 0 0" xyz="0.0018 -0.00508 0" />
       <mass value="0.1" />
-      <inertia ixx="0.00001" ixy="0" ixz="0"
-               iyy="0.00001" iyz="0"
-               izz="0.00001" />
+      <inertia ixx="0.000165887" ixy="0.000009593" ixz="0.000008307"
+               iyy="0.001979493" iyz="-0.000000187"
+               izz="0.001819711" />
     </inertial>
     <visual>
@@ -68,5 +71,5 @@
     <child link="${name}_right_finger_link" />
     <axis xyz="0 -1 0" />
-    <limit effort="28.0" lower="0.0" upper="0.05" velocity="0.1" />
+    <limit effort="25" lower="0.0" upper="0.05" velocity="0.1" />
     <calibration rising="0.0" />
     <dynamics damping="2500" />
@@ -76,7 +79,7 @@
       <origin rpy="0 0 0" xyz="0.0018 0.00508 0" />
       <mass value="0.1" />
-      <inertia ixx="0.0001" ixy="0" ixz="0"
-               iyy="0.0001" iyz="0"
-               izz="0.0001" />
+      <inertia ixx="0.000165887" ixy="0.000009593" ixz="0.000008307"
+               iyy="0.001979493" iyz="-0.000000187"
+               izz="0.001819711" />
     </inertial>
     <visual>
@@ -99,5 +102,5 @@
     <child link="${name}_left_finger_link" />
     <axis xyz="0 1 0" />
-    <limit effort="28.0" lower="0" upper="0.05" velocity="0.1" />
+    <limit effort="25" lower="0" upper="0.05" velocity="0.1" />
     <calibration rising="0.0" />
     <dynamics damping="2500" />
@@ -122,5 +125,5 @@
   <xacro:finger_gazebo name="${name}_left_finger"/>
   <xacro:finger_gazebo name="${name}_right_finger"/>
-  <xacro:gripper_grasping_hack name="${name}"/>
+  <!-- <xacro:gripper_grasping_hack name="${name}"/> -->
  </xacro:macro>
 </robot>
