Commit message: Fix optical frame alignment

File: tiago_description/urdf/head/head.urdf.xacro (robot description, xacro)
@@ -107,5 +107,5 @@
     <xacro:xtion_pro_live name="xtion" parent="${name}_2">
       <origin xyz="0 -0.03 0" rpy="${90 * deg_to_rad} 0 0" />
-      <origin xyz="0 -0.03 0" rpy="${90 * deg_to_rad} 0 0" />
+      <origin xyz="0 -0.03 0" rpy="0 ${90 * deg_to_rad} 0" />
     </xacro:xtion_pro_live>
   </xacro:macro>

Commit message: Add head based on v2 drawing

File: tiago_description/urdf/head/head.urdf.xacro (robot description, xacro)
@@ -28,16 +28,16 @@
       </inertial>
       <visual>
-        <origin rpy="0 0 0" xyz="0.03 0 0"/>
+        <origin xyz="0.0305 0 0.0175" rpy="0 0 0"/>
         <geometry>
-          <box size="0.06 0.04 0.04"/>
+          <box size="0.05 0.035 0.035"/>
         </geometry>
-        <material name="Grey" />
+        <material name="DarkGrey" />
       </visual>
       <collision>
-        <origin xyz="0.03 0 0" rpy="0 0 0" />
+        <origin xyz="0.0305 0 0.0175" rpy="0 0 0" />
         <geometry>
-          <box size="0.06 0.04 0.04"/>
+          <box size="0.05 0.035 0.035"/>
         </geometry>
-        <material name="Grey" />
+        <material name="DarkGrey" />
       </collision>
     </link>
@@ -45,12 +45,12 @@
       <parent link="${parent}"/>
       <child link="${name}_link"/>
-      <origin xyz="0 0 0.04" rpy="${0.0 * deg_to_rad} 0 0" />
+      <origin xyz="0.193 0 0.04" rpy="${0.0 * deg_to_rad} 0 0" />
       <axis xyz="0 0 1" />
-      <limit lower="${-75.0 * deg_to_rad}" upper="${75.0 * deg_to_rad}" effort="3.4" velocity="${head_max_vel}" />
+      <limit lower="${-90.0 * deg_to_rad}" upper="${90.0 * deg_to_rad}" effort="3.4" velocity="${head_max_vel}" />
       <dynamics damping="${head_damping}" friction="${head_friction}"/>
       <safety_controller k_position="20"
                          k_velocity="20"
-                         soft_lower_limit="${-75.0 * deg_to_rad + head_eps}"
-                         soft_upper_limit="${ 75.0 * deg_to_rad - head_eps}" />
+                         soft_lower_limit="${-90.0 * deg_to_rad + head_eps}"
+                         soft_upper_limit="${ 90.0 * deg_to_rad - head_eps}" />
     </joint>
     <gazebo reference="${name}_link">
@@ -74,30 +74,16 @@
         <inertia ixx="0.00640199093"  ixy="0.00012197067"  ixz="-0.00000897011" iyy="0.00676228591" iyz="-0.0000552329" izz="0.00614192438" />
       </inertial>
-      <visual>
-        <origin xyz="-0.035 0 0" rpy="0 0 0"/>
-        <geometry>
-          <box size="0.035 0.035 0.05"/>
-        </geometry>
-        <material name="DarkGrey" />
-      </visual>
-      <collision>
-        <origin xyz="-0.035 0 0" rpy="0 0 0" />
-        <geometry>
-          <box size="0.035 0.035 0.05"/>
-        </geometry>
-        <material name="DarkGrey" />
-      </collision>
     </link>
     <joint name="${name}_joint" type="revolute">
       <parent link="${parent}"/>
         <child link="${name}_link"/>
-      <origin xyz="0.0845 0 0.03" rpy="${-90.0 * deg_to_rad} 0 0" />
+      <origin xyz="0.0355 0 0.023" rpy="${-90.0 * deg_to_rad} 0 0" />
       <axis xyz="0 0 1" />
-      <limit lower="${-15.0 * deg_to_rad}" upper="${45.0 * deg_to_rad}" effort="3.26" velocity="${head_max_vel}" />
+      <limit lower="${-45.0 * deg_to_rad}" upper="${90.0 * deg_to_rad}" effort="3.26" velocity="${head_max_vel}" />
       <dynamics damping="${head_damping}" friction="${head_friction}"/>
       <safety_controller k_position="20"
                          k_velocity="20"
-                         soft_lower_limit="${-15.0 * deg_to_rad + head_eps}"
-                         soft_upper_limit="${ 20.0 * deg_to_rad}" />
+                         soft_lower_limit="${-45.0 * deg_to_rad + head_eps}"
+                         soft_upper_limit="${ 90.0 * deg_to_rad}" />
     </joint>
   </xacro:macro>
@@ -106,6 +92,6 @@
     <xacro:head_2 name="${name}_2" parent="${name}_1_link"/>
     <xacro:xtion_pro_live name="xtion" parent="${name}_2">
-      <origin xyz="0 -0.03 0" rpy="${90 * deg_to_rad} 0 0" />
-      <origin xyz="0 -0.03 0" rpy="0 ${90 * deg_to_rad} 0" />
+      <origin xyz="0.064192 -0.017614 0" rpy="${90 * deg_to_rad} 0 0" />
+      <origin xyz="0.064192 -0.017641 0" rpy="0 ${90 * deg_to_rad} 0" />
     </xacro:xtion_pro_live>
   </xacro:macro>

File: tiago_description/urdf/torso/torso.urdf.xacro (robot description, xacro)
@@ -17,7 +17,7 @@
     </inertial>
   <visual>
-      <origin rpy="0 0 0" xyz="0 0 0.2315" />
+      <origin rpy="0 0 0" xyz="0 0 0.2235" />
       <geometry>
-        <box size="0.1 0.14 0.463"/>
+        <box size="0.14 0.1 0.463"/>
       </geometry>
       <material name="LightGrey"/>
@@ -26,5 +26,5 @@
       <origin rpy="0 0 0" xyz="0.0 0.0 0.2315" />
       <geometry>
-        <box size="0.1 0.14 0.463"/>
+        <box size="0.14 0.1 0.463"/>
       </geometry>
       <material name="LightGrey"/>
@@ -32,5 +32,5 @@
   </link>
   <joint name="${name}_fixed_joint" type="fixed">
-    <origin rpy="0 0 0" xyz="-0.053 0 0.2015" />
+    <origin rpy="0 0 0" xyz="-0.068 0 0.2235" />
     <parent link="${parent}_link" />
     <child link="${name}_fixed_link" />
@@ -45,25 +45,41 @@
                izz="0.0376084656328484" />
     </inertial>
+    <!-- Lifting body -->
     <visual>
-      <origin rpy="0 0 0" xyz="0 0 -0.2315" />
+      <origin rpy="0 0 0" xyz="0 0 -0.25125" />
        <geometry>
-        <box size="0.106 0.15 0.463"/>
+        <box size="0.16 0.106 0.5025"/>
       </geometry>
       <material name="White"/>
     </visual>
     <collision>
-      <origin rpy="0 0 0" xyz="0 0 -0.2315" />
+      <origin rpy="0 0 0" xyz="0 0 -0.25125" />
        <geometry>
-        <box size="0.106 0.15 0.463"/>
+        <box size="0.16 0.106 0.5025"/>
       </geometry>
       <material name="White"/>
     </collision>
+    <!-- Head pan motor -->
+    <visual>
+      <origin xyz="0.187 0 0.02" rpy="0 0 0"/>
+      <geometry>
+        <box size="0.06 0.04 0.04"/>
+      </geometry>
+      <material name="Grey" />
+    </visual>
+    <collision>
+      <origin xyz="0.187 0 0.02" rpy="0 0 0" />
+      <geometry>
+        <box size="0.06 0.04 0.04"/>
+      </geometry>
+      <material name="Grey" />
+    </collision>
   </link>
   <joint name="${name}_lift_joint" type="prismatic">
-    <origin rpy="0 0 0" xyz="0.0 0 0.463" />
+    <origin rpy="0 0 0" xyz="0.0 0 0.5025" />
     <parent link="${name}_fixed_link" />
     <child link="${name}_lift_link" />
     <axis xyz="0 0 1" />
-    <limit effort="450" lower="0.0" upper="0.3556" velocity="0.1" />
+    <limit effort="450" lower="0.0" upper="0.35" velocity="0.1" />
     <calibration rising="0.0" />
     <dynamics damping="1000" />

Commit message: Update joint limits of head, 45degs up, 90degs down

File: tiago_description/urdf/head/head.urdf.xacro (robot description, xacro)
@@ -80,10 +80,10 @@
       <origin xyz="0.0355 0 0.023" rpy="${-90.0 * deg_to_rad} 0 0" />
       <axis xyz="0 0 1" />
-      <limit lower="${-90 * deg_to_rad}" upper="${45.0 * deg_to_rad}" effort="2.77" velocity="${head_max_vel}" />
+      <limit lower="${-45 * deg_to_rad}" upper="${90.0 * deg_to_rad}" effort="2.77" velocity="${head_max_vel}" />
       <dynamics damping="${head_damping}" friction="${head_friction}"/>
       <safety_controller k_position="20"
                          k_velocity="20"
-                         soft_lower_limit="${-90.0 * deg_to_rad + head_eps}"
-                         soft_upper_limit="${ 45.0 * deg_to_rad}" />
+                         soft_lower_limit="${-45.0 * deg_to_rad + head_eps}"
+                         soft_upper_limit="${ 90.0 * deg_to_rad}" />
     </joint>
   </xacro:macro>
@@ -91,7 +91,7 @@
     <xacro:head_1 name="${name}_1" parent="${parent}" />
     <xacro:head_2 name="${name}_2" parent="${name}_1_link"/>
-    <xacro:xtion_pro_live name="xtion" parent="${name}_2">
+    <xacro:xtion_pro_live name="xtion" parent="${name}_2_link">
       <origin xyz="0.064192 -0.017614 0" rpy="${90 * deg_to_rad} 0 0" />
-      <origin xyz="0.064192 -0.017641 0" rpy="0 ${90 * deg_to_rad} 0" />
+      <origin xyz="0 0 0" rpy="${-90 * deg_to_rad} ${0 * deg_to_rad} ${-90 * deg_to_rad}" />
     </xacro:xtion_pro_live>
   </xacro:macro>

Commit message: Fix orientation of head joint

File: tiago_description/urdf/head/head.urdf.xacro (robot description, xacro)
@@ -78,12 +78,12 @@
       <parent link="${parent}"/>
         <child link="${name}_link"/>
-      <origin xyz="0.0355 0 0.023" rpy="${-90.0 * deg_to_rad} 0 0" />
+      <origin xyz="0.0355 0 0.023" rpy="${90.0 * deg_to_rad} 0 0" />
       <axis xyz="0 0 1" />
-      <limit lower="${-45 * deg_to_rad}" upper="${90.0 * deg_to_rad}" effort="2.77" velocity="${head_max_vel}" />
+      <limit lower="${-90 * deg_to_rad}" upper="${45.0 * deg_to_rad}" effort="2.77" velocity="${head_max_vel}" />
       <dynamics damping="${head_damping}" friction="${head_friction}"/>
       <safety_controller k_position="20"
                          k_velocity="20"
-                         soft_lower_limit="${-45.0 * deg_to_rad + head_eps}"
-                         soft_upper_limit="${ 90.0 * deg_to_rad}" />
+                         soft_lower_limit="${-90.0 * deg_to_rad + head_eps}"
+                         soft_upper_limit="${ 45.0 * deg_to_rad}" />
     </joint>
   </xacro:macro>
@@ -92,5 +92,5 @@
     <xacro:head_2 name="${name}_2" parent="${name}_1_link"/>
     <xacro:xtion_pro_live name="xtion" parent="${name}_2_link">
-      <origin xyz="0.064192 -0.017614 0" rpy="${90 * deg_to_rad} 0 0" />
+      <origin xyz="0.064192 0.017614 0" rpy="${-90 * deg_to_rad} 0 0" />
       <origin xyz="0 0 0" rpy="${-90 * deg_to_rad} ${0 * deg_to_rad} ${-90 * deg_to_rad}" />
     </xacro:xtion_pro_live>

Commit message: Add nice visual to head2

File: tiago_description/urdf/head/head.urdf.xacro (robot description, xacro)
@@ -74,4 +74,11 @@
         <inertia ixx="0.0000498057"  ixy="-0.00012697329"  ixz="0.00000011444" iyy="0.00044922137" iyz="-0.00000065525" izz="0.00048113173" />
       </inertial>
+      <visual>
+        <origin xyz="0.070192 0.017614 0" rpy="0 ${90 * deg_to_rad} 0" />
+        <geometry>
+          <mesh filename="package://tiago_description/meshes/head.dae" scale="1 1 1"/>
+        </geometry>
+        <material name="LightGrey"/>
+      </visual>
     </link>
     <joint name="${name}_joint" type="revolute">

Commit message: Update xtion with inertias and adding _link to parent inside

File: tiago_description/urdf/head/head.urdf.xacro (robot description, xacro)
@@ -98,5 +98,5 @@
     <xacro:head_1 name="${name}_1" parent="${parent}" />
     <xacro:head_2 name="${name}_2" parent="${name}_1_link"/>
-    <xacro:xtion_pro_live name="xtion" parent="${name}_2_link">
+    <xacro:xtion_pro_live name="xtion" parent="${name}_2">
       <origin xyz="0.064192 0.017614 0" rpy="${-90 * deg_to_rad} 0 0" />
       <origin xyz="0 0 0" rpy="${-90 * deg_to_rad} ${0 * deg_to_rad} ${-90 * deg_to_rad}" />

File: tiago_description/urdf/sensors/xtion_pro_live.urdf.xacro (robot description, xacro)
@@ -20,18 +20,18 @@
   <xacro:include filename="$(find tiago_description)/urdf/sensors/openni.gazebo.xacro" />
   <!-- Macro -->
-  <xacro:macro name="xtion_pro_live" params="name parent *origin *calibration_origin">
-    <!-- BEGIN frames in the center of the camera -->
-    <joint name="${name}_frame_joint" type="fixed">
-      <insert_block name="origin" />
-      <parent link="${parent}"/>
+  <xacro:macro name="xtion_pro_live" params="name parent *origin *optical_origin">
+    <!-- frames in the center of the camera -->
+    <joint name="${name}_joint" type="fixed">
+      <insert_block name="origin"/>
+      <parent link="${parent}_link"/>
       <child link="${name}_link"/>
     </joint>
     <link name="${name}_link">
       <inertial>
-        <mass value="0.01" />
-        <origin xyz="0 0 0" rpy="0 0 0"/>
-        <inertia ixx="0.0"  ixy="0.0"  ixz="0.0"
-                 iyy="0.0"  iyz="0.0"
-                 izz="0.0" />
+        <origin xyz="-0.00936000000 -0.00003000000 -0.00273000000" rpy="0 0 0"/>
+        <mass value="0.21970000000"/>
+        <inertia ixx="0.00000429247" ixy="0.00000000000" ixz="0.00000002565"
+                 iyy="0.00000008027" iyz="0.00000000000"
+                 izz="0.00000427339"/>
       </inertial>
       <visual>
@@ -52,19 +52,10 @@
     </link>
     <joint name="${name}_optical_joint" type="fixed">
-      <insert_block name="calibration_origin" />
+      <insert_block name="optical_origin" />
       <parent link="${name}_link"/>
       <child link="${name}_optical_frame"/>
     </joint>
-    <link name="${name}_optical_frame">
-      <inertial>
-        <mass value="0.01" />
-        <origin xyz="0 0 0" rpy="0 0 0"/>
-        <inertia ixx="0.0"  ixy="0.0"  ixz="0.0"
-                 iyy="0.0"  iyz="0.0"
-                 izz="0.0" />
-      </inertial>
-    </link>
-    <!-- END frames in the center of the camera -->
-    <!-- BEGIN frames of the depth sensor -->
+    <link name="${name}_optical_frame"/>
+    <!-- frames of the depth sensor -->
     <joint name="${name}_depth_joint" type="fixed">
       <origin xyz="0.0 0.049 0.0" rpy="0 0 0" />
@@ -73,12 +64,11 @@
     </joint>
     <link name="${name}_depth_frame"/>
-      <joint name="${name}_depth_optical_joint" type="fixed">
-        <origin xyz="0 0 0" rpy="${-M_PI/2} 0.0 ${-M_PI/2}" />
-        <parent link="${name}_depth_frame" />
-        <child link="${name}_depth_optical_frame"/>
-      </joint>
+    <joint name="${name}_depth_optical_joint" type="fixed">
+      <origin xyz="0 0 0" rpy="${-90.0 * deg_to_rad} 0.0 ${-90.0 * deg_to_rad}" />
+      <parent link="${name}_depth_frame" />
+      <child link="${name}_depth_optical_frame"/>
+    </joint>
     <link name="${name}_depth_optical_frame"/>
-    <!-- END frames of the depth sensor -->
-    <!-- BEGIN frames of the rgb sensor -->
+    <!-- frames of the rgb sensor -->
     <joint name="${name}_rgb_joint" type="fixed">
       <origin xyz="0.0 0.022 0.0" rpy="0 0 0" />
@@ -88,10 +78,9 @@
     <link name="${name}_rgb_frame"/>
     <joint name="${name}_rgb_optical_joint" type="fixed">
-      <origin xyz="0 0 0" rpy="${-M_PI/2} 0.0 ${-M_PI/2}" />
+      <origin xyz="0 0 0" rpy="${-90.0 * deg_to_rad} 0.0 ${-90.0 * deg_to_rad}" />
       <parent link="${name}_rgb_frame" />
       <child link="${name}_rgb_optical_frame"/>
     </joint>
     <link name="${name}_rgb_optical_frame"/>
-    <!-- END frames of the rgb sensor -->
     <!-- extensions -->
     <xacro:openni_camera_gazebo_v0 name="${name}" />

Commit message: Update head joint limits

File: tiago_description/urdf/head/head.urdf.xacro (robot description, xacro)
@@ -49,10 +49,10 @@
       <origin xyz="0.193 0 0.04" rpy="${0.0 * deg_to_rad} 0 0" />
       <axis xyz="0 0 1" />
-      <limit lower="${-90.0 * deg_to_rad}" upper="${90.0 * deg_to_rad}" effort="5.197" velocity="${head_max_vel}" />
+      <limit lower="${-75.0 * deg_to_rad}" upper="${75.0 * deg_to_rad}" effort="5.197" velocity="${head_max_vel}" />
       <dynamics damping="${head_damping}" friction="${head_friction}"/>
       <safety_controller k_position="20"
                          k_velocity="20"
-                         soft_lower_limit="${-90.0 * deg_to_rad + head_eps}"
-                         soft_upper_limit="${ 90.0 * deg_to_rad - head_eps}" />
+                         soft_lower_limit="${-75.0 * deg_to_rad + head_eps}"
+                         soft_upper_limit="${ 75.0 * deg_to_rad - head_eps}" />
     </joint>
     <gazebo reference="${name}_link">
@@ -91,10 +91,10 @@
       <origin xyz="0.0355 0 0.023" rpy="${90.0 * deg_to_rad} 0 0" />
       <axis xyz="0 0 1" />
-      <limit lower="${-90 * deg_to_rad}" upper="${45.0 * deg_to_rad}" effort="2.77" velocity="${head_max_vel}" />
+      <limit lower="${-60 * deg_to_rad}" upper="${60.0 * deg_to_rad}" effort="2.77" velocity="${head_max_vel}" />
       <dynamics damping="${head_damping}" friction="${head_friction}"/>
       <safety_controller k_position="20"
                          k_velocity="20"
-                         soft_lower_limit="${-90.0 * deg_to_rad + head_eps}"
-                         soft_upper_limit="${ 45.0 * deg_to_rad}" />
+                         soft_lower_limit="${-60.0 * deg_to_rad + head_eps}"
+                         soft_upper_limit="${ 60.0 * deg_to_rad}" />
     </joint>
   </xacro:macro>

Commit message: Updated limits

File: tiago_description/urdf/head/head.urdf.xacro (robot description, xacro)
@@ -17,4 +17,8 @@
   <xacro:property name="head_max_vel"  value="3.0" />
   <xacro:property name="head_eps"      value="0.02" />
+  <xacro:property name="head_1_lower_limit" value="-75"/>
+  <xacro:property name="head_1_upper_limit" value="75"/>
+  <xacro:property name="head_2_lower_limit" value="-60"/>
+  <xacro:property name="head_2_upper_limit" value="36.25"/>
   <!--************************-->
   <!--     HEAD_1 (PAN)       -->
@@ -49,10 +53,10 @@
       <origin xyz="0.193 0 0.04" rpy="${0.0 * deg_to_rad} 0 0" />
       <axis xyz="0 0 1" />
-      <limit lower="${-75.0 * deg_to_rad}" upper="${75.0 * deg_to_rad}" effort="5.197" velocity="${head_max_vel}" />
+      <limit lower="${head_1_lower_limit * deg_to_rad}" upper="${head_1_upper_limit * deg_to_rad}" effort="5.197" velocity="${head_max_vel}" />
       <dynamics damping="${head_damping}" friction="${head_friction}"/>
       <safety_controller k_position="20"
                          k_velocity="20"
-                         soft_lower_limit="${-75.0 * deg_to_rad + head_eps}"
-                         soft_upper_limit="${ 75.0 * deg_to_rad - head_eps}" />
+                         soft_lower_limit="${head_1_lower_limit * deg_to_rad + head_eps}"
+                         soft_upper_limit="${head_1_upper_limit * deg_to_rad - head_eps}" />
     </joint>
     <gazebo reference="${name}_link">
@@ -91,10 +95,10 @@
       <origin xyz="0.0355 0 0.023" rpy="${90.0 * deg_to_rad} 0 0" />
       <axis xyz="0 0 1" />
-      <limit lower="${-60 * deg_to_rad}" upper="${60.0 * deg_to_rad}" effort="2.77" velocity="${head_max_vel}" />
+      <limit lower="${head_2_lower_limit * deg_to_rad}" upper="${head_2_upper_limit * deg_to_rad}" effort="2.77" velocity="${head_max_vel}" />
       <dynamics damping="${head_damping}" friction="${head_friction}"/>
       <safety_controller k_position="20"
                          k_velocity="20"
-                         soft_lower_limit="${-60.0 * deg_to_rad + head_eps}"
-                         soft_upper_limit="${ 60.0 * deg_to_rad}" />
+                         soft_lower_limit="${head_2_lower_limit * deg_to_rad + head_eps}"
+                         soft_upper_limit="${head_2_upper_limit * deg_to_rad}" />
     </joint>
   </xacro:macro>

Commit message: Update head

File: tiago_description/urdf/head/head.urdf.xacro (robot description, xacro)
@@ -20,5 +20,5 @@
   <xacro:property name="head_1_upper_limit" value="75"/>
   <xacro:property name="head_2_lower_limit" value="-60"/>
-  <xacro:property name="head_2_upper_limit" value="36.25"/>
+  <xacro:property name="head_2_upper_limit" value="50"/>
   <!--************************-->
   <!--     HEAD_1 (PAN)       -->
@@ -27,16 +27,16 @@
     <link name="${name}_link">
       <inertial>
-        <origin xyz="0.0208 -0.00025 0.0215" rpy="0 0 0" />
-        <mass value="0.09793" />
-        <inertia ixx="0.00005844626"  ixy="-0.00000051494"  ixz="0.00004662971"
-                 iyy="0.00001161435" iyz="0.000000001"
-                 izz="0.00005236593" />
+        <origin xyz="-0.016151 -0.000132 0.041903" rpy="0 0 0"/>
+        <mass value="0.406285"/>
+        <inertia ixx="0.000506" ixy="-0.000001" ixz="-0.000061"
+                 iyy="0.000552" iyz="0.000002"
+                 izz="0.000381"/>
       </inertial>
       <visual>
-        <origin xyz="0.0305 0 0.0175" rpy="0 0 0"/>
+        <origin xyz="0 0 0" rpy="0 0 0"/>
         <geometry>
-          <box size="0.05 0.035 0.035"/>
+          <mesh filename="package://tiago_description/meshes/head_1.stl" scale="1 1 1"/>
         </geometry>
-        <material name="DarkGrey" />
+        <material name="White" />
       </visual>
       <collision>
@@ -45,5 +45,5 @@
           <box size="0.05 0.035 0.035"/>
         </geometry>
-        <material name="DarkGrey" />
+        <material name="White" />
       </collision>
     </link>
@@ -51,5 +51,5 @@
       <parent link="${parent}"/>
       <child link="${name}_link"/>
-      <origin xyz="0.193 0 0.04" rpy="${0.0 * deg_to_rad} 0 0" />
+      <origin xyz="0.122 0 0.0425" rpy="0 0 0" />
       <axis xyz="0 0 1" />
       <limit lower="${head_1_lower_limit * deg_to_rad}" upper="${head_1_upper_limit * deg_to_rad}" effort="5.197" velocity="${head_max_vel}" />
@@ -76,14 +76,14 @@
     <link name="${name}_link">
       <inertial>
-        <origin xyz="0.04149 -0.01221 0.001" rpy="0 0 0" />
-        <mass value="0.24875" />
-        <inertia ixx="0.0000498057" ixy="0" ixz="0"
-                 iyy="0.0004492213" iyz="0"
-                 izz="0.00048113173" />
+        <origin xyz="0.013345 0.03824 0.000058" rpy="0 0 0"/>
+        <mass value="0.852579"/>
+        <inertia ixx="0.003677" ixy="-0.000003" ixz="0.000001"
+                 iyy="0.003853" iyz="0"
+                 izz="0.002551"/>
       </inertial>
       <visual>
-        <origin xyz="0.070192 0.017614 0" rpy="0 ${90 * deg_to_rad} 0" />
+        <origin xyz="0 0 0" rpy="0 0 0" />
         <geometry>
-          <mesh filename="package://tiago_description/meshes/head.dae" scale="1 1 1"/>
+          <mesh filename="package://tiago_description/meshes/head_2.stl" scale="1 1 1"/>
         </geometry>
         <material name="LightGrey"/>
@@ -92,6 +92,6 @@
     <joint name="${name}_joint" type="revolute">
       <parent link="${parent}"/>
-        <child link="${name}_link"/>
-      <origin xyz="0.0355 0 0.023" rpy="${90.0 * deg_to_rad} 0 0" />
+      <child link="${name}_link"/>
+      <origin xyz="0.0038 0 0.0596" rpy="${90.0 * deg_to_rad} 0 0" />
       <axis xyz="0 0 1" />
       <limit lower="${head_2_lower_limit * deg_to_rad}" upper="${head_2_upper_limit * deg_to_rad}" effort="2.77" velocity="${head_max_vel}" />
@@ -107,5 +107,5 @@
     <xacro:head_2 name="${name}_2" parent="${name}_1_link"/>
     <xacro:xtion_pro_live name="xtion" parent="${name}_2">
-      <origin xyz="0.064192 0.017614 0" rpy="${-90 * deg_to_rad} 0 0" />
+      <origin xyz="0.07 0.0633 0" rpy="${-90 * deg_to_rad} 0 0" />
       <origin xyz="0 0 0" rpy="${-90 * deg_to_rad} ${0 * deg_to_rad} ${-90 * deg_to_rad}" />
     </xacro:xtion_pro_live>

Commit message: Update head distance from torso_lift_link

File: tiago_description/urdf/head/head.urdf.xacro (robot description, xacro)
@@ -51,5 +51,5 @@
       <parent link="${parent}"/>
       <child link="${name}_link"/>
-      <origin xyz="0.122 0 0.0425" rpy="0 0 0" />
+      <origin xyz="0.189 0 0.0425" rpy="0 0 0" />
       <axis xyz="0 0 1" />
       <limit lower="${head_1_lower_limit * deg_to_rad}" upper="${head_1_upper_limit * deg_to_rad}" effort="5.197" velocity="${head_max_vel}" />
