Commit message: Update collision & meshes

File: tiago_description/urdf/head/head.urdf.xacro (robot description, xacro)
@@ -41,7 +41,7 @@
       </visual>
       <collision>
-        <origin xyz="0.0305 0 0.0175" rpy="0 0 0" />
+        <origin xyz="-0.025 0 0" rpy="0 0 0.07" />
         <geometry>
-          <box size="0.05 0.035 0.035"/>
+          <box size="0.11 0.1 0.14"/>
         </geometry>
         <material name="White" />
@@ -89,4 +89,11 @@
         <material name="LightGrey"/>
       </visual>
+      <collision>
+        <origin xyz="0 0 0" rpy="0 0 0" />
+        <geometry>
+          <mesh filename="package://tiago_description/meshes/head_2.stl" scale="1 1 1"/>
+        </geometry>
+        <material name="LightGrey"/>
+      </collision>
     </link>
     <joint name="${name}_joint" type="revolute">

Commit message: Update joint limit

File: tiago_description/urdf/head/head.urdf.xacro (robot description, xacro)
@@ -1,5 +1,5 @@
 <?xml version="1.0"?>
 <!--
-  Copyright (c) 2011-2012, PAL Robotics, S.L.
+  Copyright (c) 2015, PAL Robotics, S.L.
   All rights reserved.
   This work is licensed under the Creative Commons Attribution-NonCommercial-NoDerivs 3.0 Unported License.
@@ -20,5 +20,5 @@
   <xacro:property name="head_1_upper_limit" value="75"/>
   <xacro:property name="head_2_lower_limit" value="-60"/>
-  <xacro:property name="head_2_upper_limit" value="50"/>
+  <xacro:property name="head_2_upper_limit" value="45"/>
   <!--************************-->
   <!--     HEAD_1 (PAN)       -->

Commit message: Update head, todo: dae coloring for the head_2

File: tiago_description/urdf/head/head.urdf.xacro (robot description, xacro)
@@ -51,5 +51,5 @@
       <parent link="${parent}"/>
       <child link="${name}_link"/>
-      <origin xyz="0.189 0 0.0425" rpy="0 0 0" />
+      <origin xyz="0.18735 0 0.0325" rpy="0 0 0" />
       <axis xyz="0 0 1" />
       <limit lower="${head_1_lower_limit * deg_to_rad}" upper="${head_1_upper_limit * deg_to_rad}" effort="5.197" velocity="${head_max_vel}" />
@@ -85,7 +85,6 @@
         <origin xyz="0 0 0" rpy="0 0 0" />
         <geometry>
-          <mesh filename="package://tiago_description/meshes/head_2.stl" scale="1 1 1"/>
+          <mesh filename="package://tiago_description/meshes/head_2.dae" scale="1 1 1"/>
         </geometry>
-        <material name="LightGrey"/>
       </visual>
       <collision>
@@ -94,5 +93,4 @@
           <mesh filename="package://tiago_description/meshes/head_2.stl" scale="1 1 1"/>
         </geometry>
-        <material name="LightGrey"/>
       </collision>
     </link>

File: tiago_description/urdf/sensors/xtion_pro_live.urdf.xacro (robot description, xacro)
@@ -35,4 +35,5 @@
                  izz="0.00000427339"/>
       </inertial>
+      <!--
       <visual>
         <origin xyz="0 0 0" rpy="0 0 0"/>
@@ -50,4 +51,5 @@
         </geometry>
       </collision>
+      -->
     </link>
     <joint name="${name}_optical_joint" type="fixed">

Commit message: Fix frames for orbbec astra

File: tiago_description/urdf/head/head.urdf.xacro (robot description, xacro)
@@ -12,4 +12,5 @@
   <xacro:include filename="$(find tiago_description)/urdf/head/head.transmission.xacro" />
   <xacro:include filename="$(find tiago_description)/urdf/sensors/xtion_pro_live.urdf.xacro" />
+  <xacro:include filename="$(find tiago_description)/urdf/sensors/orbbec_astra.urdf.xacro" />
   <xacro:include filename="$(find tiago_description_calibration)/urdf/calibration/calibration_constants.urdf.xacro" />
   <!--Constant parameters-->
@@ -114,9 +115,18 @@
     <xacro:head_1 name="${name}_1" parent="${parent}" />
     <xacro:head_2 name="${name}_2" parent="${name}_1_link"/>
-    <xacro:xtion_pro_live name="xtion" parent="${name}_2" camera_model="${camera_model}">
-      <origin xyz="${camera_position_x} ${camera_position_y} ${camera_position_z}" rpy="${camera_orientation_r} ${camera_orientation_p} ${camera_orientation_y}" />
-      <!-- optical origin -->
-      <origin xyz="0 0 0" rpy="${-90 * deg_to_rad} ${0 * deg_to_rad} ${-90 * deg_to_rad}" />
-    </xacro:xtion_pro_live>
+    <xacro:if value="${camera_model == 'asus-xtion'}">
+      <xacro:xtion_pro_live name="xtion" parent="${name}_2" camera_model="${camera_model}">
+        <origin xyz="${camera_position_x} ${camera_position_y} ${camera_position_z}" rpy="${camera_orientation_r} ${camera_orientation_p} ${camera_orientation_y}" />
+        <!-- optical origin -->
+        <origin xyz="0 0 0" rpy="${-90 * deg_to_rad} ${0 * deg_to_rad} ${-90 * deg_to_rad}" />
+      </xacro:xtion_pro_live>
+    </xacro:if>
+    <xacro:if value="${camera_model in ['orbbec-astra', 'orbbec-astra-pro']}">
+      <xacro:orbbec_astra name="xtion" parent="${name}_2" camera_model="${camera_model}">
+        <origin xyz="${camera_position_x} ${camera_position_y} ${camera_position_z}" rpy="${camera_orientation_r} ${camera_orientation_p} ${camera_orientation_y}" />
+        <!-- optical origin -->
+        <origin xyz="0 0 0" rpy="${-90 * deg_to_rad} ${0 * deg_to_rad} ${-90 * deg_to_rad}" />
+      </xacro:orbbec_astra>
+    </xacro:if>
   </xacro:macro>
 </robot>

Commit message: remove default description_calibration_package argument in head

File: tiago_description/urdf/head/head.urdf.xacro (robot description, xacro)
@@ -111,5 +111,5 @@
     <xacro:head_transmission name="${name}" reduction="1" offset_value="${head_2_joint_offset}"/>
   </xacro:macro>
-  <xacro:macro name="head" params="name parent camera_model description_calibration_package:=tiago_description_calibration">
+  <xacro:macro name="head" params="name parent camera_model description_calibration_package">
     <!-- includes -->
     <xacro:include filename="$(find ${description_calibration_package})/urdf/calibration/calibration_constants.urdf.xacro" />

Commit message: fix the no_safety_epc head macro issue

File: tiago_description/urdf/head/head.urdf.xacro (robot description, xacro)
@@ -24,6 +24,5 @@
   <!--     HEAD_1 (PAN)       -->
   <!--************************-->
-  <xacro:macro name="head_1" params="name parent no_safety_eps:=False">
-    <xacro:property name="head_eps"      value="${0.00 if no_safety_eps else 0.07}" />
+  <xacro:macro name="head_1" params="name parent">
     <link name="${name}_link">
       <inertial>
@@ -111,5 +110,6 @@
     <xacro:head_transmission name="${name}" reduction="1" offset_value="${head_2_joint_offset}"/>
   </xacro:macro>
-  <xacro:macro name="head" params="name parent camera_model description_calibration_dir extrinsic_calibration_dir">
+  <xacro:macro name="head" params="name parent camera_model description_calibration_dir extrinsic_calibration_dir no_safety_eps:=False">
+    <xacro:property name="head_eps"      value="${0.00 if no_safety_eps else 0.07}" />
     <!-- includes -->
     <xacro:include filename="$(arg description_calibration_dir)/calibration_constants.urdf.xacro" />
