Commit message: Add yellow

File: tiago_description/urdf/materials.urdf.xacro (robot description, xacro)
@@ -29,3 +29,6 @@
     <color rgba="1.0 1.0 1.0 1.0"/>
   </material>
+  <material name="Yellow">
+    <color rgba="0.96 0.88 0.14 1.0"/>
+  </material>
 </robot>

Commit message: Fix materials

File: tiago_description/urdf/materials.urdf.xacro (robot description, xacro)
@@ -37,3 +37,12 @@
     <color rgba="0.96 0.88 0.14 1.0"/>
   </material>
+  <material name="Orange">
+    <color rgba="1.0 0.487 0 1.0"/>
+  </material>
+  <material name="Black">
+    <color rgba="0.0 0.0 0.0 1.0"/>
+  </material>
+  <material name="FlatBlack">
+    <color rgba="0.09 0.09 0.09 1.0"/>
+  </material>
 </robot>

Commit message: add missing materials

File: tiago_description/urdf/materials.urdf.xacro (robot description, xacro)
@@ -32,3 +32,12 @@
     <color rgba="0.96 0.88 0.14 1.0"/>
   </material>
+  <material name="Orange">
+    <color rgba="1.0 0.69 0.0 1.0"/>
+  </material>
+  <material name="Black">
+    <color rgba="0.0 0.0 0.0 1.0"/>
+  </material>
+  <material name="FlatBlack">
+    <color rgba="0.09 0.09 0.09 1.0"/>
+  </material>
 </robot>
