Commit message: Add role param to plugin urdf

File: tiago_description/urdf/arm/arm.ros2_control.xacro (robot description, xacro)
@@ -18,6 +18,6 @@
     <!--
     <transmission name="${name}_${number}_trans">
-      <type>transmission_interface/SimpleTransmission</type>
-      <actuator name="${name}_${number}_motor" >
+      <plugin>transmission_interface/SimpleTransmission</plugin>
+      <actuator name="${name}_${number}_motor" role="actuator1">
         <mechanicalReduction>${reduction}</mechanicalReduction>
       </actuator>

File: tiago_description/urdf/arm/arm.transmission.xacro (robot description, xacro)
@@ -10,9 +10,9 @@
   <xacro:macro name="arm_simple_transmission" params="name number reduction offset_value" >
     <transmission name="${name}_${number}_trans">
-      <type>transmission_interface/SimpleTransmission</type>
-      <actuator name="${name}_${number}_motor" >
+      <plugin>transmission_interface/SimpleTransmission</plugin>
+      <actuator name="${name}_${number}_motor"  role="actuator1">
         <mechanicalReduction>${reduction}</mechanicalReduction>
       </actuator>
-      <joint name="${name}_${number}_joint">
+      <joint name="${name}_${number}_joint" role="joint1">
         <offset>${offset_value}</offset>
         <hardwareInterface>hardware_interface/PositionJointInterface</hardwareInterface>

File: tiago_description/urdf/arm/wrist.ros2_control.xacro (robot description, xacro)
@@ -18,6 +18,6 @@
     <!--
     <transmission name="${name}_${number}_trans">
-      <type>transmission_interface/SimpleTransmission</type>
-      <actuator name="${name}_${number}_motor" >
+      <plugin>transmission_interface/SimpleTransmission</plugin>
+      <actuator name="${name}_${number}_motor" role="actuator1">
         <mechanicalReduction>${reduction}</mechanicalReduction>
       </actuator>
@@ -48,15 +48,12 @@
     <!--
     <transmission name="${name1}_${name2}_wrist_trans">
-      <type>transmission_interface/DifferentialTransmission</type>
-      <actuator name="${name_1}_motor">
-        <role>actuator1</role>
+      <plugin>transmission_interface/DifferentialTransmission</plugin>
+      <actuator name="${name_1}_motor" role="actuator1">
         <mechanicalReduction>${act_reduction_1}</mechanicalReduction>
       </actuator>
-      <actuator name="${name_2}_motor">
-        <role>actuator2</role>
+      <actuator name="${name_2}_motor" role="actuator2">
         <mechanicalReduction>${act_reduction_2}</mechanicalReduction>
       </actuator>
-      <joint name="${name_1}_joint">
-        <role>joint1</role>
+      <joint name="${name_1}_joint" role="joint1">
         <offset>${number_1_offset}</offset>
         <mechanicalReduction>${jnt_reduction_1}</mechanicalReduction>
@@ -66,6 +63,5 @@
         <ignoreTransmissionAbsoluteEncoder>1</ignoreTransmissionAbsoluteEncoder>
       </joint>
-      <joint name="${name_2}_joint">
-        <role>joint2</role>
+      <joint name="${name_2}_joint" role="joint2">
         <offset>${number_2_offset}</offset>
         <mechanicalReduction>${jnt_reduction_2}</mechanicalReduction>

File: tiago_description/urdf/arm/wrist.transmission.xacro (robot description, xacro)
@@ -11,9 +11,9 @@
   <xacro:macro name="wrist_simple_transmission" params="name number reduction offset" >
     <transmission name="${name}_${number}_trans">
-      <type>transmission_interface/SimpleTransmission</type>
-      <actuator name="${name}_${number}_motor" >
+      <plugin>transmission_interface/SimpleTransmission</plugin>
+      <actuator name="${name}_${number}_motor"  role="actuator1">
         <mechanicalReduction>${reduction}</mechanicalReduction>
       </actuator>
-      <joint name="${name}_${number}_joint">
+      <joint name="${name}_${number}_joint" role="joint1">
         <offset>${offset}</offset>
         <hardwareInterface>hardware_interface/JointStateInterface</hardwareInterface>
@@ -26,15 +26,12 @@
                params="name number_1 number_2 act_reduction_1 act_reduction_2 jnt_reduction_1 jnt_reduction_2 number_1_offset number_2_offset" >
   <transmission name="${name}_wrist_trans">
-      <type>transmission_interface/DifferentialTransmission</type>
-      <actuator name="${name}_${number_1}_motor">
-        <role>actuator1</role>
+      <plugin>transmission_interface/DifferentialTransmission</plugin>
+      <actuator name="${name}_${number_1}_motor" role="actuator1">
         <mechanicalReduction>${act_reduction_1}</mechanicalReduction>
       </actuator>
-      <actuator name="${name}_${number_2}_motor">
-        <role>actuator2</role>
+      <actuator name="${name}_${number_2}_motor" role="actuator2">
         <mechanicalReduction>${act_reduction_2}</mechanicalReduction>
       </actuator>
-      <joint name="${name}_${number_1}_joint">
-        <role>joint1</role>
+      <joint name="${name}_${number_1}_joint" role="joint1">
         <offset>${number_1_offset}</offset>
         <mechanicalReduction>${jnt_reduction_1}</mechanicalReduction>
@@ -44,6 +41,5 @@
         <ignoreTransmissionAbsoluteEncoder>1</ignoreTransmissionAbsoluteEncoder>
       </joint>
-      <joint name="${name}_${number_2}_joint">
-        <role>joint2</role>
+      <joint name="${name}_${number_2}_joint" role="joint2">
         <offset>${number_2_offset}</offset>
         <mechanicalReduction>${jnt_reduction_2}</mechanicalReduction>

File: tiago_description/urdf/head/head.ros2_control.xacro (robot description, xacro)
@@ -18,6 +18,6 @@
     <!--
     <transmission name="${name}_trans">
-      <type>transmission_interface/SimpleTransmission</type>
-      <actuator name="${name}_motor" >
+      <plugin>transmission_interface/SimpleTransmission</plugin>
+      <actuator name="${name}_motor" role="actuator1">
         <mechanicalReduction>${reduction}</mechanicalReduction>
       </actuator>

File: tiago_description/urdf/head/head.transmission.xacro (robot description, xacro)
@@ -10,9 +10,9 @@
   <xacro:macro name="head_transmission" params="name reduction offset_value">
     <transmission name="${name}_trans">
-      <type>transmission_interface/SimpleTransmission</type>
-      <actuator name="${name}_motor" >
+      <plugin>transmission_interface/SimpleTransmission</plugin>
+      <actuator name="${name}_motor"  role="actuator1">
         <mechanicalReduction>${reduction}</mechanicalReduction>
       </actuator>
-      <joint name="${name}_joint" >
+      <joint name="${name}_joint"  role="joint1">
         <offset>${offset_value}</offset>
         <hardwareInterface>hardware_interface/JointStateInterface</hardwareInterface>

File: tiago_description/urdf/torso/torso.ros2_control.xacro (robot description, xacro)
@@ -18,6 +18,6 @@
     <!--
     <transmission name="${name}_trans">
-      <type>transmission_interface/SimpleTransmission</type>
-      <actuator name="${name}_motor" >
+      <plugin>transmission_interface/SimpleTransmission</plugin>
+      <actuator name="${name}_motor" role="actuator1">
         <mechanicalReduction>${reduction}</mechanicalReduction>
       </actuator>

File: tiago_description/urdf/torso/torso.transmission.xacro (robot description, xacro)
@@ -10,9 +10,9 @@
   <xacro:macro name="torso_simple_transmission" params="name reduction" >
     <transmission name="${name}_trans">
-      <type>transmission_interface/SimpleTransmission</type>
-      <actuator name="${name}_motor" >
+      <plugin>transmission_interface/SimpleTransmission</plugin>
+      <actuator name="${name}_motor" role="actuator1">
         <mechanicalReduction>${reduction}</mechanicalReduction>
       </actuator>
-      <joint name="${name}_joint">
+      <joint name="${name}_joint" role="joint1">
         <hardwareInterface>hardware_interface/PositionJointInterface</hardwareInterface>
         <hardwareInterface>hardware_interface/JointStateInterface</hardwareInterface>

Commit message: set transmissions inside the ros2_control tag

File: tiago_description/urdf/arm/arm.ros2_control.xacro (robot description, xacro)
@@ -20,19 +20,5 @@
       <state_interface name="effort" />
     </joint>
-    <!-- @TODO transmissions for ros2 system -->
-    <!--
-    <transmission name="${name}_${number}_trans">
-      <plugin>transmission_interface/SimpleTransmission</plugin>
-      <actuator name="${name}_${number}_motor" role="actuator1">
-        <mechanicalReduction>${reduction}</mechanicalReduction>
-      </actuator>
-      <joint name="${name}_${number}_joint">
-        <offset>${offset}</offset>
-        <hardwareInterface>hardware_interface/PositionJointInterface</hardwareInterface>
-        <hardwareInterface>hardware_interface/EffortJointInterface</hardwareInterface>
-        <hardwareInterface>hardware_interface/JointStateInterface</hardwareInterface>
-      </joint>
-    </transmission>
-    -->
+    <xacro:arm_simple_transmission name="${name}" reduction="${reduction}" offset_value="${offset}"/>
   </xacro:macro>
 </robot>

File: tiago_description/urdf/arm/arm.transmission.xacro (robot description, xacro)
@@ -13,11 +13,11 @@
  -->
 <robot xmlns:xacro="http://ros.org/wiki/xacro">
-  <xacro:macro name="arm_simple_transmission" params="name number reduction offset_value" >
-    <transmission name="${name}_${number}_trans">
+  <xacro:macro name="arm_simple_transmission" params="name reduction offset_value" >
+    <transmission name="${name}_trans">
       <plugin>transmission_interface/SimpleTransmission</plugin>
-      <actuator name="${name}_${number}_motor"  role="actuator1">
+      <actuator name="${name}_motor"  role="actuator1">
         <mechanicalReduction>${reduction}</mechanicalReduction>
       </actuator>
-      <joint name="${name}_${number}_joint" role="joint1">
+      <joint name="${name}_joint" role="joint1">
         <offset>${offset_value}</offset>
         <hardwareInterface>hardware_interface/PositionJointInterface</hardwareInterface>

File: tiago_description/urdf/arm/wrist.ros2_control.xacro (robot description, xacro)
@@ -20,23 +20,9 @@
       <state_interface name="effort" />
     </joint>
-    <!-- @TODO transmissions for ros2 system -->
-    <!--
-    <transmission name="${name}_${number}_trans">
-      <plugin>transmission_interface/SimpleTransmission</plugin>
-      <actuator name="${name}_${number}_motor" role="actuator1">
-        <mechanicalReduction>${reduction}</mechanicalReduction>
-      </actuator>
-      <joint name="${name}_${number}_joint">
-        <offset>${offset}</offset>
-        <hardwareInterface>hardware_interface/JointStateInterface</hardwareInterface>
-        <hardwareInterface>hardware_interface/PositionJointInterface</hardwareInterface>
-        <hardwareInterface>hardware_interface/EffortJointInterface</hardwareInterface>
-      </joint>
-    </transmission>
-    -->
+    <xacro:wrist_simple_transmission name="${name}" reduction="${reduction}" offset="${offset}"/>
   </xacro:macro>
   <xacro:macro name="ros2_control_wrist_differential"
-               params="name_1 name_2 act_reduction_1 act_reduction_2 jnt_reduction_1 jnt_reduction_2 number_1_offset number_2_offset" >
-    <joint name="${name_1}_joint">
+               params="name number_1 number_2 act_reduction_1 act_reduction_2 jnt_reduction_1 jnt_reduction_2 number_1_offset number_2_offset" >
+    <joint name="${name}_${number_1}_joint">
       <command_interface name="position" />
       <state_interface name="position" />
@@ -44,5 +30,5 @@
       <state_interface name="effort" />
     </joint>
-    <joint name="${name_2}_joint">
+    <joint name="${name}_${number_2}_joint">
       <command_interface name="position" />
       <state_interface name="position" />
@@ -50,32 +36,4 @@
       <state_interface name="effort" />
     </joint>
-    <!-- @TODO transmissions for ros2 system -->
-    <!--
-    <transmission name="${name1}_${name2}_wrist_trans">
-      <plugin>transmission_interface/DifferentialTransmission</plugin>
-      <actuator name="${name_1}_motor" role="actuator1">
-        <mechanicalReduction>${act_reduction_1}</mechanicalReduction>
-      </actuator>
-      <actuator name="${name_2}_motor" role="actuator2">
-        <mechanicalReduction>${act_reduction_2}</mechanicalReduction>
-      </actuator>
-      <joint name="${name_1}_joint" role="joint1">
-        <offset>${number_1_offset}</offset>
-        <mechanicalReduction>${jnt_reduction_1}</mechanicalReduction>
-        <hardwareInterface>hardware_interface/JointStateInterface</hardwareInterface>
-        <hardwareInterface>hardware_interface/PositionJointInterface</hardwareInterface>
-        <hardwareInterface>hardware_interface/EffortJointInterface</hardwareInterface>
-        <ignoreTransmissionAbsoluteEncoder>1</ignoreTransmissionAbsoluteEncoder>
-      </joint>
-      <joint name="${name_2}_joint" role="joint2">
-        <offset>${number_2_offset}</offset>
-        <mechanicalReduction>${jnt_reduction_2}</mechanicalReduction>
-        <hardwareInterface>hardware_interface/JointStateInterface</hardwareInterface>
-        <hardwareInterface>hardware_interface/PositionJointInterface</hardwareInterface>
-        <hardwareInterface>hardware_interface/EffortJointInterface</hardwareInterface>
-        <ignoreTransmissionAbsoluteEncoder>1</ignoreTransmissionAbsoluteEncoder>
-      </joint>
-    </transmission>
-    -->
   </xacro:macro>
 </robot>

File: tiago_description/urdf/arm/wrist.transmission.xacro (robot description, xacro)
@@ -13,11 +13,11 @@
  -->
 <robot xmlns:xacro="http://ros.org/wiki/xacro">
-  <xacro:macro name="wrist_simple_transmission" params="name number reduction offset" >
-    <transmission name="${name}_${number}_trans">
+  <xacro:macro name="wrist_simple_transmission" params="name reduction offset" >
+    <transmission name="${name}_trans">
       <plugin>transmission_interface/SimpleTransmission</plugin>
-      <actuator name="${name}_${number}_motor"  role="actuator1">
+      <actuator name="${name}_motor"  role="actuator1">
         <mechanicalReduction>${reduction}</mechanicalReduction>
       </actuator>
-      <joint name="${name}_${number}_joint" role="joint1">
+      <joint name="${name}_joint" role="joint1">
         <offset>${offset}</offset>
         <hardwareInterface>hardware_interface/JointStateInterface</hardwareInterface>
@@ -29,5 +29,5 @@
   <xacro:macro name="wrist_differential_transmission"
                params="name number_1 number_2 act_reduction_1 act_reduction_2 jnt_reduction_1 jnt_reduction_2 number_1_offset number_2_offset" >
-  <transmission name="${name}_wrist_trans">
+  <transmission name="${name}_${number_1}_${name}_${number_2}_wrist_trans">
       <plugin>transmission_interface/DifferentialTransmission</plugin>
       <actuator name="${name}_${number_1}_motor" role="actuator1">
