Commit message: Update license

File: tiago_description/urdf/arm/arm.transmission.xacro (robot description, xacro)
@@ -1,5 +1,5 @@
 <?xml version="1.0"?>
 <!--
-  Copyright (c) 2011, PAL Robotics, S.L.
+  Copyright (c) 2015, PAL Robotics, S.L.
   All rights reserved.
   This work is licensed under the Creative Commons Attribution-NonCommercial-NoDerivs 3.0 Unported License.

File: tiago_description/urdf/arm/arm.urdf.xacro (robot description, xacro)
@@ -1,5 +1,5 @@
 <?xml version="1.0"?>
 <!--
-  Copyright (c) 2014, PAL Robotics, S.L.
+  Copyright (c) 2014-2015, PAL Robotics, S.L.
   All rights reserved.
   This work is licensed under the Creative Commons Attribution-NonCommercial-NoDerivs 3.0 Unported License.

File: tiago_description/urdf/arm/wrist.transmission.xacro (robot description, xacro)
@@ -1,5 +1,5 @@
 <?xml version="1.0"?>
 <!--
-  Copyright (c) 2011, PAL Robotics, S.L.
+  Copyright (c) 2015, PAL Robotics, S.L.
   All rights reserved.
   This work is licensed under the Creative Commons Attribution-NonCommercial-NoDerivs 3.0 Unported License.

File: tiago_description/urdf/arm/wrist.urdf.xacro (robot description, xacro)
@@ -1,5 +1,5 @@
 <?xml version="1.0"?>
 <!--
-  Copyright (c) 2011-2012, PAL Robotics, S.L.
+  Copyright (c) 2015, PAL Robotics, S.L.
   All rights reserved.
   This work is licensed under the Creative Commons Attribution-NonCommercial-NoDerivs 3.0 Unported License.
@@ -21,5 +21,4 @@
   <xacro:property name="wrist_3_max_effort"   value="6.6" />
   <xacro:property name="wrist_eps"          value="0.02" />
-  <!-- TODO: Update dynamic models -->
   <xacro:macro name="wrist" params="name parent reflect">
     <!--************************-->
@@ -51,5 +50,5 @@
       <origin xyz="-0.168 0.02 0" rpy="${0 * deg_to_rad} ${-90 * deg_to_rad} ${0 * deg_to_rad}" />
       <axis xyz="0 0 1" />
-      <limit lower="${-120.0 * deg_to_rad}" upper="${120.0 * deg_to_rad}" effort="${wrist_1_max_effort}" velocity="${wrist_1_max_vel}" /> <!--TODO: Check effort value!-->
+      <limit lower="${-120.0 * deg_to_rad}" upper="${120.0 * deg_to_rad}" effort="${wrist_1_max_effort}" velocity="${wrist_1_max_vel}" />
       <dynamics friction="${wrist_friction}" damping="${wrist_damping}"/>
       <safety_controller k_position="20"

File: tiago_description/urdf/head/head.transmission.xacro (robot description, xacro)
@@ -1,5 +1,5 @@
 <?xml version="1.0"?>
 <!--
-  Copyright (c) 2011, PAL Robotics, S.L.
+  Copyright (c) 2015, PAL Robotics, S.L.
   All rights reserved.
   This work is licensed under the Creative Commons Attribution-NonCommercial-NoDerivs 3.0 Unported License.

File: tiago_description/urdf/materials.urdf.xacro (robot description, xacro)
@@ -1,5 +1,5 @@
 <?xml version="1.0"?>
 <!--
-  Copyright (c) 2011, PAL Robotics, S.L.
+  Copyright (c) 2011-2015, PAL Robotics, S.L.
   All rights reserved.
   This work is licensed under the Creative Commons Attribution-NonCommercial-NoDerivs 3.0 Unported License.

File: tiago_description/urdf/torso/torso.urdf.xacro (robot description, xacro)
@@ -1,3 +1,10 @@
 <?xml version="1.0" ?>
+<!--
+  Copyright (c) 2015, PAL Robotics, S.L.
+  All rights reserved.
+  This work is licensed under the Creative Commons Attribution-NonCommercial-NoDerivs 3.0 Unported License.
+  To view a copy of this license, visit http://creativecommons.org/licenses/by-nc-nd/3.0/ or send a letter to
+  Creative Commons, 444 Castro Street, Suite 900, Mountain View, California, 94041, USA.
+-->
 <robot xmlns:xacro="http://ros.org/wiki/xacro">
   <!--File includes-->
@@ -43,4 +50,5 @@
     <axis xyz="0 0 0" />
   </joint>
+  <!-- Middle extending  -->
   <link name="${name}_fixed_column_link">
     <inertial>

Commit message: Modify the offset to allow the automatic calibration

File: tiago_description/urdf/arm/arm.transmission.xacro (robot description, xacro)
@@ -8,5 +8,5 @@
 -->
 <robot xmlns:xacro="http://ros.org/wiki/xacro">
-  <xacro:macro name="arm_simple_transmission" params="name number reduction" >
+  <xacro:macro name="arm_simple_transmission" params="name number reduction offset_value" >
     <transmission name="${name}_${number}_trans">
       <type>transmission_interface/SimpleTransmission</type>
@@ -15,4 +15,5 @@
       </actuator>
       <joint name="${name}_${number}_joint">
+        <offset>${offset_value}</offset>
         <hardwareInterface>hardware_interface/PositionJointInterface</hardwareInterface>
         <hardwareInterface>hardware_interface/EffortJointInterface</hardwareInterface>

File: tiago_description/urdf/arm/arm.urdf.xacro (robot description, xacro)
@@ -12,4 +12,5 @@
   <xacro:include filename="$(find tiago_description)/urdf/arm/wrist.urdf.xacro" />
   <xacro:include filename="$(find tiago_description)/urdf/arm/arm.transmission.xacro" />
+  <xacro:include filename="$(find tiago_description)/urdf/calibration/calibration_constants.urdf.xacro" />
   <!--Constant parameters-->
   <xacro:property name="arm_friction"       value="1.0" />
@@ -240,8 +241,8 @@
     </joint>
     <!-- extensions -->
-    <xacro:arm_simple_transmission name="${name}" number="1" reduction="1.0" />
-    <xacro:arm_simple_transmission name="${name}" number="2" reduction="1.0" />
-    <xacro:arm_simple_transmission name="${name}" number="3" reduction="1.0" />
-    <xacro:arm_simple_transmission name="${name}" number="4" reduction="1.0" />
+    <xacro:arm_simple_transmission name="${name}" number="1" reduction="1.0" offset_value="${arm_1_joint_offset}"/>
+    <xacro:arm_simple_transmission name="${name}" number="2" reduction="1.0" offset_value="${arm_2_joint_offset}"/>
+    <xacro:arm_simple_transmission name="${name}" number="3" reduction="1.0" offset_value="${arm_3_joint_offset}"/>
+    <xacro:arm_simple_transmission name="${name}" number="4" reduction="1.0" offset_value="${arm_4_joint_offset}"/>
   </xacro:macro>
 </robot>

File: tiago_description/urdf/arm/wrist.transmission.xacro (robot description, xacro)
@@ -8,4 +8,6 @@
 -->
 <robot xmlns:xacro="http://ros.org/wiki/xacro">
+  <!--File includes-->
+  <xacro:include filename="$(find tiago_description)/urdf/calibration/calibration_constants.urdf.xacro" />
   <xacro:macro name="wrist_simple_transmission" params="name number reduction" >
     <transmission name="${name}_${number}_trans">
@@ -15,4 +17,5 @@
       </actuator>
       <joint name="${name}_${number}_joint">
+        <offset>${arm_5_joint_offset}</offset>
         <hardwareInterface>hardware_interface/PositionJointInterface</hardwareInterface>
       </joint>
@@ -33,5 +36,5 @@
       <joint name="${name}_${number_1}_joint">
         <role>joint1</role>
-        <offset>0.0</offset>
+        <offset>${arm_6_joint_offset}</offset>
         <mechanicalReduction>${jnt_reduction_1}</mechanicalReduction>
         <hardwareInterface>hardware_interface/PositionJointInterface</hardwareInterface>
@@ -39,5 +42,5 @@
       <joint name="${name}_${number_2}_joint">
         <role>joint2</role>
-        <offset>0.0</offset>
+        <offset>${arm_7_joint_offset}</offset>
         <mechanicalReduction>${jnt_reduction_2}</mechanicalReduction>
         <hardwareInterface>hardware_interface/PositionJointInterface</hardwareInterface>

File: tiago_description/urdf/head/head.transmission.xacro (robot description, xacro)
@@ -8,5 +8,5 @@
 -->
 <robot xmlns:xacro="http://ros.org/wiki/xacro">
-  <xacro:macro name="head_transmission" params="name reduction">
+  <xacro:macro name="head_transmission" params="name reduction offset_value">
     <transmission name="${name}_trans">
       <type>transmission_interface/SimpleTransmission</type>
@@ -15,4 +15,5 @@
       </actuator>
       <joint name="${name}_joint" >
+        <offset>${offset_value}</offset>
         <hardwareInterface>hardware_interface/PositionJointInterface</hardwareInterface>
       </joint>

File: tiago_description/urdf/head/head.urdf.xacro (robot description, xacro)
@@ -12,4 +12,5 @@
   <xacro:include filename="$(find tiago_description)/urdf/head/head.transmission.xacro" />
   <xacro:include filename="$(find tiago_description)/urdf/sensors/xtion_pro_live.urdf.xacro" />
+  <xacro:include filename="$(find tiago_description)/urdf/calibration/calibration_constants.urdf.xacro" />
   <!--Constant parameters-->
   <xacro:property name="head_friction" value="1.0" />
@@ -68,5 +69,5 @@
     </gazebo>
     <!-- extensions -->
-    <xacro:head_transmission name="${name}" reduction="1" />
+    <xacro:head_transmission name="${name}" reduction="1" offset_value="${head_1_joint_offset}"/>
   </xacro:macro>
   <!--************************-->
@@ -108,5 +109,5 @@
                          soft_upper_limit="${head_2_upper_limit * deg_to_rad}" />
     </joint>
-    <xacro:head_transmission name="${name}" reduction="1" />
+    <xacro:head_transmission name="${name}" reduction="1" offset_value="${head_2_joint_offset}"/>
   </xacro:macro>
   <xacro:macro name="head" params="name parent">
@@ -114,5 +115,5 @@
     <xacro:head_2 name="${name}_2" parent="${name}_1_link"/>
     <xacro:xtion_pro_live name="xtion" parent="${name}_2">
-      <origin xyz="0.0908 0.08 0" rpy="${-90 * deg_to_rad} 0 0" />
+      <origin xyz="${camera_position_x} ${camera_position_y} ${camera_position_z}" rpy="${camera_orientation_r} ${camera_orientation_p} ${camera_orientation_y}" />
       <!-- optical origin -->
       <origin xyz="0 0 0" rpy="${-90 * deg_to_rad} ${0 * deg_to_rad} ${-90 * deg_to_rad}" />

Commit message: update transmission tags for ros2

File: tiago_description/urdf/arm/arm.transmission.xacro (robot description, xacro)
@@ -16,13 +16,9 @@
     <transmission name="${name}_trans">
       <plugin>transmission_interface/SimpleTransmission</plugin>
-      <actuator name="${name}_motor"  role="actuator1">
-        <mechanicalReduction>${reduction}</mechanicalReduction>
-      </actuator>
+      <actuator name="${name}_motor"  role="actuator1"/>
       <joint name="${name}_joint" role="joint1">
+        <mechanical_reduction>${reduction}</mechanical_reduction>
         <offset>${offset_value}</offset>
-        <hardwareInterface>hardware_interface/PositionJointInterface</hardwareInterface>
-        <hardwareInterface>hardware_interface/EffortJointInterface</hardwareInterface>
-        <hardwareInterface>hardware_interface/JointStateInterface</hardwareInterface>
-      </joint>
+     </joint>
     </transmission>
   </xacro:macro>

File: tiago_description/urdf/arm/wrist.transmission.xacro (robot description, xacro)
@@ -16,12 +16,8 @@
     <transmission name="${name}_trans">
       <plugin>transmission_interface/SimpleTransmission</plugin>
-      <actuator name="${name}_motor"  role="actuator1">
-        <mechanicalReduction>${reduction}</mechanicalReduction>
-      </actuator>
+      <actuator name="${name}_motor"  role="actuator1"/>
       <joint name="${name}_joint" role="joint1">
+        <mechanical_reduction>${reduction}</mechanical_reduction>
         <offset>${offset}</offset>
-        <hardwareInterface>hardware_interface/JointStateInterface</hardwareInterface>
-        <hardwareInterface>hardware_interface/PositionJointInterface</hardwareInterface>
-        <hardwareInterface>hardware_interface/EffortJointInterface</hardwareInterface>
       </joint>
     </transmission>
@@ -32,24 +28,16 @@
       <plugin>transmission_interface/DifferentialTransmission</plugin>
       <actuator name="${name}_${number_1}_motor" role="actuator1">
-        <mechanicalReduction>${act_reduction_1}</mechanicalReduction>
+      <mechanical_reduction>${act_reduction_1}</mechanical_reduction>
       </actuator>
       <actuator name="${name}_${number_2}_motor" role="actuator2">
-        <mechanicalReduction>${act_reduction_2}</mechanicalReduction>
+        <mechanical_reduction>${act_reduction_2}</mechanical_reduction>
       </actuator>
       <joint name="${name}_${number_1}_joint" role="joint1">
+        <mechanical_reduction>${jnt_reduction_1}</mechanical_reduction>
         <offset>${number_1_offset}</offset>
-        <mechanicalReduction>${jnt_reduction_1}</mechanicalReduction>
-        <hardwareInterface>hardware_interface/JointStateInterface</hardwareInterface>
-        <hardwareInterface>hardware_interface/PositionJointInterface</hardwareInterface>
-        <hardwareInterface>hardware_interface/EffortJointInterface</hardwareInterface>
-        <ignoreTransmissionAbsoluteEncoder>1</ignoreTransmissionAbsoluteEncoder>
       </joint>
       <joint name="${name}_${number_2}_joint" role="joint2">
+        <mechanical_reduction>${jnt_reduction_2}</mechanical_reduction>
         <offset>${number_2_offset}</offset>
-        <mechanicalReduction>${jnt_reduction_2}</mechanicalReduction>
-        <hardwareInterface>hardware_interface/JointStateInterface</hardwareInterface>
-        <hardwareInterface>hardware_interface/PositionJointInterface</hardwareInterface>
-        <hardwareInterface>hardware_interface/EffortJointInterface</hardwareInterface>
-        <ignoreTransmissionAbsoluteEncoder>1</ignoreTransmissionAbsoluteEncoder>
       </joint>
     </transmission>
