Commit message: Fix visuals on arm

File: tiago_description/urdf/arm/arm.urdf.xacro (robot description, xacro)
@@ -36,14 +36,14 @@
       </inertial>
       <visual>
-        <origin xyz="0 0 0" rpy="0 0 0" />
-        <geometry>
-          <mesh filename="package://tiago_description/meshes/arm/arm_1.dae" scale="1 1 -1"/>
-        </geometry>
-        <material name="DarkGrey" />
-      </visual>
-      <collision>
-       <origin xyz="0 0 0" rpy="0 0 0" />
-        <geometry>
-          <mesh filename="package://tiago_description/meshes/arm/arm_1_collision.stl" scale="1 1 -1"/>
+        <origin xyz="0.11 0 0.13" rpy="0 0 ${90 * deg_to_rad}" />
+        <geometry>
+          <mesh filename="package://tiago_description/meshes/arm/arm_1.dae" scale="1 1 1"/>
+        </geometry>
+        <material name="DarkGrey" />
+      </visual>
+      <collision>
+       <origin xyz="0.11 0 0.13" rpy="0 0 0" />
+        <geometry>
+          <mesh filename="package://tiago_description/meshes/arm/arm_1_collision.stl" scale="1 1 1"/>
         </geometry>
       </collision>
@@ -68,14 +68,14 @@
       </inertial>
       <visual>
-        <origin xyz="0 0 0" rpy="0 0 0" />
-        <geometry>
-          <mesh filename="package://tiago_description/meshes/arm/arm_2.dae" scale="1 1 -1"/>
-        </geometry>
-        <material name="DarkGrey" />
-      </visual>
-      <collision>
-        <origin xyz="0 0 0" rpy="0 0 0" />
-        <geometry>
-          <mesh filename="package://tiago_description/meshes/arm/arm_2_collision.stl" scale="1 1 -1"/>
+        <origin xyz="0 0 0" rpy="${180 * deg_to_rad} ${0 * deg_to_rad} ${-90 * deg_to_rad}" />
+        <geometry>
+          <mesh filename="package://tiago_description/meshes/arm/arm_2.dae" scale="1 1 1"/>
+        </geometry>
+        <material name="DarkGrey" />
+      </visual>
+      <collision>
+        <origin xyz="0 0 0" rpy="${180 * deg_to_rad} ${0 * deg_to_rad} ${-90 * deg_to_rad}" />
+        <geometry>
+          <mesh filename="package://tiago_description/meshes/arm/arm_2_collision.stl" scale="1 1 1"/>
         </geometry>
       </collision>
@@ -100,14 +100,21 @@
       </inertial>
       <visual>
-        <origin xyz="0 0 0" rpy="0 0 0" />
-        <geometry>
-          <mesh filename="package://tiago_description/meshes/arm/arm_3.dae" scale="1 1 -1"/>
-        </geometry>
-        <material name="DarkGrey" />
-      </visual>
-      <collision>
-        <origin xyz="0 0 0" rpy="0 0 0" />
-        <geometry>
-          <mesh filename="package://tiago_description/meshes/arm/arm_3_collision.stl" scale="1 1 -1"/>
+        <origin xyz="0 0 -0.1" rpy="0 0 0" />
+        <geometry>
+          <mesh filename="package://tiago_description/meshes/arm/arm_3.dae" scale="1 1 1"/>
+        </geometry>
+        <material name="DarkGrey" />
+      </visual>
+      <visual>
+        <origin xyz="0 0 0" rpy="0 0 0" />
+        <geometry>
+          <cylinder length="0.12" radius="0.06" />
+        </geometry>
+        <material name="DarkGrey" />
+      </visual>
+      <collision>
+        <origin xyz="0 0 0" rpy="0 0 0" />
+        <geometry>
+          <mesh filename="package://tiago_description/meshes/arm/arm_3_collision.stl" scale="1 1 1"/>
         </geometry>
       </collision>
@@ -137,12 +144,12 @@
         <origin xyz="0 0 0" rpy="0 0 0" />
         <geometry>
-          <mesh filename="package://tiago_description/meshes/arm/arm_4.dae" scale="1 1 -1"/>
-        </geometry>
-        <material name="DarkGrey" />
-      </visual>
-      <collision>
-        <origin xyz="0 0 0" rpy="0 0 0" />
-        <geometry>
-          <mesh filename="package://tiago_description/meshes/arm/arm_4_collision.stl" scale="1 1 -1"/>
+          <mesh filename="package://tiago_description/meshes/arm/arm_4.dae" scale="1 1 1"/>
+        </geometry>
+        <material name="DarkGrey" />
+      </visual>
+      <collision>
+        <origin xyz="0 0 0" rpy="0 0 0" />
+        <geometry>
+          <mesh filename="package://tiago_description/meshes/arm/arm_4_collision.stl" scale="1 1 1"/>
         </geometry>
       </collision>

Commit message: Add visual & collision before wrist

File: tiago_description/urdf/arm/arm.urdf.xacro (robot description, xacro)
@@ -43,5 +43,5 @@
       </visual>
       <collision>
-       <origin xyz="0.11 0 0.13" rpy="0 0 0" />
+       <origin xyz="0.11 0 0.13" rpy="0 0 ${90 * deg_to_rad}" />
         <geometry>
           <mesh filename="package://tiago_description/meshes/arm/arm_1_collision.stl" scale="1 1 1"/>
@@ -107,15 +107,22 @@
       </visual>
       <visual>
-        <origin xyz="0 0 0" rpy="0 0 0" />
-        <geometry>
-          <cylinder length="0.12" radius="0.06" />
-        </geometry>
-        <material name="DarkGrey" />
-      </visual>
-      <collision>
-        <origin xyz="0 0 0" rpy="0 0 0" />
+        <origin xyz="0 0 -0.025" rpy="0 0 0" />
+        <geometry>
+          <cylinder length="0.11" radius="0.05" />
+        </geometry>
+        <material name="DarkGrey" />
+      </visual>
+      <collision>
+        <origin xyz="0 0 -0.1" rpy="0 0 0" />
         <geometry>
           <mesh filename="package://tiago_description/meshes/arm/arm_3_collision.stl" scale="1 1 1"/>
         </geometry>
+      </collision>
+      <collision>
+        <origin xyz="0 0 -0.025" rpy="0 0 0" />
+        <geometry>
+          <cylinder length="0.11" radius="0.05" />
+        </geometry>
+        <material name="DarkGrey" />
       </collision>
     </link>
@@ -148,4 +155,11 @@
         <material name="DarkGrey" />
       </visual>
+      <visual>
+        <origin xyz="-0.13 0.02 0" rpy="0 ${90 * deg_to_rad} 0" />
+        <geometry>
+          <cylinder length="0.05" radius="0.05" />
+        </geometry>
+        <material name="DarkGrey" />
+      </visual>
       <collision>
         <origin xyz="0 0 0" rpy="0 0 0" />
@@ -153,4 +167,11 @@
           <mesh filename="package://tiago_description/meshes/arm/arm_4_collision.stl" scale="1 1 1"/>
         </geometry>
+      </collision>
+      <collision>
+        <origin xyz="-0.13 0.02 0" rpy="0 ${90 * deg_to_rad} 0" />
+        <geometry>
+          <cylinder length="0.05" radius="0.05" />
+        </geometry>
+        <material name="DarkGrey" />
       </collision>
     </link>

Commit message: Update joint limits

File: tiago_description/urdf/arm/arm.urdf.xacro (robot description, xacro)
@@ -54,5 +54,5 @@
       <origin xyz="0.1 0.07 0" rpy="${0 * deg_to_rad} ${0 * deg_to_rad} ${-90 * deg_to_rad}" />
       <axis xyz="0 0 1" />
-      <limit lower="${-45.0 * deg_to_rad}" upper="${180.0 * deg_to_rad}" effort="${arm_1_max_effort}" velocity="${arm_1_max_vel}" />
+      <limit lower="${0.0 * deg_to_rad}" upper="${180.0 * deg_to_rad}" effort="${arm_1_max_effort}" velocity="${arm_1_max_vel}" />
       <dynamics friction="${arm_friction}" damping="${arm_damping}"/>
       <safety_controller k_position="20"
@@ -86,10 +86,10 @@
       <origin xyz="0.11 0 -0.08" rpy="${90.0 * deg_to_rad} ${0 * deg_to_rad} ${0 * deg_to_rad}" />
       <axis xyz="0 0 1" />
-      <limit lower="${-15.0 * deg_to_rad}" upper="${120.0 * deg_to_rad}" effort="${arm_2_max_effort}" velocity="${arm_2_max_vel}" />
-      <dynamics friction="${arm_friction}" damping="${arm_damping}"/>
-      <safety_controller k_position="20"
-                         k_velocity="20"
-                         soft_lower_limit="${-15.0 * deg_to_rad  + arm_eps}"
-                         soft_upper_limit="${ 120.0 * deg_to_rad - arm_eps}" />
+      <limit lower="${-120.0 * deg_to_rad}" upper="${60.0 * deg_to_rad}" effort="${arm_2_max_effort}" velocity="${arm_2_max_vel}" />
+      <dynamics friction="${arm_friction}" damping="${arm_damping}"/>
+      <safety_controller k_position="20"
+                         k_velocity="20"
+                         soft_lower_limit="${-120.0 * deg_to_rad  + arm_eps}"
+                         soft_upper_limit="${ 60.0 * deg_to_rad - arm_eps}" />
     </joint>
     <link name="${name}_3_link">
@@ -181,9 +181,9 @@
       <origin xyz="0 -0.02 -0.183" rpy="0 ${-90.0 * deg_to_rad} 0" />
       <axis xyz="0 0 1" />
-      <limit lower="0" upper="${130.0 * deg_to_rad}" effort="${arm_4_max_effort}" velocity="${arm_4_max_vel}" />
-      <dynamics friction="${arm_friction}" damping="${arm_damping}"/>
-      <safety_controller k_position="20"
-                         k_velocity="20"
-                         soft_lower_limit="0.0"
+      <limit lower="${-110 * deg_to_rad}" upper="${130.0 * deg_to_rad}" effort="${arm_4_max_effort}" velocity="${arm_4_max_vel}" />
+      <dynamics friction="${arm_friction}" damping="${arm_damping}"/>
+      <safety_controller k_position="20"
+                         k_velocity="20"
+                         soft_lower_limit="${ -110.0 * deg_to_rad - arm_eps}"
                          soft_upper_limit="${ 130.0 * deg_to_rad - arm_eps}" />
     </joint>

Commit message: arm v2, extensions of the same length

File: tiago_description/urdf/arm/arm.urdf.xacro (robot description, xacro)
@@ -19,6 +19,6 @@
   <xacro:property name="arm_3_max_vel"      value="4.58" />
   <xacro:property name="arm_4_max_vel"      value="4.58" />
-  <xacro:property name="arm_1_max_effort"   value="44.64" />
-  <xacro:property name="arm_2_max_effort"   value="22.32" />
+  <xacro:property name="arm_1_max_effort"   value="39.0" />
+  <xacro:property name="arm_2_max_effort"   value="39.0" />
   <xacro:property name="arm_3_max_effort"   value="17.86" />
   <xacro:property name="arm_4_max_effort"   value="17.86" />
@@ -35,15 +35,46 @@
         <inertia ixx="0.00327313329"  ixy="-0.00000460054"  ixz="-0.00025121368" iyy="0.00316047802" iyz="0.00000313158" izz="0.00157642528" />
       </inertial>
-      <visual>
-        <origin xyz="0.11 0 0.13" rpy="0 0 ${90 * deg_to_rad}" />
-        <geometry>
-          <mesh filename="package://tiago_description/meshes/arm/arm_1.dae" scale="1 1 1"/>
-        </geometry>
-        <material name="DarkGrey" />
-      </visual>
-      <collision>
-       <origin xyz="0.11 0 0.13" rpy="0 0 ${90 * deg_to_rad}" />
-        <geometry>
-          <mesh filename="package://tiago_description/meshes/arm/arm_1_collision.stl" scale="1 1 1"/>
+      <!-- M90 module -->
+      <visual>
+        <origin xyz="0 0 -0.0425" rpy="0 0 0" />
+        <geometry>
+          <cylinder length="0.085" radius="0.045" />
+        </geometry>
+        <material name="DarkGrey" />
+      </visual>
+      <collision>
+        <origin xyz="0 0 -0.0425" rpy="0 0 0" />
+        <geometry>
+          <cylinder length="0.085" radius="0.045" />
+        </geometry>
+        <material name="DarkGrey" />
+      </collision>
+      <!-- Connecting plate -->
+      <visual>
+        <origin xyz="0.05 0 0.01" rpy="0 0 0" />
+        <geometry>
+          <box size="0.2 0.09 0.02" />
+        </geometry>
+        <material name="Blue" />
+      </visual>
+      <collision>
+        <origin xyz="0 0 -0.0425" rpy="0 0 0" />
+        <geometry>
+          <cylinder length="0.02" radius="0.045" />
+        </geometry>
+        <material name="Blue" />
+      </collision>
+      <!-- Root of arm -->
+      <visual>
+        <origin xyz="0.12 0 -0.107" rpy="${-90 * deg_to_rad} 0 ${180 * deg_to_rad}" />
+        <geometry>
+          <mesh filename="package://tiago_description/meshes/arm/arm_2.dae" scale="1 1 1"/>
+        </geometry>
+        <material name="DarkGrey" />
+      </visual>
+      <collision>
+       <origin xyz="0.12 0 -0.107" rpy="${-90 * deg_to_rad} 0 ${180 * deg_to_rad}" />
+        <geometry>
+          <mesh filename="package://tiago_description/meshes/arm/arm_2_collision.stl" scale="1 1 1"/>
         </geometry>
       </collision>
@@ -52,5 +83,5 @@
       <parent link="${parent}" />
       <child link="${name}_1_link" />
-      <origin xyz="0.1 0.07 0" rpy="${0 * deg_to_rad} ${0 * deg_to_rad} ${-90 * deg_to_rad}" />
+      <origin xyz="0.157 0.064625 0" rpy="${0 * deg_to_rad} ${0 * deg_to_rad} ${-90 * deg_to_rad}" />
       <axis xyz="0 0 1" />
       <limit lower="${0.0 * deg_to_rad}" upper="${180.0 * deg_to_rad}" effort="${arm_1_max_effort}" velocity="${arm_1_max_vel}" />
@@ -84,5 +115,5 @@
       <parent link="${name}_1_link" />
       <child link="${name}_2_link" />
-      <origin xyz="0.11 0 -0.08" rpy="${90.0 * deg_to_rad} ${0 * deg_to_rad} ${0 * deg_to_rad}" />
+      <origin xyz="0.12 0.006 -0.107" rpy="${90.0 * deg_to_rad} ${0 * deg_to_rad} ${0 * deg_to_rad}" />
       <axis xyz="0 0 1" />
       <limit lower="${-120.0 * deg_to_rad}" upper="${60.0 * deg_to_rad}" effort="${arm_2_max_effort}" velocity="${arm_2_max_vel}" />
@@ -156,7 +187,7 @@
       </visual>
       <visual>
-        <origin xyz="-0.13 0.02 0" rpy="0 ${90 * deg_to_rad} 0" />
-        <geometry>
-          <cylinder length="0.05" radius="0.05" />
+        <origin xyz="-0.15 0.02 0" rpy="0 ${90 * deg_to_rad} 0" />
+        <geometry>
+          <cylinder length="0.07" radius="0.05" />
         </geometry>
         <material name="DarkGrey" />
@@ -169,7 +200,7 @@
       </collision>
       <collision>
-        <origin xyz="-0.13 0.02 0" rpy="0 ${90 * deg_to_rad} 0" />
-        <geometry>
-          <cylinder length="0.05" radius="0.05" />
+        <origin xyz="-0.15 0.02 0" rpy="0 ${90 * deg_to_rad} 0" />
+        <geometry>
+          <cylinder length="0.07" radius="0.05" />
         </geometry>
         <material name="DarkGrey" />
@@ -179,5 +210,5 @@
       <parent link="${name}_3_link" />
       <child link="${name}_4_link" />
-      <origin xyz="0 -0.02 -0.183" rpy="0 ${-90.0 * deg_to_rad} 0" />
+      <origin xyz="0 -0.02 -0.153" rpy="0 ${-90.0 * deg_to_rad} 0" />
       <axis xyz="0 0 1" />
       <limit lower="${-110 * deg_to_rad}" upper="${130.0 * deg_to_rad}" effort="${arm_4_max_effort}" velocity="${arm_4_max_vel}" />

File: tiago_description/urdf/arm/wrist.urdf.xacro (robot description, xacro)
@@ -52,5 +52,5 @@
       <parent link="${parent}" />
       <child link="${name}_5_link" />
-      <origin xyz="-0.1245 0.02 0" rpy="${-90 * deg_to_rad} ${180 * deg_to_rad} ${90 * deg_to_rad}" />
+      <origin xyz="-0.153 0.02 0" rpy="${-90 * deg_to_rad} ${180 * deg_to_rad} ${90 * deg_to_rad}" />
       <axis xyz="0 0 1" />
       <limit lower="${-120.0 * deg_to_rad}" upper="${120.0 * deg_to_rad}" effort="${wrist_1_max_effort}" velocity="${wrist_1_max_vel}" /> <!--TODO: Check effort value!-->

Commit message: Add joint limits and rotate wrist according to v3

File: tiago_description/urdf/arm/arm.urdf.xacro (robot description, xacro)
@@ -89,6 +89,6 @@
       <safety_controller k_position="20"
                          k_velocity="20"
-                         soft_lower_limit="${-45.0 * deg_to_rad  + arm_eps}"
-                         soft_upper_limit="${ 180.0 * deg_to_rad - arm_eps}" />
+                         soft_lower_limit="${0 * deg_to_rad  + arm_eps}"
+                         soft_upper_limit="${180.0 * deg_to_rad - arm_eps}" />
     </joint>
    <link name="${name}_2_link">
@@ -117,10 +117,10 @@
       <origin xyz="0.12 0.006 -0.107" rpy="${90.0 * deg_to_rad} ${0 * deg_to_rad} ${0 * deg_to_rad}" />
       <axis xyz="0 0 1" />
-      <limit lower="${-120.0 * deg_to_rad}" upper="${60.0 * deg_to_rad}" effort="${arm_2_max_effort}" velocity="${arm_2_max_vel}" />
-      <dynamics friction="${arm_friction}" damping="${arm_damping}"/>
-      <safety_controller k_position="20"
-                         k_velocity="20"
-                         soft_lower_limit="${-120.0 * deg_to_rad  + arm_eps}"
-                         soft_upper_limit="${ 60.0 * deg_to_rad - arm_eps}" />
+      <limit lower="${-112.5 * deg_to_rad}" upper="${22.5 * deg_to_rad}" effort="${arm_2_max_effort}" velocity="${arm_2_max_vel}" />
+      <dynamics friction="${arm_friction}" damping="${arm_damping}"/>
+      <safety_controller k_position="20"
+                         k_velocity="20"
+                         soft_lower_limit="${-112.5 * deg_to_rad  + arm_eps}"
+                         soft_upper_limit="${ 22.5 * deg_to_rad - arm_eps}" />
     </joint>
     <link name="${name}_3_link">
@@ -210,12 +210,12 @@
       <parent link="${name}_3_link" />
       <child link="${name}_4_link" />
-      <origin xyz="0 -0.02 -0.153" rpy="0 ${-90.0 * deg_to_rad} 0" />
-      <axis xyz="0 0 1" />
-      <limit lower="${-110 * deg_to_rad}" upper="${130.0 * deg_to_rad}" effort="${arm_4_max_effort}" velocity="${arm_4_max_vel}" />
-      <dynamics friction="${arm_friction}" damping="${arm_damping}"/>
-      <safety_controller k_position="20"
-                         k_velocity="20"
-                         soft_lower_limit="${ -110.0 * deg_to_rad - arm_eps}"
-                         soft_upper_limit="${ 130.0 * deg_to_rad - arm_eps}" />
+      <origin xyz="0 -0.02 -0.142" rpy="0 ${-90.0 * deg_to_rad} 0" />
+      <axis xyz="0 0 1" />
+      <limit lower="${-130 * deg_to_rad}" upper="${0 * deg_to_rad}" effort="${arm_4_max_effort}" velocity="${arm_4_max_vel}" />
+      <dynamics friction="${arm_friction}" damping="${arm_damping}"/>
+      <safety_controller k_position="20"
+                         k_velocity="20"
+                         soft_lower_limit="${ -130.0 * deg_to_rad - arm_eps}"
+                         soft_upper_limit="${ 0 * deg_to_rad - arm_eps}" />
     </joint>
    <gazebo reference="${name}_1_link">

File: tiago_description/urdf/arm/wrist.urdf.xacro (robot description, xacro)
@@ -52,5 +52,5 @@
       <parent link="${parent}" />
       <child link="${name}_5_link" />
-      <origin xyz="-0.153 0.02 0" rpy="${-90 * deg_to_rad} ${180 * deg_to_rad} ${90 * deg_to_rad}" />
+      <origin xyz="-0.153 0.02 0" rpy="${0 * deg_to_rad} ${-90 * deg_to_rad} ${0 * deg_to_rad}" />
       <axis xyz="0 0 1" />
       <limit lower="${-120.0 * deg_to_rad}" upper="${120.0 * deg_to_rad}" effort="${wrist_1_max_effort}" velocity="${wrist_1_max_vel}" /> <!--TODO: Check effort value!-->

Commit message: Fix arm location

File: tiago_description/urdf/arm/arm.urdf.xacro (robot description, xacro)
@@ -83,5 +83,5 @@
       <parent link="${parent}" />
       <child link="${name}_1_link" />
-      <origin xyz="0.157 0.064625 0" rpy="${0 * deg_to_rad} ${0 * deg_to_rad} ${-90 * deg_to_rad}" />
+      <origin xyz="0.157 0.064625 -0.045" rpy="${0 * deg_to_rad} ${0 * deg_to_rad} ${-90 * deg_to_rad}" />
       <axis xyz="0 0 1" />
       <limit lower="${0.0 * deg_to_rad}" upper="${180.0 * deg_to_rad}" effort="${arm_1_max_effort}" velocity="${arm_1_max_vel}" />

Commit message: Update distances

File: tiago_description/urdf/arm/arm.urdf.xacro (robot description, xacro)
@@ -131,5 +131,5 @@
       </inertial>
       <visual>
-        <origin xyz="0 0 -0.1" rpy="0 0 0" />
+        <origin xyz="0 0 -0.055" rpy="0 0 0" />
         <geometry>
           <mesh filename="package://tiago_description/meshes/arm/arm_3.dae" scale="1 1 1"/>
@@ -138,12 +138,12 @@
       </visual>
       <visual>
-        <origin xyz="0 0 -0.025" rpy="0 0 0" />
-        <geometry>
-          <cylinder length="0.11" radius="0.05" />
-        </geometry>
-        <material name="DarkGrey" />
-      </visual>
-      <collision>
-        <origin xyz="0 0 -0.1" rpy="0 0 0" />
+        <origin xyz="0 0 0" rpy="0 0 0" />
+        <geometry>
+          <cylinder length="0.07" radius="0.05" />
+        </geometry>
+        <material name="DarkGrey" />
+      </visual>
+      <collision>
+        <origin xyz="0 0 -0.055" rpy="0 0 0" />
         <geometry>
           <mesh filename="package://tiago_description/meshes/arm/arm_3_collision.stl" scale="1 1 1"/>
@@ -151,7 +151,7 @@
       </collision>
       <collision>
-        <origin xyz="0 0 -0.025" rpy="0 0 0" />
-        <geometry>
-          <cylinder length="0.11" radius="0.05" />
+        <origin xyz="0 0 0" rpy="0 0 0" />
+        <geometry>
+          <cylinder length="0.07" radius="0.05" />
         </geometry>
         <material name="DarkGrey" />
@@ -212,10 +212,10 @@
       <origin xyz="0 -0.02 -0.142" rpy="0 ${-90.0 * deg_to_rad} 0" />
       <axis xyz="0 0 1" />
-      <limit lower="${-130 * deg_to_rad}" upper="${0 * deg_to_rad}" effort="${arm_4_max_effort}" velocity="${arm_4_max_vel}" />
-      <dynamics friction="${arm_friction}" damping="${arm_damping}"/>
-      <safety_controller k_position="20"
-                         k_velocity="20"
-                         soft_lower_limit="${ -130.0 * deg_to_rad - arm_eps}"
-                         soft_upper_limit="${ 0 * deg_to_rad - arm_eps}" />
+      <limit lower="${0 * deg_to_rad}" upper="${130 * deg_to_rad}" effort="${arm_4_max_effort}" velocity="${arm_4_max_vel}" />
+      <dynamics friction="${arm_friction}" damping="${arm_damping}"/>
+      <safety_controller k_position="20"
+                         k_velocity="20"
+                         soft_lower_limit="${ 0 * deg_to_rad - arm_eps}"
+                         soft_upper_limit="${ 130 * deg_to_rad - arm_eps}" />
     </joint>
    <gazebo reference="${name}_1_link">

File: tiago_description/urdf/head/head.urdf.xacro (robot description, xacro)
@@ -80,10 +80,10 @@
       <origin xyz="0.0355 0 0.023" rpy="${-90.0 * deg_to_rad} 0 0" />
       <axis xyz="0 0 1" />
-      <limit lower="${-45.0 * deg_to_rad}" upper="${90.0 * deg_to_rad}" effort="3.26" velocity="${head_max_vel}" />
+      <limit lower="${-90 * deg_to_rad}" upper="${45.0 * deg_to_rad}" effort="3.26" velocity="${head_max_vel}" />
       <dynamics damping="${head_damping}" friction="${head_friction}"/>
       <safety_controller k_position="20"
                          k_velocity="20"
-                         soft_lower_limit="${-45.0 * deg_to_rad + head_eps}"
-                         soft_upper_limit="${ 90.0 * deg_to_rad}" />
+                         soft_lower_limit="${-90.0 * deg_to_rad + head_eps}"
+                         soft_upper_limit="${ 45.0 * deg_to_rad}" />
     </joint>
   </xacro:macro>

Commit message: Update elbow joint limits

File: tiago_description/urdf/arm/arm.urdf.xacro (robot description, xacro)
@@ -212,10 +212,10 @@
       <origin xyz="0 -0.02 -0.142" rpy="0 ${-90.0 * deg_to_rad} 0" />
       <axis xyz="0 0 1" />
-      <limit lower="${0 * deg_to_rad}" upper="${130 * deg_to_rad}" effort="${arm_4_max_effort}" velocity="${arm_4_max_vel}" />
-      <dynamics friction="${arm_friction}" damping="${arm_damping}"/>
-      <safety_controller k_position="20"
-                         k_velocity="20"
-                         soft_lower_limit="${ 0 * deg_to_rad - arm_eps}"
-                         soft_upper_limit="${ 130 * deg_to_rad - arm_eps}" />
+      <limit lower="${-90 * deg_to_rad}" upper="${135 * deg_to_rad}" effort="${arm_4_max_effort}" velocity="${arm_4_max_vel}" />
+      <dynamics friction="${arm_friction}" damping="${arm_damping}"/>
+      <safety_controller k_position="20"
+                         k_velocity="20"
+                         soft_lower_limit="${ -90 * deg_to_rad - arm_eps}"
+                         soft_upper_limit="${ 135 * deg_to_rad - arm_eps}" />
     </joint>
    <gazebo reference="${name}_1_link">
