Commit message: Update joint limit to real

File: tiago_description/urdf/arm/arm.urdf.xacro (robot description, xacro)
@@ -163,10 +163,10 @@
       <origin xyz="0.142 -0.02 0" rpy="${0.0 * deg_to_rad} ${-90.0 * deg_to_rad} 0" />
       <axis xyz="0 0 1" />
-      <limit lower="${-135.0 * deg_to_rad}" upper="${157.5 * deg_to_rad}" effort="${arm_3_max_effort}" velocity="${arm_3_max_vel}" />
-      <dynamics friction="${arm_friction}" damping="${arm_damping}"/>
-      <safety_controller k_position="20"
-                         k_velocity="20"
-                         soft_lower_limit="${-135.0 * deg_to_rad + arm_eps}"
-                         soft_upper_limit="${ 157.5 * deg_to_rad - arm_eps}" />
+      <limit lower="${-200.0 * deg_to_rad}" upper="${90 * deg_to_rad}" effort="${arm_3_max_effort}" velocity="${arm_3_max_vel}" />
+      <dynamics friction="${arm_friction}" damping="${arm_damping}"/>
+      <safety_controller k_position="20"
+                         k_velocity="20"
+                         soft_lower_limit="${-200.0 * deg_to_rad + arm_eps}"
+                         soft_upper_limit="${ 90 * deg_to_rad - arm_eps}" />
     </joint>
     <!--************************-->

Commit message: DarkGrey for all arm parts in gazebo

File: tiago_description/urdf/arm/arm.urdf.xacro (robot description, xacro)
@@ -222,16 +222,20 @@
      <mu1>0.9</mu1>
      <mu2>0.9</mu2>
+     <material>Gazebo/DarkGrey</material>
    </gazebo>
    <gazebo reference="${name}_2_link">
      <mu1>0.9</mu1>
      <mu2>0.9</mu2>
+     <material>Gazebo/DarkGrey</material>
    </gazebo>
    <gazebo reference="${name}_3_link">
      <mu1>0.9</mu1>
      <mu2>0.9</mu2>
+     <material>Gazebo/DarkGrey</material>
    </gazebo>
    <gazebo reference="${name}_4_link">
      <mu1>0.9</mu1>
      <mu2>0.9</mu2>
+     <material>Gazebo/DarkGrey</material>
    </gazebo>
    <gazebo reference="${name}_1_joint">

Commit message: New arm distances, more to come

File: tiago_description/urdf/arm/arm.urdf.xacro (robot description, xacro)
@@ -50,20 +50,6 @@
         <material name="DarkGrey" />
       </collision>
-      <!-- Connecting plate -->
-      <visual>
-        <origin xyz="0.05 0 0.01" rpy="0 0 0" />
-        <geometry>
-          <box size="0.2 0.09 0.02" />
-        </geometry>
-        <material name="Blue" />
-      </visual>
-      <collision>
-        <origin xyz="0 0 -0.0425" rpy="0 0 0" />
-        <geometry>
-          <cylinder length="0.02" radius="0.045" />
-        </geometry>
-        <material name="Blue" />
-      </collision>
       <!-- Root of arm -->
+      <!--
       <visual>
         <origin xyz="0.12 0 -0.107" rpy="${-90 * deg_to_rad} 0 ${180 * deg_to_rad}" />
@@ -79,9 +65,10 @@
         </geometry>
       </collision>
+      -->
     </link>
     <joint name="${name}_1_joint" type="revolute">
       <parent link="${parent}" />
       <child link="${name}_1_link" />
-      <origin xyz="0.157 0.064625 -0.045" rpy="${0 * deg_to_rad} ${0 * deg_to_rad} ${-90 * deg_to_rad}" />
+      <origin xyz="0.155 0.011 -0.152" rpy="${0 * deg_to_rad} ${0 * deg_to_rad} ${-90 * deg_to_rad}" />
       <axis xyz="0 0 1" />
       <limit lower="${0.0 * deg_to_rad}" upper="${180.0 * deg_to_rad}" effort="${arm_1_max_effort}" velocity="${arm_1_max_vel}" />
@@ -115,5 +102,5 @@
       <parent link="${name}_1_link" />
       <child link="${name}_2_link" />
-      <origin xyz="0.12 0.006 -0.107" rpy="${90.0 * deg_to_rad} ${0 * deg_to_rad} ${0 * deg_to_rad}" />
+      <origin xyz="0.125 0.009 -0.032" rpy="${90.0 * deg_to_rad} ${0 * deg_to_rad} ${0 * deg_to_rad}" />
       <axis xyz="0 0 1" />
       <limit lower="${-112.5 * deg_to_rad}" upper="${22.5 * deg_to_rad}" effort="${arm_2_max_effort}" velocity="${arm_2_max_vel}" />
@@ -210,5 +197,5 @@
       <parent link="${name}_3_link" />
       <child link="${name}_4_link" />
-      <origin xyz="0 -0.02 -0.142" rpy="0 ${-90.0 * deg_to_rad} 0" />
+      <origin xyz="0 -0.02 -0.168" rpy="0 ${-90.0 * deg_to_rad} 0" />
       <axis xyz="0 0 1" />
       <limit lower="${-90 * deg_to_rad}" upper="${135 * deg_to_rad}" effort="${arm_4_max_effort}" velocity="${arm_4_max_vel}" />

File: tiago_description/urdf/arm/wrist.urdf.xacro (robot description, xacro)
@@ -49,5 +49,5 @@
       <parent link="${parent}" />
       <child link="${name}_5_link" />
-      <origin xyz="-0.153 0.02 0" rpy="${0 * deg_to_rad} ${-90 * deg_to_rad} ${0 * deg_to_rad}" />
+      <origin xyz="-0.168 0.02 0" rpy="${0 * deg_to_rad} ${-90 * deg_to_rad} ${0 * deg_to_rad}" />
       <axis xyz="0 0 1" />
       <limit lower="${-120.0 * deg_to_rad}" upper="${120.0 * deg_to_rad}" effort="${wrist_1_max_effort}" velocity="${wrist_1_max_vel}" /> <!--TODO: Check effort value!-->

Commit message: Update arm

File: tiago_description/urdf/arm/arm.urdf.xacro (robot description, xacro)
@@ -37,45 +37,32 @@
       <!-- M90 module -->
       <visual>
+        <origin xyz="0 0 0" rpy="0 0 0" />
+        <geometry>
+          <mesh filename="package://tiago_description/meshes/arm/arm_1.stl" scale="1 1 1"/>
+        </geometry>
+        <material name="Orange" />
+      </visual>
+      <collision>
         <origin xyz="0 0 -0.0425" rpy="0 0 0" />
         <geometry>
           <cylinder length="0.085" radius="0.045" />
         </geometry>
-        <material name="DarkGrey" />
-      </visual>
-      <collision>
-        <origin xyz="0 0 -0.0425" rpy="0 0 0" />
-        <geometry>
-          <cylinder length="0.085" radius="0.045" />
-        </geometry>
-        <material name="DarkGrey" />
-      </collision>
-      <!-- Root of arm -->
-      <!--
-      <visual>
-        <origin xyz="0.12 0 -0.107" rpy="${-90 * deg_to_rad} 0 ${180 * deg_to_rad}" />
-        <geometry>
-          <mesh filename="package://tiago_description/meshes/arm/arm_2.dae" scale="1 1 1"/>
-        </geometry>
-        <material name="DarkGrey" />
-      </visual>
-      <collision>
-       <origin xyz="0.12 0 -0.107" rpy="${-90 * deg_to_rad} 0 ${180 * deg_to_rad}" />
-        <geometry>
-          <mesh filename="package://tiago_description/meshes/arm/arm_2_collision.stl" scale="1 1 1"/>
-        </geometry>
-      </collision>
-      -->
-    </link>
+        <material name="Orange" />
+      </collision>
+    </link>
+    <gazebo reference="${name}_1_link">
+      <material>Gazebo/Orange</material>
+    </gazebo>
     <joint name="${name}_1_joint" type="revolute">
       <parent link="${parent}" />
       <child link="${name}_1_link" />
-      <origin xyz="0.155 0.011 -0.152" rpy="${0 * deg_to_rad} ${0 * deg_to_rad} ${-90 * deg_to_rad}" />
-      <axis xyz="0 0 1" />
-      <limit lower="${0.0 * deg_to_rad}" upper="${180.0 * deg_to_rad}" effort="${arm_1_max_effort}" velocity="${arm_1_max_vel}" />
+      <origin xyz="0.155 0.011 -0.152" rpy="${0 * deg_to_rad} ${0 * deg_to_rad} ${0 * deg_to_rad}" />
+      <axis xyz="0 0 1" />
+      <limit lower="${0.0 * deg_to_rad}" upper="${165.0 * deg_to_rad}" effort="${arm_1_max_effort}" velocity="${arm_1_max_vel}" />
       <dynamics friction="${arm_friction}" damping="${arm_damping}"/>
       <safety_controller k_position="20"
                          k_velocity="20"
                          soft_lower_limit="${0 * deg_to_rad}"
-                         soft_upper_limit="${180.0 * deg_to_rad - arm_eps}" />
+                         soft_upper_limit="${165.0 * deg_to_rad - arm_eps}" />
     </joint>
    <link name="${name}_2_link">
@@ -102,12 +89,12 @@
       <parent link="${name}_1_link" />
       <child link="${name}_2_link" />
-      <origin xyz="0.125 0.009 -0.032" rpy="${90.0 * deg_to_rad} ${0 * deg_to_rad} ${0 * deg_to_rad}" />
-      <axis xyz="0 0 1" />
-      <limit lower="${-112.5 * deg_to_rad}" upper="${22.5 * deg_to_rad}" effort="${arm_2_max_effort}" velocity="${arm_2_max_vel}" />
-      <dynamics friction="${arm_friction}" damping="${arm_damping}"/>
-      <safety_controller k_position="20"
-                         k_velocity="20"
-                         soft_lower_limit="${-112.5 * deg_to_rad  + arm_eps}"
-                         soft_upper_limit="${ 22.5 * deg_to_rad - arm_eps}" />
+      <origin xyz="0.009 -0.125 -0.032" rpy="${90.0 * deg_to_rad} ${0 * deg_to_rad} ${-90 * deg_to_rad}" />
+      <axis xyz="0 0 1" />
+      <limit lower="${-93 * deg_to_rad}" upper="${86 * deg_to_rad}" effort="${arm_2_max_effort}" velocity="${arm_2_max_vel}" />
+      <dynamics friction="${arm_friction}" damping="${arm_damping}"/>
+      <safety_controller k_position="20"
+                         k_velocity="20"
+                         soft_lower_limit="${-93 * deg_to_rad  + arm_eps}"
+                         soft_upper_limit="${ 86 * deg_to_rad - arm_eps}" />
     </joint>
     <link name="${name}_3_link">

Commit message: Review of joint limits

File: tiago_description/urdf/arm/arm.urdf.xacro (robot description, xacro)
@@ -91,10 +91,10 @@
       <origin xyz="0.009 -0.125 -0.032" rpy="${90.0 * deg_to_rad} ${0 * deg_to_rad} ${-90 * deg_to_rad}" />
       <axis xyz="0 0 1" />
-      <limit lower="${-93 * deg_to_rad}" upper="${86 * deg_to_rad}" effort="${arm_2_max_effort}" velocity="${arm_2_max_vel}" />
+      <limit lower="${-93 * deg_to_rad}" upper="${75 * deg_to_rad}" effort="${arm_2_max_effort}" velocity="${arm_2_max_vel}" />
       <dynamics friction="${arm_friction}" damping="${arm_damping}"/>
       <safety_controller k_position="20"
                          k_velocity="20"
                          soft_lower_limit="${-93 * deg_to_rad  + arm_eps}"
-                         soft_upper_limit="${ 86 * deg_to_rad - arm_eps}" />
+                         soft_upper_limit="${ 75 * deg_to_rad - arm_eps}" />
     </joint>
     <link name="${name}_3_link">

Commit message: Arm 1 collision added

File: tiago_description/urdf/arm/arm.urdf.xacro (robot description, xacro)
@@ -44,9 +44,8 @@
       </visual>
       <collision>
-        <origin xyz="0 0 -0.0425" rpy="0 0 0" />
-        <geometry>
-          <cylinder length="0.085" radius="0.045" />
-        </geometry>
-        <material name="Orange" />
+        <origin xyz="0 0 0" rpy="0 0 0" />
+        <geometry>
+          <mesh filename="package://tiago_description/meshes/arm/arm_1.stl" scale="1 1 1"/>
+        </geometry>
       </collision>
     </link>

Commit message: Update inertial params

File: tiago_description/urdf/arm/arm.urdf.xacro (robot description, xacro)
@@ -24,5 +24,4 @@
   <xacro:property name="arm_4_max_effort"   value="17.86" />
   <xacro:property name="arm_eps"            value="0.02" />
-  <!-- TODO: Update dynamic models -->
   <xacro:macro name="tiago_arm" params="name parent">
     <!--************************-->
@@ -31,7 +30,9 @@
     <link name="${name}_1_link">
       <inertial>
-        <origin xyz="0.08375 0.00308 -0.04965" rpy="0 0 0"/>
-        <mass value="2.64731" />
-        <inertia ixx="0.01488823102"  ixy="0.00097928027"  ixz="-0.014599404" iyy="0.03785812845" iyz="-0.0008663619" izz="0.0261720489" />
+        <origin xyz="0.019568 -0.052265 0.008219" rpy="0 0 0"/>
+        <mass value="2.108556" />
+        <inertia ixx="0.005489" ixy="-0.001537" ixz="-0.000404"
+                 iyy="0.002232" iyz="0.000996"
+                 izz="0.006068" />
       </inertial>
       <!-- M90 module -->
@@ -56,5 +57,5 @@
       <parent link="${parent}" />
       <child link="${name}_1_link" />
-      <origin xyz="0.155 0.011 -0.152" rpy="${0 * deg_to_rad} ${0 * deg_to_rad} ${0 * deg_to_rad}" />
+      <origin xyz="0.155 0.011 -0.152" rpy="0 0 0" />
       <axis xyz="0 0 1" />
       <limit lower="${0.0 * deg_to_rad}" upper="${165.0 * deg_to_rad}" effort="${arm_1_max_effort}" velocity="${arm_1_max_vel}" />

File: tiago_description/urdf/torso/torso.urdf.xacro (robot description, xacro)
@@ -18,9 +18,9 @@
   <link name="${name}_fixed_link">
     <inertial>
-      <origin rpy="0 0 0" xyz="0.01929 -0.01317 0.0798" />
-      <mass value="7.22876" />
-      <inertia ixx="0.16941095831" ixy="-0.00114443001" ixz="0.00090167218"
-               iyy="0.15113888533" iyz="-0.00744737659"
-               izz="0.04165307088" />
+      <origin rpy="0 0 0" xyz="0.012654 -0.003497 0.257258" />
+      <mass value="21.34739" />
+      <inertia ixx="0.587525" ixy="0.00091" ixz="-0.02817"
+               iyy="0.591558" iyz="0.002331"
+               izz="0.214263" />
     </inertial>
     <visual>
@@ -85,9 +85,9 @@
   <link name="${name}_lift_link">
     <inertial>
-      <origin rpy="0 0 0" xyz="-0.04761 0.01408 -0.12387" />
-      <mass value="6.54467" />
-      <inertia ixx="0.0641960264706125" ixy="0.001128617953499" ixz="0.00203364821006436"
-               iyy="0.061658561971383" iyz="-3.14401755382909E-05"
-               izz="0.0376084656328484" />
+      <origin rpy="0 0 0" xyz="-0.044629 -0.000126 -0.16836" />
+      <mass value="6.713942" />
+      <inertia ixx="0.220103" ixy="-0.000808" ixz="-0.015835"
+               iyy="0.223461" iyz="0.008905"
+               izz="0.083575" />
     </inertial>
     <!-- Lifting body -->
