Commit message: Update urdf

File: tiago_description/urdf/arm/arm.urdf.xacro (robot description, xacro)
@@ -30,9 +30,9 @@
     <link name="${name}_1_link">
       <inertial>
-        <origin xyz="0.019568 -0.052265 0.008219" rpy="0 0 0"/>
-        <mass value="2.108556" />
-        <inertia ixx="0.005489" ixy="-0.001537" ixz="-0.000404"
-                 iyy="0.002232" iyz="0.000996"
-                 izz="0.006068" />
+        <origin xyz="0.08169 0.01822 -0.01884" rpy="0.00000 0.00000 0.00000"/>
+        <mass value="2.31325"/>
+        <inertia ixx="0.00269400000" ixy="0.00115700000" ixz="-0.00142300000"
+                 iyy="0.00704100000" iyz="-0.00031200000"
+                 izz="0.00731200000"/>
       </inertial>
       <!-- M90 module -->
@@ -42,10 +42,10 @@
           <mesh filename="package://tiago_description/meshes/arm/arm_1.stl" scale="1 1 1"/>
         </geometry>
-        <material name="Orange" />
-      </visual>
-      <collision>
-        <origin xyz="0 0 0" rpy="0 0 0" />
-        <geometry>
-          <mesh filename="package://tiago_description/meshes/arm/arm_1.stl" scale="1 1 1"/>
+        <material name="White"/>
+      </visual>
+      <collision>
+        <origin xyz="0 0 0" rpy="0 0 0" />
+        <geometry>
+          <mesh filename="package://tiago_description/meshes/arm/arm_1_collision.dae" scale="1 1 1"/>
         </geometry>
       </collision>
@@ -57,30 +57,34 @@
       <parent link="${parent}" />
       <child link="${name}_1_link" />
-      <origin xyz="0.155 0.011 -0.152" rpy="0 0 0" />
-      <axis xyz="0 0 1" />
-      <limit lower="${0.0 * deg_to_rad}" upper="${165.0 * deg_to_rad}" effort="${arm_1_max_effort}" velocity="${arm_1_max_vel}" />
-      <dynamics friction="${arm_friction}" damping="${arm_damping}"/>
-      <safety_controller k_position="20"
-                         k_velocity="20"
-                         soft_lower_limit="${0 * deg_to_rad}"
-                         soft_upper_limit="${165.0 * deg_to_rad - arm_eps}" />
+      <origin xyz="0.15505 0.014 -0.151" rpy="0 0 ${-90 * deg_to_rad}" />
+      <axis xyz="0 0 1" />
+      <limit lower="${0.0 * deg_to_rad}" upper="${157.5 * deg_to_rad}" effort="${arm_1_max_effort}" velocity="${arm_1_max_vel}" />
+      <dynamics friction="${arm_friction}" damping="${arm_damping}"/>
+      <safety_controller k_position="20"
+                         k_velocity="20"
+                         soft_lower_limit="${0.0 * deg_to_rad + arm_eps}"
+                         soft_upper_limit="${157.5 * deg_to_rad - arm_eps}" />
     </joint>
    <link name="${name}_2_link">
       <inertial>
-        <origin xyz="0.01435 -0.06294 ${0.01039}" rpy="0 0 0"/>
-        <mass value="1.58751" />
-        <inertia ixx="0.002253374"  ixy="-0.00185617271"  ixz="0.00023094382" iyy="0.01079198201" iyz="-0.00004741252" izz="0.0112248261" />
-      </inertial>
-      <visual>
-        <origin xyz="0 0 0" rpy="${180 * deg_to_rad} ${0 * deg_to_rad} ${-90 * deg_to_rad}" />
-        <geometry>
-          <mesh filename="package://tiago_description/meshes/arm/arm_2.dae" scale="1 1 1"/>
+        <origin xyz="-0.03609 -0.00006 0.01649" rpy="0.00000 0.00000 0.00000"/>
+        <mass value="1.10224"/>
+        <inertia ixx="0.00114600000" ixy="0.00000100000" ixz="0.00043500000"
+                 iyy="0.00218200000" iyz="-0.00000100000"
+                 izz="0.00237300000"/>
+      </inertial>
+      <visual>
+        <!-- <origin xyz="0 0 0" rpy="${180 * deg_to_rad} ${0 * deg_to_rad} ${-90 * deg_to_rad}" /> -->
+        <origin xyz="0 0 0" rpy="${0 * deg_to_rad} ${0 * deg_to_rad} ${0 * deg_to_rad}" />
+        <geometry>
+          <mesh filename="package://tiago_description/meshes/arm/arm_2.stl" scale="1 1 1"/>
         </geometry>
         <material name="DarkGrey" />
       </visual>
       <collision>
-        <origin xyz="0 0 0" rpy="${180 * deg_to_rad} ${0 * deg_to_rad} ${-90 * deg_to_rad}" />
-        <geometry>
-          <mesh filename="package://tiago_description/meshes/arm/arm_2_collision.stl" scale="1 1 1"/>
+        <!-- <origin xyz="0 0 0" rpy="${180 * deg_to_rad} ${0 * deg_to_rad} ${-90 * deg_to_rad}" /> -->
+        <origin xyz="0 0 0" rpy="${0 * deg_to_rad} ${0 * deg_to_rad} ${0 * deg_to_rad}" />
+        <geometry>
+          <mesh filename="package://tiago_description/meshes/arm/arm_2_collision.dae" scale="1 1 1"/>
         </geometry>
       </collision>
@@ -89,45 +93,34 @@
       <parent link="${name}_1_link" />
       <child link="${name}_2_link" />
-      <origin xyz="0.009 -0.125 -0.032" rpy="${90.0 * deg_to_rad} ${0 * deg_to_rad} ${-90 * deg_to_rad}" />
-      <axis xyz="0 0 1" />
-      <limit lower="${-93 * deg_to_rad}" upper="${75 * deg_to_rad}" effort="${arm_2_max_effort}" velocity="${arm_2_max_vel}" />
-      <dynamics friction="${arm_friction}" damping="${arm_damping}"/>
-      <safety_controller k_position="20"
-                         k_velocity="20"
-                         soft_lower_limit="${-93 * deg_to_rad  + arm_eps}"
-                         soft_upper_limit="${ 75 * deg_to_rad - arm_eps}" />
+      <origin xyz="0.125 0.0165 -0.031"
+              rpy="${90.0 * deg_to_rad} 0.0 0.0"/>
+      <axis xyz="0 0 1" />
+      <limit lower="${-87.5 * deg_to_rad}" upper="${65.0 * deg_to_rad}" effort="${arm_2_max_effort}" velocity="${arm_2_max_vel}" />
+      <dynamics friction="${arm_friction}" damping="${arm_damping}"/>
+      <safety_controller k_position="20"
+                         k_velocity="20"
+                         soft_lower_limit="${-87.5 * deg_to_rad  + arm_eps}"
+                         soft_upper_limit="${ 65.0 * deg_to_rad - arm_eps}" />
     </joint>
     <link name="${name}_3_link">
       <inertial>
-        <origin xyz="0.00557 -0.01042 -0.10388" rpy="0 0 0"/>
-        <mass value="1.79881" />
-         <inertia ixx="0.02682610467"  ixy="-0.00019692212"  ixz="-0.0015045329" iyy="0.02638053578" iyz="0.00263989274" izz="0.002385016" />
-      </inertial>
-      <visual>
-        <origin xyz="0 0 -0.055" rpy="0 0 0" />
-        <geometry>
-          <mesh filename="package://tiago_description/meshes/arm/arm_3.dae" scale="1 1 1"/>
+        <origin xyz="0.00752 0.00244 0.12957" rpy="0.00000 0.00000 0.00000"/>
+        <mass value="2.42460"/>
+        <inertia ixx="0.01441800000" ixy="0.00008400000" ixz="0.00114300000"
+                 iyy="0.01478800000" iyz="0.00064200000"
+                 izz="0.00256000000"/>
+      </inertial>
+      <visual>
+        <origin xyz="0 0 0" rpy="0 0 0" />
+        <geometry>
+          <mesh filename="package://tiago_description/meshes/arm/arm_3.stl" scale="1 1 1"/>
         </geometry>
         <material name="DarkGrey" />
       </visual>
-      <visual>
-        <origin xyz="0 0 0" rpy="0 0 0" />
-        <geometry>
-          <cylinder length="0.07" radius="0.05" />
-        </geometry>
-        <material name="DarkGrey" />
-      </visual>
-      <collision>
-        <origin xyz="0 0 -0.055" rpy="0 0 0" />
-        <geometry>
-          <mesh filename="package://tiago_description/meshes/arm/arm_3_collision.stl" scale="1 1 1"/>
-        </geometry>
-      </collision>
-      <collision>
-        <origin xyz="0 0 0" rpy="0 0 0" />
-        <geometry>
-          <cylinder length="0.07" radius="0.05" />
-        </geometry>
-        <material name="DarkGrey" />
+      <collision>
+        <origin xyz="0 0 0" rpy="0 0 0" />
+        <geometry>
+          <mesh filename="package://tiago_description/meshes/arm/arm_3_collision.dae" scale="1 1 1"/>
+        </geometry>
       </collision>
     </link>
@@ -135,12 +128,13 @@
       <parent link="${name}_2_link" />
       <child link="${name}_3_link" />
-      <origin xyz="0.142 -0.02 0" rpy="${0.0 * deg_to_rad} ${-90.0 * deg_to_rad} 0" />
-      <axis xyz="0 0 1" />
-      <limit lower="${-200.0 * deg_to_rad}" upper="${90 * deg_to_rad}" effort="${arm_3_max_effort}" velocity="${arm_3_max_vel}" />
-      <dynamics friction="${arm_friction}" damping="${arm_damping}"/>
-      <safety_controller k_position="20"
-                         k_velocity="20"
-                         soft_lower_limit="${-200.0 * deg_to_rad + arm_eps}"
-                         soft_upper_limit="${ 90 * deg_to_rad - arm_eps}" />
+      <origin xyz="0.0895 0.0 0.0015"
+              rpy="${-90.0 * deg_to_rad} ${0.0 * deg_to_rad} ${90.0 * deg_to_rad}"/>
+      <axis xyz="0 0 1" />
+      <limit lower="${-202.5 * deg_to_rad}" upper="${90.0 * deg_to_rad}" effort="${arm_3_max_effort}" velocity="${arm_3_max_vel}" />
+      <dynamics friction="${arm_friction}" damping="${arm_damping}"/>
+      <safety_controller k_position="20"
+                         k_velocity="20"
+                         soft_lower_limit="${-202.5 * deg_to_rad + arm_eps}"
+                         soft_upper_limit="${ 90.0 * deg_to_rad - arm_eps}" />
     </joint>
     <!--************************-->
@@ -149,34 +143,22 @@
     <link name="${name}_4_link">
       <inertial>
-        <origin xyz="-0.06578 0.0126 0.01194" rpy="0 0 0"/>
-        <mass value="1.35076" />
-        <inertia ixx="0.00220509703"  ixy="-0.00165490069" ixz="-0.0002277335" iyy="0.01177626386" iyz="0.00003472435" izz="0.0120918757" />
-      </inertial>
-      <visual>
-        <origin xyz="0 0 0" rpy="0 0 0" />
-        <geometry>
-          <mesh filename="package://tiago_description/meshes/arm/arm_4.dae" scale="1 1 1"/>
+        <origin xyz="0.07426 -0.01306 0.01549" rpy="0.00000 0.00000 0.00000"/>
+        <mass value="1.45429"/>
+        <inertia ixx="0.00195300000" ixy="-0.00059600000" ixz="0.00088000000"
+                 iyy="0.00709700000" iyz="-0.00017100000"
+                 izz="0.00740500000"/>
+      </inertial>
+      <visual>
+        <origin xyz="0 0 0" rpy="0 0 0" />
+        <geometry>
+          <mesh filename="package://tiago_description/meshes/arm/arm_4.stl" scale="1 1 1"/>
         </geometry>
         <material name="DarkGrey" />
       </visual>
-      <visual>
-        <origin xyz="-0.15 0.02 0" rpy="0 ${90 * deg_to_rad} 0" />
-        <geometry>
-          <cylinder length="0.07" radius="0.05" />
-        </geometry>
-        <material name="DarkGrey" />
-      </visual>
-      <collision>
-        <origin xyz="0 0 0" rpy="0 0 0" />
-        <geometry>
-          <mesh filename="package://tiago_description/meshes/arm/arm_4_collision.stl" scale="1 1 1"/>
-        </geometry>
-      </collision>
-      <collision>
-        <origin xyz="-0.15 0.02 0" rpy="0 ${90 * deg_to_rad} 0" />
-        <geometry>
-          <cylinder length="0.07" radius="0.05" />
-        </geometry>
-        <material name="DarkGrey" />
+      <collision>
+        <origin xyz="0 0 0" rpy="0 0 0" />
+        <geometry>
+          <mesh filename="package://tiago_description/meshes/arm/arm_4_collision.dae" scale="1 1 1"/>
+        </geometry>
       </collision>
     </link>
@@ -184,11 +166,12 @@
       <parent link="${name}_3_link" />
       <child link="${name}_4_link" />
-      <origin xyz="0 -0.02 -0.168" rpy="0 ${-90.0 * deg_to_rad} 0" />
-      <axis xyz="0 0 1" />
-      <limit lower="${-90 * deg_to_rad}" upper="${135 * deg_to_rad}" effort="${arm_4_max_effort}" velocity="${arm_4_max_vel}" />
-      <dynamics friction="${arm_friction}" damping="${arm_damping}"/>
-      <safety_controller k_position="20"
-                         k_velocity="20"
-                         soft_lower_limit="${ -90 * deg_to_rad - arm_eps}"
+      <origin xyz="-0.02 -0.027 -0.222"
+              rpy="${-90.0 * deg_to_rad} ${-90.0 * deg_to_rad} ${0.0 * deg_to_rad}"/>
+      <axis xyz="0 0 1" />
+      <limit lower="${-35 * deg_to_rad}" upper="${135 * deg_to_rad}" effort="${arm_4_max_effort}" velocity="${arm_4_max_vel}" />
+      <dynamics friction="${arm_friction}" damping="${arm_damping}"/>
+      <safety_controller k_position="20"
+                         k_velocity="20"
+                         soft_lower_limit="${ -35 * deg_to_rad + arm_eps}"
                          soft_upper_limit="${ 135 * deg_to_rad - arm_eps}" />
     </joint>

File: tiago_description/urdf/arm/wrist.urdf.xacro (robot description, xacro)
@@ -27,12 +27,14 @@
     <link name="${name}_5_link">
       <inertial>
-        <origin xyz="-0.00084 0.00001 ${reflect * 0.07797}" rpy="0 0 0"/>
-        <mass value="1.32698" />
-        <inertia ixx="0.01049566566"  ixy="-0.00000316264"  ixz="-0.00012548144" iyy="0.01028836655" iyz="0.0000027891" izz="0.00094419873" />
+        <origin xyz="0.00003 -0.00028 0.07831" rpy="0.00000 0.00000 0.00000"/>
+        <mass value="1.07424"/>
+        <inertia ixx="0.00168000000" ixy="0.00000100000" ixz="-0.00001500000"
+                 iyy="0.00160300000" iyz="-0.00001900000"
+                 izz="0.00040400000"/>
       </inertial>
       <visual>
         <origin xyz="0 0 0" rpy="0 0 0" />
         <geometry>
-          <mesh filename="package://tiago_description/meshes/arm/arm_5.dae" scale="1 1 ${-1*reflect}"/>
+          <mesh filename="package://tiago_description/meshes/arm/arm_5.stl" scale="1 1 1"/>
         </geometry>
         <material name="LightGrey" />
@@ -41,5 +43,5 @@
         <origin xyz="0 0 0" rpy="0 0 0" />
         <geometry>
-          <mesh filename="package://tiago_description/meshes/arm/arm_5_collision.stl" scale="1 1 ${-1*reflect}"/>
+          <mesh filename="package://tiago_description/meshes/arm/arm_5_collision.dae" scale="1 1 1"/>
         </geometry>
       </collision>
@@ -48,5 +50,5 @@
       <parent link="${parent}" />
       <child link="${name}_5_link" />
-      <origin xyz="-0.168 0.02 0" rpy="${0 * deg_to_rad} ${-90 * deg_to_rad} ${0 * deg_to_rad}" />
+      <origin xyz="-0.162 0.02 0.027" rpy="${0.0 * deg_to_rad} ${-90.0 * deg_to_rad} ${0.0 * deg_to_rad}" />
       <axis xyz="0 0 1" />
       <limit lower="${-120.0 * deg_to_rad}" upper="${120.0 * deg_to_rad}" effort="${wrist_1_max_effort}" velocity="${wrist_1_max_vel}" />
@@ -59,12 +61,14 @@
     <link name="${name}_6_link">
       <inertial>
-        <origin xyz="-0.000014 -0.00368 ${reflect * 0.00001}" rpy="0 0 0"/>
-        <mass value="0.35781" />
-         <inertia ixx="0.00016489507"  ixy="0.0000002779"  ixz="0.00000009308" iyy="0.00013154987" iyz="0.00000007106" izz="0.00011998795" />
+        <origin xyz="0.00531 0.00021 0.00002" rpy="0.00000 0.00000 0.00000"/>
+        <mass value="0.28722"/>
+        <inertia ixx="0.00005900000" ixy="-0.00000000000" ixz="-0.00000000000"
+                 iyy="0.00010600000" iyz="0.00000000000"
+                 izz="0.00012600000"/>
       </inertial>
       <visual>
         <origin xyz="0 0 0" rpy="0 0 0" />
         <geometry>
-          <mesh filename="package://tiago_description/meshes/arm/arm_6.dae" scale="1 1 ${-1*reflect}"/>
+          <mesh filename="package://tiago_description/meshes/arm/arm_6.stl" scale="1 1 1"/>
         </geometry>
         <material name="LightGrey" />
@@ -73,5 +77,5 @@
         <origin xyz="0 0 0" rpy="0 0 0" />
         <geometry>
-          <cylinder radius="0.04" length="0.0385"/>
+          <mesh filename="package://tiago_description/meshes/arm/arm_6_collision.dae" scale="1 1 1"/>
         </geometry>
       </collision>
@@ -80,5 +84,5 @@
       <parent link="${name}_5_link" />
       <child link="${name}_6_link" />
-      <origin xyz="0 0 0.15" rpy="${-90.0 * reflect * deg_to_rad} 0 0" />
+      <origin xyz="0 0 0.15" rpy="${0.0 * deg_to_rad} ${-90.0 * deg_to_rad} ${-90.0 * deg_to_rad}" />
       <axis xyz="0 0 1" />
       <limit lower="${-90.0 * deg_to_rad}" upper="${90.0 * deg_to_rad}" effort="${wrist_2_max_effort}" velocity="${wrist_2_max_vel}" />
@@ -91,26 +95,15 @@
     <link name="${name}_7_link">
       <inertial>
-        <origin xyz="0 -0.00005 ${reflect * -0.01573}" rpy="0 0 0"/>
-        <mass value="0.10721" />
-         <inertia ixx="0.00008977003"  ixy="-0.00000000001"  ixz="0.0" iyy="0.00008968773" iyz="-0.00000021816" izz="0.00000951878" />
+        <origin xyz="0.00011 -0.00034 0.02405" rpy="0.00000 0.00000 0.00000"/>
+        <mass value="0.05935"/>
+        <inertia ixx="0.00001400000" ixy="-0.00000000000" ixz="-0.00000000000"
+                 iyy="0.00001400000" iyz="0.00000000000"
+                 izz="0.00000400000"/>
       </inertial>
-      <visual>
-        <origin xyz="0 0 ${0.046 * reflect}" rpy="0 0 0" />
-        <geometry>
-          <cylinder radius="0.02" length="0.005"/>
-        </geometry>
-        <material name="DarkGrey" />
-      </visual>
-      <collision>
-        <origin xyz="0 0 ${0.046 * 0.75 * reflect}" rpy="0 0 0" />
-        <geometry>
-          <cylinder radius="0.02" length="0.023"/>
-        </geometry>
-      </collision>
     </link>
     <joint name="${name}_7_joint" type="revolute">
       <parent link="${name}_6_link" />
       <child link="${name}_7_link" />
-      <origin xyz="0 0 0" rpy="${90.0 * reflect * deg_to_rad} 0 0" />
+      <origin xyz="0 0 0" rpy="${90.0 * deg_to_rad} ${0.0 * deg_to_rad} ${90.0 * deg_to_rad}" />
       <axis xyz="0 0 1" />
       <limit lower="${-120.0 * deg_to_rad}" upper="${120.0 * deg_to_rad}" effort="${wrist_3_max_effort}" velocity="${wrist_3_max_vel}" />

File: tiago_description/urdf/head/head.urdf.xacro (robot description, xacro)
@@ -27,21 +27,21 @@
     <link name="${name}_link">
       <inertial>
-        <origin xyz="-0.016151 -0.000132 0.041903" rpy="0 0 0"/>
-        <mass value="0.406285"/>
-        <inertia ixx="0.000506" ixy="-0.000001" ixz="-0.000061"
-                 iyy="0.000552" iyz="0.000002"
-                 izz="0.000381"/>
+        <origin xyz="-0.00508 0.00237 0.07229" rpy="0.00000 0.00000 0.00000"/>
+        <mass value="0.62220"/>
+        <inertia ixx="0.00119200000" ixy="-0.00000700000" ixz="0.00009600000"
+                 iyy="0.00140200000" iyz="0.00000400000"
+                 izz="0.00088900000"/>
       </inertial>
       <visual>
         <origin xyz="0 0 0" rpy="0 0 0"/>
         <geometry>
-          <mesh filename="package://tiago_description/meshes/head_1.stl" scale="1 1 1"/>
+          <mesh filename="package://tiago_description/meshes/head/head_1.stl" scale="1 1 1"/>
         </geometry>
         <material name="White" />
       </visual>
       <collision>
-        <origin xyz="-0.025 0 0" rpy="0 0 0.07" />
+        <origin xyz="0.0 0 0" rpy="0 0 0.0" />
         <geometry>
-          <box size="0.11 0.1 0.14"/>
+          <mesh filename="package://tiago_description/meshes/head/head_1_collision.dae" scale="1 1 1"/>
         </geometry>
         <material name="White" />
@@ -51,5 +51,5 @@
       <parent link="${parent}"/>
       <child link="${name}_link"/>
-      <origin xyz="0.18735 0 0.0325" rpy="0 0 0" />
+      <origin xyz="0.182 0.0 0.0"  rpy="0 0 0" />
       <axis xyz="0 0 1" />
       <limit lower="${head_1_lower_limit * deg_to_rad}" upper="${head_1_upper_limit * deg_to_rad}" effort="5.197" velocity="${head_max_vel}" />
@@ -76,20 +76,21 @@
     <link name="${name}_link">
       <inertial>
-        <origin xyz="0.013345 0.03824 0.000058" rpy="0 0 0"/>
-        <mass value="0.852579"/>
-        <inertia ixx="0.003677" ixy="-0.000003" ixz="0.000001"
-                 iyy="0.003853" iyz="0"
-                 izz="0.002551"/>
+        <origin xyz="0.04700 0.05542 0.00022" rpy="0.00000 0.00000 0.00000"/>
+        <mass value="0.66123"/>
+        <inertia ixx="0.00462000000" ixy="0.00068900000" ixz="0.00000600000"
+                 iyy="0.00486100000" iyz="0.00000600000"
+                 izz="0.00313200000"/>
       </inertial>
       <visual>
         <origin xyz="0 0 0" rpy="0 0 0" />
         <geometry>
-          <mesh filename="package://tiago_description/meshes/head_2.dae" scale="1 1 1"/>
+          <mesh filename="package://tiago_description/meshes/head/head_2.stl" scale="1 1 1"/>
         </geometry>
+        <material name="White" />
       </visual>
       <collision>
         <origin xyz="0 0 0" rpy="0 0 0" />
         <geometry>
-          <mesh filename="package://tiago_description/meshes/head_2.stl" scale="1 1 1"/>
+          <mesh filename="package://tiago_description/meshes/head/head_2_collision.dae" scale="1 1 1"/>
         </geometry>
       </collision>
@@ -98,5 +99,5 @@
       <parent link="${parent}"/>
       <child link="${name}_link"/>
-      <origin xyz="0.0038 0 0.0596" rpy="${90.0 * deg_to_rad} 0 0" />
+      <origin xyz="0.005 0.0 0.098"  rpy="${90.0 * deg_to_rad} 0 0" />
       <axis xyz="0 0 1" />
       <limit lower="${head_2_lower_limit * deg_to_rad}" upper="${head_2_upper_limit * deg_to_rad}" effort="2.77" velocity="${head_max_vel}" />
@@ -113,5 +114,6 @@
     <xacro:head_2 name="${name}_2" parent="${name}_1_link"/>
     <xacro:xtion_pro_live name="xtion" parent="${name}_2">
-      <origin xyz="0.07 0.0633 0" rpy="${-90 * deg_to_rad} 0 0" />
+      <origin xyz="0.0908 0.08 0" rpy="${-90 * deg_to_rad} 0 0" />
+      <!-- optical origin -->
       <origin xyz="0 0 0" rpy="${-90 * deg_to_rad} ${0 * deg_to_rad} ${-90 * deg_to_rad}" />
     </xacro:xtion_pro_live>
