Commit message: Update urdf

File: tiago_description/urdf/torso/torso.urdf.xacro (robot description, xacro)
@@ -18,9 +18,9 @@
   <link name="${name}_fixed_link">
     <inertial>
-      <origin rpy="0 0 0" xyz="0.012654 -0.003497 0.257258" />
-      <mass value="21.34739" />
-      <inertia ixx="0.587525" ixy="0.00091" ixz="-0.02817"
-               iyy="0.591558" iyz="0.002331"
-               izz="0.214263" />
+      <origin xyz="0.02435 -0.00464 0.15900" rpy="0.00000 0.00000 0.00000"/>
+      <mass value="14.01360"/>
+      <inertia ixx="0.38341100000" ixy="0.00036400000" ixz="-0.02438900000"
+               iyy="0.40577300000" iyz="-0.00078200000"
+               izz="0.07699800000"/>
     </inertial>
     <visual>
@@ -45,5 +45,5 @@
   </link>
   <joint name="${name}_fixed_joint" type="fixed">
-    <origin rpy="0 0 0" xyz="-0.062 0 0.195" />
+    <origin rpy="0 0 0" xyz="-0.062 0.0 0.193" />
     <parent link="${parent}" />
     <child link="${name}_fixed_link" />
@@ -85,9 +85,9 @@
   <link name="${name}_lift_link">
     <inertial>
-      <origin rpy="0 0 0" xyz="-0.044629 -0.000126 -0.16836" />
-      <mass value="6.713942" />
-      <inertia ixx="0.220103" ixy="-0.000808" ixz="-0.015835"
-               iyy="0.223461" iyz="0.008905"
-               izz="0.083575" />
+      <origin xyz="0.04361 -0.00116 -0.17334" rpy="0.00000 0.00000 0.00000"/>
+      <mass value="6.93198"/>
+      <inertia ixx="0.24487000000" ixy="-0.00145600000" ixz="-0.00974200000"
+               iyy="0.24926900000" iyz="0.00828100000"
+               izz="0.09039500000"/>
     </inertial>
     <!-- Lifting body -->
@@ -95,5 +95,5 @@
       <origin rpy="0 0 0" xyz="0 0 0" />
        <geometry>
-        <mesh filename="package://tiago_description/meshes/torso/torso_lift.stl" scale="1 1 1"/>
+        <mesh filename="package://tiago_description/meshes/torso/torso_lift_with_arm.stl" scale="1 1 1"/>
       </geometry>
       <material name="White"/>
@@ -102,11 +102,11 @@
       <origin rpy="0 0 0" xyz="0 0 0" />
        <geometry>
-        <mesh filename="package://tiago_description/meshes/torso/torso_lift_collision.stl" scale="1 1 1"/>
+        <mesh filename="package://tiago_description/meshes/torso/torso_lift_collision.dae" scale="1 1 1"/>
       </geometry>
-      <material name="White"/>
+      <material name="LightGrey"/>
     </collision>
   </link>
   <joint name="${name}_lift_joint" type="prismatic">
-    <origin rpy="0 0 0" xyz="0.0 0 0.589" />
+    <origin rpy="0.0 0.0 0.0" xyz="0.0 0.0 0.587" />
     <parent link="${name}_fixed_link" />
     <child link="${name}_lift_link" />

Commit message: Updated joint limits as per errors found by Louis

File: tiago_description/urdf/arm/arm.urdf.xacro (robot description, xacro)
@@ -96,10 +96,10 @@
               rpy="${90.0 * deg_to_rad} 0.0 0.0"/>
       <axis xyz="0 0 1" />
-      <limit lower="${-87.5 * deg_to_rad}" upper="${65.0 * deg_to_rad}" effort="${arm_2_max_effort}" velocity="${arm_2_max_vel}" />
-      <dynamics friction="${arm_friction}" damping="${arm_damping}"/>
-      <safety_controller k_position="20"
-                         k_velocity="20"
-                         soft_lower_limit="${-87.5 * deg_to_rad  + arm_eps}"
-                         soft_upper_limit="${ 65.0 * deg_to_rad - arm_eps}" />
+      <limit lower="${-90.0 * deg_to_rad}" upper="${62.5 * deg_to_rad}" effort="${arm_2_max_effort}" velocity="${arm_2_max_vel}" />
+      <dynamics friction="${arm_friction}" damping="${arm_damping}"/>
+      <safety_controller k_position="20"
+                         k_velocity="20"
+                         soft_lower_limit="${-90.0 * deg_to_rad  + arm_eps}"
+                         soft_upper_limit="${ 62.5 * deg_to_rad - arm_eps}" />
     </joint>
     <link name="${name}_3_link">
@@ -169,9 +169,9 @@
               rpy="${-90.0 * deg_to_rad} ${-90.0 * deg_to_rad} ${0.0 * deg_to_rad}"/>
       <axis xyz="0 0 1" />
-      <limit lower="${-35 * deg_to_rad}" upper="${135 * deg_to_rad}" effort="${arm_4_max_effort}" velocity="${arm_4_max_vel}" />
-      <dynamics friction="${arm_friction}" damping="${arm_damping}"/>
-      <safety_controller k_position="20"
-                         k_velocity="20"
-                         soft_lower_limit="${ -35 * deg_to_rad + arm_eps}"
+      <limit lower="${-22.5 * deg_to_rad}" upper="${135 * deg_to_rad}" effort="${arm_4_max_effort}" velocity="${arm_4_max_vel}" />
+      <dynamics friction="${arm_friction}" damping="${arm_damping}"/>
+      <safety_controller k_position="20"
+                         k_velocity="20"
+                         soft_lower_limit="${ -22.5 * deg_to_rad + arm_eps}"
                          soft_upper_limit="${ 135 * deg_to_rad - arm_eps}" />
     </joint>

Commit message: update urdf arm model for CoM position fix

File: tiago_description/urdf/arm/arm.urdf.xacro (robot description, xacro)
@@ -30,9 +30,9 @@
     <link name="${name}_1_link">
       <inertial>
-        <origin xyz="0.08169 0.01822 -0.01884" rpy="0.00000 0.00000 0.00000"/>
-        <mass value="2.31325"/>
-        <inertia ixx="0.00269400000" ixy="0.00115700000" ixz="-0.00142300000"
-                 iyy="0.00704100000" iyz="-0.00031200000"
-                 izz="0.00731200000"/>
+        <origin xyz="0.063989 0.022546 -0.014608" rpy="0.00000 0.00000 0.00000"/>
+        <mass value="2.083078"/>
+        <inertia ixx="0.003003" ixy="0.002396" ixz="0.001531"
+                 iyy="0.008613" iyz="0.000588"
+                 izz="0.009348"/>
       </inertial>
       <!-- M90 module -->
@@ -68,9 +68,9 @@
    <link name="${name}_2_link">
       <inertial>
-        <origin xyz="-0.03609 -0.00006 0.01649" rpy="0.00000 0.00000 0.00000"/>
-        <mass value="1.10224"/>
-        <inertia ixx="0.00114600000" ixy="0.00000100000" ixz="0.00043500000"
-                 iyy="0.00218200000" iyz="-0.00000100000"
-                 izz="0.00237300000"/>
+        <origin xyz="0.035264 0.000327 0.008489" rpy="0.00000 0.00000 0.00000"/>
+        <mass value="1.792499"/>
+        <inertia ixx="0.001683" ixy="-0.000010" ixz="-0.000387"
+                 iyy="0.004708" iyz="-0.000028"
+                 izz="0.004780"/>
       </inertial>
       <visual>
@@ -105,9 +105,9 @@
     <link name="${name}_3_link">
       <inertial>
-        <origin xyz="0.00752 0.00244 0.12957" rpy="0.00000 0.00000 0.00000"/>
-        <mass value="2.42460"/>
-        <inertia ixx="0.01441800000" ixy="0.00008400000" ixz="0.00114300000"
-                 iyy="0.01478800000" iyz="0.00064200000"
-                 izz="0.00256000000"/>
+        <origin xyz="-0.007956 0.005368 -0.136320" rpy="0.00000 0.00000 0.00000"/>
+        <mass value="2.275860"/>
+        <inertia ixx="0.018178" ixy="-0.000143" ixz="0.001379"
+                 iyy="0.018552" iyz="-0.000888"
+                 izz="0.002774"/>
       </inertial>
       <visual>
@@ -143,9 +143,9 @@
     <link name="${name}_4_link">
       <inertial>
-        <origin xyz="0.07426 -0.01306 0.01549" rpy="0.00000 0.00000 0.00000"/>
-        <mass value="1.45429"/>
-        <inertia ixx="0.00195300000" ixy="-0.00059600000" ixz="0.00088000000"
-                 iyy="0.00709700000" iyz="-0.00017100000"
-                 izz="0.00740500000"/>
+        <origin xyz="-0.095658 0.014666 0.018133" rpy="0.00000 0.00000 0.00000"/>
+        <mass value="1.892788"/>
+        <inertia ixx="0.002542" ixy="-0.000956" ixz="-0.001457"
+                 iyy="0.011789" iyz="0.000229"
+                 izz="0.012058"/>
       </inertial>
       <visual>

Commit message: increase eps in arm and head joints' ranges
To prevent reaching mechanical limits after eye-hand calibration, which changes the offsets of these joints

File: tiago_description/urdf/arm/arm.urdf.xacro (robot description, xacro)
@@ -24,5 +24,5 @@
   <xacro:property name="arm_3_max_effort"   value="17.86" />
   <xacro:property name="arm_4_max_effort"   value="17.86" />
-  <xacro:property name="arm_eps"            value="0.02" />
+  <xacro:property name="arm_eps"            value="0.07" />
   <xacro:macro name="tiago_arm" params="name parent wrist_6_range">
     <!--************************-->

File: tiago_description/urdf/head/head.urdf.xacro (robot description, xacro)
@@ -17,5 +17,5 @@
   <xacro:property name="head_damping"  value="0.5" />
   <xacro:property name="head_max_vel"  value="3.0" />
-  <xacro:property name="head_eps"      value="0.02" />
+  <xacro:property name="head_eps"      value="0.07" />
   <xacro:property name="head_1_lower_limit" value="-75"/>
   <xacro:property name="head_1_upper_limit" value="75"/>

Commit message: review link 4-5-6-7

File: tiago_description/urdf/arm/arm.urdf.xacro (robot description, xacro)
@@ -33,6 +33,6 @@
         <origin xyz="0.063989 0.022546 -0.014608" rpy="0.00000 0.00000 0.00000"/>
         <mass value="2.083078"/>
-        <inertia ixx="0.003003" ixy="0.002396" ixz="0.001531"
-                 iyy="0.008613" iyz="0.000588"
+        <inertia ixx="0.003003" ixy="0.002396" ixz="-0.001531"
+                 iyy="0.008613" iyz="-0.000588"
                  izz="0.009348"/>
       </inertial>

File: tiago_description/urdf/arm/wrist.urdf.xacro (robot description, xacro)
@@ -27,9 +27,9 @@
     <link name="${name}_5_link">
       <inertial>
-        <origin xyz="0.00003 -0.00028 0.07831" rpy="0.00000 0.00000 0.00000"/>
-        <mass value="1.07424"/>
-        <inertia ixx="0.00168000000" ixy="0.00000100000" ixz="-0.00001500000"
-                 iyy="0.00160300000" iyz="-0.00001900000"
-                 izz="0.00040400000"/>
+        <origin xyz="0.000366 -0.000150 -0.062" rpy="0.00000 0.00000 0.00000"/>
+        <mass value="1.655819"/>
+        <inertia ixx="0.00613800000" ixy="-0.00000400000" ixz="0.00015600000"
+                 iyy="0.00564000000" iyz="0.00002200000"
+                 izz="0.00179700000"/>
       </inertial>
       <visual>
@@ -61,9 +61,9 @@
     <link name="${name}_6_link">
       <inertial>
-        <origin xyz="0.00531 0.00021 0.00002" rpy="0.00000 0.00000 0.00000"/>
-        <mass value="0.28722"/>
-        <inertia ixx="0.00005900000" ixy="-0.00000000000" ixz="-0.00000000000"
-                 iyy="0.00010600000" iyz="0.00000000000"
-                 izz="0.00012600000"/>
+        <origin xyz="-0.000153 -0.003122 0.000183" rpy="0.00000 0.00000 0.00000"/>
+        <mass value="0.370063"/>
+        <inertia ixx="0.00021500000" ixy="0.00000000000" ixz="0.00000000000"
+                 iyy="0.00017000000" iyz="0.00000200000"
+                 izz="0.00017400000"/>
       </inertial>
       <visual>
@@ -95,9 +95,9 @@
     <link name="${name}_7_link">
       <inertial>
-        <origin xyz="0.00011 -0.00034 0.02405" rpy="0.00000 0.00000 0.00000"/>
-        <mass value="0.05935"/>
-        <inertia ixx="0.00001400000" ixy="-0.00000000000" ixz="-0.00000000000"
-                 iyy="0.00001400000" iyz="0.00000000000"
-                 izz="0.00000400000"/>
+        <origin xyz="0.000010 -0.000003 -0.007774" rpy="0.00000 0.00000 0.00000"/>
+        <mass value="0.234252"/>
+        <inertia ixx="0.00014200000" ixy="0.00000000000" ixz="0.00000000000"
+                 iyy="0.00011300000" iyz="0.00000000000"
+                 izz="0.00005200000"/>
       </inertial>
     </link>

Commit message: Fixed torque and speed limits for arm

File: tiago_description/urdf/arm/arm.urdf.xacro (robot description, xacro)
@@ -17,11 +17,11 @@
   <xacro:property name="arm_damping"        value="1.0" />
   <xacro:property name="arm_1_max_vel"      value="2.7" />
-  <xacro:property name="arm_2_max_vel"      value="3.66" />
-  <xacro:property name="arm_3_max_vel"      value="4.58" />
-  <xacro:property name="arm_4_max_vel"      value="4.58" />
+  <xacro:property name="arm_2_max_vel"      value="2.7" />
+  <xacro:property name="arm_3_max_vel"      value="3.14" />
+  <xacro:property name="arm_4_max_vel"      value="3.14" />
   <xacro:property name="arm_1_max_effort"   value="39.0" />
   <xacro:property name="arm_2_max_effort"   value="39.0" />
-  <xacro:property name="arm_3_max_effort"   value="17.86" />
-  <xacro:property name="arm_4_max_effort"   value="17.86" />
+  <xacro:property name="arm_3_max_effort"   value="22" />
+  <xacro:property name="arm_4_max_effort"   value="22" />
   <xacro:property name="arm_eps"            value="0.07" />
   <xacro:macro name="tiago_arm" params="name parent wrist_6_range *origin">

Commit message: fix max vel and adjust max efforts

File: tiago_description/urdf/arm/arm.urdf.xacro (robot description, xacro)
@@ -16,12 +16,12 @@
   <xacro:property name="arm_friction"       value="1.0" />
   <xacro:property name="arm_damping"        value="1.0" />
-  <xacro:property name="arm_1_max_vel"      value="2.7" />
-  <xacro:property name="arm_2_max_vel"      value="2.7" />
-  <xacro:property name="arm_3_max_vel"      value="3.14" />
-  <xacro:property name="arm_4_max_vel"      value="3.14" />
-  <xacro:property name="arm_1_max_effort"   value="39.0" />
-  <xacro:property name="arm_2_max_effort"   value="39.0" />
-  <xacro:property name="arm_3_max_effort"   value="22" />
-  <xacro:property name="arm_4_max_effort"   value="22" />
+  <xacro:property name="arm_1_max_vel"      value="1.95" />
+  <xacro:property name="arm_2_max_vel"      value="1.95" />
+  <xacro:property name="arm_3_max_vel"      value="2.35" />
+  <xacro:property name="arm_4_max_vel"      value="2.35" />
+  <xacro:property name="arm_1_max_effort"   value="43.0" />
+  <xacro:property name="arm_2_max_effort"   value="43.0" />
+  <xacro:property name="arm_3_max_effort"   value="26" />
+  <xacro:property name="arm_4_max_effort"   value="26" />
   <xacro:property name="arm_eps"            value="0.07" />
   <xacro:macro name="tiago_arm" params="name parent wrist_6_range *origin">

Commit message: remove gazebo property overwrite

File: tiago_description/urdf/arm/arm.urdf.xacro (robot description, xacro)
@@ -52,7 +52,4 @@
       </collision>
     </link>
-    <gazebo reference="${name}_1_link">
-      <material>Gazebo/Orange</material>
-    </gazebo>
     <joint name="${name}_1_joint" type="revolute">
       <parent link="${parent}" />

Commit message: Almost finished dual arms

File: tiago_description/urdf/arm/arm.urdf.xacro (robot description, xacro)
@@ -33,8 +33,8 @@
       <inertial>
         <origin xyz="0.063989 0.022546 -0.014608" rpy="0.00000 0.00000 0.00000"/>
-        <mass value="2.083078"/>
-        <inertia ixx="0.003003" ixy="0.002396" ixz="0.001531"
-                 iyy="0.008613" iyz="0.000588"
-                 izz="0.009348"/>
+        <mass value="1.563428"/>
+        <inertia ixx="0.002471" ixy="${reflect * -0.001809}" ixz="-0.001202"
+                 iyy="0.006132" iyz="${reflect * 0.000494}"
+                 izz="0.006704"/>
       </inertial>
       <!-- M90 module -->
@@ -42,5 +42,5 @@
         <origin xyz="0 0 0" rpy="0 0 0" />
         <geometry>
-          <mesh filename="package://tiago_description/meshes/arm/arm_1.stl" scale="1 1 1"/>
+          <mesh filename="package://tiago_description/meshes/arm/arm_1.stl" scale="1 1 ${reflect}"/>
         </geometry>
         <material name="White"/>
@@ -49,5 +49,5 @@
         <origin xyz="0 0 0" rpy="0 0 0" />
         <geometry>
-          <mesh filename="package://tiago_description/meshes/arm/arm_1_collision.dae" scale="1 1 1"/>
+          <mesh filename="package://tiago_description/meshes/arm/arm_1_collision.dae" scale="1 1 ${reflect}"/>
         </geometry>
       </collision>
@@ -68,8 +68,8 @@
       <inertial>
         <origin xyz="0.035264 0.000327 0.008489" rpy="0.00000 0.00000 0.00000"/>
-        <mass value="1.792499"/>
-        <inertia ixx="0.001683" ixy="-0.000010" ixz="-0.000387"
-                 iyy="0.004708" iyz="-0.000028"
-                 izz="0.004780"/>
+        <mass value="1.800397"/>
+        <inertia ixx="0.001809" ixy="${reflect * 0.000015}" ixz="${reflect * 0.000254}"
+                 iyy="0.004333" iyz="${reflect * 0.000014}"
+                 izz="0.004341"/>
       </inertial>
       <visual>
@@ -92,6 +92,6 @@
       <parent link="${name}_1_link" />
       <child link="${name}_2_link" />
-      <origin xyz="0.125 0.0165 -0.031"
-              rpy="${90.0 * deg_to_rad} 0.0 0.0"/>
+      <origin xyz="0.125 0.0195 ${reflect * -0.031}"
+              rpy="${reflect * 90.0 * deg_to_rad} 0.0 0.0"/>
       <axis xyz="0 0 1" />
       <limit lower="${-90.0 * deg_to_rad}" upper="${62.5 * deg_to_rad}" effort="${arm_2_max_effort}" velocity="${arm_2_max_vel}" />
@@ -105,8 +105,8 @@
       <inertial>
         <origin xyz="-0.007956 0.005368 -0.136320" rpy="0.00000 0.00000 0.00000"/>
-        <mass value="2.275860"/>
-        <inertia ixx="0.018178" ixy="-0.000143" ixz="0.001379"
-                 iyy="0.018552" iyz="-0.000888"
-                 izz="0.002774"/>
+        <mass value="2.343502"/>
+        <inertia ixx="0.019541" ixy="${-reflect * 0.000105}" ixz="-0.001717"
+          iyy="0.019936" iyz="${reflect * 0.000852}"
+                 izz="0.002864"/>
       </inertial>
       <visual>
@@ -127,6 +127,6 @@
       <parent link="${name}_2_link" />
       <child link="${name}_3_link" />
-      <origin xyz="0.0895 0.0 ${reflect*0.0015}"
-              rpy="${-90.0 * deg_to_rad} ${0.0 * deg_to_rad} ${90.0 * deg_to_rad}"/>
+      <origin xyz="0.0895 0.0 -0.0015"
+              rpy="${reflect * -90.0 * deg_to_rad} ${0.0 * deg_to_rad} ${reflect * 90.0 * deg_to_rad}"/>
       <axis xyz="0 0 1" />
       <limit lower="${-202.5 * deg_to_rad}" upper="${90.0 * deg_to_rad}" effort="${arm_3_max_effort}" velocity="${arm_3_max_vel}" />
@@ -143,8 +143,8 @@
       <inertial>
         <origin xyz="-0.095658 0.014666 0.018133" rpy="0.00000 0.00000 0.00000"/>
-        <mass value="1.892788"/>
-        <inertia ixx="0.002542" ixy="-0.000956" ixz="-0.001457"
-                 iyy="0.011789" iyz="0.000229"
-                 izz="0.012058"/>
+        <mass value="1.432697"/>
+        <inertia ixx="0.002040" ixy="${reflect * 0.000725}" ixz="${-reflect * 0.001150}"
+                 iyy="0.008424" iyz="-0.000204"
+                 izz="0.008686"/>
       </inertial>
       <visual>

File: tiago_description/urdf/arm/wrist.urdf.xacro (robot description, xacro)
@@ -36,5 +36,5 @@
         <origin xyz="0 0 0" rpy="0 0 0" />
         <geometry>
-          <mesh filename="package://tiago_description/meshes/arm/arm_5.stl" scale="1 1 1"/>
+          <mesh filename="package://tiago_description/meshes/arm/arm_5.stl" scale="1 1 ${reflect}"/>
         </geometry>
         <material name="LightGrey" />
@@ -43,5 +43,5 @@
         <origin xyz="0 0 0" rpy="0 0 0" />
         <geometry>
-          <mesh filename="package://tiago_description/meshes/arm/arm_5_collision.dae" scale="1 1 1"/>
+          <mesh filename="package://tiago_description/meshes/arm/arm_5_collision.dae" scale="1 1 ${reflect}"/>
         </geometry>
       </collision>
@@ -50,5 +50,5 @@
       <parent link="${parent}" />
       <child link="${name}_5_link" />
-      <origin xyz="-0.162 0.02 0.027" rpy="${90.0 * deg_to_rad} ${reflect * -90.0 * deg_to_rad} ${-90.0 * deg_to_rad}" />
+      <origin xyz="-0.162 0.02 0.027" rpy="${90.0 * deg_to_rad} ${-90.0 * deg_to_rad} ${reflect * -90.0 * deg_to_rad}" />
       <axis xyz="0 0 1" />
       <limit lower="${-120.0 * deg_to_rad}" upper="${120.0 * deg_to_rad}" effort="${wrist_1_max_effort}" velocity="${wrist_1_max_vel}" />
@@ -84,5 +84,5 @@
       <parent link="${name}_5_link" />
       <child link="${name}_6_link" />
-      <origin xyz="0 0 0.15" rpy="${0.0 * deg_to_rad} ${-90.0 * deg_to_rad} ${-90.0 * deg_to_rad}" />
+      <origin xyz="0 0 ${reflect * 0.15}" rpy="${0.0 * deg_to_rad} ${reflect * -90.0 * deg_to_rad} ${-90.0 * deg_to_rad}" />
       <axis xyz="0 0 1" />
       <limit lower="${-wrist_6_range * deg_to_rad}" upper="${wrist_6_range * deg_to_rad}" effort="${wrist_2_max_effort}" velocity="${wrist_2_max_vel}" />
