Commit message: Finish dual arm urdf

File: tiago_description/urdf/arm/arm.urdf.xacro (robot description, xacro)
@@ -77,5 +77,5 @@
         <origin xyz="0 0 0" rpy="${0 * deg_to_rad} ${0 * deg_to_rad} ${0 * deg_to_rad}" />
         <geometry>
-          <mesh filename="package://tiago_description/meshes/arm/arm_2.stl" scale="1 1 1"/>
+          <mesh filename="package://tiago_description/meshes/arm/arm_2.stl" scale="1 1 ${reflect}"/>
         </geometry>
         <material name="DarkGrey" />
@@ -85,5 +85,5 @@
         <origin xyz="0 0 0" rpy="${0 * deg_to_rad} ${0 * deg_to_rad} ${0 * deg_to_rad}" />
         <geometry>
-          <mesh filename="package://tiago_description/meshes/arm/arm_2_collision.dae" scale="1 1 1"/>
+          <mesh filename="package://tiago_description/meshes/arm/arm_2_collision.dae" scale="1 1 ${reflect}"/>
         </geometry>
       </collision>
@@ -113,5 +113,5 @@
         <origin xyz="0 0 0" rpy="0 0 0" />
         <geometry>
-          <mesh filename="package://tiago_description/meshes/arm/arm_3.stl" scale="1 1 1"/>
+          <mesh filename="package://tiago_description/meshes/arm/arm_3.stl" scale="1 1 ${reflect}"/>
         </geometry>
         <material name="DarkGrey" />
@@ -120,5 +120,5 @@
         <origin xyz="0 0 0" rpy="0 0 0" />
         <geometry>
-          <mesh filename="package://tiago_description/meshes/arm/arm_3_collision.dae" scale="1 1 1"/>
+          <mesh filename="package://tiago_description/meshes/arm/arm_3_collision.dae" scale="1 1 ${reflect}"/>
         </geometry>
       </collision>
@@ -128,5 +128,5 @@
       <child link="${name}_3_link" />
       <origin xyz="0.0895 0.0 -0.0015"
-              rpy="${reflect * -90.0 * deg_to_rad} ${0.0 * deg_to_rad} ${reflect * 90.0 * deg_to_rad}"/>
+              rpy="${0.0 * deg_to_rad} ${reflect * -90.0 * deg_to_rad} ${0.0 * deg_to_rad}"/>
       <axis xyz="0 0 1" />
       <limit lower="${-202.5 * deg_to_rad}" upper="${90.0 * deg_to_rad}" effort="${arm_3_max_effort}" velocity="${arm_3_max_vel}" />
@@ -151,5 +151,5 @@
         <origin xyz="0 0 0" rpy="0 0 0" />
         <geometry>
-          <mesh filename="package://tiago_description/meshes/arm/arm_4.stl" scale="1 1 1"/>
+          <mesh filename="package://tiago_description/meshes/arm/arm_4.stl" scale="${reflect} ${reflect} ${reflect}"/>
         </geometry>
         <material name="DarkGrey" />
@@ -158,5 +158,5 @@
         <origin xyz="0 0 0" rpy="0 0 0" />
         <geometry>
-          <mesh filename="package://tiago_description/meshes/arm/arm_4_collision.dae" scale="1 1 1"/>
+          <mesh filename="package://tiago_description/meshes/arm/arm_4_collision.dae" scale="${reflect} ${reflect} ${reflect}"/>
         </geometry>
       </collision>
@@ -165,6 +165,6 @@
       <parent link="${name}_3_link" />
       <child link="${name}_4_link" />
-      <origin xyz="-0.02 -0.027 -0.222"
-              rpy="${-90.0 * deg_to_rad} ${-90.0 * deg_to_rad} ${0.0 * deg_to_rad}"/>
+      <origin xyz="-0.02 -0.027 ${reflect * -0.222}"
+              rpy="${reflect * -90.0 * deg_to_rad} ${-90.0 * deg_to_rad} ${0.0 * deg_to_rad}"/>
       <axis xyz="0 0 1" />
       <limit lower="${-22.5 * deg_to_rad}" upper="${135 * deg_to_rad}" effort="${arm_4_max_effort}" velocity="${arm_4_max_vel}" />
@@ -236,5 +236,5 @@
       <parent link="${name}_7_link" />
       <child link="${name}_tool_link" />
-      <origin xyz="0 0 0.046" rpy="${90.0 * deg_to_rad} ${-90.0 * deg_to_rad} ${180 * deg_to_rad}" />
+      <origin xyz="0 0 ${reflect*0.046}" rpy="${90.0 * deg_to_rad} ${reflect * -90.0 * deg_to_rad} ${180 * deg_to_rad}" />
     </joint>
     <!-- extensions -->

File: tiago_description/urdf/arm/wrist.urdf.xacro (robot description, xacro)
@@ -36,5 +36,5 @@
         <origin xyz="0 0 0" rpy="0 0 0" />
         <geometry>
-          <mesh filename="package://tiago_description/meshes/arm/arm_5.stl" scale="1 1 ${reflect}"/>
+          <mesh filename="package://tiago_description/meshes/arm/arm_5.stl" scale="${reflect} ${reflect} ${reflect}"/>
         </geometry>
         <material name="LightGrey" />
@@ -43,5 +43,5 @@
         <origin xyz="0 0 0" rpy="0 0 0" />
         <geometry>
-          <mesh filename="package://tiago_description/meshes/arm/arm_5_collision.dae" scale="1 1 ${reflect}"/>
+          <mesh filename="package://tiago_description/meshes/arm/arm_5_collision.dae" scale="${reflect} ${reflect} ${reflect}"/>
         </geometry>
       </collision>
@@ -50,5 +50,5 @@
       <parent link="${parent}" />
       <child link="${name}_5_link" />
-      <origin xyz="-0.162 0.02 0.027" rpy="${90.0 * deg_to_rad} ${-90.0 * deg_to_rad} ${reflect * -90.0 * deg_to_rad}" />
+      <origin xyz="${reflect * -0.162} ${reflect*0.02} ${reflect * 0.027}" rpy="${90.0 * deg_to_rad} ${-90.0 * deg_to_rad} ${-90.0 * deg_to_rad}" />
       <axis xyz="0 0 1" />
       <limit lower="${-120.0 * deg_to_rad}" upper="${120.0 * deg_to_rad}" effort="${wrist_1_max_effort}" velocity="${wrist_1_max_vel}" />
@@ -70,5 +70,5 @@
         <origin xyz="0 0 0" rpy="0 0 0" />
         <geometry>
-          <mesh filename="package://tiago_description/meshes/arm/arm_6.stl" scale="1 1 1"/>
+          <mesh filename="package://tiago_description/meshes/arm/arm_6.stl" scale="${reflect} 1 1"/>
         </geometry>
         <material name="LightGrey" />
@@ -77,5 +77,5 @@
         <origin xyz="0 0 0" rpy="0 0 0" />
         <geometry>
-          <mesh filename="package://tiago_description/meshes/arm/arm_6_collision.dae" scale="1 1 1"/>
+          <mesh filename="package://tiago_description/meshes/arm/arm_6_collision.dae" scale="${reflect} 1 1"/>
         </geometry>
       </collision>
@@ -84,5 +84,5 @@
       <parent link="${name}_5_link" />
       <child link="${name}_6_link" />
-      <origin xyz="0 0 ${reflect * 0.15}" rpy="${0.0 * deg_to_rad} ${reflect * -90.0 * deg_to_rad} ${-90.0 * deg_to_rad}" />
+      <origin xyz="0 0 ${reflect * 0.15}" rpy="${0.0 * deg_to_rad} ${-90.0 * deg_to_rad} ${-90.0 * deg_to_rad}" />
       <axis xyz="0 0 1" />
       <limit lower="${-wrist_6_range * deg_to_rad}" upper="${wrist_6_range * deg_to_rad}" effort="${wrist_2_max_effort}" velocity="${wrist_2_max_vel}" />

File: tiago_description/urdf/end_effector/end_effector.urdf.xacro (robot description, xacro)
@@ -48,5 +48,5 @@
       <parent link="${parent}"/>
       <child link="${name}_safety_box"/>
-      <origin xyz="0.1 0.02 0.02" rpy="0 0 0"/>
+      <origin xyz="0.1 0.02 ${reflect * 0.02}" rpy="0 0 0"/>
     </joint>
     <link name="${name}_safety_box">

Commit message: Corrected com positions and some inertias

File: tiago_description/urdf/arm/arm.urdf.xacro (robot description, xacro)
@@ -32,5 +32,6 @@
     <link name="${name}_1_link">
       <inertial>
-        <origin xyz="0.063989 0.022546 -0.014608" rpy="0.00000 0.00000 0.00000"/>
+        <!--<origin xyz="0.061191 ${reflect * -0.022397} -0.012835" rpy="0.00000 0.00000 0.00000"/>-->
+        <origin xyz="0.061191 -0.022397 ${reflect * -0.012835}" rpy="0.00000 0.00000 0.00000"/>
         <mass value="1.563428"/>
         <inertia ixx="0.002471" ixy="${reflect * -0.001809}" ixz="-0.001202"
@@ -67,5 +68,5 @@
    <link name="${name}_2_link">
       <inertial>
-        <origin xyz="0.035264 0.000327 0.008489" rpy="0.00000 0.00000 0.00000"/>
+        <origin xyz="0.030432 0.000229 ${reflect * -0.005942}" rpy="0.00000 0.00000 0.00000"/>
         <mass value="1.800397"/>
         <inertia ixx="0.001809" ixy="${reflect * 0.000015}" ixz="${reflect * 0.000254}"
@@ -104,7 +105,7 @@
     <link name="${name}_3_link">
       <inertial>
-        <origin xyz="-0.007956 0.005368 -0.136320" rpy="0.00000 0.00000 0.00000"/>
+        <origin xyz="0.007418 -0.004361 ${reflect * -0.134194}" rpy="0.00000 0.00000 0.00000"/>
         <mass value="2.343502"/>
-        <inertia ixx="0.019541" ixy="${-reflect * 0.000105}" ixz="-0.001717"
+        <inertia ixx="0.019541" ixy="${1 * -0.000105}" ixz="-0.001717"
           iyy="0.019936" iyz="${reflect * 0.000852}"
                  izz="0.002864"/>
@@ -142,5 +143,5 @@
     <link name="${name}_4_link">
       <inertial>
-        <origin xyz="-0.095658 0.014666 0.018133" rpy="0.00000 0.00000 0.00000"/>
+        <origin xyz="${reflect * -0.095658} ${reflect * 0.014666} 0.018133" rpy="0.00000 0.00000 0.00000"/>
         <mass value="1.432697"/>
         <inertia ixx="0.002040" ixy="${reflect * 0.000725}" ixz="${-reflect * 0.001150}"

File: tiago_description/urdf/arm/wrist.urdf.xacro (robot description, xacro)
@@ -27,5 +27,5 @@
     <link name="${name}_5_link">
       <inertial>
-        <origin xyz="0.000366 -0.000150 -0.062" rpy="0.00000 0.00000 0.00000"/>
+        <origin xyz="0.001078 -0.000151 ${reflect * -0.077173}" rpy="0.00000 0.00000 0.00000"/>
         <mass value="1.655819"/>
         <inertia ixx="0.00613800000" ixy="-0.00000400000" ixz="0.00015600000"

Commit message: Fix joint limits for tiago 2 arm

File: tiago_description/urdf/arm/arm.urdf.xacro (robot description, xacro)
@@ -60,6 +60,6 @@
       <xacro:insert_block name="origin"/>
       <axis xyz="0 0 1" />
-      <xacro:property name="arm_1_upper_limit"       value="${180.0 if tiago_dual == 1 else 157.5}"/>
-      <xacro:property name="arm_1_lower_limit"       value="${22.5 if tiago_dual == 1 else 0.0}"/>
+      <xacro:property name="arm_1_upper_limit"       value="${90.0 if tiago_dual == 1 else 157.5}"/>
+      <xacro:property name="arm_1_lower_limit"       value="${-67.5 if tiago_dual == 1 else 0.0}"/>
       <limit lower="${arm_1_lower_limit * deg_to_rad}" upper="${arm_1_upper_limit * deg_to_rad}" effort="${arm_1_max_effort}" velocity="${arm_1_max_vel}" />
       <dynamics friction="${arm_friction}" damping="${arm_damping}"/>

Commit message: Fix dual arm 2 lower limit

File: tiago_description/urdf/arm/arm.urdf.xacro (robot description, xacro)
@@ -100,9 +100,10 @@
       <axis xyz="0 0 1" />
       <xacro:property name="arm_2_upper_limit"       value="${90.0 if tiago_dual == 1 else 62.5}"/>
-      <limit lower="${-90.0 * deg_to_rad}" upper="${arm_2_upper_limit * deg_to_rad}" effort="${arm_2_max_effort}" velocity="${arm_2_max_vel}" />
-      <dynamics friction="${arm_friction}" damping="${arm_damping}"/>
-      <safety_controller k_position="20"
-                         k_velocity="20"
-                         soft_lower_limit="${-90.0 * deg_to_rad  + arm_eps}"
+      <xacro:property name="arm_2_lower_limit"       value="${-67.5 if tiago_dual == 1 else -90.0}"/>
+      <limit lower="${arm_2_lower_limit * deg_to_rad}" upper="${arm_2_upper_limit * deg_to_rad}" effort="${arm_2_max_effort}" velocity="${arm_2_max_vel}" />
+      <dynamics friction="${arm_friction}" damping="${arm_damping}"/>
+      <safety_controller k_position="20"
+                         k_velocity="20"
+                         soft_lower_limit="${arm_2_lower_limit * deg_to_rad  + arm_eps}"
                          soft_upper_limit="${ arm_2_upper_limit * deg_to_rad - arm_eps}" />
     </joint>

Commit message: Adjust end_effector-wrist distance without FT sensor

File: tiago_description/urdf/arm/arm.urdf.xacro (robot description, xacro)
@@ -250,5 +250,5 @@
     </xacro:if>
     <xacro:if value="${wrist_model == 'wrist-2017'}">
-     <xacro:property name="tool_link_z_offset"           value="${ 0.046 if has_ft_sensor else 0.06825 }"/>
+     <xacro:property name="tool_link_z_offset"           value="${ 0.046 if has_ft_sensor else 0.0573 }"/>
     </xacro:if>
     <joint name="${name}_tool_joint" type="fixed">

Commit message: Use different meshes for wrist 2017

File: tiago_description/urdf/arm/arm.urdf.xacro (robot description, xacro)
@@ -223,5 +223,5 @@
      <xacro:property name="wrist_6_range"           value="81"/>
    </xacro:if>
-   <xacro:wrist name="${name}" parent="${name}_4_link" reflect="${reflect}" wrist_6_range="${wrist_6_range}" arm_5_offset="${arm_5_offset}" arm_6_offset="${arm_6_offset}" arm_7_offset="${arm_7_offset}"/>
+   <xacro:wrist name="${name}" parent="${name}_4_link" reflect="${reflect}" wrist_model="${wrist_model}" has_ft_sensor="${has_ft_sensor}" arm_5_offset="${arm_5_offset}" arm_6_offset="${arm_6_offset}" arm_7_offset="${arm_7_offset}"/>
     <!--***********************-->
     <!--        TOOL           -->

File: tiago_description/urdf/arm/wrist.urdf.xacro (robot description, xacro)
@@ -21,5 +21,5 @@
   <xacro:property name="wrist_3_max_effort"   value="6.6" />
   <xacro:property name="wrist_eps"          value="0.02" />
-  <xacro:macro name="wrist" params="name parent reflect wrist_6_range arm_5_offset arm_6_offset arm_7_offset">
+  <xacro:macro name="wrist" params="name parent reflect wrist_model has_ft_sensor arm_5_offset arm_6_offset arm_7_offset">
     <!--************************-->
     <!--        WRIST           -->
@@ -36,5 +36,5 @@
         <origin xyz="0 0 0" rpy="0 0 0" />
         <geometry>
-          <mesh filename="package://tiago_description/meshes/arm/arm_5.stl" scale="${reflect} ${reflect} ${reflect}"/>
+          <mesh filename="package://tiago_description/meshes/arm/arm_5-${wrist_model}.stl" scale="${reflect} ${reflect} ${reflect}"/>
         </geometry>
         <material name="LightGrey" />
@@ -43,5 +43,5 @@
         <origin xyz="0 0 0" rpy="0 0 0" />
         <geometry>
-          <mesh filename="package://tiago_description/meshes/arm/arm_5_collision.dae" scale="${reflect} ${reflect} ${reflect}"/>
+          <mesh filename="package://tiago_description/meshes/arm/arm_5_collision-${wrist_model}.dae" scale="${reflect} ${reflect} ${reflect}"/>
         </geometry>
       </collision>
@@ -70,5 +70,5 @@
         <origin xyz="0 0 0" rpy="0 0 0" />
         <geometry>
-          <mesh filename="package://tiago_description/meshes/arm/arm_6.stl" scale="${reflect} 1 1"/>
+          <mesh filename="package://tiago_description/meshes/arm/arm_6-${wrist_model}.stl" scale="${reflect} 1 1"/>
         </geometry>
         <material name="LightGrey" />
@@ -77,8 +77,14 @@
         <origin xyz="0 0 0" rpy="0 0 0" />
         <geometry>
-          <mesh filename="package://tiago_description/meshes/arm/arm_6_collision.dae" scale="${reflect} 1 1"/>
+          <mesh filename="package://tiago_description/meshes/arm/arm_6_collision-${wrist_model}.dae" scale="${reflect} 1 1"/>
         </geometry>
       </collision>
     </link>
+    <xacro:if value="${wrist_model == 'wrist-2010'}">
+      <xacro:property name="wrist_6_range"           value="${ 81 if has_ft_sensor else 90 }"/>
+    </xacro:if>
+    <xacro:if value="${wrist_model == 'wrist-2017'}">
+      <xacro:property name="wrist_6_range"           value="81"/>
+    </xacro:if>
     <joint name="${name}_6_joint" type="revolute">
       <parent link="${name}_5_link" />

Commit message: Remove unused properties

File: tiago_description/urdf/arm/arm.urdf.xacro (robot description, xacro)
@@ -217,10 +217,4 @@
     <!--        WRIST           -->
     <!--************************-->
-   <xacro:if value="${wrist_model == 'wrist-2010'}">
-     <xacro:property name="wrist_6_range"           value="${ 81 if has_ft_sensor else 90 }"/>
-   </xacro:if>
-   <xacro:if value="${wrist_model == 'wrist-2017'}">
-     <xacro:property name="wrist_6_range"           value="81"/>
-   </xacro:if>
    <xacro:wrist name="${name}" parent="${name}_4_link" reflect="${reflect}" wrist_model="${wrist_model}" has_ft_sensor="${has_ft_sensor}" arm_5_offset="${arm_5_offset}" arm_6_offset="${arm_6_offset}" arm_7_offset="${arm_7_offset}"/>
     <!--***********************-->

Commit message: Fix default no_safety_eps value

File: tiago_description/urdf/arm/arm.urdf.xacro (robot description, xacro)
@@ -25,5 +25,5 @@
   <!-- reflect: Set to 1 for a right arm, or to -1 for a left arm-->
   <!-- tiago_dual: Set to 1 for tiago dual, -1 for original tiago, changes joints 1 and 2 -->
-  <xacro:macro name="tiago_arm" params="name parent wrist_model has_ft_sensor reflect tiago_dual *origin arm_1_offset arm_2_offset arm_3_offset arm_4_offset arm_5_offset arm_6_offset arm_7_offset no_safety_eps:=${no_safety_eps}">
+  <xacro:macro name="tiago_arm" params="name parent wrist_model has_ft_sensor reflect tiago_dual *origin arm_1_offset arm_2_offset arm_3_offset arm_4_offset arm_5_offset arm_6_offset arm_7_offset no_safety_eps:=False">
    <xacro:property name="arm_eps"       value="${0.00 if no_safety_eps else 0.07}"/>
     <!--************************-->

Commit message: Update arm_3_link weight for gravity compensation

File: tiago_description/urdf/arm/arm.urdf.xacro (robot description, xacro)
@@ -110,5 +110,5 @@
       <inertial>
         <origin xyz="0.007418 -0.004361 ${reflect * -0.134194}" rpy="0.00000 0.00000 0.00000"/>
-        <mass value="2.343502"/>
+        <mass value="1.8"/>
         <inertia ixx="0.019541" ixy="${1 * -0.000105}" ixz="-0.001717"
           iyy="0.019936" iyz="${reflect * 0.000852}"

Commit message: Add reflect for 4th link CoM

File: tiago_description/urdf/arm/arm.urdf.xacro (robot description, xacro)
@@ -149,5 +149,5 @@
     <link name="${name}_4_link">
       <inertial>
-        <origin xyz="${reflect * -0.095658} ${reflect * 0.014666} 0.018133" rpy="0.00000 0.00000 0.00000"/>
+        <origin xyz="${reflect * -0.095658} ${reflect * 0.014666} ${reflect * 0.018133}" rpy="0.00000 0.00000 0.00000"/>
         <mass value="1.432697"/>
         <inertia ixx="0.002040" ixy="${reflect * 0.000725}" ixz="${-reflect * 0.001150}"

Commit message: fix the inertia matrices of arm_tool_link and of force torque sensor

File: tiago_description/urdf/arm/arm.urdf.xacro (robot description, xacro)
@@ -229,5 +229,5 @@
       <inertial>
         <mass value="0.1" />
-        <inertia ixx="0.0" ixy="0.0" ixz="0.0" iyy="0.0" iyz="0.0" izz="0.0" />
+        <inertia ixx="8.33E-07" ixy="0.0" ixz="0.0" iyy="8.33E-07" iyz="0.0" izz="1.25E-06" />
       </inertial>
       <visual>

File: tiago_description/urdf/sensors/ftsensor.urdf.xacro (robot description, xacro)
@@ -20,5 +20,5 @@
       <inertial>
         <mass value="0.1" />
-        <inertia ixx="0.0" ixy="0.0" ixz="0.0" iyy="0.0" iyz="0.0" izz="0.0" />
+        <inertia ixx="1.6E-05" ixy="-2.0E-06" ixz="0.0" iyy="1.6E-05" iyz="0.0" izz="2.7E-05" />
       </inertial>
       <visual>
@@ -47,5 +47,5 @@
       <inertial>
         <mass value="0.1" />
-        <inertia ixx="0.0" ixy="0.0" ixz="0.0" iyy="0.0" iyz="0.0" izz="0.0" />
+        <inertia ixx="1.64E-05" ixy="0.0" ixz="0.0" iyy="1.64E-05" iyz="0.0" izz="3.125E-05" />
       </inertial>
       <visual>

Commit message: update arm friction and damping

File: tiago_description/urdf/arm/arm.urdf.xacro (robot description, xacro)
@@ -13,6 +13,6 @@
   <xacro:include filename="$(find tiago_description)/urdf/arm/arm.transmission.xacro" />
   <!--Constant parameters-->
-  <xacro:property name="arm_friction"       value="1.0" />
-  <xacro:property name="arm_damping"        value="1.0" />
+  <xacro:property name="arm_friction"       value="4.0" />
+  <xacro:property name="arm_damping"        value="60.0" />
   <xacro:property name="arm_1_max_vel"      value="1.95" />
   <xacro:property name="arm_2_max_vel"      value="1.95" />

Commit message: adjust arm friction and dumping

File: tiago_description/urdf/arm/arm.urdf.xacro (robot description, xacro)
@@ -18,6 +18,6 @@
   <xacro:include filename="$(find tiago_description)/urdf/arm/arm.transmission.xacro" />
   <!--Constant parameters-->
-  <xacro:property name="arm_friction"       value="4.0" />
-  <xacro:property name="arm_damping"        value="60.0" />
+  <xacro:property name="arm_friction"       value="1.0" />
+  <xacro:property name="arm_damping"        value="40.0" />
   <xacro:property name="arm_1_max_vel"      value="1.95" />
   <xacro:property name="arm_2_max_vel"      value="1.95" />

Commit message: Fix inertia values for arm_1_link to pass Gazebo Fortress validation.

File: tiago_description/urdf/arm/arm.urdf.xacro (robot description, xacro)
@@ -43,5 +43,5 @@
         <origin xyz="0.061191 -0.022397 ${reflect * -0.012835}" rpy="0.00000 0.00000 0.00000"/>
         <mass value="1.563428"/>
-        <inertia ixx="0.002471" ixy="${reflect * -0.001809}" ixz="-0.001202" iyy="0.006132" iyz="${reflect * 0.000494}" izz="0.006704"/>
+        <inertia ixx="0.002471" ixy="0.001809" ixz="0.001202" iyy="0.006132" iyz="0.000494" izz="0.006704"/>
       </inertial>
       <!-- M90 module -->

Commit message: Fix link position

File: tiago_description/urdf/arm/arm.urdf.xacro (robot description, xacro)
@@ -128,5 +128,5 @@
       <parent link="${name}_2_link" />
       <child link="${name}_3_link" />
-      <origin xyz="0.0895 0.0 -0.0015" rpy="${-90.0 * deg_to_rad} ${(90.0 - reflect * 90.0) * deg_to_rad} ${reflect * 90.0 * deg_to_rad}"/>
+      <origin xyz="0.0895 0.0 ${reflect * 0.0015}" rpy="${-90.0 * deg_to_rad} ${(90.0 - reflect * 90.0) * deg_to_rad} ${reflect * 90.0 * deg_to_rad}"/>
       <axis xyz="0 0 1" />
       <xacro:property name="arm_3_lower_limit" value="${-45. if tiago_dual == 1 else -202.5}"/>
