Commit message: Use package instead of find for meshes lookup
This change avoids errors when visualizing the robot in rviz2 from a
remote host instead of directly inside the robot

File: tiago_description/urdf/arm/arm.urdf.xacro (robot description, xacro)
@@ -49,5 +49,5 @@
         <origin xyz="0 0 0" rpy="0 0 0" />
         <geometry>
-          <mesh filename="file://$(find tiago_description)/meshes/arm/arm_1.stl" scale="1 ${-1 * tiago_dual} ${reflect}"/>
+          <mesh filename="package://tiago_description/meshes/arm/arm_1.stl" scale="1 ${-1 * tiago_dual} ${reflect}"/>
         </geometry>
         <material name="White"/>
@@ -56,5 +56,5 @@
         <origin xyz="0 0 0" rpy="0 0 0" />
         <geometry>
-          <mesh filename="file://$(find tiago_description)/meshes/arm/arm_1_collision.dae" scale="1 ${-1 * tiago_dual} ${reflect}"/>
+          <mesh filename="package://tiago_description/meshes/arm/arm_1_collision.dae" scale="1 ${-1 * tiago_dual} ${reflect}"/>
         </geometry>
       </collision>
@@ -81,5 +81,5 @@
         <origin xyz="0 0 0" rpy="${0 * deg_to_rad} ${0 * deg_to_rad} ${0 * deg_to_rad}" />
         <geometry>
-          <mesh filename="file://$(find tiago_description)/meshes/arm/arm_2.stl" scale="1 1 ${reflect}"/>
+          <mesh filename="package://tiago_description/meshes/arm/arm_2.stl" scale="1 1 ${reflect}"/>
         </geometry>
         <material name="DarkGrey" />
@@ -89,5 +89,5 @@
         <origin xyz="0 0 0" rpy="${0 * deg_to_rad} ${0 * deg_to_rad} ${0 * deg_to_rad}" />
         <geometry>
-          <mesh filename="file://$(find tiago_description)/meshes/arm/arm_2_collision.dae" scale="1 1 ${reflect}"/>
+          <mesh filename="package://tiago_description/meshes/arm/arm_2_collision.dae" scale="1 1 ${reflect}"/>
         </geometry>
       </collision>
@@ -113,5 +113,5 @@
         <origin xyz="0 0 0" rpy="0 0 0" />
         <geometry>
-          <mesh filename="file://$(find tiago_description)/meshes/arm/arm_3.stl" scale="1 1 ${reflect}"/>
+          <mesh filename="package://tiago_description/meshes/arm/arm_3.stl" scale="1 1 ${reflect}"/>
         </geometry>
         <material name="DarkGrey" />
@@ -120,5 +120,5 @@
         <origin xyz="0 0 0" rpy="0 0 0" />
         <geometry>
-          <mesh filename="file://$(find tiago_description)/meshes/arm/arm_3_collision.dae" scale="1 1 ${reflect}"/>
+          <mesh filename="package://tiago_description/meshes/arm/arm_3_collision.dae" scale="1 1 ${reflect}"/>
         </geometry>
       </collision>
@@ -145,5 +145,5 @@
         <origin xyz="0 0 0" rpy="0 0 0" />
         <geometry>
-          <mesh filename="file://$(find tiago_description)/meshes/arm/arm_4.stl" scale="${reflect} ${reflect} ${reflect}"/>
+          <mesh filename="package://tiago_description/meshes/arm/arm_4.stl" scale="${reflect} ${reflect} ${reflect}"/>
         </geometry>
         <material name="DarkGrey" />
@@ -152,5 +152,5 @@
         <origin xyz="0 0 0" rpy="0 0 0" />
         <geometry>
-          <mesh filename="file://$(find tiago_description)/meshes/arm/arm_4_collision.dae" scale="${reflect} ${reflect} ${reflect}"/>
+          <mesh filename="package://tiago_description/meshes/arm/arm_4_collision.dae" scale="${reflect} ${reflect} ${reflect}"/>
         </geometry>
       </collision>

File: tiago_description/urdf/arm/wrist.urdf.xacro (robot description, xacro)
@@ -50,5 +50,5 @@
         <origin xyz="0 0 0" rpy="0 0 0" />
         <geometry>
-          <mesh filename="file://$(find tiago_description)/meshes/arm/arm_5-${wrist_model}.stl" scale="${reflect} ${reflect} ${reflect}"/>
+          <mesh filename="package://tiago_description/meshes/arm/arm_5-${wrist_model}.stl" scale="${reflect} ${reflect} ${reflect}"/>
         </geometry>
         <material name="LightGrey" />
@@ -57,5 +57,5 @@
         <origin xyz="0 0 0" rpy="0 0 0" />
         <geometry>
-          <mesh filename="file://$(find tiago_description)/meshes/arm/arm_5_collision-${wrist_model}.dae" scale="${reflect} ${reflect} ${reflect}"/>
+          <mesh filename="package://tiago_description/meshes/arm/arm_5_collision-${wrist_model}.dae" scale="${reflect} ${reflect} ${reflect}"/>
         </geometry>
       </collision>
@@ -85,5 +85,5 @@
         <origin xyz="0 0 0" rpy="0 0 0" />
         <geometry>
-          <mesh filename="file://$(find tiago_description)/meshes/arm/arm_6-${wrist_model}.stl" scale="${reflect} 1 1"/>
+          <mesh filename="package://tiago_description/meshes/arm/arm_6-${wrist_model}.stl" scale="${reflect} 1 1"/>
         </geometry>
         <material name="LightGrey" />
@@ -92,5 +92,5 @@
         <origin xyz="0 0 0" rpy="0 0 0" />
         <geometry>
-          <mesh filename="file://$(find tiago_description)/meshes/arm/arm_6_collision-${wrist_model}.dae" scale="${reflect} 1 1"/>
+          <mesh filename="package://tiago_description/meshes/arm/arm_6_collision-${wrist_model}.dae" scale="${reflect} 1 1"/>
         </geometry>
       </collision>

File: tiago_description/urdf/head/head.urdf.xacro (robot description, xacro)
@@ -40,5 +40,5 @@
         <origin xyz="0 0 0" rpy="0 0 0"/>
         <geometry>
-          <mesh filename="file://$(find tiago_description)/meshes/head/head_1.stl" scale="1 1 1"/>
+          <mesh filename="package://tiago_description/meshes/head/head_1.stl" scale="1 1 1"/>
         </geometry>
         <material name="White" />
@@ -47,5 +47,5 @@
         <origin xyz="0.0 0 0" rpy="0 0 0.0" />
         <geometry>
-          <mesh filename="file://$(find tiago_description)/meshes/head/head_1_collision.dae" scale="1 1 1"/>
+          <mesh filename="package://tiago_description/meshes/head/head_1_collision.dae" scale="1 1 1"/>
         </geometry>
         <material name="White" />
@@ -80,5 +80,5 @@
         <origin xyz="0 0 0" rpy="0 0 0" />
         <geometry>
-          <mesh filename="file://$(find tiago_description)/meshes/head/head_2.stl" scale="1 1 1"/>
+          <mesh filename="package://tiago_description/meshes/head/head_2.stl" scale="1 1 1"/>
         </geometry>
         <material name="White" />
@@ -87,5 +87,5 @@
         <origin xyz="0 0 0" rpy="0 0 0" />
         <geometry>
-          <mesh filename="file://$(find tiago_description)/meshes/head/head_2_collision.dae" scale="1 1 1"/>
+          <mesh filename="package://tiago_description/meshes/head/head_2_collision.dae" scale="1 1 1"/>
         </geometry>
       </collision>

File: tiago_description/urdf/torso/torso.urdf.xacro (robot description, xacro)
@@ -30,5 +30,5 @@
         <origin rpy="0 0 0" xyz="0 0 0" />
         <geometry>
-          <mesh filename="file://$(find tiago_description)/meshes/torso/torso_fix.stl" scale="1 1 1"/>
+          <mesh filename="package://tiago_description/meshes/torso/torso_fix.stl" scale="1 1 1"/>
         </geometry>
         <material name="LightGrey"/>
@@ -94,5 +94,5 @@
         <origin rpy="0 0 0" xyz="0 0 0" />
         <geometry>
-          <mesh filename="file://$(find tiago_description)/meshes/torso/torso_lift_with_arm.stl" scale="1 1 1"/>
+          <mesh filename="package://tiago_description/meshes/torso/torso_lift_with_arm.stl" scale="1 1 1"/>
         </geometry>
         <material name="White"/>
@@ -101,5 +101,5 @@
         <origin rpy="0 0 0" xyz="0 0 0" />
         <geometry>
-          <mesh filename="file://$(find tiago_description)/meshes/torso/torso_lift_collision_core.dae" scale="1 1 1"/>
+          <mesh filename="package://tiago_description/meshes/torso/torso_lift_collision_core.dae" scale="1 1 1"/>
         </geometry>
         <material name="LightGrey"/>
@@ -108,5 +108,5 @@
         <origin rpy="0 0 0" xyz="0 0 0" />
         <geometry>
-          <mesh filename="file://$(find tiago_description)/meshes/torso/torso_lift_collision_shoulder.dae" scale="1 1 1"/>
+          <mesh filename="package://tiago_description/meshes/torso/torso_lift_collision_shoulder.dae" scale="1 1 1"/>
         </geometry>
         <material name="LightGrey"/>
@@ -115,5 +115,5 @@
         <origin rpy="0 0 0" xyz="0 0 0" />
         <geometry>
-          <mesh filename="file://$(find tiago_description)/meshes/torso/torso_lift_collision_neck.dae" scale="1 1 1"/>
+          <mesh filename="package://tiago_description/meshes/torso/torso_lift_collision_neck.dae" scale="1 1 1"/>
         </geometry>
         <material name="LightGrey"/>
@@ -123,5 +123,5 @@
         <origin rpy="0 0 -1.57" xyz="-0.01 0.125 -0.27" />
         <geometry>
-          <mesh filename="file://$(find tiago_description)/meshes/torso/tiago_screen.stl" scale="1 1 1"/>
+          <mesh filename="package://tiago_description/meshes/torso/tiago_screen.stl" scale="1 1 1"/>
         </geometry>
         <material name="White"/>
@@ -130,5 +130,5 @@
         <origin rpy="0 0 -1.57" xyz="-0.01 0.125 -0.27" />
         <geometry>
-          <mesh filename="file://$(find tiago_description)/meshes/torso/tiago_screen_collision.stl" scale="1 1 1"/>
+          <mesh filename="package://tiago_description/meshes/torso/tiago_screen_collision.stl" scale="1 1 1"/>
         </geometry>
         <material name="LightGrey"/>

Commit message: Add support for new gazebo

File: tiago_description/urdf/arm/arm.urdf.xacro (robot description, xacro)
@@ -49,5 +49,6 @@
         <origin xyz="0 0 0" rpy="0 0 0" />
         <geometry>
-          <mesh filename="package://tiago_description/meshes/arm/arm_1.stl" scale="1 ${-1 * tiago_dual} ${reflect}"/>
+          <!-- TODO Remove reflected meshes https://github.com/gazebosim/ros_gz/issues/587 -->
+          <mesh filename="package://tiago_description/meshes/arm/arm_1${'_dual' if tiago_dual == 1 else ''}${'_reflected' if reflect == -1 else ''}.stl" scale="1 1 1"/>
         </geometry>
         <material name="White"/>
@@ -56,5 +57,5 @@
         <origin xyz="0 0 0" rpy="0 0 0" />
         <geometry>
-          <mesh filename="package://tiago_description/meshes/arm/arm_1_collision.dae" scale="1 ${-1 * tiago_dual} ${reflect}"/>
+          <mesh filename="package://tiago_description/meshes/arm/arm_1_collision${'_dual' if tiago_dual == 1 else ''}${'_reflected' if reflect == -1 else ''}.stl" scale="1 1 1"/>
         </geometry>
       </collision>
@@ -81,5 +82,5 @@
         <origin xyz="0 0 0" rpy="${0 * deg_to_rad} ${0 * deg_to_rad} ${0 * deg_to_rad}" />
         <geometry>
-          <mesh filename="package://tiago_description/meshes/arm/arm_2.stl" scale="1 1 ${reflect}"/>
+          <mesh filename="package://tiago_description/meshes/arm/arm_2${'_reflected' if reflect == -1 else ''}.stl" scale="1 1 1"/>
         </geometry>
         <material name="DarkGrey" />
@@ -89,5 +90,5 @@
         <origin xyz="0 0 0" rpy="${0 * deg_to_rad} ${0 * deg_to_rad} ${0 * deg_to_rad}" />
         <geometry>
-          <mesh filename="package://tiago_description/meshes/arm/arm_2_collision.dae" scale="1 1 ${reflect}"/>
+          <mesh filename="package://tiago_description/meshes/arm/arm_2_collision${'_reflected' if reflect == -1 else ''}.stl" scale="1 1 1"/>
         </geometry>
       </collision>
@@ -113,5 +114,5 @@
         <origin xyz="0 0 0" rpy="0 0 0" />
         <geometry>
-          <mesh filename="package://tiago_description/meshes/arm/arm_3.stl" scale="1 1 ${reflect}"/>
+          <mesh filename="package://tiago_description/meshes/arm/arm_3${'_reflected' if reflect == -1 else ''}.stl" scale="1 1 1"/>
         </geometry>
         <material name="DarkGrey" />
@@ -120,5 +121,5 @@
         <origin xyz="0 0 0" rpy="0 0 0" />
         <geometry>
-          <mesh filename="package://tiago_description/meshes/arm/arm_3_collision.dae" scale="1 1 ${reflect}"/>
+          <mesh filename="package://tiago_description/meshes/arm/arm_3_collision${'_reflected' if reflect == -1 else ''}.stl" scale="1 1 1"/>
         </geometry>
       </collision>
@@ -145,5 +146,5 @@
         <origin xyz="0 0 0" rpy="0 0 0" />
         <geometry>
-          <mesh filename="package://tiago_description/meshes/arm/arm_4.stl" scale="${reflect} ${reflect} ${reflect}"/>
+          <mesh filename="package://tiago_description/meshes/arm/arm_4${'_reflected' if reflect == -1 else ''}.stl" scale="1 1 1"/>
         </geometry>
         <material name="DarkGrey" />
@@ -152,5 +153,5 @@
         <origin xyz="0 0 0" rpy="0 0 0" />
         <geometry>
-          <mesh filename="package://tiago_description/meshes/arm/arm_4_collision.dae" scale="${reflect} ${reflect} ${reflect}"/>
+          <mesh filename="package://tiago_description/meshes/arm/arm_4_collision${'_reflected' if reflect == -1 else ''}.stl" scale="1 1 1"/>
         </geometry>
       </collision>

File: tiago_description/urdf/arm/wrist.urdf.xacro (robot description, xacro)
@@ -50,5 +50,5 @@
         <origin xyz="0 0 0" rpy="0 0 0" />
         <geometry>
-          <mesh filename="package://tiago_description/meshes/arm/arm_5-${wrist_model}.stl" scale="${reflect} ${reflect} ${reflect}"/>
+          <mesh filename="package://tiago_description/meshes/arm/arm_5-${wrist_model}${'_reflected' if reflect == -1 else ''}.stl" scale="1 1 1"/>
         </geometry>
         <material name="LightGrey" />
@@ -57,5 +57,5 @@
         <origin xyz="0 0 0" rpy="0 0 0" />
         <geometry>
-          <mesh filename="package://tiago_description/meshes/arm/arm_5_collision-${wrist_model}.dae" scale="${reflect} ${reflect} ${reflect}"/>
+          <mesh filename="package://tiago_description/meshes/arm/arm_5_collision-${wrist_model}${'_reflected' if reflect == -1 else ''}.stl" scale="1 1 1"/>
         </geometry>
       </collision>
@@ -85,5 +85,5 @@
         <origin xyz="0 0 0" rpy="0 0 0" />
         <geometry>
-          <mesh filename="package://tiago_description/meshes/arm/arm_6-${wrist_model}.stl" scale="${reflect} 1 1"/>
+          <mesh filename="package://tiago_description/meshes/arm/arm_6-${wrist_model}${'_reflected' if reflect == -1 else ''}.stl" scale="1 1 1"/>
         </geometry>
         <material name="LightGrey" />
@@ -92,5 +92,5 @@
         <origin xyz="0 0 0" rpy="0 0 0" />
         <geometry>
-          <mesh filename="package://tiago_description/meshes/arm/arm_6_collision-${wrist_model}.dae" scale="${reflect} 1 1"/>
+          <mesh filename="package://tiago_description/meshes/arm/arm_6_collision-${wrist_model}${'_reflected' if reflect == -1 else ''}.stl" scale="1 1 1"/>
         </geometry>
       </collision>
