Commit message: fix: xacro negation

File: tiago_description/urdf/end_effector/end_effector.urdf.xacro (robot description, xacro)
@@ -18,5 +18,5 @@
     - reflect: Set to 1 for a right end effector, or to -1 for a left end effector
   -->
-  <xacro:macro name="tiago_end_effector" params="name parent type reflect">
+  <xacro:macro name="tiago_end_effector" params="name parent type reflect is_dual:='false'">
   <!-- PAL Gripper -->
   <xacro:if value="${type == 'pal-gripper'}">
@@ -74,6 +74,18 @@
   </xacro:if>
   <!-- Custom -->
-  <xacro:if value="${type == 'custom'}">
+  <xacro:if value="${type == 'custom' and not is_dual}">
     <xacro:include filename="$(find custom_ee_description)/urdf/end-effector.urdf.xacro" />
+    <xacro:end_effector parent="${parent}">
+      <origin xyz="0.01 0 0" rpy="${90*deg_to_rad} ${90*deg_to_rad} ${-90*deg_to_rad}"/>
+    </xacro:end_effector>
+  </xacro:if>
+  <!-- Custom dual-->
+  <xacro:if value="${type == 'custom' and is_dual}">
+    <xacro:if value="${reflect}"> <!-- If right -->
+    <xacro:include filename="$(find custom_dual_ee_description)/urdf/end-effector-right.urdf.xacro" />
+    </xacro:if>
+    <xacro:if value="${reflect == -1}"> <!-- If left -->
+    <xacro:include filename="$(find custom_dual_ee_description)/urdf/end-effector-left.urdf.xacro" />
+    </xacro:if>
     <xacro:end_effector parent="${parent}">
       <origin xyz="0.01 0 0" rpy="${90*deg_to_rad} ${90*deg_to_rad} ${-90*deg_to_rad}"/>

Commit message: fix: duplicating right ee causing error link

File: tiago_description/urdf/end_effector/end_effector.urdf.xacro (robot description, xacro)
@@ -82,13 +82,16 @@
   <!-- Custom dual-->
   <xacro:if value="${type == 'custom' and is_dual}">
-    <xacro:if value="${reflect}"> <!-- If right -->
+    <xacro:if value="${reflect == 1}"> <!-- If right -->
     <xacro:include filename="$(find custom_dual_ee_description)/urdf/end-effector-right.urdf.xacro" />
+    <xacro:end_effector_right parent="${parent}">
+      <origin xyz="0.01 0 0" rpy="${90*deg_to_rad} ${90*deg_to_rad} ${-90*deg_to_rad}"/>
+    </xacro:end_effector_right>
     </xacro:if>
     <xacro:if value="${reflect == -1}"> <!-- If left -->
     <xacro:include filename="$(find custom_dual_ee_description)/urdf/end-effector-left.urdf.xacro" />
+    <xacro:end_effector_left parent="${parent}">
+      <origin xyz="0.01 0 0" rpy="${90*deg_to_rad} ${90*deg_to_rad} ${-90*deg_to_rad}"/>
+    </xacro:end_effector_left>
     </xacro:if>
-    <xacro:end_effector parent="${parent}">
-      <origin xyz="0.01 0 0" rpy="${90*deg_to_rad} ${90*deg_to_rad} ${-90*deg_to_rad}"/>
-    </xacro:end_effector>
   </xacro:if>
   </xacro:macro>

Commit message: fix: load custom urdfs

File: tiago_description/urdf/end_effector/end_effector.urdf.xacro (robot description, xacro)
@@ -18,5 +18,5 @@
     - reflect: Set to 1 for a right end effector, or to -1 for a left end effector
   -->
-  <xacro:macro name="tiago_end_effector" params="name parent type reflect is_dual:='false'">
+  <xacro:macro name="tiago_end_effector" params="name parent type reflect is_dual:=false">
   <!-- PAL Gripper -->
   <xacro:if value="${type == 'pal-gripper'}">
@@ -74,5 +74,5 @@
   </xacro:if>
   <!-- Custom -->
-  <xacro:if value="${type == 'custom' and is_dual == 'false'}">
+  <xacro:if value="${type == 'custom' and is not is_dual}">
     <xacro:include filename="$(find custom_ee_description)/urdf/end-effector.urdf.xacro" />
     <xacro:end_effector parent="${parent}">
@@ -81,5 +81,5 @@
   </xacro:if>
   <!-- Custom dual-->
-  <xacro:if value="${type == 'custom' and is_dual == 'true'}">
+  <xacro:if value="${type == 'custom' and is_dual}">
     <xacro:if value="${reflect == 1}"> <!-- If right -->
     <xacro:include filename="$(find custom_dual_ee_description)/urdf/end-effector-right.urdf.xacro" />

Commit message: Match the code with the other robotiq gripper

File: tiago_description/urdf/end_effector/end_effector.urdf.xacro (robot description, xacro)
@@ -95,5 +95,6 @@
   <xacro:if value="${type == 'robotiq-epick'}">
     <xacro:include filename="$(find pal_robotiq_epick_description)/urdf/robotiq_epick_model_macro.xacro" />
-    <xacro:epick_hand  hand_link_name="epick" robot_name="robotiq" prefix="${name}_" parent="${parent}">
+    <xacro:epick_hand  prefix="${name}_" parent="${parent}">
+      <origin xyz="0.01 0 0" rpy="${90*deg_to_rad} ${0*deg_to_rad} ${90*deg_to_rad}"/>
     </xacro:epick_hand>
   </xacro:if>

Commit message: fix faulty if statement in urdf

File: tiago_description/urdf/end_effector/end_effector.urdf.xacro (robot description, xacro)
@@ -24,27 +24,29 @@
   -->
   <xacro:macro name="tiago_end_effector" params="name parent type has_end_effector reflect is_dual:=false">
-  <!-- No end-effector -->
   <!-- For now the custom end-effector is used in the case of no end-effector -->
-  <xacro:unless value="${has_end_effector}">
-    <xacro:include filename="$(find custom_ee_description)/urdf/end-effector.urdf.xacro" />
-    <xacro:end_effector parent="${parent}">
-      <origin xyz="0.01 0 0" rpy="${90*deg_to_rad} ${90*deg_to_rad} ${-90*deg_to_rad}"/>
-    </xacro:end_effector>
-  </xacro:unless>
-    <!-- No end-effector dual-->
-  <xacro:unless value="${has_end_effector and is_dual}">
-    <xacro:if value="${reflect == 1}"> <!-- If right -->
-    <xacro:include filename="$(find custom_dual_ee_description)/urdf/end-effector-right.urdf.xacro" />
-    <xacro:end_effector_right parent="${parent}">
-      <origin xyz="0.01 0 0" rpy="${90*deg_to_rad} ${90*deg_to_rad} ${-90*deg_to_rad}"/>
-    </xacro:end_effector_right>
+  <xacro:if value="${not has_end_effector}">
+    <!-- No end-effector single-->
+    <xacro:if values="${not is_dual}">
+      <xacro:include filename="$(find custom_ee_description)/urdf/end-effector.urdf.xacro" />
+      <xacro:end_effector parent="${parent}">
+        <origin xyz="0.01 0 0" rpy="${90*deg_to_rad} ${90*deg_to_rad} ${-90*deg_to_rad}"/>
+      </xacro:end_effector>
     </xacro:if>
-    <xacro:if value="${reflect == -1}"> <!-- If left -->
-    <xacro:include filename="$(find custom_dual_ee_description)/urdf/end-effector-left.urdf.xacro" />
-    <xacro:end_effector_left parent="${parent}">
-      <origin xyz="0.01 0 0" rpy="${90*deg_to_rad} ${90*deg_to_rad} ${-90*deg_to_rad}"/>
-    </xacro:end_effector_left>
+  <!-- No end-effector dual -->
+    <xacro:if value="${is_dual}">
+      <xacro:if value="${reflect == 1}"> <!-- If right -->
+        <xacro:include filename="$(find custom_dual_ee_description)/urdf/end-effector-right.urdf.xacro" />
+        <xacro:end_effector_right parent="${parent}">
+          <origin xyz="0.01 0 0" rpy="${90*deg_to_rad} ${90*deg_to_rad} ${-90*deg_to_rad}"/>
+        </xacro:end_effector_right>
+      </xacro:if>
+      <xacro:if value="${reflect == -1}"> <!-- If left -->
+        <xacro:include filename="$(find custom_dual_ee_description)/urdf/end-effector-left.urdf.xacro" />
+        <xacro:end_effector_left parent="${parent}">
+          <origin xyz="0.01 0 0" rpy="${90*deg_to_rad} ${90*deg_to_rad} ${-90*deg_to_rad}"/>
+        </xacro:end_effector_left>
+      </xacro:if>
     </xacro:if>
-  </xacro:unless>
+  </xacro:if>
   <!-- PAL Gripper -->
   <xacro:if value="${type == 'pal-gripper'}">

Commit message: fix faulty if statement in urdf

File: tiago_description/urdf/end_effector/end_effector.urdf.xacro (robot description, xacro)
@@ -96,11 +96,4 @@
     </xacro:robotiq_140_gripper>
   </xacro:if>
-  <!-- Robotiq Epick Gripper -->
-  <xacro:if value="${type == 'robotiq-epick'}">
-    <xacro:include filename="$(find pal_robotiq_epick_description)/urdf/robotiq_epick_model_macro.xacro" />
-    <xacro:epick_hand  prefix="${name}_" parent="${parent}">
-      <origin xyz="0.01 0 0" rpy="${90*deg_to_rad} ${0*deg_to_rad} ${90*deg_to_rad}"/>
-    </xacro:epick_hand>
-  </xacro:if>
   <!-- Custom -->
   <xacro:if value="${type == 'custom' and not is_dual}">

Commit message: add no-ee to urdf

File: tiago_description/urdf/end_effector/end_effector.urdf.xacro (robot description, xacro)
@@ -24,28 +24,7 @@
   -->
   <xacro:macro name="tiago_end_effector" params="name parent type has_end_effector reflect is_dual:=false">
-  <!-- For now the custom end-effector is used in the case of no end-effector -->
+  <!-- No end-effector -->
   <xacro:if value="${not has_end_effector}">
-    <!-- No end-effector single-->
-    <xacro:if values="${not is_dual}">
-      <xacro:include filename="$(find custom_ee_description)/urdf/end-effector.urdf.xacro" />
-      <xacro:end_effector parent="${parent}">
-        <origin xyz="0.01 0 0" rpy="${90*deg_to_rad} ${90*deg_to_rad} ${-90*deg_to_rad}"/>
-      </xacro:end_effector>
-    </xacro:if>
-  <!-- No end-effector dual -->
-    <xacro:if value="${is_dual}">
-      <xacro:if value="${reflect == 1}">
-        <xacro:include filename="$(find custom_dual_ee_description)/urdf/end-effector-right.urdf.xacro" />
-        <xacro:end_effector_right parent="${parent}">
-          <origin xyz="0.01 0 0" rpy="${90*deg_to_rad} ${90*deg_to_rad} ${-90*deg_to_rad}"/>
-        </xacro:end_effector_right>
-      </xacro:if>
-      <xacro:if value="${reflect == -1}">
-        <xacro:include filename="$(find custom_dual_ee_description)/urdf/end-effector-left.urdf.xacro" />
-        <xacro:end_effector_left parent="${parent}">
-          <origin xyz="0.01 0 0" rpy="${90*deg_to_rad} ${90*deg_to_rad} ${-90*deg_to_rad}"/>
-        </xacro:end_effector_left>
-      </xacro:if>
-    </xacro:if>
+    <!-- Add nothing -->
   </xacro:if>
   <!-- PAL Gripper -->

Commit message: add epick end-effector

File: tiago_description/urdf/end_effector/end_effector.urdf.xacro (robot description, xacro)
@@ -96,4 +96,11 @@
     </xacro:robotiq_140_gripper>
   </xacro:if>
+  <!-- Robotiq Epick Gripper -->
+  <xacro:if value="${type == 'robotiq-epick'}">
+    <xacro:include filename="$(find pal_robotiq_epick_description)/urdf/robotiq_epick_model_macro.xacro" />
+    <xacro:epick_hand  prefix="${name}_" parent="${parent}">
+      <origin xyz="0.01 0 0" rpy="${90*deg_to_rad} ${0*deg_to_rad} ${90*deg_to_rad}"/>
+    </xacro:epick_hand>
+  </xacro:if>
   <!-- Custom -->
   <xacro:if value="${type == 'custom' and not is_dual}">

Commit message: Add is_dual arg to arm.urdf.xacro

File: tiago_description/urdf/end_effector/end_effector.urdf.xacro (robot description, xacro)
@@ -23,5 +23,5 @@
     - reflect: Set to 1 for a right end effector, or to -1 for a left end effector
   -->
-  <xacro:macro name="tiago_end_effector" params="name parent type reflect">
+  <xacro:macro name="tiago_end_effector" params="name parent type reflect is_dual:=false">
   <!-- PAL Gripper -->
   <xacro:if value="${type == 'pal-gripper'}">
@@ -64,10 +64,25 @@
   </xacro:if>
   <!-- Custom -->
-  <!-- <xacro:if value="${type == 'custom'}">
+  <!--xacro:if value="${type == 'custom' and not is_dual}">
     <xacro:include filename="$(find custom_ee_description)/urdf/end-effector.urdf.xacro" />
     <xacro:end_effector parent="${parent}">
       <origin xyz="0.01 0 0" rpy="${90*deg_to_rad} ${90*deg_to_rad} ${-90*deg_to_rad}"/>
     </xacro:end_effector>
-  </xacro:if> -->
+  </xacro:if-->
+  <!-- Custom dual-->
+  <!--xacro:if value="${type == 'custom' and is_dual}">
+    <xacro:if value="${reflect == 1}"--> <!-- If right -->
+    <!--xacro:include filename="$(find custom_dual_ee_description)/urdf/end-effector-right.urdf.xacro" />
+    <xacro:end_effector_right parent="${parent}">
+      <origin xyz="0.01 0 0" rpy="${90*deg_to_rad} ${90*deg_to_rad} ${-90*deg_to_rad}"/>
+    </xacro:end_effector_right>
+    </xacro:if>
+    <xacro:if value="${reflect == -1}"--> <!-- If left -->
+    <!--xacro:include filename="$(find custom_dual_ee_description)/urdf/end-effector-left.urdf.xacro" />
+    <xacro:end_effector_left parent="${parent}">
+      <origin xyz="0.01 0 0" rpy="${90*deg_to_rad} ${90*deg_to_rad} ${-90*deg_to_rad}"/>
+    </xacro:end_effector_left>
+    </xacro:if>
+  </xacro:if-->
   </xacro:macro>
 </robot>

Commit message: Rename end-effector xacro arg

File: tiago_description/urdf/end_effector/end_effector.urdf.xacro (robot description, xacro)
@@ -23,5 +23,5 @@
     - reflect: Set to 1 for a right end effector, or to -1 for a left end effector
   -->
-  <xacro:macro name="tiago_end_effector" params="name parent type reflect is_dual:=false">
+  <xacro:macro name="tiago_end_effector" params="name parent type reflect tiago_dual:=false">
   <!-- PAL Gripper -->
   <xacro:if value="${type == 'pal-gripper'}">
@@ -64,5 +64,5 @@
   </xacro:if>
   <!-- Custom -->
-  <!--xacro:if value="${type == 'custom' and not is_dual}">
+  <!--xacro:if value="${type == 'custom' and not tiago_dual}">
     <xacro:include filename="$(find custom_ee_description)/urdf/end-effector.urdf.xacro" />
     <xacro:end_effector parent="${parent}">
@@ -71,5 +71,5 @@
   </xacro:if-->
   <!-- Custom dual-->
-  <!--xacro:if value="${type == 'custom' and is_dual}">
+  <!--xacro:if value="${type == 'custom' and tiago_dual}">
     <xacro:if value="${reflect == 1}"--> <!-- If right -->
     <!--xacro:include filename="$(find custom_dual_ee_description)/urdf/end-effector-right.urdf.xacro" />
