Commit message: Allow multiple Tiagos on Gazebo
Refs #15402

File: tiago_description/gazebo/gazebo.urdf.xacro (robot description, xacro)
@@ -7,10 +7,15 @@
   Creative Commons, 444 Castro Street, Suite 900, Mountain View, California, 94041, USA.
 -->
-<robot name="tiago">
+<robot name="tiago" xmlns:xacro="http://www.ros.org/wiki/xacro">
   <gazebo>
     <plugin filename="libgazebo_ros_control.so" name="gazebo_ros_control">
       <ns></ns>
       <robotSimType>pal_hardware_gazebo/PalHardwareGazebo</robotSimType>
-      <robotNamespace></robotNamespace>
+      <xacro:if value="${is_multiple}">
+          <robotNamespace>/${nsp}</robotNamespace>
+      </xacro:if>
+      <xacro:unless value="${is_multiple}">
+          <robotNamespace></robotNamespace>
+      </xacro:unless>
       <controlPeriod>0.001</controlPeriod>
     </plugin>
@@ -20,10 +25,16 @@
       <alwaysOn>true</alwaysOn>
       <updateRate>100.0</updateRate>
+      <xacro:if value="${is_multiple}">
+          <robotNamespace>/${nsp}</robotNamespace>
+      </xacro:if>
     </plugin>
   </gazebo>
   <gazebo>
     <plugin filename="libgazebo_world_odometry.so" name="gazebo_ros_odometry">
-    <frameName>base_footprint</frameName>
-    <topicName>floating_base_pose_simulated</topicName>
+      <frameName>base_footprint</frameName>
+      <topicName>floating_base_pose_simulated</topicName>
+      <xacro:if value="${is_multiple}">
+          <robotNamespace>/${nsp}</robotNamespace>
+      </xacro:if>
     </plugin>
   </gazebo>

File: tiago_description/robots/tiago_steel.urdf.xacro (robot description, xacro)
@@ -9,4 +9,8 @@
 <robot  xmlns:xacro="http://www.ros.org/wiki/xacro"
         name="tiago" >
+  <xacro:arg name="multiple" default="false"/>
+  <xacro:arg name="namespace" default=""/>
+  <xacro:property name="is_multiple" value="$(arg multiple)" />
+  <xacro:property name="nsp" value="$(arg namespace)" />
   <!-- The following included files set up definitions of parts of the robot body -->
   <!-- Base -->

File: tiago_description/robots/tiago_titanium.urdf.xacro (robot description, xacro)
@@ -9,4 +9,8 @@
 <robot  xmlns:xacro="http://www.ros.org/wiki/xacro"
         name="tiago" >
+  <xacro:arg name="multiple" default="false"/>
+  <xacro:arg name="namespace" default=""/>
+  <xacro:property name="is_multiple" value="$(arg multiple)" />
+  <xacro:property name="nsp" value="$(arg namespace)" />
   <!-- The following included files set up definitions of parts of the robot body -->
   <!-- Base -->

Commit message: fix xacro warning
  deprecated: xacro tags should be prepended with 'xacro' xml namespace.
    Use the following script to fix incorrect usage:
              find . -iname "*.xacro" | xargs sed -i 's#<\([/]\?\)\(if\|unless\|include\|arg\|property\|macro\|insert_block\)#<\1xacro:\2#g'

File: tiago_description/gazebo/gazebo.urdf.xacro (robot description, xacro)
@@ -82,4 +82,4 @@
   </gazebo>
   <!-- define global properties -->
-  <property name="M_PI" value="3.1415926535897931" />
+  <xacro:property name="M_PI" value="3.1415926535897931" />
 </robot>

Commit message: make possible the possibility to choose the control period for gazebo

File: tiago_description/gazebo/gazebo.urdf.xacro (robot description, xacro)
@@ -23,5 +23,5 @@
           <robotNamespace></robotNamespace>
       </xacro:unless>
-      <controlPeriod>0.01</controlPeriod>
+      <controlPeriod>${gazebo_control_period}</controlPeriod>
     </plugin>
     <xacro:if value="${base_type == 'omni_base'}">

File: tiago_description/robots/tiago.urdf.xacro (robot description, xacro)
@@ -28,4 +28,5 @@
     <xacro:arg name="base_type" default="pmb2"/> <!-- pmb2, omni_base -->
     <xacro:arg name="fixed_torso" default="false" />
+    <xacro:arg name="gazebo_control_period" default="0.001"/> <!-- 1000Hz or 100 Hz-->
     <xacro:property name="wrist_model" value="$(arg wrist_model)" />
     <xacro:property name="end_effector" value="$(arg end_effector)" />
@@ -38,4 +39,5 @@
     <xacro:property name="no_safety_eps" value="$(arg no_safety_eps)" />
     <xacro:property name="fixed_torso" value="$(arg fixed_torso)" />
+    <xacro:property name="gazebo_control_period" value="$(arg gazebo_control_period)" />
   <xacro:if value="$(arg arm)">
     <xacro:if value="${wrist_model not in ['wrist-2010', 'wrist-2017']}">
