Commit message: Updated torso

File: tiago_description/urdf/torso/torso.urdf.xacro (robot description, xacro)
@@ -16,13 +16,19 @@
                izz="0.04165307088" />
     </inertial>
+    <visual>
+      <origin rpy="0 0 0" xyz="0.0 0.0 0" />
+      <geometry>
+        <box size="0.10 0.22 0.4"/>
+      </geometry>
+    </visual>
     <collision>
-      <origin rpy="0 0 0" xyz="0.13 0.45 0" />
+      <origin rpy="0 0 0" xyz="0.0 0.0 0" />
       <geometry>
-        <box size="0.20 0.40 0.32"/>
+        <box size="0.10 0.22 0.4"/>
       </geometry>
     </collision>
   </link>
   <joint name="${name}_fixed_joint" type="fixed">
-    <origin rpy="0 0 0" xyz="-0.053 0 0" />
+    <origin rpy="0 0 0" xyz="0 0 0.3" />
     <parent link="${parent}_link" />
     <child link="${name}_fixed_link" />
@@ -37,8 +43,14 @@
                izz="0.0376084656328484" />
     </inertial>
+    <visual>
+      <origin rpy="0 0 0" xyz="0 0 -0.35" />
+       <geometry>
+        <box size="0.10 0.22 0.7"/>
+      </geometry>
+    </visual>
     <collision>
-      <origin rpy="0 0 0" xyz="0 -.02 0" />
+      <origin rpy="0 0 0" xyz="0 0 0" />
        <geometry>
-        <box size="0.20 0.40 0.32"/>
+        <box size="0.10 0.22 0.7"/>
       </geometry>
     </collision>

Commit message: Fix torso

File: tiago_description/urdf/torso/torso.urdf.xacro (robot description, xacro)
@@ -16,19 +16,21 @@
                izz="0.04165307088" />
     </inertial>
-    <visual>
-      <origin rpy="0 0 0" xyz="0.0 0.0 0" />
+  <visual>
+      <origin rpy="0 0 0" xyz="0 0 0.2315" />
       <geometry>
-        <box size="0.10 0.22 0.4"/>
+        <box size="0.1 0.14 0.463"/>
       </geometry>
+      <material name="LightGrey"/>
     </visual>
     <collision>
-      <origin rpy="0 0 0" xyz="0.0 0.0 0" />
+      <origin rpy="0 0 0" xyz="0.0 0.0 0.2315" />
       <geometry>
-        <box size="0.10 0.22 0.4"/>
+        <box size="0.1 0.14 0.463"/>
       </geometry>
+      <material name="LightGrey"/>
     </collision>
   </link>
   <joint name="${name}_fixed_joint" type="fixed">
-    <origin rpy="0 0 0" xyz="-0.053 0 0.3" />
+    <origin rpy="0 0 0" xyz="-0.053 0 0.2015" />
     <parent link="${parent}_link" />
     <child link="${name}_fixed_link" />
@@ -44,18 +46,20 @@
     </inertial>
     <visual>
-      <origin rpy="0 0 0" xyz="0 0 -0.35" />
+      <origin rpy="0 0 0" xyz="0 0 -0.2315" />
        <geometry>
-        <box size="0.10 0.22 0.7"/>
+        <box size="0.106 0.15 0.463"/>
       </geometry>
+      <material name="White"/>
     </visual>
     <collision>
-      <origin rpy="0 0 0" xyz="0 0 0" />
+      <origin rpy="0 0 0" xyz="0 0 -0.2315" />
        <geometry>
-        <box size="0.10 0.22 0.7"/>
+        <box size="0.106 0.15 0.463"/>
       </geometry>
+      <material name="White"/>
     </collision>
   </link>
   <joint name="${name}_lift_joint" type="prismatic">
-    <origin rpy="0 0 0" xyz="0.0 0 0.26428" />
+    <origin rpy="0 0 0" xyz="0.0 0 0.463" />
     <parent link="${name}_fixed_link" />
     <child link="${name}_lift_link" />

Commit message: Update torso with reviewed inertial params

File: tiago_description/urdf/torso/torso.urdf.xacro (robot description, xacro)
@@ -11,6 +11,6 @@
   <link name="${name}_fixed_link">
     <inertial>
-      <origin rpy="0 0 0" xyz="0.00635 -0.01673 0.10662" />
-      <mass value="14.52876" />
+      <origin rpy="0 0 0" xyz="0.01929 -0.01317 0.0798" />
+      <mass value="7.22876" />
       <inertia ixx="0.17621875653" ixy="-0.00154333947"   ixz="0.00980172504"
                iyy="0.18995293862" iyz="-0.0259201152"
@@ -40,6 +40,6 @@
   <link name="${name}_lift_link">
     <inertial>
-      <origin rpy="0 0 0" xyz="0.02909 0.01068 -0.14826" />
-      <mass value="8.62177" />
+      <origin rpy="0 0 0" xyz="0.04761 0.01408 -0.12387" />
+      <mass value="6.54467" />
       <inertia ixx="0.19639986797" ixy="0.00528625771" ixz="-0.04018414421"
                iyy="0.212736527" iyz="-0.01564349386"

Commit message: Increase speed of torso joint

File: tiago_description/urdf/torso/torso.urdf.xacro (robot description, xacro)
@@ -87,5 +87,5 @@
     <child link="${name}_lift_link" />
     <axis xyz="0 0 1" />
-    <limit effort="2000" lower="0.0" upper="0.35" velocity="0.01" />
+    <limit effort="2000" lower="0.0" upper="0.35" velocity="0.02" />
     <calibration rising="0.0" />
     <dynamics damping="1000" />

Commit message: Add more collision geometries representing boxes and cable carriers on first tiago

File: tiago_description/urdf/torso/torso.urdf.xacro (robot description, xacro)
@@ -17,5 +17,5 @@
                izz="0.04165307088" />
     </inertial>
-  <visual>
+    <visual>
       <origin rpy="0 0 0" xyz="0 0 0.2235" />
       <geometry>
@@ -30,4 +30,51 @@
       </geometry>
       <material name="LightGrey"/>
+    </collision>
+    <!-- TODO: REMOVE -->
+    <!-- Preseries tiago boxes on the outside, these should go away in series version -->
+    <!-- column motor -->
+    <visual>
+      <origin rpy="${90*deg_to_rad} 0 0" xyz="-0.02 -0.09 0.035" />
+      <geometry>
+        <cylinder radius="0.035" length="0.09"/>
+      </geometry>
+      <material name="Yellow"/>
+    </visual>
+    <collision>
+      <origin rpy="${90*deg_to_rad} 0 0" xyz="-0.02 -0.09 0.035" />
+      <geometry>
+        <cylinder radius="0.035" length="0.09"/>
+      </geometry>
+      <material name="Yellow"/>
+    </collision>
+    <!-- column electronics box -->
+    <visual>
+      <origin rpy="0 0 0" xyz="0.04 -0.175 0.03" />
+      <geometry>
+        <box size="0.13 0.13 0.06"/>
+      </geometry>
+      <material name="Yellow"/>
+    </visual>
+    <collision>
+      <origin rpy="0 0 0" xyz="0.04 -0.175 0.03" />
+      <geometry>
+        <box size="0.13 0.13 0.06"/>
+      </geometry>
+      <material name="Yellow"/>
+    </collision>
+    <!-- cable carrier -->
+    <visual>
+      <origin rpy="0 0 0" xyz="0.045 -0.1 0.2" />
+      <geometry>
+        <box size="0.04 0.10 0.4"/>
+      </geometry>
+      <material name="Yellow"/>
+    </visual>
+    <collision>
+      <origin rpy="0 0 0" xyz="0.045 -0.1 0.2" />
+      <geometry>
+        <box size="0.04 0.10 0.4"/>
+      </geometry>
+      <material name="Yellow"/>
     </collision>
   </link>
@@ -81,4 +128,21 @@
       <material name="Grey" />
     </collision>
+    <!-- TODO: REMOVE -->
+    <!-- Preseries tiago boxes on the outside, these should go away in series version -->
+    <!-- cable carrier -->
+    <visual>
+      <origin rpy="0 0 0" xyz="0.045 -0.1 -0.4" />
+      <geometry>
+        <box size="0.04 0.10 0.4"/>
+      </geometry>
+      <material name="Yellow"/>
+    </visual>
+    <collision>
+      <origin rpy="0 0 0" xyz="0.045 -0.1 -0.4" />
+      <geometry>
+        <box size="0.04 0.10 0.4"/>
+      </geometry>
+      <material name="Yellow"/>
+    </collision>
   </link>
   <joint name="${name}_lift_joint" type="prismatic">

Commit message: Increase speed of torso

File: tiago_description/urdf/torso/torso.urdf.xacro (robot description, xacro)
@@ -151,5 +151,5 @@
     <child link="${name}_lift_link" />
     <axis xyz="0 0 1" />
-    <limit effort="2000" lower="0.0" upper="0.35" velocity="0.02" />
+    <limit effort="2000" lower="0.0" upper="0.35" velocity="0.05" />
     <calibration rising="0.0" />
     <dynamics damping="1000" />

Commit message: Add cable channel to the front of the column

File: tiago_description/urdf/torso/torso.urdf.xacro (robot description, xacro)
@@ -145,4 +145,11 @@
       <material name="Yellow"/>
     </collision>
+    <visual>
+      <origin rpy="0 0 0" xyz="0.085 -0.025 -0.25" />
+      <geometry>
+        <box size="0.025 0.05 0.5"/>
+      </geometry>
+      <material name="Yellow"/>
+    </visual>
   </link>
   <joint name="${name}_lift_joint" type="prismatic">

Commit message: restrict lifter joint to go lower than 5 cm
Take into account new mobile base covers that are 5 cm high

File: tiago_description/urdf/torso/torso.urdf.xacro (robot description, xacro)
@@ -158,5 +158,5 @@
     <child link="${name}_lift_link" />
     <axis xyz="0 0 1" />
-    <limit effort="2000" lower="0.0" upper="0.35" velocity="0.05" />
+    <limit effort="2000" lower="0.05" upper="0.35" velocity="0.05" />
     <calibration rising="0.0" />
     <dynamics damping="1000" />

Commit message: add cover on top of mobile base
Define collision and visual elements needed for the motion planning of TIAGo proof-of-concept

File: tiago_description/urdf/torso/torso.urdf.xacro (robot description, xacro)
@@ -75,4 +75,19 @@
       <geometry>
         <box size="0.04 0.10 0.4"/>
+      </geometry>
+      <material name="Yellow"/>
+    </collision>
+    <!-- mobile base top cover -->
+    <visual>
+      <origin rpy="0 0 0" xyz="0.068 0 0.01" />
+      <geometry>
+        <cylinder radius="0.25" length="0.05"/>
+      </geometry>
+      <material name="Yellow"/>
+    </visual>
+    <collision>
+      <origin rpy="0 0 0" xyz="0.068 0 0.01" />
+      <geometry>
+        <cylinder radius="0.25" length="0.05"/>
       </geometry>
       <material name="Yellow"/>

Commit message: change torso limits and update motions

File: tiago_description/urdf/torso/torso.urdf.xacro (robot description, xacro)
@@ -173,5 +173,5 @@
     <child link="${name}_lift_link" />
     <axis xyz="0 0 1" />
-    <limit effort="2000" lower="0.05" upper="0.35" velocity="0.05" />
+    <limit effort="2000" lower="0.06" upper="0.35" velocity="0.05" />
     <calibration rising="0.0" />
     <dynamics damping="1000" />

Commit message: Remove temporary cabling boxes

File: tiago_description/urdf/torso/torso.urdf.xacro (robot description, xacro)
@@ -17,4 +17,5 @@
                izz="0.04165307088" />
     </inertial>
+    <!-- Bottom fixed part of column -->
     <visual>
       <origin rpy="0 0 0" xyz="0 0 0.2235" />
@@ -31,66 +32,4 @@
       <material name="LightGrey"/>
     </collision>
-    <!-- TODO: REMOVE -->
-    <!-- Preseries tiago boxes on the outside, these should go away in series version -->
-    <!-- column motor -->
-    <visual>
-      <origin rpy="${90*deg_to_rad} 0 0" xyz="-0.02 -0.09 0.035" />
-      <geometry>
-        <cylinder radius="0.035" length="0.09"/>
-      </geometry>
-      <material name="Yellow"/>
-    </visual>
-    <collision>
-      <origin rpy="${90*deg_to_rad} 0 0" xyz="-0.02 -0.09 0.035" />
-      <geometry>
-        <cylinder radius="0.035" length="0.09"/>
-      </geometry>
-      <material name="Yellow"/>
-    </collision>
-    <!-- column electronics box -->
-    <visual>
-      <origin rpy="0 0 0" xyz="0.04 -0.175 0.03" />
-      <geometry>
-        <box size="0.13 0.13 0.06"/>
-      </geometry>
-      <material name="Yellow"/>
-    </visual>
-    <collision>
-      <origin rpy="0 0 0" xyz="0.04 -0.175 0.03" />
-      <geometry>
-        <box size="0.13 0.13 0.06"/>
-      </geometry>
-      <material name="Yellow"/>
-    </collision>
-    <!-- cable carrier -->
-    <visual>
-      <origin rpy="0 0 0" xyz="0.045 -0.1 0.2" />
-      <geometry>
-        <box size="0.04 0.10 0.4"/>
-      </geometry>
-      <material name="Yellow"/>
-    </visual>
-    <collision>
-      <origin rpy="0 0 0" xyz="0.045 -0.1 0.2" />
-      <geometry>
-        <box size="0.04 0.10 0.4"/>
-      </geometry>
-      <material name="Yellow"/>
-    </collision>
-    <!-- mobile base top cover -->
-    <visual>
-      <origin rpy="0 0 0" xyz="0.068 0 0.01" />
-      <geometry>
-        <cylinder radius="0.25" length="0.05"/>
-      </geometry>
-      <material name="Yellow"/>
-    </visual>
-    <collision>
-      <origin rpy="0 0 0" xyz="0.068 0 0.01" />
-      <geometry>
-        <cylinder radius="0.25" length="0.05"/>
-      </geometry>
-      <material name="Yellow"/>
-    </collision>
   </link>
   <joint name="${name}_fixed_joint" type="fixed">
@@ -104,9 +43,4 @@
       <origin rpy="0 0 0" xyz="-0.04761 0.01408 -0.12387" />
       <mass value="6.54467" />
-      <!--
-      <inertia ixx="0.19792" ixy="0" ixz="0"
-               iyy="0.21204" iyz="0"
-               izz="0.00332" />
-               -->
       <inertia ixx="0.0641960264706125" ixy="0.001128617953499" ixz="0.00203364821006436"
                iyy="0.061658561971383" iyz="-3.14401755382909E-05"
@@ -128,43 +62,4 @@
       <material name="White"/>
     </collision>
-    <!-- Head pan motor -->
-    <visual>
-      <origin xyz="0.187 0 0.02" rpy="0 0 0"/>
-      <geometry>
-        <box size="0.06 0.04 0.04"/>
-      </geometry>
-      <material name="Grey" />
-    </visual>
-    <collision>
-      <origin xyz="0.187 0 0.02" rpy="0 0 0" />
-      <geometry>
-        <box size="0.06 0.04 0.04"/>
-      </geometry>
-      <material name="Grey" />
-    </collision>
-    <!-- TODO: REMOVE -->
-    <!-- Preseries tiago boxes on the outside, these should go away in series version -->
-    <!-- cable carrier -->
-    <visual>
-      <origin rpy="0 0 0" xyz="0.045 -0.1 -0.4" />
-      <geometry>
-        <box size="0.04 0.10 0.4"/>
-      </geometry>
-      <material name="Yellow"/>
-    </visual>
-    <collision>
-      <origin rpy="0 0 0" xyz="0.045 -0.1 -0.4" />
-      <geometry>
-        <box size="0.04 0.10 0.4"/>
-      </geometry>
-      <material name="Yellow"/>
-    </collision>
-    <visual>
-      <origin rpy="0 0 0" xyz="0.085 -0.025 -0.25" />
-      <geometry>
-        <box size="0.025 0.05 0.5"/>
-      </geometry>
-      <material name="Yellow"/>
-    </visual>
   </link>
   <joint name="${name}_lift_joint" type="prismatic">

Commit message: Update torso

File: tiago_description/urdf/torso/torso.urdf.xacro (robot description, xacro)
@@ -4,9 +4,9 @@
   <xacro:include filename="$(find tiago_description)/urdf/deg_to_rad.xacro" />
   <xacro:include filename="$(find tiago_description)/urdf/torso/torso.transmission.xacro" />
- <!--Constant parameters-->
-  <xacro:property name="torso_max_vel"  value="5.4" />
-  <xacro:property name="torso_max_effort"  value="78.0" />
+  <!--Constant parameters-->
+  <xacro:property name="torso_max_vel"  value="0.1" />
   <xacro:property name="torso_eps"      value="0.02" />
   <xacro:macro name="tiago_torso" params="name parent">
+  <!-- Bottom fixed part of column -->
   <link name="${name}_fixed_link">
     <inertial>
@@ -17,9 +17,8 @@
                izz="0.04165307088" />
     </inertial>
-    <!-- Bottom fixed part of column -->
     <visual>
-      <origin rpy="0 0 0" xyz="0 0 0.2235" />
+      <origin rpy="0 0 0" xyz="0 0 0" />
       <geometry>
-        <box size="0.14 0.1 0.463"/>
+        <mesh filename="package://tiago_description/meshes/torso/torso_fix.stl" scale="1 1 1"/>
       </geometry>
       <material name="LightGrey"/>
@@ -34,7 +33,39 @@
   </link>
   <joint name="${name}_fixed_joint" type="fixed">
-    <origin rpy="0 0 0" xyz="-0.068 0 0.2235" />
+    <origin rpy="0 0 0" xyz="-0.062 0 0.195" />
     <parent link="${parent}" />
     <child link="${name}_fixed_link" />
+    <axis xyz="0 0 0" />
+  </joint>
+  <link name="${name}_fixed_column_link">
+    <inertial>
+      <origin rpy="0 0 0" xyz="0 0 0" />
+      <mass value="0.01" />
+      <inertia ixx="0.000001" ixy="0" ixz="0"
+               iyy="0.000001" iyz="0"
+               izz="0.000001" />
+    </inertial>
+    <visual>
+      <origin rpy="0 0 0" xyz="0 0 0.275" />
+      <geometry>
+        <box size="0.18 0.2 0.55"/>
+      </geometry>
+      <material name="DarkGrey"/>
+    </visual>
+    <collision>
+      <origin rpy="0 0 0" xyz="0 0 0.275" />
+      <geometry>
+        <box size="0.23 0.23 0.55"/>
+      </geometry>
+      <material name="DarkGrey"/>
+    </collision>
+  </link>
+  <gazebo reference="${name}_fixed_column_link">
+    <material>Gazebo/DarkGrey</material>
+  </gazebo>
+  <joint name="${name}_fixed_column_joint" type="fixed">
+    <origin rpy="0 0 0" xyz="-0.062 0 0.195" />
+    <parent link="${parent}" />
+    <child link="${name}_fixed_column_link" />
     <axis xyz="0 0 0" />
   </joint>
@@ -49,7 +80,7 @@
     <!-- Lifting body -->
     <visual>
-      <origin rpy="0 0 0" xyz="0 0 -0.25125" />
+      <origin rpy="0 0 0" xyz="0 0 0" />
        <geometry>
-        <box size="0.16 0.106 0.5025"/>
+        <mesh filename="package://tiago_description/meshes/torso/torso_lift.stl" scale="1 1 1"/>
       </geometry>
       <material name="White"/>
@@ -64,9 +95,9 @@
   </link>
   <joint name="${name}_lift_joint" type="prismatic">
-    <origin rpy="0 0 0" xyz="0.0 0 0.5025" />
+    <origin rpy="0 0 0" xyz="0.0 0 0.589" />
     <parent link="${name}_fixed_link" />
     <child link="${name}_lift_link" />
     <axis xyz="0 0 1" />
-    <limit effort="2000" lower="0.06" upper="0.35" velocity="0.05" />
+    <limit effort="2000" lower="0" upper="0.35" velocity="${torso_max_vel}" />
     <calibration rising="0.0" />
     <dynamics damping="1000" />

Commit message: Update torso meshes &  collision

File: tiago_description/urdf/torso/torso.urdf.xacro (robot description, xacro)
@@ -25,9 +25,14 @@
     </visual>
     <collision>
-      <origin rpy="0 0 0" xyz="0.0 0.0 0.2315" />
+      <origin rpy="0 0 0" xyz="0.085 0.0 0.02" />
       <geometry>
-        <box size="0.14 0.1 0.463"/>
+        <box size="0.4 0.25 0.04"/>
       </geometry>
-      <material name="LightGrey"/>
+    </collision>
+    <collision>
+      <origin rpy="0 0 0" xyz="0 0 0.05" />
+      <geometry>
+        <box size="0.25 0.25 0.1"/>
+      </geometry>
     </collision>
   </link>
@@ -87,7 +92,7 @@
     </visual>
     <collision>
-      <origin rpy="0 0 0" xyz="0 0 -0.25125" />
+      <origin rpy="0 0 0" xyz="0 0 0" />
        <geometry>
-        <box size="0.16 0.106 0.5025"/>
+        <mesh filename="package://tiago_description/meshes/torso/torso_lift_collision.stl" scale="1 1 1"/>
       </geometry>
       <material name="White"/>

Commit message: 7 cm / sec torso speed

File: tiago_description/urdf/torso/torso.urdf.xacro (robot description, xacro)
@@ -12,5 +12,5 @@
   <xacro:include filename="$(find tiago_description)/urdf/torso/torso.transmission.xacro" />
   <!--Constant parameters-->
-  <xacro:property name="torso_max_vel"  value="0.1" />
+  <xacro:property name="torso_max_vel"  value="0.07" />
   <xacro:property name="torso_eps"      value="0.02" />
   <xacro:macro name="tiago_torso" params="name parent">

Commit message: move torso 0 position 1 cm upwards

File: tiago_description/urdf/torso/torso.urdf.xacro (robot description, xacro)
@@ -108,5 +108,5 @@
   </link>
   <joint name="${name}_lift_joint" type="prismatic">
-    <origin rpy="0.0 0.0 0.0" xyz="0.0 0.0 0.587" />
+    <origin rpy="0.0 0.0 0.0" xyz="0.0 0.0 0.597" />
     <parent link="${name}_fixed_link" />
     <child link="${name}_lift_link" />

Commit message: Split torso collision into multiple elements for better convex hulls

File: tiago_description/urdf/torso/torso.urdf.xacro (robot description, xacro)
@@ -102,5 +102,19 @@
       <origin rpy="0 0 0" xyz="0 0 0" />
        <geometry>
-        <mesh filename="package://tiago_description/meshes/torso/torso_lift_collision.dae" scale="1 1 1"/>
+        <mesh filename="package://tiago_description/meshes/torso/torso_lift_collision_core.dae" scale="1 1 1"/>
+      </geometry>
+      <material name="LightGrey"/>
+    </collision>
+    <collision>
+      <origin rpy="0 0 0" xyz="0 0 0" />
+       <geometry>
+        <mesh filename="package://tiago_description/meshes/torso/torso_lift_collision_shoulder.dae" scale="1 1 1"/>
+      </geometry>
+      <material name="LightGrey"/>
+    </collision>
+    <collision>
+      <origin rpy="0 0 0" xyz="0 0 0" />
+       <geometry>
+        <mesh filename="package://tiago_description/meshes/torso/torso_lift_collision_neck.dae" scale="1 1 1"/>
       </geometry>
       <material name="LightGrey"/>

Commit message: Fix collision boxes for the torso

File: tiago_description/urdf/torso/torso.urdf.xacro (robot description, xacro)
@@ -39,5 +39,5 @@
       <origin rpy="0 0 0" xyz="0.085 0.0 0.02" />
       <geometry>
-        <box size="0.4 0.25 0.04"/>
+        <box size="0.4 0.265 0.05"/>
       </geometry>
     </collision>
@@ -45,5 +45,5 @@
       <origin rpy="0 0 0" xyz="0 0 0.05" />
       <geometry>
-        <box size="0.25 0.25 0.1"/>
+        <box size="0.255 0.255 0.117"/>
       </geometry>
     </collision>
@@ -74,5 +74,5 @@
       <origin rpy="0 0 0" xyz="0 0 0.275" />
       <geometry>
-        <box size="0.23 0.23 0.55"/>
+        <box size="0.23 0.253 0.45"/>
       </geometry>
       <material name="DarkGrey"/>

Commit message: Added if condition in torso xacro related to fixed_torso parameter

File: tiago_description/urdf/torso/torso.urdf.xacro (robot description, xacro)
@@ -126,4 +126,12 @@
     </collision>
   </link>
+  <xacro:if value="$(arg fixed_torso)">
+  <joint name="${name}_lift_joint" type="fixed">
+    <origin rpy="0.0 0.0 0.0" xyz="0.0 0.0 0.597" />
+    <parent link="${name}_fixed_link" />
+    <child link="${name}_lift_link" />
+  </joint>
+</xacro:if>
+<xacro:unless value="$(arg fixed_torso)">
   <joint name="${name}_lift_joint" type="prismatic">
     <origin rpy="0.0 0.0 0.0" xyz="0.0 0.0 0.597" />
@@ -135,9 +143,10 @@
     <dynamics damping="1000" />
     <safety_controller k_position="20"
-                         k_velocity="20"
-                         soft_lower_limit="0.0"
-                         soft_upper_limit="0.35" />
+      k_velocity="20"
+      soft_lower_limit="0.0"
+      soft_upper_limit="0.35" />
   </joint>
-  <xacro:torso_simple_transmission name="torso_lift" reduction="1.0"/>
+  <xacro:torso_simple_transmission name="torso_lift" reduction="1.0" />
+</xacro:unless>
  </xacro:macro>
 </robot>
