Commit message: Manual formating

File: tiago_description/urdf/torso/torso.urdf.xacro (robot description, xacro)
@@ -127,26 +127,26 @@
   </link>
   <xacro:if value="$(arg fixed_torso)">
-  <joint name="${name}_lift_joint" type="fixed">
-    <origin rpy="0.0 0.0 0.0" xyz="0.0 0.0 0.597" />
-    <parent link="${name}_fixed_link" />
-    <child link="${name}_lift_link" />
-  </joint>
-</xacro:if>
-<xacro:unless value="$(arg fixed_torso)">
-  <joint name="${name}_lift_joint" type="prismatic">
-    <origin rpy="0.0 0.0 0.0" xyz="0.0 0.0 0.597" />
-    <parent link="${name}_fixed_link" />
-    <child link="${name}_lift_link" />
-    <axis xyz="0 0 1" />
-    <limit effort="2000" lower="0" upper="0.35" velocity="${torso_max_vel}" />
-    <calibration rising="0.0" />
-    <dynamics damping="1000" />
-    <safety_controller k_position="20"
+    <joint name="${name}_lift_joint" type="fixed">
+      <origin rpy="0.0 0.0 0.0" xyz="0.0 0.0 0.597" />
+      <parent link="${name}_fixed_link" />
+      <child link="${name}_lift_link" />
+    </joint>
+  </xacro:if>
+  <xacro:unless value="$(arg fixed_torso)">
+    <joint name="${name}_lift_joint" type="prismatic">
+      <origin rpy="0.0 0.0 0.0" xyz="0.0 0.0 0.597" />
+      <parent link="${name}_fixed_link" />
+      <child link="${name}_lift_link" />
+      <axis xyz="0 0 1" />
+      <limit effort="2000" lower="0" upper="0.35" velocity="${torso_max_vel}" />
+      <calibration rising="0.0" />
+      <dynamics damping="1000" />
+      <safety_controller k_position="20"
       k_velocity="20"
       soft_lower_limit="0.0"
       soft_upper_limit="0.35" />
-  </joint>
-  <xacro:torso_simple_transmission name="torso_lift" reduction="1.0" />
-</xacro:unless>
+    </joint>
+    <xacro:torso_simple_transmission name="torso_lift" reduction="1.0" />
+  </xacro:unless>
  </xacro:macro>
 </robot>

Commit message: updated the torso to be at half it's range when fixed

File: tiago_description/urdf/torso/torso.urdf.xacro (robot description, xacro)
@@ -128,5 +128,6 @@
   <xacro:if value="$(arg fixed_torso)">
     <joint name="${name}_lift_joint" type="fixed">
-      <origin rpy="0.0 0.0 0.0" xyz="0.0 0.0 0.597" />
+      <!-- Torso fixed height is set to half it's range -->
+      <origin rpy="0.0 0.0 0.0" xyz="0.0 0.0 0.772" />
       <parent link="${name}_fixed_link" />
       <child link="${name}_lift_link" />

Commit message: Slightly increase the torso fix link collisoin model to avoid self collision

File: tiago_description/urdf/torso/torso.urdf.xacro (robot description, xacro)
@@ -36,7 +36,7 @@
     </visual>
     <collision>
-      <origin rpy="0 0 0" xyz="0.085 0.0 0.02" />
+      <origin rpy="0 0 0" xyz="0.105 0.0 0.04" />
       <geometry>
-        <box size="0.4 0.265 0.05"/>
+        <box size="0.4 0.3 0.1"/>
       </geometry>
     </collision>

Commit message: Slightly reduce the torso collision link size

File: tiago_description/urdf/torso/torso.urdf.xacro (robot description, xacro)
@@ -36,7 +36,7 @@
     </visual>
     <collision>
-      <origin rpy="0 0 0" xyz="0.105 0.0 0.04" />
+      <origin rpy="0 0 0" xyz="0.09 0.0 0.02" />
       <geometry>
-        <box size="0.4 0.3 0.1"/>
+        <box size="0.4 0.28 0.075"/>
       </geometry>
     </collision>

Commit message: add screen link in torso lift link

File: tiago_description/urdf/torso/torso.urdf.xacro (robot description, xacro)
@@ -124,4 +124,20 @@
       <material name="LightGrey"/>
     </collision>
+    <xacro:if value="$(arg has_screen)">
+      <visual>
+        <origin rpy="0 0 -1.57" xyz="-0.01 0.125 -0.27" />
+        <geometry>
+          <mesh filename="package://tiago_description/meshes/torso/tiago_screen.STL" scale="1 1 1"/>
+        </geometry>
+        <material name="White"/>
+      </visual>
+      <collision>
+        <origin rpy="0 0 -1.57" xyz="-0.01 0.125 -0.27" />
+        <geometry>
+          <mesh filename="package://tiago_description/meshes/torso/screen_collision.stl" scale="1 1 1"/>
+        </geometry>
+        <material name="LightGrey"/>
+      </collision>
+    </xacro:if>
   </link>
   <xacro:if value="$(arg fixed_torso)">
@@ -149,34 +165,4 @@
     <xacro:torso_simple_transmission name="torso_lift" reduction="1.0" />
   </xacro:unless>
-  <xacro:if value="$(arg has_screen)">
-    <link name="${name}_screen_link">
-      <inertial>
-        <origin xyz="0.00004923 0.000001  -0.00000308" rpy="0.00000 0.00000 0.00000"/>
-        <mass value="0.96841"/>
-        <inertia ixx="0.0" ixy="1.0" ixz="0.0"
-                iyy="0.24926900000" iyz="0.00828100000"
-                izz="0.09039500000"/>
-      </inertial>
-      <visual>
-        <origin rpy="3.14159 0 0" xyz="-0.0425 0.1275 0.065" />
-        <geometry>
-          <mesh filename="package://tiago_description/meshes/torso/tiago_screen.STL" scale="0.001 0.001 0.001"/>
-        </geometry>
-        <material name="White"/>
-      </visual>
-      <collision>
-        <origin rpy="3.14159 0 0" xyz="-0.040 0.1275 0.065" />
-        <geometry>
-          <mesh filename="package://tiago_description/meshes/torso/tiago_screen.STL" scale="0.001 0.001 0.001"/>
-        </geometry>
-        <material name="LightGrey"/>
-      </collision>
-    </link>
-    <joint name="${name}_screen_joint" type="fixed">
-      <origin rpy="0.0 0.0 1.57" xyz="-0.02 0.125 -0.27" />
-      <parent link="${name}_lift_link" />
-      <child link="${name}_screen_link" />
-    </joint>
-  </xacro:if>
  </xacro:macro>
 </robot>

Commit message: idkl

File: tiago_description/urdf/torso/torso.urdf.xacro (robot description, xacro)
@@ -41,5 +41,5 @@
       </collision>
       <collision>
-        <origin rpy="0 0 0" xyz="0 0 0.05" />
+        <origin rpy="0 0 0" xyz="0 0 0.25" />
         <geometry>
           <box size="0.25 0.25 0.1"/>

Commit message: find installed tiago_description package

File: tiago_description/urdf/torso/torso.urdf.xacro (robot description, xacro)
@@ -31,5 +31,5 @@
       <origin rpy="0 0 0" xyz="0 0 0" />
       <geometry>
-        <mesh filename="package://tiago_description/meshes/torso/torso_fix.stl" scale="1 1 1"/>
+        <mesh filename="$(find tiago_description)/meshes/torso/torso_fix.stl" scale="1 1 1"/>
       </geometry>
       <material name="LightGrey"/>
@@ -99,5 +99,5 @@
       <origin rpy="0 0 0" xyz="0 0 0" />
        <geometry>
-        <mesh filename="package://tiago_description/meshes/torso/torso_lift_with_arm.stl" scale="1 1 1"/>
+        <mesh filename="$(find tiago_description)/meshes/torso/torso_lift_with_arm.stl" scale="1 1 1"/>
       </geometry>
       <material name="White"/>
@@ -106,5 +106,5 @@
       <origin rpy="0 0 0" xyz="0 0 0" />
        <geometry>
-        <mesh filename="package://tiago_description/meshes/torso/torso_lift_collision_core.dae" scale="1 1 1"/>
+        <mesh filename="$(find tiago_description)/meshes/torso/torso_lift_collision_core.dae" scale="1 1 1"/>
       </geometry>
       <material name="LightGrey"/>
@@ -113,5 +113,5 @@
       <origin rpy="0 0 0" xyz="0 0 0" />
        <geometry>
-        <mesh filename="package://tiago_description/meshes/torso/torso_lift_collision_shoulder.dae" scale="1 1 1"/>
+        <mesh filename="$(find tiago_description)/meshes/torso/torso_lift_collision_shoulder.dae" scale="1 1 1"/>
       </geometry>
       <material name="LightGrey"/>
@@ -120,5 +120,5 @@
       <origin rpy="0 0 0" xyz="0 0 0" />
        <geometry>
-        <mesh filename="package://tiago_description/meshes/torso/torso_lift_collision_neck.dae" scale="1 1 1"/>
+        <mesh filename="$(find tiago_description)/meshes/torso/torso_lift_collision_neck.dae" scale="1 1 1"/>
       </geometry>
       <material name="LightGrey"/>
@@ -128,5 +128,5 @@
         <origin rpy="0 0 -1.57" xyz="-0.01 0.125 -0.27" />
         <geometry>
-          <mesh filename="package://tiago_description/meshes/torso/tiago_screen.STL" scale="1 1 1"/>
+          <mesh filename="$(find tiago_description)/meshes/torso/tiago_screen.STL" scale="1 1 1"/>
         </geometry>
         <material name="White"/>
@@ -135,5 +135,5 @@
         <origin rpy="0 0 -1.57" xyz="-0.01 0.125 -0.27" />
         <geometry>
-          <mesh filename="package://tiago_description/meshes/torso/screen_collision.stl" scale="1 1 1"/>
+          <mesh filename="$(find tiago_description)/meshes/torso/screen_collision.stl" scale="1 1 1"/>
         </geometry>
         <material name="LightGrey"/>

Commit message: Fix package path for meshes

File: tiago_description/urdf/torso/torso.urdf.xacro (robot description, xacro)
@@ -31,5 +31,5 @@
       <origin rpy="0 0 0" xyz="0 0 0" />
       <geometry>
-        <mesh filename="$(find tiago_description)/meshes/torso/torso_fix.stl" scale="1 1 1"/>
+        <mesh filename="package://tiago_description/meshes/torso/torso_fix.stl" scale="1 1 1"/>
       </geometry>
       <material name="LightGrey"/>
@@ -99,5 +99,5 @@
       <origin rpy="0 0 0" xyz="0 0 0" />
        <geometry>
-        <mesh filename="$(find tiago_description)/meshes/torso/torso_lift_with_arm.stl" scale="1 1 1"/>
+        <mesh filename="package://tiago_description/meshes/torso/torso_lift_with_arm.stl" scale="1 1 1"/>
       </geometry>
       <material name="White"/>
@@ -106,5 +106,5 @@
       <origin rpy="0 0 0" xyz="0 0 0" />
        <geometry>
-        <mesh filename="$(find tiago_description)/meshes/torso/torso_lift_collision_core.dae" scale="1 1 1"/>
+        <mesh filename="package://tiago_description/meshes/torso/torso_lift_collision_core.dae" scale="1 1 1"/>
       </geometry>
       <material name="LightGrey"/>
@@ -113,5 +113,5 @@
       <origin rpy="0 0 0" xyz="0 0 0" />
        <geometry>
-        <mesh filename="$(find tiago_description)/meshes/torso/torso_lift_collision_shoulder.dae" scale="1 1 1"/>
+        <mesh filename="package://tiago_description/meshes/torso/torso_lift_collision_shoulder.dae" scale="1 1 1"/>
       </geometry>
       <material name="LightGrey"/>
@@ -120,5 +120,5 @@
       <origin rpy="0 0 0" xyz="0 0 0" />
        <geometry>
-        <mesh filename="$(find tiago_description)/meshes/torso/torso_lift_collision_neck.dae" scale="1 1 1"/>
+        <mesh filename="package://tiago_description/meshes/torso/torso_lift_collision_neck.dae" scale="1 1 1"/>
       </geometry>
       <material name="LightGrey"/>
@@ -128,5 +128,5 @@
         <origin rpy="0 0 -1.57" xyz="-0.01 0.125 -0.27" />
         <geometry>
-          <mesh filename="$(find tiago_description)/meshes/torso/tiago_screen.STL" scale="1 1 1"/>
+          <mesh filename="package://tiago_description/meshes/torso/tiago_screen.STL" scale="1 1 1"/>
         </geometry>
         <material name="White"/>
@@ -135,5 +135,5 @@
         <origin rpy="0 0 -1.57" xyz="-0.01 0.125 -0.27" />
         <geometry>
-          <mesh filename="$(find tiago_description)/meshes/torso/screen_collision.stl" scale="1 1 1"/>
+          <mesh filename="package://tiago_description/meshes/torso/screen_collision.stl" scale="1 1 1"/>
         </geometry>
         <material name="LightGrey"/>

Commit message: Add side screen to URDF

File: tiago_description/urdf/torso/torso.urdf.xacro (robot description, xacro)
@@ -19,5 +19,5 @@
   <xacro:include filename="$(find pal_urdf_utils)/urdf/deg_to_rad.urdf.xacro" />
   <!-- MACRO DEFINITION-->
-  <xacro:macro name="tiago_torso" params="name parent *origin">
+  <xacro:macro name="tiago_torso" params="name parent *origin has_screen">
     <!-- Bottom fixed part of column -->
     <link name="${name}_fixed_link">
@@ -119,4 +119,20 @@
         <material name="LightGrey"/>
       </collision>
+    <xacro:if value="$(arg has_screen)">
+      <visual>
+        <origin rpy="0 0 -1.57" xyz="-0.01 0.125 -0.27" />
+        <geometry>
+          <mesh filename="package://tiago_description/meshes/torso/tiago_screen.stl" scale="1 1 1"/>
+        </geometry>
+        <material name="White"/>
+      </visual>
+      <collision>
+        <origin rpy="0 0 -1.57" xyz="-0.01 0.125 -0.27" />
+        <geometry>
+          <mesh filename="package://tiago_description/meshes/torso/tiago_screen_collision.stl" scale="1 1 1"/>
+        </geometry>
+        <material name="LightGrey"/>
+      </collision>
+    </xacro:if>
     </link>
     <joint name="${name}_lift_joint" type="prismatic">

Commit message: Fix torso collision

File: tiago_description/urdf/torso/torso.urdf.xacro (robot description, xacro)
@@ -70,5 +70,5 @@
         <origin rpy="0 0 0" xyz="0 0 0.275" />
         <geometry>
-          <box size="0.23 0.23 0.55"/>
+          <box size="0.232 0.265 0.45"/>
         </geometry>
         <material name="DarkGrey"/>
