Commit message: Added wrist to arm_controller

File: tiago_description/ros2_control/ros2_control.urdf.xacro (robot description, xacro)
@@ -11,8 +11,9 @@
   <xacro:arg name="description_calibration_dir" default="$(find tiago_description_calibration)/urdf/calibration"/>
   <!-- TODO has_arm param -->
-  <xacro:include filename="$(find pmb2_description)/urdf/wheels/wheel.ros2_control.xacro"/>
-  <xacro:include filename="$(find tiago_description)/urdf/torso/torso.ros2_control.xacro"/>
-  <xacro:include filename="$(find tiago_description)/urdf/head/head.ros2_control.xacro"/>
-  <xacro:include filename="$(find tiago_description)/urdf/arm/arm.ros2_control.xacro"/>
+  <xacro:include filename="$(find pmb2_description)/urdf/wheels/wheel.ros2_control.xacro" />
+  <xacro:include filename="$(find tiago_description)/urdf/torso/torso.ros2_control.xacro" />
+  <xacro:include filename="$(find tiago_description)/urdf/head/head.ros2_control.xacro" />
+  <xacro:include filename="$(find tiago_description)/urdf/arm/arm.ros2_control.xacro" />
+  <xacro:include filename="$(find tiago_description)/urdf/arm/wrist.ros2_control.xacro" />
   <!-- calibration offsets -->
   <xacro:include filename="$(arg description_calibration_dir)/calibration_constants.urdf.xacro" />
@@ -27,11 +28,17 @@
     <xacro:ros2_control_torso name="torso_lift" reduction="1.0" />
     <!-- head -->
-    <xacro:ros2_control_head name="head_1" reduction="1.0" offset_value="${head_1_joint_offset}"/>
-    <xacro:ros2_control_head name="head_2" reduction="1.0" offset_value="${head_2_joint_offset}"/>
+    <xacro:ros2_control_head name="head_1" reduction="1.0" offset="${head_1_joint_offset}" />
+    <xacro:ros2_control_head name="head_2" reduction="1.0" offset="${head_2_joint_offset}" />
     <!-- arm -->
-    <xacro:ros2_control_arm name="arm_1" reduction="1.0" offset_value="${arm_1_joint_offset}"/>
-    <xacro:ros2_control_arm name="arm_2" reduction="1.0" offset_value="${arm_2_joint_offset}"/>
-    <xacro:ros2_control_arm name="arm_3" reduction="1.0" offset_value="${arm_3_joint_offset}"/>
-    <xacro:ros2_control_arm name="arm_4" reduction="1.0" offset_value="${arm_4_joint_offset}"/>
+    <xacro:ros2_control_arm name="arm_1" reduction="1.0" offset="${arm_1_joint_offset}" />
+    <xacro:ros2_control_arm name="arm_2" reduction="1.0" offset="${arm_2_joint_offset}" />
+    <xacro:ros2_control_arm name="arm_3" reduction="1.0" offset="${arm_3_joint_offset}" />
+    <xacro:ros2_control_arm name="arm_4" reduction="1.0" offset="${arm_4_joint_offset}" />
+    <!-- wrist -->
+    <xacro:ros2_control_wrist_rotational name="arm_5" reduction="1.0" offset="${arm_5_joint_offset}" />
+    <xacro:ros2_control_wrist_differential name_1="arm_6" name_2="arm_7"
+                                           act_reduction_1="-1.0" act_reduction_2="1.0"
+                                           jnt_reduction_1="1.0" jnt_reduction_2="1.0"
+                                           number_1_offset="${arm_6_joint_offset}" number_2_offset="${arm_7_joint_offset}" />
   </ros2_control>
 </robot>

File: tiago_description/urdf/arm/arm.ros2_control.xacro (robot description, xacro)
@@ -8,5 +8,5 @@
 -->
 <robot xmlns:xacro="http://ros.org/wiki/xacro">
-  <xacro:macro name="ros2_control_arm" params="name reduction offset_value" >
+  <xacro:macro name="ros2_control_arm" params="name reduction offset" >
     <joint name="${name}_joint">
       <command_interface name="position" />
@@ -23,5 +23,5 @@
       </actuator>
       <joint name="${name}_${number}_joint">
-        <offset>${offset_value}</offset>
+        <offset>${offset}</offset>
         <hardwareInterface>hardware_interface/PositionJointInterface</hardwareInterface>
         <hardwareInterface>hardware_interface/EffortJointInterface</hardwareInterface>

File: tiago_description/urdf/head/head.ros2_control.xacro (robot description, xacro)
@@ -8,5 +8,5 @@
 -->
 <robot xmlns:xacro="http://ros.org/wiki/xacro">
-  <xacro:macro name="ros2_control_head" params="name reduction offset_value" >
+  <xacro:macro name="ros2_control_head" params="name reduction offset" >
     <joint name="${name}_joint">
       <command_interface name="position" />

Commit message: Added support for arm and ft_sensor args

File: tiago_description/ros2_control/ros2_control.urdf.xacro (robot description, xacro)
@@ -9,11 +9,14 @@
 <robot xmlns:xacro="http://ros.org/wiki/xacro"
        name="tiago" >
-  <xacro:arg name="description_calibration_dir" default="$(find tiago_description_calibration)/urdf/calibration"/>
-  <!-- TODO has_arm param -->
+  <xacro:arg name="arm" default="true" />
+  <xacro:arg name="description_calibration_dir" default="$(find tiago_description_calibration)/urdf/calibration" />
+  <xacro:property name="has_arm" value="$(arg arm)" />
   <xacro:include filename="$(find pmb2_description)/urdf/wheels/wheel.ros2_control.xacro" />
   <xacro:include filename="$(find tiago_description)/urdf/torso/torso.ros2_control.xacro" />
   <xacro:include filename="$(find tiago_description)/urdf/head/head.ros2_control.xacro" />
-  <xacro:include filename="$(find tiago_description)/urdf/arm/arm.ros2_control.xacro" />
-  <xacro:include filename="$(find tiago_description)/urdf/arm/wrist.ros2_control.xacro" />
+  <xacro:if value="${has_arm}">
+    <xacro:include filename="$(find tiago_description)/urdf/arm/arm.ros2_control.xacro" />
+    <xacro:include filename="$(find tiago_description)/urdf/arm/wrist.ros2_control.xacro" />
+  </xacro:if>
   <!-- calibration offsets -->
   <xacro:include filename="$(arg description_calibration_dir)/calibration_constants.urdf.xacro" />
@@ -30,15 +33,17 @@
     <xacro:ros2_control_head name="head_1" reduction="1.0" offset="${head_1_joint_offset}" />
     <xacro:ros2_control_head name="head_2" reduction="1.0" offset="${head_2_joint_offset}" />
-    <!-- arm -->
-    <xacro:ros2_control_arm name="arm_1" reduction="1.0" offset="${arm_1_joint_offset}" />
-    <xacro:ros2_control_arm name="arm_2" reduction="1.0" offset="${arm_2_joint_offset}" />
-    <xacro:ros2_control_arm name="arm_3" reduction="1.0" offset="${arm_3_joint_offset}" />
-    <xacro:ros2_control_arm name="arm_4" reduction="1.0" offset="${arm_4_joint_offset}" />
-    <!-- wrist -->
-    <xacro:ros2_control_wrist_rotational name="arm_5" reduction="1.0" offset="${arm_5_joint_offset}" />
-    <xacro:ros2_control_wrist_differential name_1="arm_6" name_2="arm_7"
-                                           act_reduction_1="-1.0" act_reduction_2="1.0"
-                                           jnt_reduction_1="1.0" jnt_reduction_2="1.0"
-                                           number_1_offset="${arm_6_joint_offset}" number_2_offset="${arm_7_joint_offset}" />
+    <xacro:if value="${has_arm}">
+      <!-- arm -->
+      <xacro:ros2_control_arm name="arm_1" reduction="1.0" offset="${arm_1_joint_offset}" />
+      <xacro:ros2_control_arm name="arm_2" reduction="1.0" offset="${arm_2_joint_offset}" />
+      <xacro:ros2_control_arm name="arm_3" reduction="1.0" offset="${arm_3_joint_offset}" />
+      <xacro:ros2_control_arm name="arm_4" reduction="1.0" offset="${arm_4_joint_offset}" />
+      <!-- wrist -->
+      <xacro:ros2_control_wrist_rotational name="arm_5" reduction="1.0" offset="${arm_5_joint_offset}" />
+      <xacro:ros2_control_wrist_differential name_1="arm_6" name_2="arm_7"
+                                             act_reduction_1="-1.0" act_reduction_2="1.0"
+                                             jnt_reduction_1="1.0" jnt_reduction_2="1.0"
+                                             number_1_offset="${arm_6_joint_offset}" number_2_offset="${arm_7_joint_offset}" />
+    </xacro:if>
   </ros2_control>
 </robot>

Commit message: Support for pal-gripper end effector

File: tiago_description/ros2_control/ros2_control.urdf.xacro (robot description, xacro)
@@ -10,6 +10,8 @@
        name="tiago" >
   <xacro:arg name="arm" default="true" />
+  <xacro:arg name="end_effector" default="pal-hey5"/>
   <xacro:arg name="description_calibration_dir" default="$(find tiago_description_calibration)/urdf/calibration" />
   <xacro:property name="has_arm" value="$(arg arm)" />
+  <xacro:property name="end_effector" value="$(arg end_effector)" />
   <xacro:include filename="$(find pmb2_description)/urdf/wheels/wheel.ros2_control.xacro" />
   <xacro:include filename="$(find tiago_description)/urdf/torso/torso.ros2_control.xacro" />
@@ -18,4 +20,7 @@
     <xacro:include filename="$(find tiago_description)/urdf/arm/arm.ros2_control.xacro" />
     <xacro:include filename="$(find tiago_description)/urdf/arm/wrist.ros2_control.xacro" />
+    <xacro:if value="${end_effector == 'pal-gripper'}">
+      <xacro:include filename="$(find pal_gripper_description)/urdf/gripper.ros2_control.xacro" />
+    </xacro:if>
   </xacro:if>
   <!-- calibration offsets -->
@@ -45,4 +50,9 @@
                                              jnt_reduction_1="1.0" jnt_reduction_2="1.0"
                                              number_1_offset="${arm_6_joint_offset}" number_2_offset="${arm_7_joint_offset}" />
+      <xacro:if value="${end_effector == 'pal-gripper'}">
+        <!-- pal-gripper -->
+        <xacro:ros2_control_gripper name="gripper_left_finger" reduction="1.0" />
+        <xacro:ros2_control_gripper name="gripper_right_finger" reduction="1.0" />
+      </xacro:if>
     </xacro:if>
   </ros2_control>

Commit message: Add support for new gazebo

File: tiago_description/ros2_control/ros2_control.urdf.xacro (robot description, xacro)
@@ -44,7 +44,16 @@
     <xacro:if value="${use_sim_time}">
       <gazebo>
-        <plugin filename="libgazebo_ros2_control.so" name="gazebo_ros2_control">
-          <parameters>$(find tiago_description)/ros2_control/gazebo_controller_manager_cfg.yaml</parameters>
-        </plugin>
+        <xacro:if value="${gazebo_version == 'classic'}">
+          <plugin filename="libgazebo_ros2_control.so" name="gazebo_ros2_control">
+            <parameters>$(find tiago_description)/ros2_control/gazebo_controller_manager_cfg.yaml</parameters>
+          </plugin>
+        </xacro:if>
+        <xacro:if value="${gazebo_version == 'gazebo'}">
+          <plugin filename="gz_ros2_control-system" name="gz_ros2_control::GazeboSimROS2ControlPlugin">
+            <robot_param>robot_description</robot_param>
+            <robot_param_node>robot_state_publisher</robot_param_node>
+            <parameters>$(find tiago_description)/ros2_control/gazebo_controller_manager_cfg.yaml</parameters>
+          </plugin>
+        </xacro:if>
       </gazebo>
     </xacro:if>
@@ -54,5 +63,10 @@
       <hardware>
         <xacro:if value="${use_sim_time}">
-          <plugin>gazebo_ros2_control/GazeboSystem</plugin>
+          <xacro:if value="${gazebo_version == 'classic'}">
+            <plugin>gazebo_ros2_control/GazeboSystem</plugin>
+          </xacro:if>
+          <xacro:if value="${gazebo_version == 'gazebo'}">
+            <plugin>gz_ros2_control/GazeboSimSystem</plugin>
+          </xacro:if>
         </xacro:if>
         <xacro:unless value="${use_sim_time}">

File: tiago_description/urdf/arm/arm.ros2_control.xacro (robot description, xacro)
@@ -19,6 +19,11 @@
     <joint name="${name}_joint">
       <command_interface name="position" />
-      <command_interface name="velocity" />
-      <command_interface name="effort" />
+      <!-- TODO: Remove when moving to Gazebo Harmonic or ROS 2 Jazzy -->
+      <!-- Multiple command interfaces not working on Gazebo Fortress -->
+      <!-- https://github.com/ros-controls/gz_ros2_control/issues/182 -->
+      <xacro:if value="${gazebo_version == 'classic'}">
+        <command_interface name="velocity" />
+        <command_interface name="effort" />
+      </xacro:if>
       <state_interface name="position" />
       <state_interface name="velocity" />

File: tiago_description/urdf/arm/arm.urdf.xacro (robot description, xacro)
@@ -43,5 +43,5 @@
         <origin xyz="0.061191 -0.022397 ${reflect * -0.012835}" rpy="0.00000 0.00000 0.00000"/>
         <mass value="1.563428"/>
-        <inertia ixx="0.002471" ixy="${reflect * -0.001809}" ixz="-0.001202" iyy="0.006132" iyz="${reflect * 0.000494}" izz="0.006704"/>
+        <inertia ixx="0.002471" ixy="${-reflect * -0.001809}" ixz="-0.001202" iyy="0.006132" iyz="${reflect * 0.000494}" izz="0.006704"/>
       </inertial>
       <!-- M90 module -->
@@ -49,5 +49,5 @@
         <origin xyz="0 0 0" rpy="0 0 0" />
         <geometry>
-          <mesh filename="package://tiago_description/meshes/arm/arm_1.stl" scale="1 ${-1 * tiago_dual} ${reflect}"/>
+          <mesh filename="file://$(find tiago_description)/meshes/arm/arm_1.stl" scale="1 ${-1 * tiago_dual} ${reflect}"/>
         </geometry>
         <material name="White"/>
@@ -56,5 +56,5 @@
         <origin xyz="0 0 0" rpy="0 0 0" />
         <geometry>
-          <mesh filename="package://tiago_description/meshes/arm/arm_1_collision.dae" scale="1 ${-1 * tiago_dual} ${reflect}"/>
+          <mesh filename="file://$(find tiago_description)/meshes/arm/arm_1_collision.dae" scale="1 ${-1 * tiago_dual} ${reflect}"/>
         </geometry>
       </collision>
@@ -81,5 +81,5 @@
         <origin xyz="0 0 0" rpy="${0 * deg_to_rad} ${0 * deg_to_rad} ${0 * deg_to_rad}" />
         <geometry>
-          <mesh filename="package://tiago_description/meshes/arm/arm_2.stl" scale="1 1 ${reflect}"/>
+          <mesh filename="file://$(find tiago_description)/meshes/arm/arm_2.stl" scale="1 1 ${reflect}"/>
         </geometry>
         <material name="DarkGrey" />
@@ -89,5 +89,5 @@
         <origin xyz="0 0 0" rpy="${0 * deg_to_rad} ${0 * deg_to_rad} ${0 * deg_to_rad}" />
         <geometry>
-          <mesh filename="package://tiago_description/meshes/arm/arm_2_collision.dae" scale="1 1 ${reflect}"/>
+          <mesh filename="file://$(find tiago_description)/meshes/arm/arm_2_collision.dae" scale="1 1 ${reflect}"/>
         </geometry>
       </collision>
@@ -113,5 +113,5 @@
         <origin xyz="0 0 0" rpy="0 0 0" />
         <geometry>
-          <mesh filename="package://tiago_description/meshes/arm/arm_3.stl" scale="1 1 ${reflect}"/>
+          <mesh filename="file://$(find tiago_description)/meshes/arm/arm_3.stl" scale="1 1 ${reflect}"/>
         </geometry>
         <material name="DarkGrey" />
@@ -120,5 +120,5 @@
         <origin xyz="0 0 0" rpy="0 0 0" />
         <geometry>
-          <mesh filename="package://tiago_description/meshes/arm/arm_3_collision.dae" scale="1 1 ${reflect}"/>
+          <mesh filename="file://$(find tiago_description)/meshes/arm/arm_3_collision.dae" scale="1 1 ${reflect}"/>
         </geometry>
       </collision>
@@ -145,5 +145,5 @@
         <origin xyz="0 0 0" rpy="0 0 0" />
         <geometry>
-          <mesh filename="package://tiago_description/meshes/arm/arm_4.stl" scale="${reflect} ${reflect} ${reflect}"/>
+          <mesh filename="file://$(find tiago_description)/meshes/arm/arm_4.stl" scale="${reflect} ${reflect} ${reflect}"/>
         </geometry>
         <material name="DarkGrey" />
@@ -152,5 +152,5 @@
         <origin xyz="0 0 0" rpy="0 0 0" />
         <geometry>
-          <mesh filename="package://tiago_description/meshes/arm/arm_4_collision.dae" scale="${reflect} ${reflect} ${reflect}"/>
+          <mesh filename="file://$(find tiago_description)/meshes/arm/arm_4_collision.dae" scale="${reflect} ${reflect} ${reflect}"/>
         </geometry>
       </collision>

File: tiago_description/urdf/arm/wrist.ros2_control.xacro (robot description, xacro)
@@ -19,6 +19,11 @@
     <joint name="${name}_joint">
       <command_interface name="position" />
-      <command_interface name="velocity" />
-      <command_interface name="effort" />
+      <!-- TODO: Remove when moving to Gazebo Harmonic or ROS 2 Jazzy -->
+      <!-- Multiple command interfaces not working on Gazebo Fortress -->
+      <!-- https://github.com/ros-controls/gz_ros2_control/issues/182 -->
+      <xacro:if value="${gazebo_version == 'classic'}">
+        <command_interface name="velocity" />
+        <command_interface name="effort" />
+      </xacro:if>
       <state_interface name="position" />
       <state_interface name="velocity" />
@@ -30,6 +35,11 @@
     <joint name="${name}_${number_1}_joint">
       <command_interface name="position" />
-      <command_interface name="velocity" />
-      <command_interface name="effort" />
+      <!-- TODO: Remove when moving to Gazebo Harmonic or ROS 2 Jazzy -->
+      <!-- Multiple command interfaces not working on Gazebo Fortress -->
+      <!-- https://github.com/ros-controls/gz_ros2_control/issues/182 -->
+      <xacro:if value="${gazebo_version == 'classic'}">
+        <command_interface name="velocity" />
+        <command_interface name="effort" />
+      </xacro:if>
       <state_interface name="position" />
       <state_interface name="velocity" />
@@ -38,6 +48,11 @@
     <joint name="${name}_${number_2}_joint">
       <command_interface name="position" />
-      <command_interface name="velocity" />
-      <command_interface name="effort" />
+      <!-- TODO: Remove when moving to Gazebo Harmonic or ROS 2 Jazzy -->
+      <!-- Multiple command interfaces not working on Gazebo Fortress -->
+      <!-- https://github.com/ros-controls/gz_ros2_control/issues/182 -->
+      <xacro:if value="${gazebo_version == 'classic'}">
+        <command_interface name="velocity" />
+        <command_interface name="effort" />
+      </xacro:if>
       <state_interface name="position" />
       <state_interface name="velocity" />

File: tiago_description/urdf/head/head.urdf.xacro (robot description, xacro)
@@ -40,5 +40,5 @@
         <origin xyz="0 0 0" rpy="0 0 0"/>
         <geometry>
-          <mesh filename="package://tiago_description/meshes/head/head_1.stl" scale="1 1 1"/>
+          <mesh filename="file://$(find tiago_description)/meshes/head/head_1.stl" scale="1 1 1"/>
         </geometry>
         <material name="White" />
@@ -47,5 +47,5 @@
         <origin xyz="0.0 0 0" rpy="0 0 0.0" />
         <geometry>
-          <mesh filename="package://tiago_description/meshes/head/head_1_collision.dae" scale="1 1 1"/>
+          <mesh filename="file://$(find tiago_description)/meshes/head/head_1_collision.dae" scale="1 1 1"/>
         </geometry>
         <material name="White" />
@@ -80,5 +80,5 @@
         <origin xyz="0 0 0" rpy="0 0 0" />
         <geometry>
-          <mesh filename="package://tiago_description/meshes/head/head_2.stl" scale="1 1 1"/>
+          <mesh filename="file://$(find tiago_description)/meshes/head/head_2.stl" scale="1 1 1"/>
         </geometry>
         <material name="White" />
@@ -87,5 +87,5 @@
         <origin xyz="0 0 0" rpy="0 0 0" />
         <geometry>
-          <mesh filename="package://tiago_description/meshes/head/head_2_collision.dae" scale="1 1 1"/>
+          <mesh filename="file://$(find tiago_description)/meshes/head/head_2_collision.dae" scale="1 1 1"/>
         </geometry>
       </collision>

File: tiago_description/urdf/torso/torso.urdf.xacro (robot description, xacro)
@@ -30,5 +30,5 @@
         <origin rpy="0 0 0" xyz="0 0 0" />
         <geometry>
-          <mesh filename="package://tiago_description/meshes/torso/torso_fix.stl" scale="1 1 1"/>
+          <mesh filename="file://$(find tiago_description)/meshes/torso/torso_fix.stl" scale="1 1 1"/>
         </geometry>
         <material name="LightGrey"/>
@@ -94,5 +94,5 @@
         <origin rpy="0 0 0" xyz="0 0 0" />
         <geometry>
-          <mesh filename="package://tiago_description/meshes/torso/torso_lift_with_arm.stl" scale="1 1 1"/>
+          <mesh filename="file://$(find tiago_description)/meshes/torso/torso_lift_with_arm.stl" scale="1 1 1"/>
         </geometry>
         <material name="White"/>
@@ -101,5 +101,5 @@
         <origin rpy="0 0 0" xyz="0 0 0" />
         <geometry>
-          <mesh filename="package://tiago_description/meshes/torso/torso_lift_collision_core.dae" scale="1 1 1"/>
+          <mesh filename="file://$(find tiago_description)/meshes/torso/torso_lift_collision_core.dae" scale="1 1 1"/>
         </geometry>
         <material name="LightGrey"/>
@@ -108,5 +108,5 @@
         <origin rpy="0 0 0" xyz="0 0 0" />
         <geometry>
-          <mesh filename="package://tiago_description/meshes/torso/torso_lift_collision_shoulder.dae" scale="1 1 1"/>
+          <mesh filename="file://$(find tiago_description)/meshes/torso/torso_lift_collision_shoulder.dae" scale="1 1 1"/>
         </geometry>
         <material name="LightGrey"/>
@@ -115,5 +115,5 @@
         <origin rpy="0 0 0" xyz="0 0 0" />
         <geometry>
-          <mesh filename="package://tiago_description/meshes/torso/torso_lift_collision_neck.dae" scale="1 1 1"/>
+          <mesh filename="file://$(find tiago_description)/meshes/torso/torso_lift_collision_neck.dae" scale="1 1 1"/>
         </geometry>
         <material name="LightGrey"/>
@@ -123,5 +123,5 @@
         <origin rpy="0 0 -1.57" xyz="-0.01 0.125 -0.27" />
         <geometry>
-          <mesh filename="package://tiago_description/meshes/torso/tiago_screen.stl" scale="1 1 1"/>
+          <mesh filename="file://$(find tiago_description)/meshes/torso/tiago_screen.stl" scale="1 1 1"/>
         </geometry>
         <material name="White"/>
@@ -130,5 +130,5 @@
         <origin rpy="0 0 -1.57" xyz="-0.01 0.125 -0.27" />
         <geometry>
-          <mesh filename="package://tiago_description/meshes/torso/tiago_screen_collision.stl" scale="1 1 1"/>
+          <mesh filename="file://$(find tiago_description)/meshes/torso/tiago_screen_collision.stl" scale="1 1 1"/>
         </geometry>
         <material name="LightGrey"/>
@@ -136,4 +136,12 @@
     </xacro:if>
     </link>
+    <!-- TODO: set lower limit back to 0 when moving to Gazebo Harmonic or ROS 2 Jazzy -->
+    <!-- See https://github.com/gazebosim/gz-sim/issues/1684 for more information -->
+    <xacro:if value="${gazebo_version == 'classic'}">
+      <xacro:property name="torso_lower_limit" value="0.0"/>
+    </xacro:if>
+    <xacro:if value="${gazebo_version == 'gazebo'}">
+      <xacro:property name="torso_lower_limit" value="-1e-3"/>
+    </xacro:if>
     <joint name="${name}_lift_joint" type="prismatic">
       <origin rpy="0.0 0.0 0.0" xyz="0.0 0.0 0.597" />
@@ -141,5 +149,5 @@
       <child link="${name}_lift_link" />
       <axis xyz="0 0 1" />
-      <limit effort="2000" lower="0" upper="0.35" velocity="${torso_max_vel}" />
+      <limit effort="2000" lower="${torso_lower_limit}" upper="0.35" velocity="${torso_max_vel}" />
       <calibration rising="0.0" />
       <dynamics damping="1000" />
