Commit message: revert sign on arm_6_joint wrt standards

File: tiago_description/urdf/calibration/eye_hand_calibration.urdf.xacro (robot description, xacro)
@@ -27,5 +27,5 @@
   <xacro:property name="arm_4_joint_offset" value="0.0" />
   <xacro:property name="arm_5_joint_offset" value="0.0" />
-  <xacro:property name="arm_6_joint_offset" value="-0.0" />
+  <xacro:property name="arm_6_joint_offset" value="0.0" />
   <xacro:property name="arm_7_joint_offset" value="0.0" />
   <xacro:property name="head_1_joint_offset" value="0.0" />
